Commit message: Add fiction,trigger actuators in standard.yaml, fix shooter.urdf.xacro

File: urdf/standard/shooter.urdf.xacro (robot description, xacro)
@@ -29,5 +29,5 @@
     </link>
     <joint name="trigger_joint"  type="continuous">
-        <origin xyz="-0.073838 -0.037028 0"  rpy="0 0 0" />
+        <origin xyz="-0.064 0 0" rpy="0 0 0"/>
         <parent link="pitch" />
         <child link="trigger" />

File: urdf/standard/standard.urdf.xacro (robot description, xacro)
@@ -17,4 +17,5 @@
     <xacro:include filename="$(find rm_description)/urdf/standard/shooter.urdf.xacro"/>
   </xacro:if>
+  <xacro:include filename="$(find rm_description)/urdf/standard/standard.transmission.urdf.xacro"/>
   <xacro:if value="$(arg load_gazebo)">
     <xacro:if value="$(arg use_rm_gazebo)">
