Commit message: Add limit and test

File: urdf/standard/gimbal.transmission.urdf.xacro (robot description, xacro)
@@ -13,5 +13,5 @@
     </transmission>
     <transmission name="trans_pitch_joint">
-        <type>transmission_interface/SimpleTransmission</type>
+        <type>transmission_interface/RevoluteTransmission</type>
         <actuator name="pitch_joint_motor">
             <hardwareInterface>hardware_interface/EffortJointInterface</hardwareInterface>

File: urdf/standard/gimbal.urdf.xacro (robot description, xacro)
@@ -2,6 +2,6 @@
 <robot xmlns:xacro="http://www.ros.org/wiki/xacro">
     <xacro:property name="threshold" value="0.1"/>
-    <xacro:property name="lower_limit" value="-0.79"/>
-    <xacro:property name="upper_limit" value="0.79"/>
+    <xacro:property name="pitch_lower_limit" value="-0.716"/>
+    <xacro:property name="pitch_upper_limit" value="0.487"/>
     <link name="yaw">
         <inertial>
@@ -14,5 +14,5 @@
             <origin xyz="0 0 0" rpy="0 0 0"/>
             <geometry>
-                <mesh filename="package://rm_description/meshes/standard/yaw.stl" scale="0.001 0.001 0.001" />
+                <mesh filename="package://rm_description/meshes/standard/yaw.stl" scale="0.001 0.001 0.001"/>
             </geometry>
         </visual>
@@ -20,5 +20,5 @@
             <origin xyz="0 0 0" rpy="0 0 0"/>
             <geometry>
-                <mesh filename="package://rm_description/meshes/standard/yaw.stl"  scale="0.001 0.001 0.001" />
+                <mesh filename="package://rm_description/meshes/standard/yaw.stl" scale="0.001 0.001 0.001"/>
             </geometry>
         </collision>
@@ -28,9 +28,5 @@
                 rpy="0 0 0"/>
         <dynamics damping="0.0" friction="0.1"/>
-        <limit effort="1.2" velocity="31" lower="${lower_limit}" upper="${upper_limit}"/>
-        <safety_controller k_velocity="0.01"
-                           k_position="10000000"
-                           soft_lower_limit="${lower_limit+threshold}"
-                           soft_upper_limit="${upper_limit-threshold}"/>
+        <limit effort="1.2" velocity="31" lower="-1e10" upper="1e10"/>
         <parent link="base_link"/>
         <child link="yaw"/>
@@ -47,5 +43,5 @@
             <origin xyz="0 0 0" rpy="0 0 0"/>
             <geometry>
-                <mesh filename="package://rm_description/meshes/standard/pitch.stl" scale="0.001 0.001 0.001" />
+                <mesh filename="package://rm_description/meshes/standard/pitch.stl" scale="0.001 0.001 0.001"/>
             </geometry>
         </visual>
@@ -60,9 +56,8 @@
         <origin xyz="0 0 0.189" rpy="0 0 0"/>
         <dynamics damping="0.0" friction="0.1"/>
-        <limit effort="1.2" velocity="13.82" lower="${lower_limit}" upper="${upper_limit}"/>
-        <!--        <safety_controller k_velocity="10"-->
-        <!--                           k_position="15"-->
-        <!--                           soft_lower_limit="${lower_limit+threshold}"-->
-        <!--                           soft_upper_limit="${upper_limit-threshold}"/>-->
+        <limit effort="1.2" velocity="13.82" lower="${pitch_lower_limit}" upper="${pitch_upper_limit}"/>
+        <safety_controller k_position="100" k_velocity="0.1"
+                           soft_lower_limit="${pitch_lower_limit+threshold}"
+                           soft_upper_limit="${pitch_upper_limit-threshold}"/>
         <parent link="yaw"/>
         <child link="pitch"/>
