Commit message: Correct the word "infantry" to "standard"

File: urdf/standard/chassis.urdf.xacro (robot description, xacro)
@@ -18,5 +18,5 @@
         <origin xyz="0 0 0" rpy="0 0 0"/>
         <geometry>
-          <mesh filename="package://rm_description/meshes/infantry/base.stl" scale="0.001 0.001 0.001"/>
+          <mesh filename="package://rm_description/meshes/standard/base.stl" scale="0.001 0.001 0.001"/>
         </geometry>
       </visual>
@@ -24,5 +24,5 @@
         <origin xyz="0 0 0" rpy="0 0 0"/>
         <geometry>
-          <mesh filename="package://rm_description/meshes/infantry/base.stl" scale="0.001 0.001 0.001"/>
+          <mesh filename="package://rm_description/meshes/standard/base.stl" scale="0.001 0.001 0.001"/>
         </geometry>
       </collision>

File: urdf/standard/gimbal.urdf.xacro (robot description, xacro)
@@ -1,4 +1,3 @@
-<robot xmlns:xacro="http://www.ros.org/wiki/xacro">
-    <xacro:include filename="$(find rm_description)/urdf/infantry/chassis.urdf.xacro"/>
+<robot>
     <!-- https://upload.wikimedia.org/wikipedia/commons/5/52/Wheelbase_and_Track.png -->
     <link name="yaw_link">
@@ -12,5 +11,5 @@
             <origin xyz="0 0 0" rpy="0 0 0"/>
             <geometry>
-                <mesh filename="package://rm_description/meshes/infantry/yaw_base.stl" scale="0.001 0.001 0.001" />
+                <mesh filename="package://rm_description/meshes/standard/yaw_base.stl" scale="0.001 0.001 0.001"/>
             </geometry>
         </visual>
@@ -18,5 +17,5 @@
             <origin xyz="0 0 0" rpy="0 0 0"/>
             <geometry>
-                <mesh filename="package://rm_description/meshes/infantry/yaw_base.stl"  scale="0.001 0.001 0.001" />
+                <mesh filename="package://rm_description/meshes/standard/yaw_base.stl" scale="0.001 0.001 0.001"/>
             </geometry>
         </collision>
@@ -39,5 +38,5 @@
             <origin xyz="0 0 0" rpy="0 0 0"/>
             <geometry>
-                <mesh filename="package://rm_description/meshes/infantry/yaw_arm.stl" scale="0.001 0.001 0.001" />
+                <mesh filename="package://rm_description/meshes/standard/yaw_arm.stl" scale="0.001 0.001 0.001"/>
             </geometry>
         </visual>
@@ -45,5 +44,5 @@
             <origin xyz="0 0 0" rpy="0 0 0"/>
             <geometry>
-                <mesh filename="package://rm_description/meshes/infantry/yaw_arm.stl"  scale="0.001 0.001 0.001" />
+                <mesh filename="package://rm_description/meshes/standard/yaw_arm.stl" scale="0.001 0.001 0.001"/>
             </geometry>
         </collision>
@@ -65,5 +64,5 @@
             <origin xyz="0 0 0" rpy="0 0 0"/>
             <geometry>
-                <mesh filename="package://rm_description/meshes/infantry/pitch.stl" scale="0.001 0.001 0.001" />
+                <mesh filename="package://rm_description/meshes/standard/pitch.stl" scale="0.001 0.001 0.001"/>
             </geometry>
         </visual>
@@ -71,5 +70,5 @@
             <origin xyz="0 0 0" rpy="0 0 0"/>
             <geometry>
-                <mesh filename="package://rm_description/meshes/infantry/pitch.stl"  scale="0.001 0.001 0.001" />
+                <mesh filename="package://rm_description/meshes/standard/pitch.stl" scale="0.001 0.001 0.001"/>
             </geometry>
         </collision>

File: urdf/standard/standard.urdf.xacro (robot description, xacro)
@@ -1,4 +1,4 @@
 <?xml version="1.0"?>
-<robot xmlns:xacro="http://www.ros.org/wiki/xacro" name="infantry">
+<robot xmlns:xacro="http://www.ros.org/wiki/xacro" name="standard">
   <xacro:arg name="load_chassis" default="true"/>
   <xacro:arg name="load_gimbal" default="true"/>
@@ -8,9 +8,9 @@
   <xacro:arg name="roller_type" default="realistic"/>
   <xacro:if value="$(arg load_chassis)">
-    <xacro:include filename="$(find rm_description)/urdf/infantry/chassis.urdf.xacro"/>
+    <xacro:include filename="$(find rm_description)/urdf/standard/chassis.urdf.xacro"/>
     <xacro:chassis roller_type="$(arg roller_type)"/>
   </xacro:if>
   <xacro:if value="$(arg load_gimbal)">
-    <xacro:include filename="$(find rm_description)/urdf/infantry/gimbal.urdf.xacro"/>
+    <xacro:include filename="$(find rm_description)/urdf/standard/gimbal.urdf.xacro"/>
   </xacro:if>
   <xacro:if value="$(arg load_shooter)">

Commit message: add chassis mass

File: urdf/standard/chassis.urdf.xacro (robot description, xacro)
@@ -10,5 +10,5 @@
     <link name="base_link">
       <inertial>
-        <mass value="10"/>
+        <mass value="10.56"/>
         <origin xyz="-0.025077  0  0.055047"/>
         <inertia ixx="2.247e-1" ixy="-1.139e-5" ixz="2.983e-2" iyy="3.771e-1"

Commit message: Use simple rectangular collision

File: urdf/standard/chassis.urdf.xacro (robot description, xacro)
@@ -1,51 +1,51 @@
 <robot xmlns:xacro="http://www.ros.org/wiki/xacro">
-  <xacro:include filename="$(find rm_description)/urdf/common/mecanum_wheel.urdf.xacro"/>
-  <!-- https://upload.wikimedia.org/wikipedia/commons/5/52/Wheelbase_and_Track.png -->
-  <xacro:property name="wheel_track" value="0.380"/>
-  <xacro:property name="wheel_base" value="0.395"/>
-  <xacro:property name="wheel_offset_z" value="0.0"/>
-  <xacro:property name="wheel_joint_damping" value="1.0"/>
-  <xacro:property name="wheel_joint_friction" value="1.0"/>
-  <xacro:macro name="chassis" params="roller_type">
-    <link name="base_link">
-      <inertial>
-        <mass value="10.56"/>
-        <origin xyz="-0.025077  0  0.055047"/>
-        <inertia ixx="2.247e-1" ixy="-1.139e-5" ixz="2.983e-2" iyy="3.771e-1"
-                 iyz="3.3454e-6" izz="4.803e-1"/>
-      </inertial>
-      <visual>
-        <origin xyz="0 0 0" rpy="0 0 0"/>
-        <geometry>
-          <mesh filename="package://rm_description/meshes/standard/base.stl" scale="0.001 0.001 0.001"/>
-        </geometry>
-      </visual>
-      <collision>
-        <origin xyz="0 0 0" rpy="0 0 0"/>
-        <geometry>
-          <mesh filename="package://rm_description/meshes/standard/base.stl" scale="0.001 0.001 0.001"/>
-        </geometry>
-      </collision>
-    </link>
-    <xacro:mecanum_wheel prefix="front_left" connected_to="base_link"
-                         wheel_x_offset="${wheel_track/2}" wheel_y_offset="${wheel_base/2}"
-                         wheel_z_offset="${wheel_offset_z}"
-                         reflect="1" roller_type="${roller_type}"/>
-    <xacro:mecanum_wheel prefix="front_right" connected_to="base_link"
-                         wheel_x_offset="${wheel_track/2}" wheel_y_offset="${-wheel_base/2}"
-                         wheel_z_offset="${wheel_offset_z}"
-                         reflect="-1" roller_type="${roller_type}"/>
-    <xacro:mecanum_wheel prefix="back_left" connected_to="base_link"
-                         wheel_x_offset="${-wheel_track/2}" wheel_y_offset="${wheel_base/2}"
-                         wheel_z_offset="${wheel_offset_z}"
-                         reflect="-1" roller_type="${roller_type}"/>
-    <xacro:mecanum_wheel prefix="back_right" connected_to="base_link"
-                         wheel_x_offset="${-wheel_track/2}" wheel_y_offset="${-wheel_base/2}"
-                         wheel_z_offset="${wheel_offset_z}"
-                         reflect="1" roller_type="${roller_type}"/>
-    <xacro:wheel_transmission prefix="front_left" mechanical_reduction="1"/>
-    <xacro:wheel_transmission prefix="front_right" mechanical_reduction="-1"/>
-    <xacro:wheel_transmission prefix="back_left" mechanical_reduction="1"/>
-    <xacro:wheel_transmission prefix="back_right" mechanical_reduction="-1"/>
-  </xacro:macro>
+    <xacro:include filename="$(find rm_description)/urdf/common/mecanum_wheel.urdf.xacro"/>
+    <!-- https://upload.wikimedia.org/wikipedia/commons/5/52/Wheelbase_and_Track.png -->
+    <xacro:property name="wheel_track" value="0.380"/>
+    <xacro:property name="wheel_base" value="0.395"/>
+    <xacro:property name="wheel_offset_z" value="0.0"/>
+    <xacro:property name="wheel_joint_damping" value="1.0"/>
+    <xacro:property name="wheel_joint_friction" value="1.0"/>
+    <xacro:macro name="chassis" params="roller_type">
+        <link name="base_link">
+            <inertial>
+                <mass value="10.56"/>
+                <origin xyz="-0.025077  0  0.055047"/>
+                <inertia ixx="2.247e-1" ixy="-1.139e-5" ixz="2.983e-2" iyy="3.771e-1"
+                         iyz="3.3454e-6" izz="4.803e-1"/>
+            </inertial>
+            <visual>
+                <origin xyz="0 0 0" rpy="0 0 0"/>
+                <geometry>
+                    <mesh filename="package://rm_description/meshes/standard/base.stl" scale="0.001 0.001 0.001"/>
+                </geometry>
+            </visual>
+            <collision>
+                <origin xyz="0 0 0" rpy="0 0 0"/>
+                <geometry>
+                    <box size="0.580 0.500 0.050"/>
+                </geometry>
+            </collision>
+        </link>
+        <xacro:mecanum_wheel prefix="front_left" connected_to="base_link"
+                             wheel_x_offset="${wheel_track/2}" wheel_y_offset="${wheel_base/2}"
+                             wheel_z_offset="${wheel_offset_z}"
+                             reflect="1" roller_type="${roller_type}"/>
+        <xacro:mecanum_wheel prefix="front_right" connected_to="base_link"
+                             wheel_x_offset="${wheel_track/2}" wheel_y_offset="${-wheel_base/2}"
+                             wheel_z_offset="${wheel_offset_z}"
+                             reflect="-1" roller_type="${roller_type}"/>
+        <xacro:mecanum_wheel prefix="back_left" connected_to="base_link"
+                             wheel_x_offset="${-wheel_track/2}" wheel_y_offset="${wheel_base/2}"
+                             wheel_z_offset="${wheel_offset_z}"
+                             reflect="-1" roller_type="${roller_type}"/>
+        <xacro:mecanum_wheel prefix="back_right" connected_to="base_link"
+                             wheel_x_offset="${-wheel_track/2}" wheel_y_offset="${-wheel_base/2}"
+                             wheel_z_offset="${wheel_offset_z}"
+                             reflect="1" roller_type="${roller_type}"/>
+        <xacro:wheel_transmission prefix="front_left" mechanical_reduction="1"/>
+        <xacro:wheel_transmission prefix="front_right" mechanical_reduction="-1"/>
+        <xacro:wheel_transmission prefix="back_left" mechanical_reduction="1"/>
+        <xacro:wheel_transmission prefix="back_right" mechanical_reduction="-1"/>
+    </xacro:macro>
 </robot>
