Commit message: Fix error of transmission in standard

File: urdf/standard/gimbal.urdf.xacro (robot description, xacro)
@@ -47,18 +47,18 @@
             <origin xyz="0 0 0" rpy="0 0 0"/>
             <geometry>
-                <mesh filename="package://rm_description/meshes/standard/pitch.stl"  scale="0.001 0.001 0.001" />
+                <mesh filename="package://rm_description/meshes/standard/pitch.stl" scale="0.001 0.001 0.001"/>
             </geometry>
         </collision>
     </link>
-    <joint name="pitch_joint"  type="revolute">
-        <origin xyz="0 0 0.189"  rpy="0 0 0" />
+    <joint name="pitch_joint" type="revolute">
+        <origin xyz="0 0 0.189" rpy="0 0 0"/>
         <limit effort="3000" velocity="1000" lower="${lower_limit}" upper="${upper_limit}"/>
-        <safety_controller k_velocity="10"
-                k_position="15"
-                soft_lower_limit="${lower_limit+threshold}"
-                soft_upper_limit="${upper_limit-threshold}" />
-        <parent link="yaw" />
-        <child link="pitch" />
-        <axis xyz="0 1 0 " />
+        <!--        <safety_controller k_position="15"-->
+        <!--                           k_velocity="0.01"-->
+        <!--                           soft_lower_limit="${lower_limit+threshold}"-->
+        <!--                           soft_upper_limit="${upper_limit-threshold}"/>-->
+        <parent link="yaw"/>
+        <child link="pitch"/>
+        <axis xyz="0 1 0 "/>
     </joint>
 </robot>

File: urdf/standard/shooter.transmission.urdf.xacro (robot description, xacro)
@@ -1,25 +1,4 @@
 <?xml version="1.0" encoding="utf-8"?>
-<robot xmlns:xacro="http://www.ros.org/wiki/xacro">
-    <!-- transmission -->
-    <transmission name="trans_yaw_joint">
-        <type>transmission_interface/SimpleTransmission</type>
-        <actuator name="yaw_joint_motor">
-            <hardwareInterface>hardware_interface/EffortJointInterface</hardwareInterface>
-            <mechanicalReduction>1</mechanicalReduction>
-        </actuator>
-        <joint name="yaw_joint">
-            <hardwareInterface>hardware_interface/EffortJointInterface</hardwareInterface>
-        </joint>
-    </transmission>
-    <transmission name="trans_pitch_joint">
-        <type>transmission_interface/SimpleTransmission</type>
-        <actuator name="pitch_joint_motor">
-            <hardwareInterface>hardware_interface/EffortJointInterface</hardwareInterface>
-            <mechanicalReduction>1</mechanicalReduction>
-        </actuator>
-        <joint name="pitch_joint">
-            <hardwareInterface>hardware_interface/EffortJointInterface</hardwareInterface>
-        </joint>
-    </transmission>
+<robot>
     <transmission name="trans_trigger_joint">
         <type>transmission_interface/SimpleTransmission</type>

File: urdf/standard/standard.urdf.xacro (robot description, xacro)
@@ -13,9 +13,10 @@
   <xacro:if value="$(arg load_gimbal)">
     <xacro:include filename="$(find rm_description)/urdf/standard/gimbal.urdf.xacro"/>
+    <xacro:include filename="$(find rm_description)/urdf/standard/gimbal.transmission.urdf.xacro"/>
   </xacro:if>
   <xacro:if value="$(arg load_shooter)">
     <xacro:include filename="$(find rm_description)/urdf/standard/shooter.urdf.xacro"/>
+    <xacro:include filename="$(find rm_description)/urdf/standard/shooter.transmission.urdf.xacro"/>
   </xacro:if>
-  <xacro:include filename="$(find rm_description)/urdf/standard/standard.transmission.urdf.xacro"/>
   <xacro:if value="$(arg load_gazebo)">
     <xacro:if value="$(arg use_rm_gazebo)">

Commit message: Set a smaller friction of pitch_joint

File: urdf/standard/gimbal.urdf.xacro (robot description, xacro)
@@ -55,5 +55,5 @@
     <joint name="pitch_joint" type="revolute">
         <origin xyz="0 0 0.189" rpy="0 0 0"/>
-        <dynamics damping="0.0" friction="0.5"/>
+        <dynamics damping="0.0" friction="0.1"/>
         <limit effort="1.2" velocity="13.82" lower="${lower_limit}" upper="${upper_limit}"/>
         <!--        <safety_controller k_velocity="10"-->

Commit message: Test satety_controller

File: urdf/standard/gimbal.urdf.xacro (robot description, xacro)
@@ -1,7 +1,7 @@
 <?xml version="1.0" encoding="utf-8"?>
 <robot xmlns:xacro="http://www.ros.org/wiki/xacro">
-    <xacro:property name="threshold" value="0.01"/>
-    <xacro:property name="lower_limit" value="-0.436323"/>
-    <xacro:property name="upper_limit" value="0.7853982"/>
+    <xacro:property name="threshold" value="0.1"/>
+    <xacro:property name="lower_limit" value="-0.79"/>
+    <xacro:property name="upper_limit" value="0.79"/>
     <link name="yaw">
         <inertial>
@@ -24,8 +24,13 @@
         </collision>
     </link>
-    <joint name="yaw_joint" type="continuous">
+    <joint name="yaw_joint" type="revolute">
         <origin xyz="0 0 0.0696"
                 rpy="0 0 0"/>
         <dynamics damping="0.0" friction="0.1"/>
+        <limit effort="1.2" velocity="31" lower="${lower_limit}" upper="${upper_limit}"/>
+        <safety_controller k_velocity="0.01"
+                           k_position="10000000"
+                           soft_lower_limit="${lower_limit+threshold}"
+                           soft_upper_limit="${upper_limit-threshold}"/>
         <parent link="base_link"/>
         <child link="yaw"/>

Commit message: Update gimbal pitch_lower_limit and pitch_upper_limit

File: urdf/standard/gimbal.urdf.xacro (robot description, xacro)
@@ -2,6 +2,6 @@
 <robot xmlns:xacro="http://www.ros.org/wiki/xacro">
     <xacro:property name="threshold" value="0.1"/>
-    <xacro:property name="pitch_lower_limit" value="-0.716"/>
-    <xacro:property name="pitch_upper_limit" value="0.487"/>
+    <xacro:property name="pitch_lower_limit" value="-0.482"/>
+    <xacro:property name="pitch_upper_limit" value="0.257"/>
     <link name="yaw">
         <inertial>

Commit message: Update standard shooter qd parameter and gimbal pid

File: urdf/standard/gimbal.urdf.xacro (robot description, xacro)
@@ -2,6 +2,6 @@
 <robot xmlns:xacro="http://www.ros.org/wiki/xacro">
     <xacro:property name="threshold" value="0.1"/>
-    <xacro:property name="pitch_lower_limit" value="-0.716"/>
-    <xacro:property name="pitch_upper_limit" value="0.487"/>
+    <xacro:property name="pitch_lower_limit" value="-0.734"/>
+    <xacro:property name="pitch_upper_limit" value="0.422"/>
     <link name="yaw">
         <inertial>

Commit message: Delete collision position of camera

File: urdf/standard/gimbal.urdf.xacro (robot description, xacro)
@@ -79,5 +79,5 @@
             </visual>
             <collision>
-                <origin xyz="0.02 0.0 0.0" rpy="0 -1.57 0"/>
+                <origin xyz="0 0 0" rpy="0 -1.57 0"/>
                 <geometry>
                     <mesh filename="package://rm_description/meshes/common/camera.stl" scale="0.001 0.001 0.001"/>

Commit message: change limit of gimbal pitch

File: urdf/standard/gimbal.urdf.xacro (robot description, xacro)
@@ -2,6 +2,6 @@
 <robot xmlns:xacro="http://www.ros.org/wiki/xacro">
     <xacro:property name="threshold" value="0.1"/>
-    <xacro:property name="pitch_lower_limit" value="-0.734"/>
-    <xacro:property name="pitch_upper_limit" value="0.422"/>
+    <xacro:property name="pitch_lower_limit" value="-0.7"/>
+    <xacro:property name="pitch_upper_limit" value="0.2"/>
     <xacro:macro name="gimbal" params="simulation">
         <link name="yaw">

Commit message: change limit of gimbal pitch

File: urdf/standard/gimbal.urdf.xacro (robot description, xacro)
@@ -3,5 +3,5 @@
     <xacro:property name="threshold" value="0.1"/>
     <xacro:property name="pitch_lower_limit" value="-0.7"/>
-    <xacro:property name="pitch_upper_limit" value="0.2"/>
+    <xacro:property name="pitch_upper_limit" value="0.4"/>
     <xacro:macro name="gimbal" params="simulation">
         <link name="yaw">

Commit message: Update camera position and time_compensation

File: urdf/standard/gimbal.urdf.xacro (robot description, xacro)
@@ -88,5 +88,5 @@
             <parent link="pitch"/>
             <child link="camera"/>
-            <origin xyz="0.064 0.0 -0.043" rpy="-1.57 0 -1.57"/>
+            <origin xyz="0.12 0.0 -0.055" rpy="-1.57 0 -1.57"/>
             <axis xyz="0 0 1"/>
         </joint>

Commit message: Change camera into camera_link

File: urdf/standard/gimbal.urdf.xacro (robot description, xacro)
@@ -65,5 +65,5 @@
             <axis xyz="0 1 0 "/>
         </joint>
-        <link name="camera">
+        <link name="camera_link">
             <inertial>
                 <mass value="0.17671"/>
@@ -87,5 +87,5 @@
         <joint name="camera_joint" type="fixed">
             <parent link="pitch"/>
-            <child link="camera"/>
+            <child link="camera_link"/>
             <origin xyz="0.12 0.0 -0.055" rpy="-1.57 0 -1.57"/>
             <axis xyz="0 0 1"/>

Commit message: Update camera_joint position

File: urdf/standard/gimbal.urdf.xacro (robot description, xacro)
@@ -88,5 +88,5 @@
             <parent link="pitch"/>
             <child link="camera_link"/>
-            <origin xyz="0.12 0.0 -0.055" rpy="-1.57 0 -1.57"/>
+            <origin xyz="0.15 0.0 -0.03" rpy="-1.57 0 -1.57"/>
             <axis xyz="0 0 1"/>
         </joint>

Commit message: Move cover from gimbal to shooter in standard

File: urdf/standard/gimbal.urdf.xacro (robot description, xacro)
@@ -64,30 +64,3 @@
             <axis xyz="0 1 0 "/>
         </joint>
-    <link name="cover">
-        <inertial>
-            <mass value="0.149"/>
-            <origin xyz="-0.008 -0.005 0.019"/>
-            <inertia ixx="2.366e-3" ixy="-2.372e-4" ixz="-7.983e-4" iyy="2.959e-3" iyz="-2.826e-4" izz="9.090e-4"/>
-        </inertial>
-        <visual>
-            <origin xyz="0 0 0" rpy="0 0 0"/>
-            <geometry>
-                <mesh filename="package://rm_description/meshes/standard/cover.stl" scale="0.001 0.001 0.001"/>
-            </geometry>
-        </visual>
-        <collision>
-            <origin xyz="0.033 0.0 -0.0" rpy="0 0.0 0"/>
-            <geometry>
-                <mesh filename="package://rm_description/meshes/standard/cover.stl" scale="0.001 0.001 0.001"/>
-            </geometry>
-        </collision>
-    </link>
-    <joint name="cover_joint" type="revolute">
-        <axis xyz="0 0 1"/>
-        <origin xyz="0.037 0.042 0.122"/>
-        <limit effort="1.0" velocity="30" lower="-3.14" upper="3.14"/>
-        <dynamics damping="0.0" friction="0.1"/>
-        <parent link="pitch"/>
-        <child link="cover"/>
-    </joint>
 </robot>

File: urdf/standard/shooter.urdf.xacro (robot description, xacro)
@@ -39,3 +39,30 @@
         <axis xyz="0 0 1 "/>
     </joint>
+    <link name="cover">
+        <inertial>
+            <mass value="0.149"/>
+            <origin xyz="-0.008 -0.005 0.019"/>
+            <inertia ixx="2.366e-3" ixy="-2.372e-4" ixz="-7.983e-4" iyy="2.959e-3" iyz="-2.826e-4" izz="9.090e-4"/>
+        </inertial>
+        <visual>
+            <origin xyz="0 0 0" rpy="0 0 0"/>
+            <geometry>
+                <mesh filename="package://rm_description/meshes/standard/cover.stl" scale="0.001 0.001 0.001"/>
+            </geometry>
+        </visual>
+        <collision>
+            <origin xyz="0.033 0.0 -0.0" rpy="0 0.0 0"/>
+            <geometry>
+                <mesh filename="package://rm_description/meshes/standard/cover.stl" scale="0.001 0.001 0.001"/>
+            </geometry>
+        </collision>
+    </link>
+    <joint name="cover_joint" type="revolute">
+        <axis xyz="0 0 1"/>
+        <origin xyz="0.037 0.042 0.122"/>
+        <limit effort="1.0" velocity="30" lower="-3.14" upper="3.14"/>
+        <dynamics damping="0.0" friction="0.1"/>
+        <parent link="pitch"/>
+        <child link="cover"/>
+    </joint>
 </robot>
