Commit message: Add limit and dynamics to joint, and fix fiction wheel same velocity direction in gazebo

File: urdf/common/friction.urdf.xacro (robot description, xacro)
@@ -23,4 +23,5 @@
         <joint name="${prefixs}_friction_wheel_joint"  type="continuous">
             <origin xyz="${wheel_x_offset} ${wheel_y_offset} ${wheel_offset_z}" rpy="0 0 0"/>"
+            <limit upper="1e16" lower="-1e16" effort="0.156" velocity="942.00"/>
             <parent link="${connected_to}" />
             <child link="${prefixs}_friction_wheel" />

File: urdf/standard/gimbal.urdf.xacro (robot description, xacro)
@@ -24,10 +24,12 @@
         </collision>
     </link>
-    <joint name="yaw_joint"  type="continuous">
+    <joint name="yaw_joint" type="continuous">
         <origin xyz="0 0 0.0696"
-                rpy="0 0 0" />
-        <parent link="base_link" />
-        <child link="yaw" />
-        <axis xyz="0 0 1" />
+                rpy="0 0 0"/>
+        <dynamics damping="0.0" friction="0.5"/>
+        <limit effort="1.2" velocity="13.82" lower="${lower_limit}" upper="${upper_limit}"/>
+        <parent link="base_link"/>
+        <child link="yaw"/>
+        <axis xyz="0 0 1"/>
     </joint>
     <link name="pitch">
@@ -47,18 +49,19 @@
             <origin xyz="0 0 0" rpy="0 0 0"/>
             <geometry>
-                <mesh filename="package://rm_description/meshes/standard/pitch.stl"  scale="0.001 0.001 0.001" />
+                <mesh filename="package://rm_description/meshes/standard/pitch.stl" scale="0.001 0.001 0.001"/>
             </geometry>
         </collision>
     </link>
-    <joint name="pitch_joint"  type="revolute">
-        <origin xyz="0 0 0.189"  rpy="0 0 0" />
-        <limit effort="3000" velocity="1000" lower="${lower_limit}" upper="${upper_limit}"/>
+    <joint name="pitch_joint" type="revolute">
+        <origin xyz="0 0 0.189" rpy="0 0 0"/>
+        <dynamics damping="0.0" friction="0.5"/>
+        <limit effort="1.2" velocity="13.82" lower="${lower_limit}" upper="${upper_limit}"/>
         <safety_controller k_velocity="10"
-                k_position="15"
-                soft_lower_limit="${lower_limit+threshold}"
-                soft_upper_limit="${upper_limit-threshold}" />
-        <parent link="yaw" />
-        <child link="pitch" />
-        <axis xyz="0 1 0 " />
+                           k_position="15"
+                           soft_lower_limit="${lower_limit+threshold}"
+                           soft_upper_limit="${upper_limit-threshold}"/>
+        <parent link="yaw"/>
+        <child link="pitch"/>
+        <axis xyz="0 1 0 "/>
     </joint>
 </robot>

File: urdf/standard/shooter.urdf.xacro (robot description, xacro)
@@ -28,9 +28,11 @@
         </collision>
     </link>
-    <joint name="trigger_joint"  type="continuous">
+    <joint name="trigger_joint" type="continuous">
         <origin xyz="-0.064 0 0" rpy="0 0 0"/>
-        <parent link="pitch" />
-        <child link="trigger" />
-        <axis xyz="0 0 1 " />
+        <dynamics damping="0.0" friction="0.01"/>
+        <limit effort="1.0" velocity="43.54" lower="-1e16" upper="1e16"/>
+        <parent link="pitch"/>
+        <child link="trigger"/>
+        <axis xyz="0 0 1 "/>
     </joint>
 </robot>

File: urdf/standard/standard.transmission.urdf.xacro (robot description, xacro)
@@ -1,4 +1,4 @@
 <?xml version="1.0" encoding="utf-8"?>
-<robot xmlns:xacro="http://www.ros.org/wiki/xacro">
+<robot>
     <!-- transmission -->
     <transmission name="trans_yaw_joint">

Commit message: Fix trigger can not rotate and fiction can not stop in gazebo

File: urdf/common/friction.urdf.xacro (robot description, xacro)
@@ -23,4 +23,5 @@
         <joint name="${prefixs}_friction_wheel_joint"  type="continuous">
             <origin xyz="${wheel_x_offset} ${wheel_y_offset} ${wheel_offset_z}" rpy="0 0 0"/>"
+            <dynamics damping="0.0" friction="0.01"/>
             <limit upper="1e16" lower="-1e16" effort="0.156" velocity="942.00"/>
             <parent link="${connected_to}" />

Commit message: Add some joint limit, dynamics about hero urdf and test shooter controller in gazebo

File: urdf/common/friction.urdf.xacro (robot description, xacro)
@@ -24,5 +24,5 @@
             <origin xyz="${wheel_x_offset} ${wheel_y_offset} ${wheel_offset_z}" rpy="0 0 0"/>"
             <dynamics damping="0.0" friction="0.01"/>
-            <limit upper="1e16" lower="-1e16" effort="0.156" velocity="942.00"/>
+            <limit upper="1e16" lower="-1e16" effort="0.156" velocity="942.66"/>
             <parent link="${connected_to}" />
             <child link="${prefixs}_friction_wheel" />

File: urdf/hero/gimbal.urdf.xacro (robot description, xacro)
@@ -27,5 +27,6 @@
         <origin xyz="0 0 0.1"
                 rpy="0 0 0"/>
-        <dynamics damping="0.0" friction="0.5"/>
+        <dynamics damping="0.0" friction="0.1"/>
+        <limit effort="1.2" velocity="13.82" lower="${lower_limit}" upper="${upper_limit}"/>
         <parent link="base_link"/>
         <child link="yaw"/>

File: urdf/hero/shooter.urdf.xacro (robot description, xacro)
@@ -31,5 +31,5 @@
         <origin xyz="-0.064 0 0" rpy="0 0 0"/>
         <dynamics damping="0.0" friction="0.01"/>
-        <limit effort="1.0" velocity="43.54" lower="-1e16" upper="1e16"/>
+        <limit effort="3.0" velocity="49.09" lower="-1e16" upper="1e16"/>
         <parent link="base_link"/>
         <child link="trigger"/>

File: urdf/standard/gimbal.urdf.xacro (robot description, xacro)
@@ -27,5 +27,5 @@
         <origin xyz="0 0 0.0696"
                 rpy="0 0 0"/>
-        <dynamics damping="0.0" friction="0.5"/>
+        <dynamics damping="0.0" friction="0.1"/>
         <parent link="base_link"/>
         <child link="yaw"/>
