Commit message: Change some name

File: urdf/common/imu.urdf.xacro (robot description, xacro)
@@ -10,13 +10,13 @@
     <xacro:property name="acceleration_drift" value="0.0 0.0 0.0"/>
     <xacro:property name="acceleration_drift_frequency" value="0.0 0.0 0.0"/>
-    <xacro:property name="acceleration_gaussian_noise" value="0.0 0.0 0.0"/>
+    <xacro:property name="acceleration_gaussian_noise" value="0.1 0.1 0.1"/>
     <xacro:property name="rate_offset" value="0.0 0.0 0.0"/>
     <xacro:property name="rate_drift" value="0.0 0.0 0.0"/>
     <xacro:property name="rate_drift_frequency" value="0.0 0.0 0.0"/>
-    <xacro:property name="rate_gaussian_noise" value="0.0 0.0 0.0"/>
+    <xacro:property name="rate_gaussian_noise" value="0.2 0.2 0.2"/>
     <xacro:property name="heading_offset" value="0.0"/>
     <xacro:property name="heading_drift" value="0.0"/>
     <xacro:property name="heading_drift_frequency" value="0.0"/>
-    <xacro:property name="heading_gaussian_noise" value="0.0"/>
+    <xacro:property name="heading_gaussian_noise" value="0.3"/>
     <xacro:if value="${simulation}">
       <gazebo>

File: urdf/engineer/hand.urdf.xacro (robot description, xacro)
@@ -2,5 +2,5 @@
 <robot xmlns:xacro="http://www.ros.org/wiki/xacro" name="hand">
   <!-- safety_distance: Minimum safety distance in [m] by which the collision volumes are expanded and which is enforced during robot motions -->
-  <xacro:macro name="hand" params="connected_to:='' rpy:='0 0 0' xyz:='0 0 0' ">
+  <xacro:macro name="hand" params="connected_to:='' xyz:='0 0 0' rpy:='0 0 0' ">
     <link name="palm">
       <inertial>

File: urdf/standard/standard.urdf.xacro (robot description, xacro)
@@ -4,5 +4,5 @@
   <xacro:arg name="load_gimbal" default="true"/>
   <xacro:arg name="load_shooter" default="true"/>
-  <xacro:arg name="load_gazebo" default="true"/>
+  <xacro:arg name="use_simulation" default="true"/>
   <xacro:arg name="use_rm_gazebo" default="false"/>
   <xacro:arg name="roller_type" default="realistic"/>
@@ -10,4 +10,6 @@
     <xacro:include filename="$(find rm_description)/urdf/standard/chassis.urdf.xacro"/>
     <xacro:chassis roller_type="$(arg roller_type)"/>
+    <xacro:include filename="$(find rm_description)/urdf/common/imu.urdf.xacro"/>
+    <xacro:IMU connected_to="base_link" imu_link_name="base_imu" simulation="$(arg use_simulation)" xyz="0 -0.12 0.03"/>
   </xacro:if>
   <xacro:if value="$(arg load_gimbal)">
@@ -19,5 +21,5 @@
     <xacro:include filename="$(find rm_description)/urdf/standard/shooter.transmission.urdf.xacro"/>
   </xacro:if>
-  <xacro:if value="$(arg load_gazebo)">
+  <xacro:if value="$(arg use_simulation)">
     <xacro:if value="$(arg use_rm_gazebo)">
       <gazebo>

Commit message: Reformat imu.urdf.xacro

File: urdf/common/imu.urdf.xacro (robot description, xacro)
@@ -3,72 +3,72 @@
 <!-- Documentation can be found at http://wiki.ros.org/hector_gazebo_plugins -->
 <robot xmlns:xacro="http://www.ros.org/wiki/xacro" name="imu">
-  <xacro:macro name="IMU" params="connected_to imu_link_name simulation xyz:='0 0 0' rpy:='0 0 0' ">
-    <xacro:property name="imu_base_link" value="${base_link}"/>
-    <xacro:property name="imu_update_rate" value="200"/>
-    <xacro:property name="imu_calibration_service_name" value="${imu_link_name}/calibrate"/>
-    <xacro:property name="acceleration_offset" value="0.0 0.0 0.0"/>
-    <xacro:property name="acceleration_drift" value="0.0 0.0 0.0"/>
-    <xacro:property name="acceleration_drift_frequency" value="0.0 0.0 0.0"/>
-    <xacro:property name="acceleration_gaussian_noise" value="0.1 0.1 0.1"/>
-    <xacro:property name="rate_offset" value="0.0 0.0 0.0"/>
-    <xacro:property name="rate_drift" value="0.0 0.0 0.0"/>
-    <xacro:property name="rate_drift_frequency" value="0.0 0.0 0.0"/>
-    <xacro:property name="rate_gaussian_noise" value="0.2 0.2 0.2"/>
-    <xacro:property name="heading_offset" value="0.0"/>
-    <xacro:property name="heading_drift" value="0.0"/>
-    <xacro:property name="heading_drift_frequency" value="0.0"/>
-    <xacro:property name="heading_gaussian_noise" value="0.3"/>
-    <xacro:if value="${simulation}">
-      <gazebo>
-        <plugin name="smb_imu_plugin" filename="libhector_gazebo_ros_imu.so">
-          <updateRate>${imu_update_rate}</updateRate>
-          <bodyName>${imu_link_name}</bodyName>
-          <frameId>${imu_link_name}</frameId>
-          <topicName>${imu_link_name}</topicName>
-          <serviceName>${imu_calibration_service_name}</serviceName>
-          <accelOffset>${acceleration_offset}</accelOffset>
-          <accelDrift>${acceleration_drift}</accelDrift>
-          <accelDriftFrequency>${acceleration_drift_frequency}</accelDriftFrequency>
-          <accelGaussianNoise>${acceleration_gaussian_noise}</accelGaussianNoise>
-          <rateOffset>${rate_offset}</rateOffset>
-          <rateDrift>${rate_drift}</rateDrift>
-          <rateDriftFrequency>${rate_drift_frequency}</rateDriftFrequency>
-          <rateGaussianNoise>${rate_gaussian_noise}</rateGaussianNoise>
-          <headingOffset>${heading_offset}</headingOffset>
-          <headingDrift>${heading_drift}</headingDrift>
-          <headingDriftFrequency>${heading_drift_frequency}</headingDriftFrequency>
-          <headingGaussianNoise>${heading_gaussian_noise}</headingGaussianNoise>
-        </plugin>
-      </gazebo>
-    </xacro:if>
-    <!-- Imu is fixed to the base link -->
-    <joint name="${imu_link_name}_joint" type="fixed">
-      <origin xyz="${xyz}" rpy="${rpy}"/>
-      <parent link="${connected_to}"/>
-      <child link="${imu_link_name}"/>
-    </joint>
-    <!-- Imu link -->
-    <link name="${imu_link_name}">
-      <inertial>
-        <mass value="0.001"/>
-        <origin rpy="0 0 0" xyz="0 0 0"/>
-        <inertia ixx="0.0001" ixy="0" ixz="0" iyy="0.000001" iyz="0" izz="0.0001"/>
-      </inertial>
-      <visual>
-        <origin rpy="0 0 0" xyz="0 0 0"/>
-        <geometry>
-          <box size="0.015 0.015 0.004"/>
-        </geometry>
-      </visual>
-      <material name="orange">
-        <color rgba="255 108 10 255"/>
-      </material>
-    </link>
-    <gazebo reference="${imu_link_name}">
-      <material>Gazebo/Orange</material>
-    </gazebo>
-    <gazebo reference="${imu_link_name}_joint">
-      <disableFixedJointLumping>true</disableFixedJointLumping>
-    </gazebo>
-  </xacro:macro>
+    <xacro:macro name="IMU" params="connected_to imu_link_name simulation xyz:='0 0 0' rpy:='0 0 0' ">
+        <xacro:property name="imu_base_link" value="${base_link}"/>
+        <xacro:property name="imu_update_rate" value="200"/>
+        <xacro:property name="imu_calibration_service_name" value="${imu_link_name}/calibrate"/>
+        <xacro:property name="acceleration_offset" value="0.0 0.0 0.0"/>
+        <xacro:property name="acceleration_drift" value="0.0 0.0 0.0"/>
+        <xacro:property name="acceleration_drift_frequency" value="0.0 0.0 0.0"/>
+        <xacro:property name="acceleration_gaussian_noise" value="0.1 0.1 0.1"/>
+        <xacro:property name="rate_offset" value="0.0 0.0 0.0"/>
+        <xacro:property name="rate_drift" value="0.0 0.0 0.0"/>
+        <xacro:property name="rate_drift_frequency" value="0.0 0.0 0.0"/>
+        <xacro:property name="rate_gaussian_noise" value="0.2 0.2 0.2"/>
+        <xacro:property name="heading_offset" value="0.0"/>
+        <xacro:property name="heading_drift" value="0.0"/>
+        <xacro:property name="heading_drift_frequency" value="0.0"/>
+        <xacro:property name="heading_gaussian_noise" value="0.3"/>
+        <!-- Imu is fixed to the base link -->
+        <joint name="${imu_link_name}_joint" type="fixed">
+            <origin xyz="${xyz}" rpy="${rpy}"/>
+            <parent link="${connected_to}"/>
+            <child link="${imu_link_name}"/>
+        </joint>
+        <!-- Imu link -->
+        <link name="${imu_link_name}">
+            <inertial>
+                <mass value="0.001"/>
+                <origin rpy="0 0 0" xyz="0 0 0"/>
+                <inertia ixx="0.0001" ixy="0" ixz="0" iyy="0.000001" iyz="0" izz="0.0001"/>
+            </inertial>
+            <visual>
+                <origin rpy="0 0 0" xyz="0 0 0"/>
+                <geometry>
+                    <box size="0.015 0.015 0.004"/>
+                </geometry>
+            </visual>
+            <material name="orange">
+                <color rgba="255 108 10 255"/>
+            </material>
+        </link>
+        <gazebo reference="${imu_link_name}">
+            <material>Gazebo/Orange</material>
+        </gazebo>
+        <gazebo reference="${imu_link_name}_joint">
+            <disableFixedJointLumping>true</disableFixedJointLumping>
+        </gazebo>
+        <xacro:if value="${simulation}">
+            <gazebo>
+                <plugin name="smb_imu_plugin" filename="libhector_gazebo_ros_imu.so">
+                    <updateRate>${imu_update_rate}</updateRate>
+                    <bodyName>${imu_link_name}</bodyName>
+                    <frameId>${imu_link_name}</frameId>
+                    <topicName>${imu_link_name}</topicName>
+                    <serviceName>${imu_calibration_service_name}</serviceName>
+                    <accelOffset>${acceleration_offset}</accelOffset>
+                    <accelDrift>${acceleration_drift}</accelDrift>
+                    <accelDriftFrequency>${acceleration_drift_frequency}</accelDriftFrequency>
+                    <accelGaussianNoise>${acceleration_gaussian_noise}</accelGaussianNoise>
+                    <rateOffset>${rate_offset}</rateOffset>
+                    <rateDrift>${rate_drift}</rateDrift>
+                    <rateDriftFrequency>${rate_drift_frequency}</rateDriftFrequency>
+                    <rateGaussianNoise>${rate_gaussian_noise}</rateGaussianNoise>
+                    <headingOffset>${heading_offset}</headingOffset>
+                    <headingDrift>${heading_drift}</headingDrift>
+                    <headingDriftFrequency>${heading_drift_frequency}</headingDriftFrequency>
+                    <headingGaussianNoise>${heading_gaussian_noise}</headingGaussianNoise>
+                </plugin>
+            </gazebo>
+        </xacro:if>
+    </xacro:macro>
 </robot>
