Commit message: Remove dark material

File: urdf/common/lidar2d.urdf.xacro (robot description, xacro)
@@ -22,5 +22,4 @@
                     <mesh filename="package://rm_description/meshes/common/lds.stl" scale="0.001 0.001 0.001"/>
                 </geometry>
-                <material name="dark"/>
             </visual>
             <collision>
