Commit message: Change name steering_wheel to swerve_drive

File: urdf/common/swerve_drive.xacro (robot description, xacro)
@@ -1,5 +1,5 @@
 <robot xmlns:xacro="http://www.ros.org/wiki/xacro">
-    <xacro:macro name="steering_wheel" params="xyz rpy parent">
-        <link name="steering_gear">
+    <xacro:macro name="swerve_drive" params="xyz rpy parent">
+        <link name="steering">
             <visual>
                 <origin xyz="0 0 0" rpy="0 0 0"/>
@@ -22,11 +22,11 @@
             </collision>
         </link>
-        <joint name="steering_gear_joint" type="continuous">
+        <joint name="steering_joint" type="continuous">
             <axis xyz="0 0 1"/>
             <origin xyz="${xyz}" rpy="${rpy}"/>
             <parent link="${parent}"/>
-            <child link="steering_gear"/>
+            <child link="steering"/>
         </joint>
-        <link name="steering_wheel">
+        <link name="wheel">
             <visual>
                 <origin xyz="0 0 0" rpy="0 0 0"/>
@@ -49,9 +49,9 @@
             </collision>
         </link>
-        <joint name="steering_wheel_joint" type="continuous">
+        <joint name="wheel_joint" type="continuous">
             <axis xyz="0 1 0"/>
             <origin xyz="0 -0.001 -0.094" rpy="0 0 0"/>
-            <parent link="steering_gear"/>
-            <child link="steering_wheel"/>
+            <parent link="steering"/>
+            <child link="wheel"/>
         </joint>
     </xacro:macro>

Commit message: Change name steering to pivot

File: urdf/common/swerve_drive.xacro (robot description, xacro)
@@ -1,9 +1,9 @@
 <robot xmlns:xacro="http://www.ros.org/wiki/xacro">
     <xacro:macro name="swerve_drive" params="xyz rpy parent">
-        <link name="steering">
+        <link name="pivot">
             <visual>
                 <origin xyz="0 0 0" rpy="0 0 0"/>
                 <geometry>
-                    <mesh filename="package://rm_description/meshes/common/steering.stl"
+                    <mesh filename="package://rm_description/meshes/common/swerve_pivot.stl"
                           scale="0.001 0.001 0.001"/>
                 </geometry>
@@ -17,14 +17,14 @@
                 <origin xyz="0 0 0" rpy="0 0 0"/>
                 <geometry>
-                    <mesh filename="package://rm_description/meshes/common/steering.stl"
+                    <mesh filename="package://rm_description/meshes/common/swerve_pivot.stl"
                           scale="0.001 0.001 0.001"/>
                 </geometry>
             </collision>
         </link>
-        <joint name="steering_joint" type="continuous">
+        <joint name="pivot_joint" type="continuous">
             <axis xyz="0 0 1"/>
             <origin xyz="${xyz}" rpy="${rpy}"/>
             <parent link="${parent}"/>
-            <child link="steering"/>
+            <child link="pivot"/>
         </joint>
         <link name="wheel">
@@ -32,5 +32,5 @@
                 <origin xyz="0 0 0" rpy="0 0 0"/>
                 <geometry>
-                    <mesh filename="package://rm_description/meshes/common/steering_wheel.stl"
+                    <mesh filename="package://rm_description/meshes/common/swerve_wheel.stl"
                           scale="0.001 0.001 0.001"/>
                 </geometry>
@@ -44,5 +44,5 @@
                 <origin xyz="0 0 0" rpy="0 0 0"/>
                 <geometry>
-                    <mesh filename="package://rm_description/meshes/common/steering_wheel.stl"
+                    <mesh filename="package://rm_description/meshes/common/swerve_wheel.stl"
                           scale="0.001 0.001 0.001"/>
                 </geometry>
@@ -52,5 +52,5 @@
             <axis xyz="0 1 0"/>
             <origin xyz="0 -0.001 -0.094" rpy="0 0 0"/>
-            <parent link="steering"/>
+            <parent link="pivot"/>
             <child link="wheel"/>
         </joint>
