Commit message: finish mecanum_wheel
Former-commit-id: 10a4c235a46e8b66270129343667b3cc14d14455

File: urdf/common/mecanum_wheel.urdf.xacro (robot description, xacro)
@@ -1,3 +1,3 @@
-<robot xmlns:xacro="http://www.ros.org/wiki/xacro">
+<robot xmlns:xacro="http://www.ros.org/wiki/xacro" name="test">
   <xacro:property name="wheel_radius" value="0.07625"/>
   <xacro:property name="M_PI" value="3.14159265359"/>
@@ -12,4 +12,8 @@
         </geometry>
       </visual>
+      <inertial>
+        <mass value="0.59"/>
+        <inertia ixx="1.416e-3" ixy="0.0" ixz="0.0" iyy="2.749e-3" iyz="0.0" izz="1.416e-3"/>
+      </inertial>
     </link>
     <link name="${prefix}_rotor">
@@ -19,4 +23,8 @@
         </geometry>
       </collision>
+      <inertial>
+        <mass value="0.036"/>
+        <inertia ixx="3128e-9" ixy="-1638.12e-9" ixz="0.0" iyy="3128e-9" iyz="0.0" izz="4766e-9"/>
+      </inertial>
     </link>
     <joint name="${prefix}_rotor_joint" type="continuous">
@@ -26,23 +34,3 @@
     </joint>
   </xacro:macro>
-  <!--  <xacro:mecanum_wheel prefix="test" reflect="1"/>-->
-  <link name="wheel">
-    <visual>
-      <geometry>
-        <mesh filename="package://rm_description/meshes/common/mecanum_wheel.stl"/>
-      </geometry>
-    </visual>
-    <collision>
-      <geometry>
-        <sphere radius="${wheel_radius}"/>
-      </geometry>
-    </collision>
-  </link>
-  <!--  <xacro:mecanum_wheel prefix="test" reflect="1"/>-->
-  <!-- Gazebo plugin for ROS Control -->
-  <gazebo>
-    <plugin name="gazebo_ros_control" filename="libgazebo_ros_control.so">
-      <robotNamespace>/</robotNamespace>
-    </plugin>
-  </gazebo>
 </robot>

Commit message: add wheel_joint to mecanum_wheel
Former-commit-id: 77edfbec2afa59e1b24d0166a654d22a07e7294b

File: urdf/common/mecanum_wheel.urdf.xacro (robot description, xacro)
@@ -1,6 +1,5 @@
-<robot xmlns:xacro="http://www.ros.org/wiki/xacro" name="test">
+<robot xmlns:xacro="http://www.ros.org/wiki/xacro">
   <xacro:property name="wheel_radius" value="0.07625"/>
-  <xacro:property name="M_PI" value="3.14159265359"/>
-  <xacro:macro name="mecanum_wheel" params="prefix reflect">
+  <xacro:macro name="mecanum_wheel" params="prefix parent wheel_x_offset wheel_y_offset wheel_z_offset reflect">
     <link name="${prefix}_wheel">
       <visual>
@@ -8,5 +7,5 @@
           <mesh filename="package://rm_description/meshes/common/mecanum_wheel.stl"/>
           <xacro:if value="${reflect == -1}">
-            <origin rpy="0 0 ${M_PI}"/>
+            <origin rpy="0 0 pi"/>
           </xacro:if>
         </geometry>
@@ -28,4 +27,10 @@
       </inertial>
     </link>
+    <joint name="${prefix}_wheel_joint" type="continuous">
+      <axis xyz="0 1 0"/>
+      <origin xyz="${wheel_x_offset} ${wheel_y_offset} ${wheel_offset_z}" rpy="0 0 0"/>
+      <parent link="${parent}"/>
+      <child link="${prefix}_wheel"/>
+    </joint>
     <joint name="${prefix}_rotor_joint" type="continuous">
       <axis xyz="${reflect * 0.70719678} ${reflect * 0.70719678} 0"/>

Commit message: fix wrong rotor joint direction
Former-commit-id: e31cf6998c6ba4eec11eccbf873bf0f265e36782

File: urdf/common/mecanum_wheel.urdf.xacro (robot description, xacro)
@@ -5,8 +5,8 @@
       <visual>
         <geometry>
+          <xacro:if value="${reflect == '-1'}">
+            <!--            //TODO: add right threaded wheel-->
+          </xacro:if>
           <mesh filename="package://rm_description/meshes/common/mecanum_wheel.stl"/>
-          <xacro:if value="${reflect == -1}">
-            <origin rpy="0 0 pi"/>
-          </xacro:if>
         </geometry>
       </visual>
@@ -30,9 +30,10 @@
       <axis xyz="0 1 0"/>
       <origin xyz="${wheel_x_offset} ${wheel_y_offset} ${wheel_offset_z}" rpy="0 0 0"/>
+      <dynamics damping="0.1" friction="0.1"/>
       <parent link="${parent}"/>
       <child link="${prefix}_wheel"/>
     </joint>
     <joint name="${prefix}_rotor_joint" type="continuous">
-      <axis xyz="${reflect * 0.70719678} ${reflect * 0.70719678} 0"/>
+      <axis xyz="${0.70719678} ${reflect * 0.70719678} 0"/>
       <parent link="${prefix}_wheel"/>
       <child link="${prefix}_rotor"/>

Commit message: add joint_state_controller replace mecanum_wheel.stl
Former-commit-id: 2be7c396ded3d800be63febd80b32e4783de2843

File: urdf/common/mecanum_wheel.urdf.xacro (robot description, xacro)
@@ -5,8 +5,12 @@
       <visual>
         <geometry>
-          <xacro:if value="${reflect == '-1'}">
-            <!--            //TODO: add right threaded wheel-->
+          <xacro:if value="${reflect == 1}">
+            <mesh filename="package://rm_description/meshes/common/left_threaded_mecanum_wheel.stl"
+                  scale="0.035 0.035 0.035"/>
           </xacro:if>
-          <mesh filename="package://rm_description/meshes/common/mecanum_wheel.stl"/>
+          <xacro:if value="${reflect == -1}">
+            <mesh filename="package://rm_description/meshes/common/right_threaded_mecanum_wheel.stl"
+                  scale="0.035 0.035 0.035"/>
+          </xacro:if>
         </geometry>
       </visual>
@@ -26,4 +30,8 @@
         <inertia ixx="3128e-9" ixy="-1638.12e-9" ixz="0.0" iyy="3128e-9" iyz="0.0" izz="4766e-9"/>
       </inertial>
+      <gazebo>
+        <mu1>0.8</mu1>
+        <mu2>0.8</mu2>
+      </gazebo>
     </link>
     <joint name="${prefix}_wheel_joint" type="continuous">

File: urdf/hero/base.urdf.xacro (robot description, xacro)
@@ -1,6 +1,4 @@
 <robot xmlns:xacro="http://www.ros.org/wiki/xacro">
   <xacro:include filename="$(find rm_description)/urdf/common/mecanum_wheel.urdf.xacro"/>
-  <!-- simplified box collision geometry for base -->
-  <xacro:property name="base_mass" value="10.0"/>
   <!-- https://upload.wikimedia.org/wikipedia/commons/5/52/Wheelbase_and_Track.png -->
   <xacro:property name="wheel_track" value="0.500"/>
@@ -11,8 +9,8 @@
   <link name="base_link">
     <inertial>
-      <mass value="${base_mass}"/>
+      <mass value="10"/>
       <origin xyz="0 0 0"/>
-      <inertia ixx="5.652232699207" ixy="-0.009719934438" ixz="1.293988226423" iyy="5.669473158652"
-               iyz="-0.007379583694" izz="3.683196351726"/>
+      <inertia ixx="1.013" ixy="1.818e-3" ixz="5.843e-2" iyy="1.516"
+               iyz="3.179e-2" izz="2.208"/>
     </inertial>
     <visual>
@@ -46,3 +44,9 @@
                        wheel_z_offset="${wheel_offset_z}"
                        reflect="-1"/>
+  <!-- Gazebo plugin for ROS Control -->
+  <gazebo>
+    <plugin name="gazebo_ros_control" filename="libgazebo_ros_control.so">
+      <robotNamespace>/</robotNamespace>
+    </plugin>
+  </gazebo>
 </robot>

Commit message: add transmission
Former-commit-id: 3a4a9d5370e74d26c414df794492c75a67dc6541

File: urdf/common/mecanum_wheel.urdf.xacro (robot description, xacro)
@@ -2,4 +2,5 @@
   <xacro:property name="wheel_radius" value="0.07625"/>
   <xacro:macro name="mecanum_wheel" params="prefix parent wheel_x_offset wheel_y_offset wheel_z_offset reflect">
+    <!--  link  -->
     <link name="${prefix}_wheel">
       <visual>
@@ -31,8 +32,9 @@
       </inertial>
       <gazebo>
-        <mu1>0.8</mu1>
-        <mu2>0.8</mu2>
+        <mu1>200</mu1>
+        <mu2>200</mu2>
       </gazebo>
     </link>
+    <!--  joint  -->
     <joint name="${prefix}_wheel_joint" type="continuous">
       <axis xyz="0 1 0"/>
@@ -47,4 +49,15 @@
       <child link="${prefix}_rotor"/>
     </joint>
+    <!-- transmission -->
+    <transmission name="${prefix}_wheel_trans">
+      <type>transmission_interface/SimpleTransmission</type>
+      <actuator name="${prefix}_wheel_actuator">
+        <hardwareInterface>hardware_interface/EffortJointInterface</hardwareInterface>
+        <mechanicalReduction>${reflect}</mechanicalReduction>
+      </actuator>
+      <joint name="${prefix}_wheel_joint">
+        <hardwareInterface>hardware_interface/EffortJointInterface</hardwareInterface>
+      </joint>
+    </transmission>
   </xacro:macro>
 </robot>

Commit message: add rotor
Former-commit-id: 5260af5f246e0cb8589a5b6245e31af731791e9a

File: urdf/common/mecanum_wheel.urdf.xacro (robot description, xacro)
@@ -1,28 +1,16 @@
 <robot xmlns:xacro="http://www.ros.org/wiki/xacro">
   <xacro:property name="wheel_radius" value="0.07625"/>
-  <xacro:macro name="mecanum_wheel" params="prefix parent wheel_x_offset wheel_y_offset wheel_z_offset reflect">
+  <xacro:property name="wheel_length" value="0.0269"/>
+  <xacro:property name="rotor_radius" value="0.006"/>
+  <xacro:macro name="rotor" params="prefix suffix theta">
     <!--  link  -->
-    <link name="${prefix}_wheel">
-      <visual>
+    <link name="${prefix}_rotor_${suffix}">
+      <collision>
+        <!--        <origin rpy="0 ${pi/2} ${-pi/4}"/>-->
+        <!--        <geometry>-->
+        <!--          <cylinder radius="${rotor_radius}" length="${wheel_length}"/>-->
+        <!--        </geometry>-->
         <geometry>
-          <xacro:if value="${reflect == 1}">
-            <mesh filename="package://rm_description/meshes/common/left_threaded_mecanum_wheel.stl"
-                  scale="0.035 0.035 0.035"/>
-          </xacro:if>
-          <xacro:if value="${reflect == -1}">
-            <mesh filename="package://rm_description/meshes/common/right_threaded_mecanum_wheel.stl"
-                  scale="0.035 0.035 0.035"/>
-          </xacro:if>
-        </geometry>
-      </visual>
-      <inertial>
-        <mass value="0.59"/>
-        <inertia ixx="1.416e-3" ixy="0.0" ixz="0.0" iyy="2.749e-3" iyz="0.0" izz="1.416e-3"/>
-      </inertial>
-    </link>
-    <link name="${prefix}_rotor">
-      <collision>
-        <geometry>
-          <sphere radius="${wheel_radius}"/>
+          <sphere radius="${rotor_radius}"/>
         </geometry>
       </collision>
@@ -36,4 +24,33 @@
       </gazebo>
     </link>
+    <joint name="${prefix}_rotor_${suffix}_joint" type="continuous">
+      <origin
+          xyz="${(wheel_radius-rotor_radius)*cos(theta-pi/2) * 0.70719678} 0 ${(wheel_radius-rotor_radius)*sin(theta-pi/2) * 0.70719678}"
+          rpy="0 0 0"/>
+      <axis xyz="${cos(theta) * 0.70719678} ${- reflect * 0.70719678} ${sin(theta) * 0.70719678}"/>
+      <parent link="${prefix}_wheel"/>
+      <child link="${prefix}_rotor_${suffix}"/>
+    </joint>
+  </xacro:macro>
+  <xacro:macro name="mecanum_wheel" params="prefix parent wheel_x_offset wheel_y_offset wheel_z_offset reflect">
+    <!--  link  -->
+    <link name="${prefix}_wheel">
+      <visual>
+        <geometry>
+          <xacro:if value="${reflect == 1}">
+            <mesh filename="package://rm_description/meshes/common/right_threaded_mecanum_wheel.stl"
+                  scale="0.035 0.035 0.035"/>
+          </xacro:if>
+          <xacro:if value="${reflect == -1}">
+            <mesh filename="package://rm_description/meshes/common/left_threaded_mecanum_wheel.stl"
+                  scale="0.035 0.035 0.035"/>
+          </xacro:if>
+        </geometry>
+      </visual>
+      <inertial>
+        <mass value="0.59"/>
+        <inertia ixx="1.416e-3" ixy="0.0" ixz="0.0" iyy="2.749e-3" iyz="0.0" izz="1.416e-3"/>
+      </inertial>
+    </link>
     <!--  joint  -->
     <joint name="${prefix}_wheel_joint" type="continuous">
@@ -44,9 +61,21 @@
       <child link="${prefix}_wheel"/>
     </joint>
-    <joint name="${prefix}_rotor_joint" type="continuous">
-      <axis xyz="${0.70719678} ${reflect * 0.70719678} 0"/>
-      <parent link="${prefix}_wheel"/>
-      <child link="${prefix}_rotor"/>
-    </joint>
+    <!-- rotor -->
+    <xacro:rotor prefix="${prefix}" suffix="0" theta="${0*0.393}"/>
+    <xacro:rotor prefix="${prefix}" suffix="1" theta="${1*0.393}"/>
+    <xacro:rotor prefix="${prefix}" suffix="2" theta="${2*0.393}"/>
+    <xacro:rotor prefix="${prefix}" suffix="3" theta="${3*0.393}"/>
+    <xacro:rotor prefix="${prefix}" suffix="4" theta="${4*0.393}"/>
+    <xacro:rotor prefix="${prefix}" suffix="5" theta="${5*0.393}"/>
+    <xacro:rotor prefix="${prefix}" suffix="6" theta="${6*0.393}"/>
+    <xacro:rotor prefix="${prefix}" suffix="7" theta="${7*0.393}"/>
+    <xacro:rotor prefix="${prefix}" suffix="8" theta="${8*0.393}"/>
+    <xacro:rotor prefix="${prefix}" suffix="9" theta="${9*0.393}"/>
+    <xacro:rotor prefix="${prefix}" suffix="10" theta="${10*0.393}"/>
+    <xacro:rotor prefix="${prefix}" suffix="11" theta="${11*0.393}"/>
+    <xacro:rotor prefix="${prefix}" suffix="12" theta="${12*0.393}"/>
+    <xacro:rotor prefix="${prefix}" suffix="13" theta="${13*0.393}"/>
+    <xacro:rotor prefix="${prefix}" suffix="14" theta="${14*0.393}"/>
+    <xacro:rotor prefix="${prefix}" suffix="15" theta="${15*0.393}"/>
     <!-- transmission -->
     <transmission name="${prefix}_wheel_trans">

File: urdf/hero/base.urdf.xacro (robot description, xacro)
@@ -29,9 +29,9 @@
   </link>
   <xacro:mecanum_wheel prefix="front_left" parent="base_link"
-                       wheel_x_offset="${wheel_track/2}" wheel_y_offset="${-wheel_base/2}"
+                       wheel_x_offset="${wheel_track/2}" wheel_y_offset="${wheel_base/2}"
                        wheel_z_offset="${wheel_offset_z}"
                        reflect="1"/>
   <xacro:mecanum_wheel prefix="front_right" parent="base_link"
-                       wheel_x_offset="${wheel_track/2}" wheel_y_offset="${wheel_base/2}"
+                       wheel_x_offset="${wheel_track/2}" wheel_y_offset="${-wheel_base/2}"
                        wheel_z_offset="${wheel_offset_z}"
                        reflect="-1"/>

Commit message: try rotor.stl
Former-commit-id: 7d31594b5eb59f80fe03518afccfac34707ae3fc

File: urdf/common/mecanum_wheel.urdf.xacro (robot description, xacro)
@@ -2,12 +2,13 @@
   <xacro:property name="wheel_radius" value="0.07625"/>
   <xacro:property name="wheel_length" value="0.0269"/>
-  <xacro:property name="rotor_radius" value="0.006"/>
+  <xacro:property name="rotor_radius" value="0.008"/>
   <xacro:macro name="rotor" params="prefix suffix theta">
     <!--  link  -->
     <link name="${prefix}_rotor_${suffix}">
       <collision>
-        <!--        <origin rpy="0 ${pi/2} ${-pi/4}"/>-->
+        <!--  still has wrong ration of rotor-->
         <!--        <geometry>-->
-        <!--          <cylinder radius="${rotor_radius}" length="${wheel_length}"/>-->
+        <!--          <mesh filename="package://rm_description/meshes/common/rotor.stl"-->
+        <!--                scale="0.001 0.001 0.001"/>-->
         <!--        </geometry>-->
         <geometry>
@@ -40,9 +41,9 @@
           <xacro:if value="${reflect == 1}">
             <mesh filename="package://rm_description/meshes/common/right_threaded_mecanum_wheel.stl"
-                  scale="0.035 0.035 0.035"/>
+                  scale="0.001 0.001 0.001"/>
           </xacro:if>
           <xacro:if value="${reflect == -1}">
             <mesh filename="package://rm_description/meshes/common/left_threaded_mecanum_wheel.stl"
-                  scale="0.035 0.035 0.035"/>
+                  scale="0.001 0.001 0.001"/>
           </xacro:if>
         </geometry>
@@ -61,5 +62,5 @@
       <child link="${prefix}_wheel"/>
     </joint>
-    <!-- rotor -->
+    <!-- 16 rotor  2pi/16=0.393-->
     <xacro:rotor prefix="${prefix}" suffix="0" theta="${0*0.393}"/>
     <xacro:rotor prefix="${prefix}" suffix="1" theta="${1*0.393}"/>

File: urdf/hero/base.urdf.xacro (robot description, xacro)
@@ -39,9 +39,9 @@
                        wheel_x_offset="${-wheel_track/2}" wheel_y_offset="${wheel_base/2}"
                        wheel_z_offset="${wheel_offset_z}"
-                       reflect="1"/>
+                       reflect="-1"/>
   <xacro:mecanum_wheel prefix="back_right" parent="base_link"
                        wheel_x_offset="${-wheel_track/2}" wheel_y_offset="${-wheel_base/2}"
                        wheel_z_offset="${wheel_offset_z}"
-                       reflect="-1"/>
+                       reflect="1"/>
   <!-- Gazebo plugin for ROS Control -->
   <gazebo>

Commit message: add material of rotors
Former-commit-id: 06cf6172fd02f8ac7aaf692e3cfdc036520a4f4f

File: urdf/common/mecanum_wheel.urdf.xacro (robot description, xacro)
@@ -1,6 +1,7 @@
 <robot xmlns:xacro="http://www.ros.org/wiki/xacro">
   <xacro:property name="wheel_radius" value="0.07625"/>
-  <xacro:property name="wheel_length" value="0.0269"/>
   <xacro:property name="rotor_radius" value="0.008"/>
+  <xacro:property name="wheel_joint_effort" value="0.1"/>
+  <xacro:property name="wheel_joint_velocity" value="100"/>
   <xacro:macro name="rotor" params="prefix suffix theta">
     <!--  link  -->
@@ -18,14 +19,10 @@
       <inertial>
         <mass value="0.036"/>
-        <inertia ixx="3128e-9" ixy="-1638.12e-9" ixz="0.0" iyy="3128e-9" iyz="0.0" izz="4766e-9"/>
+        <inertia ixx="3128e-9" ixy="0.0" ixz="0.0" iyy="3128e-9" iyz="0.0" izz="3128e-9"/>
       </inertial>
-      <gazebo>
-        <mu1>200</mu1>
-        <mu2>200</mu2>
-      </gazebo>
     </link>
     <joint name="${prefix}_rotor_${suffix}_joint" type="continuous">
       <origin
-          xyz="${(wheel_radius-rotor_radius)*cos(theta-pi/2) * 0.70719678} 0 ${(wheel_radius-rotor_radius)*sin(theta-pi/2) * 0.70719678}"
+          xyz="${(wheel_radius-rotor_radius)*cos(theta-pi/2)} 0 ${(wheel_radius-rotor_radius)*sin(theta-pi/2)}"
           rpy="0 0 0"/>
       <axis xyz="${cos(theta) * 0.70719678} ${- reflect * 0.70719678} ${sin(theta) * 0.70719678}"/>
@@ -33,4 +30,11 @@
       <child link="${prefix}_rotor_${suffix}"/>
     </joint>
+    <gazebo reference="${prefix}_rotor_${suffix}">
+      <mu1 value="2000.0"/>
+      <mu2 value="2000.0"/>
+      <kp value="1000000.0"/>
+      <kd value="100.0"/>
+      <material>Gazebo/Black</material>
+    </gazebo>
   </xacro:macro>
   <xacro:macro name="mecanum_wheel" params="prefix parent wheel_x_offset wheel_y_offset wheel_z_offset reflect">
@@ -58,5 +62,5 @@
       <axis xyz="0 1 0"/>
       <origin xyz="${wheel_x_offset} ${wheel_y_offset} ${wheel_offset_z}" rpy="0 0 0"/>
-      <dynamics damping="0.1" friction="0.1"/>
+      <limit effort="${wheel_joint_effort}" velocity="${wheel_joint_velocity}"/>
       <parent link="${parent}"/>
       <child link="${prefix}_wheel"/>
@@ -84,5 +88,5 @@
       <actuator name="${prefix}_wheel_actuator">
         <hardwareInterface>hardware_interface/EffortJointInterface</hardwareInterface>
-        <mechanicalReduction>${reflect}</mechanicalReduction>
+        <mechanicalReduction>1</mechanicalReduction>
       </actuator>
       <joint name="${prefix}_wheel_joint">

File: urdf/hero/base.urdf.xacro (robot description, xacro)
@@ -22,8 +22,8 @@
     </visual>
     <collision>
-      <origin xyz="0 0 0" rpy="0 0 0"/>
-      <geometry>
-        <mesh filename="package://rm_description/meshes/hero/base.stl" scale="0.001 0.001 0.001"/>
-      </geometry>
+      <!--      <origin xyz="0 0 0" rpy="0 0 0"/>-->
+      <!--      <geometry>-->
+      <!--        <mesh filename="package://rm_description/meshes/hero/base.stl" scale="0.001 0.001 0.001"/>-->
+      <!--      </geometry>-->
     </collision>
   </link>

Commit message: add effort, velocity limit and friction for wheel joint
Former-commit-id: ec6eefa794102240dda0eba6e960c5cc3c909ad2

File: urdf/common/mecanum_wheel.urdf.xacro (robot description, xacro)
@@ -2,6 +2,6 @@
   <xacro:property name="wheel_radius" value="0.07625"/>
   <xacro:property name="rotor_radius" value="0.008"/>
-  <xacro:property name="wheel_joint_effort" value="0.1"/>
-  <xacro:property name="wheel_joint_velocity" value="100"/>
+  <xacro:property name="wheel_joint_effort" value="5"/>
+  <xacro:property name="wheel_joint_velocity" value="50"/>
   <xacro:macro name="rotor" params="prefix suffix theta">
     <!--  link  -->
@@ -59,8 +59,10 @@
     </link>
     <!--  joint  -->
-    <joint name="${prefix}_wheel_joint" type="continuous">
+    <joint name="${prefix}_wheel_joint" type="revolute">
       <axis xyz="0 1 0"/>
       <origin xyz="${wheel_x_offset} ${wheel_y_offset} ${wheel_offset_z}" rpy="0 0 0"/>
-      <limit effort="${wheel_joint_effort}" velocity="${wheel_joint_velocity}"/>
+      <!--      limit not work while type="continuous"-->
+      <limit effort="${wheel_joint_effort}" velocity="${wheel_joint_velocity}" lower="-1e16" upper="1e16"/>
+      <dynamics damping="0.0" friction="0.05"/>
       <parent link="${parent}"/>
       <child link="${prefix}_wheel"/>
