Commit message: Try roller.stl (rotor.stl)
Former-commit-id: 8b1576c86ea8b0673a3e057f03236e21112bc787

File: urdf/common/mecanum_wheel.urdf.xacro (robot description, xacro)
@@ -1,18 +1,26 @@
 <robot xmlns:xacro="http://www.ros.org/wiki/xacro">
   <xacro:property name="wheel_radius" value="0.07625"/>
-  <xacro:property name="rotor_radius" value="0.008"/>
+  <xacro:property name="roller_radius" value="0.008"/>
   <xacro:property name="wheel_joint_effort" value="5"/>
   <xacro:property name="wheel_joint_velocity" value="50"/>
-  <xacro:macro name="rotor" params="prefix suffix theta">
+  <xacro:macro name="roller" params="prefix suffix theta">
+    <!-- rotation math: roller_joint_axis -->
+    <xacro:property name="sqrt_2_2" value="${sqrt(2)/2}"/>
+    <xacro:property name="roller_joint_axis_x" value="${cos(theta) * sqrt_2_2}"/>
+    <xacro:property name="roller_joint_axis_y" value="${-reflect * sqrt_2_2}"/>
+    <xacro:property name="roller_joint_axis_z" value="${sin(theta) * sqrt_2_2}"/>
+    <!-- rotation math: get quaternion between x_axis (1,0,0) and roller_joint_axis
+    https://stackoverflow.com/questions/1171849/finding-quaternion-representing-the-rotation-from-one-vector-to-another -->
+    <xacro:property name="quaternion_x" value="${0}"/>
+    <xacro:property name="quaternion_y" value="${roller_joint_axis_z}"/>
+    <xacro:property name="quaternion_z" value="${-roller_joint_axis_y}"/>
+    <xacro:property name="quaternion_w" value="${1+roller_joint_axis_x}"/>
     <!--  link  -->
-    <link name="${prefix}_rotor_${suffix}">
+    <link name="${prefix}_roller_${suffix}">
       <collision>
-        <!--  still has wrong ration of rotor-->
-        <!--        <geometry>-->
-        <!--          <mesh filename="package://rm_description/meshes/common/rotor.stl"-->
-        <!--                scale="0.001 0.001 0.001"/>-->
-        <!--        </geometry>-->
+        <origin
+            xyz="0 0 0" quat_xyzw="quaternion_x quaternion_y quaternion_z quaternion_w"/>
         <geometry>
-          <sphere radius="${rotor_radius}"/>
+          <mesh filename="package://rm_description/meshes/common/roller.stl" scale="0.001 0.001 0.001"/>
         </geometry>
       </collision>
@@ -22,13 +30,13 @@
       </inertial>
     </link>
-    <joint name="${prefix}_rotor_${suffix}_joint" type="continuous">
+    <joint name="${prefix}_roller_${suffix}_joint" type="continuous">
       <origin
-          xyz="${(wheel_radius-rotor_radius)*cos(theta-pi/2)} 0 ${(wheel_radius-rotor_radius)*sin(theta-pi/2)}"
+          xyz="${(wheel_radius-roller_radius)*cos(theta-pi/2)} 0 ${(wheel_radius-roller_radius)*sin(theta-pi/2)}"
           rpy="0 0 0"/>
-      <axis xyz="${cos(theta) * 0.70719678} ${- reflect * 0.70719678} ${sin(theta) * 0.70719678}"/>
+      <axis xyz="${roller_joint_axis_x} ${roller_joint_axis_y} ${roller_joint_axis_z}"/>
       <parent link="${prefix}_wheel"/>
-      <child link="${prefix}_rotor_${suffix}"/>
+      <child link="${prefix}_roller_${suffix}"/>
     </joint>
-    <gazebo reference="${prefix}_rotor_${suffix}">
+    <gazebo reference="${prefix}_roller_${suffix}">
       <mu1 value="2000.0"/>
       <mu2 value="2000.0"/>
@@ -68,21 +76,21 @@
       <child link="${prefix}_wheel"/>
     </joint>
-    <!-- 16 rotor  2pi/16=0.393-->
-    <xacro:rotor prefix="${prefix}" suffix="0" theta="${0*0.393}"/>
-    <xacro:rotor prefix="${prefix}" suffix="1" theta="${1*0.393}"/>
-    <xacro:rotor prefix="${prefix}" suffix="2" theta="${2*0.393}"/>
-    <xacro:rotor prefix="${prefix}" suffix="3" theta="${3*0.393}"/>
-    <xacro:rotor prefix="${prefix}" suffix="4" theta="${4*0.393}"/>
-    <xacro:rotor prefix="${prefix}" suffix="5" theta="${5*0.393}"/>
-    <xacro:rotor prefix="${prefix}" suffix="6" theta="${6*0.393}"/>
-    <xacro:rotor prefix="${prefix}" suffix="7" theta="${7*0.393}"/>
-    <xacro:rotor prefix="${prefix}" suffix="8" theta="${8*0.393}"/>
-    <xacro:rotor prefix="${prefix}" suffix="9" theta="${9*0.393}"/>
-    <xacro:rotor prefix="${prefix}" suffix="10" theta="${10*0.393}"/>
-    <xacro:rotor prefix="${prefix}" suffix="11" theta="${11*0.393}"/>
-    <xacro:rotor prefix="${prefix}" suffix="12" theta="${12*0.393}"/>
-    <xacro:rotor prefix="${prefix}" suffix="13" theta="${13*0.393}"/>
-    <xacro:rotor prefix="${prefix}" suffix="14" theta="${14*0.393}"/>
-    <xacro:rotor prefix="${prefix}" suffix="15" theta="${15*0.393}"/>
+    <!-- 16 roller  2pi/16=0.393-->
+    <xacro:roller prefix="${prefix}" suffix="0" theta="${0*0.393}"/>
+    <xacro:roller prefix="${prefix}" suffix="1" theta="${1*0.393}"/>
+    <xacro:roller prefix="${prefix}" suffix="2" theta="${2*0.393}"/>
+    <xacro:roller prefix="${prefix}" suffix="3" theta="${3*0.393}"/>
+    <xacro:roller prefix="${prefix}" suffix="4" theta="${4*0.393}"/>
+    <xacro:roller prefix="${prefix}" suffix="5" theta="${5*0.393}"/>
+    <xacro:roller prefix="${prefix}" suffix="6" theta="${6*0.393}"/>
+    <xacro:roller prefix="${prefix}" suffix="7" theta="${7*0.393}"/>
+    <xacro:roller prefix="${prefix}" suffix="8" theta="${8*0.393}"/>
+    <xacro:roller prefix="${prefix}" suffix="9" theta="${9*0.393}"/>
+    <xacro:roller prefix="${prefix}" suffix="10" theta="${10*0.393}"/>
+    <xacro:roller prefix="${prefix}" suffix="11" theta="${11*0.393}"/>
+    <xacro:roller prefix="${prefix}" suffix="12" theta="${12*0.393}"/>
+    <xacro:roller prefix="${prefix}" suffix="13" theta="${13*0.393}"/>
+    <xacro:roller prefix="${prefix}" suffix="14" theta="${14*0.393}"/>
+    <xacro:roller prefix="${prefix}" suffix="15" theta="${15*0.393}"/>
     <!-- transmission -->
     <transmission name="${prefix}_wheel_trans">

Commit message: Get quaternion but quat_xyzw dosen't work, try convert to rpy
Former-commit-id: e4c589a0f4805d5e29cb7e1a7f81570d5902a003

File: urdf/common/mecanum_wheel.urdf.xacro (robot description, xacro)
@@ -19,6 +19,30 @@
     <link name="${prefix}_roller_${suffix}">
       <collision>
-        <origin
-            xyz="0 0 0" quat_xyzw="quaternion_x quaternion_y quaternion_z quaternion_w"/>
+        <!--  quat_xyzw dosen't work ?! covert to rpy-->
+        <xacro:property name="t" value="${2. * (quaternion_w * quaternion_y - quaternion_z * quaternion_x)}"/>
+        <xacro:if value="${t > 1}">
+          <origin rpy="${atan2(2. * (quaternion_w * quaternion_x + quaternion_y * quaternion_z),
+                              1. - 2. * (quaternion_x * quaternion_x + quaternion_y * quaternion_y))}
+                     ${asin(1)}
+                     ${atan2(2. * (quaternion_w * quaternion_z + quaternion_x * quaternion_y),
+                              1. - 2. * (quaternion_y * quaternion_y + quaternion_z * quaternion_z))}"
+                  xyz="0 0 0"/>
+        </xacro:if>
+        <xacro:if value="${-1 > t}">
+          <origin rpy="${atan2(2. * (quaternion_w * quaternion_x + quaternion_y * quaternion_z),
+                              1. - 2. * (quaternion_x * quaternion_x + quaternion_y * quaternion_y))}
+                     ${asin(-1)}
+                     ${atan2(2. * (quaternion_w * quaternion_z + quaternion_x * quaternion_y),
+                              1. - 2. * (quaternion_y * quaternion_y + quaternion_z * quaternion_z))}"
+                  xyz="0 0 0"/>
+        </xacro:if>
+        <xacro:if value="${t > -1 and 1 > t}">
+          <origin rpy="${atan2(2. * (quaternion_w * quaternion_x + quaternion_y * quaternion_z),
+                              1. - 2. * (quaternion_x * quaternion_x + quaternion_y * quaternion_y))}
+                     ${asin(t)}
+                     ${atan2(2. * (quaternion_w * quaternion_z + quaternion_x * quaternion_y),
+                              1. - 2. * (quaternion_y * quaternion_y + quaternion_z * quaternion_z))}"
+                  xyz="0 0 0"/>
+        </xacro:if>
         <geometry>
           <mesh filename="package://rm_description/meshes/common/roller.stl" scale="0.001 0.001 0.001"/>

Commit message: Use roller.stl successfully
Former-commit-id: 2d3721d1e978263eeb0c06b352e098f27d1bb67c

File: urdf/common/mecanum_wheel.urdf.xacro (robot description, xacro)
@@ -1,5 +1,5 @@
 <robot xmlns:xacro="http://www.ros.org/wiki/xacro">
   <xacro:property name="wheel_radius" value="0.07625"/>
-  <xacro:property name="roller_radius" value="0.008"/>
+  <xacro:property name="roller_radius" value="0.009"/>
   <xacro:property name="wheel_joint_effort" value="5"/>
   <xacro:property name="wheel_joint_velocity" value="50"/>
@@ -12,37 +12,23 @@
     <!-- rotation math: get quaternion between x_axis (1,0,0) and roller_joint_axis
     https://stackoverflow.com/questions/1171849/finding-quaternion-representing-the-rotation-from-one-vector-to-another -->
-    <xacro:property name="quaternion_x" value="${0}"/>
-    <xacro:property name="quaternion_y" value="${roller_joint_axis_z}"/>
-    <xacro:property name="quaternion_z" value="${-roller_joint_axis_y}"/>
-    <xacro:property name="quaternion_w" value="${1+roller_joint_axis_x}"/>
+    <xacro:property name="quat_x" value="${0}"/>
+    <xacro:property name="quat_y" value="${roller_joint_axis_z}"/>
+    <xacro:property name="quat_z" value="${-roller_joint_axis_y}"/>
+    <xacro:property name="quat_w" value="${-(1+roller_joint_axis_x)}"/>
+    <xacro:property name="quat_length" value="${sqrt(quat_y*quat_y + quat_z * quat_z+quat_w * quat_w)}"/>
+    <xacro:property name="quat_normal_x" value="${0}"/>
+    <xacro:property name="quat_normal_y" value="${quat_y/quat_length}"/>
+    <xacro:property name="quat_normal_z" value="${quat_z/quat_length}"/>
+    <xacro:property name="quat_normal_w" value="${quat_w/quat_length}"/>
     <!--  link  -->
     <link name="${prefix}_roller_${suffix}">
       <collision>
         <!--  quat_xyzw dosen't work ?! covert to rpy-->
-        <xacro:property name="t" value="${2. * (quaternion_w * quaternion_y - quaternion_z * quaternion_x)}"/>
-        <xacro:if value="${t > 1}">
-          <origin rpy="${atan2(2. * (quaternion_w * quaternion_x + quaternion_y * quaternion_z),
-                              1. - 2. * (quaternion_x * quaternion_x + quaternion_y * quaternion_y))}
-                     ${asin(1)}
-                     ${atan2(2. * (quaternion_w * quaternion_z + quaternion_x * quaternion_y),
-                              1. - 2. * (quaternion_y * quaternion_y + quaternion_z * quaternion_z))}"
-                  xyz="0 0 0"/>
-        </xacro:if>
-        <xacro:if value="${-1 > t}">
-          <origin rpy="${atan2(2. * (quaternion_w * quaternion_x + quaternion_y * quaternion_z),
-                              1. - 2. * (quaternion_x * quaternion_x + quaternion_y * quaternion_y))}
-                     ${asin(-1)}
-                     ${atan2(2. * (quaternion_w * quaternion_z + quaternion_x * quaternion_y),
-                              1. - 2. * (quaternion_y * quaternion_y + quaternion_z * quaternion_z))}"
-                  xyz="0 0 0"/>
-        </xacro:if>
-        <xacro:if value="${t > -1 and 1 > t}">
-          <origin rpy="${atan2(2. * (quaternion_w * quaternion_x + quaternion_y * quaternion_z),
-                              1. - 2. * (quaternion_x * quaternion_x + quaternion_y * quaternion_y))}
-                     ${asin(t)}
-                     ${atan2(2. * (quaternion_w * quaternion_z + quaternion_x * quaternion_y),
-                              1. - 2. * (quaternion_y * quaternion_y + quaternion_z * quaternion_z))}"
-                  xyz="0 0 0"/>
-        </xacro:if>
+        <origin rpy="${atan2(2. * (quat_normal_w * quat_normal_x + quat_normal_y * quat_normal_z),
+                              1. - 2. * (quat_normal_x * quat_normal_x + quat_normal_y * quat_normal_y))}
+                     ${asin(2. * (quat_normal_w * quat_normal_y - quat_normal_z * quat_normal_x))}
+                     ${atan2(2. * (quat_normal_w * quat_normal_z + quat_normal_x * quat_normal_y),
+                              1. - 2. * (quat_normal_y * quat_normal_y + quat_normal_z * quat_normal_z))}"
+                xyz="0 0 0"/>
         <geometry>
           <mesh filename="package://rm_description/meshes/common/roller.stl" scale="0.001 0.001 0.001"/>
@@ -59,4 +45,5 @@
           rpy="0 0 0"/>
       <axis xyz="${roller_joint_axis_x} ${roller_joint_axis_y} ${roller_joint_axis_z}"/>
+      <dynamics damping="0.0" friction="0.001"/>
       <parent link="${prefix}_wheel"/>
       <child link="${prefix}_roller_${suffix}"/>

Commit message: Add roller_type

File: urdf/common/mecanum_wheel.urdf.xacro (robot description, xacro)
@@ -4,5 +4,5 @@
   <xacro:property name="wheel_joint_effort" value="5"/>
   <xacro:property name="wheel_joint_velocity" value="50"/>
-  <xacro:macro name="roller" params="prefix suffix theta">
+  <xacro:macro name="roller" params="prefix suffix theta roller_type">
     <!-- rotation math: roller_joint_axis -->
     <xacro:property name="sqrt_2_2" value="${sqrt(2)/2}"/>
@@ -24,14 +24,21 @@
     <link name="${prefix}_roller_${suffix}">
       <collision>
-        <!--  quat_xyzw dosen't work ?! covert to rpy-->
-        <origin rpy="${atan2(2. * (quat_normal_w * quat_normal_x + quat_normal_y * quat_normal_z),
+        <xacro:if value="${roller_type=='realistic'}">
+          <!--  quat_xyzw dosen't work ?! covert to rpy-->
+          <origin rpy="${atan2(2. * (quat_normal_w * quat_normal_x + quat_normal_y * quat_normal_z),
                               1. - 2. * (quat_normal_x * quat_normal_x + quat_normal_y * quat_normal_y))}
                      ${asin(2. * (quat_normal_w * quat_normal_y - quat_normal_z * quat_normal_x))}
                      ${atan2(2. * (quat_normal_w * quat_normal_z + quat_normal_x * quat_normal_y),
                               1. - 2. * (quat_normal_y * quat_normal_y + quat_normal_z * quat_normal_z))}"
-                xyz="0 0 0"/>
-        <geometry>
-          <mesh filename="package://rm_description/meshes/common/roller.stl" scale="0.001 0.001 0.001"/>
-        </geometry>
+                  xyz="0 0 0"/>
+          <geometry>
+            <mesh filename="package://rm_description/meshes/common/roller.stl" scale="0.001 0.001 0.001"/>
+          </geometry>
+        </xacro:if>
+        <xacro:if value="${roller_type=='simple'}">
+          <geometry>
+            <sphere radius="${roller_radius}"/>
+          </geometry>
+        </xacro:if>
       </collision>
       <inertial>
@@ -57,5 +64,6 @@
     </gazebo>
   </xacro:macro>
-  <xacro:macro name="mecanum_wheel" params="prefix parent wheel_x_offset wheel_y_offset wheel_z_offset reflect">
+  <xacro:macro name="mecanum_wheel"
+               params="prefix connected_to wheel_x_offset wheel_y_offset wheel_z_offset reflect roller_type">
     <!--  link  -->
     <link name="${prefix}_wheel">
@@ -84,24 +92,26 @@
       <limit effort="${wheel_joint_effort}" velocity="${wheel_joint_velocity}" lower="-1e16" upper="1e16"/>
       <dynamics damping="0.0" friction="0.05"/>
-      <parent link="${parent}"/>
+      <parent link="${connected_to}"/>
       <child link="${prefix}_wheel"/>
     </joint>
-    <!-- 16 roller  2pi/16=0.393-->
-    <xacro:roller prefix="${prefix}" suffix="0" theta="${0*0.393}"/>
-    <xacro:roller prefix="${prefix}" suffix="1" theta="${1*0.393}"/>
-    <xacro:roller prefix="${prefix}" suffix="2" theta="${2*0.393}"/>
-    <xacro:roller prefix="${prefix}" suffix="3" theta="${3*0.393}"/>
-    <xacro:roller prefix="${prefix}" suffix="4" theta="${4*0.393}"/>
-    <xacro:roller prefix="${prefix}" suffix="5" theta="${5*0.393}"/>
-    <xacro:roller prefix="${prefix}" suffix="6" theta="${6*0.393}"/>
-    <xacro:roller prefix="${prefix}" suffix="7" theta="${7*0.393}"/>
-    <xacro:roller prefix="${prefix}" suffix="8" theta="${8*0.393}"/>
-    <xacro:roller prefix="${prefix}" suffix="9" theta="${9*0.393}"/>
-    <xacro:roller prefix="${prefix}" suffix="10" theta="${10*0.393}"/>
-    <xacro:roller prefix="${prefix}" suffix="11" theta="${11*0.393}"/>
-    <xacro:roller prefix="${prefix}" suffix="12" theta="${12*0.393}"/>
-    <xacro:roller prefix="${prefix}" suffix="13" theta="${13*0.393}"/>
-    <xacro:roller prefix="${prefix}" suffix="14" theta="${14*0.393}"/>
-    <xacro:roller prefix="${prefix}" suffix="15" theta="${15*0.393}"/>
+    <xacro:unless value="${roller_type=='none'}">
+      <!-- 16 roller  2pi/16=0.393-->
+      <xacro:roller prefix="${prefix}" suffix="0" theta="${0*0.393}" roller_type="${roller_type}"/>
+      <xacro:roller prefix="${prefix}" suffix="1" theta="${1*0.393}" roller_type="${roller_type}"/>
+      <xacro:roller prefix="${prefix}" suffix="2" theta="${2*0.393}" roller_type="${roller_type}"/>
+      <xacro:roller prefix="${prefix}" suffix="3" theta="${3*0.393}" roller_type="${roller_type}"/>
+      <xacro:roller prefix="${prefix}" suffix="4" theta="${4*0.393}" roller_type="${roller_type}"/>
+      <xacro:roller prefix="${prefix}" suffix="5" theta="${5*0.393}" roller_type="${roller_type}"/>
+      <xacro:roller prefix="${prefix}" suffix="6" theta="${6*0.393}" roller_type="${roller_type}"/>
+      <xacro:roller prefix="${prefix}" suffix="7" theta="${7*0.393}" roller_type="${roller_type}"/>
+      <xacro:roller prefix="${prefix}" suffix="8" theta="${8*0.393}" roller_type="${roller_type}"/>
+      <xacro:roller prefix="${prefix}" suffix="9" theta="${9*0.393}" roller_type="${roller_type}"/>
+      <xacro:roller prefix="${prefix}" suffix="10" theta="${10*0.393}" roller_type="${roller_type}"/>
+      <xacro:roller prefix="${prefix}" suffix="11" theta="${11*0.393}" roller_type="${roller_type}"/>
+      <xacro:roller prefix="${prefix}" suffix="12" theta="${12*0.393}" roller_type="${roller_type}"/>
+      <xacro:roller prefix="${prefix}" suffix="13" theta="${13*0.393}" roller_type="${roller_type}"/>
+      <xacro:roller prefix="${prefix}" suffix="14" theta="${14*0.393}" roller_type="${roller_type}"/>
+      <xacro:roller prefix="${prefix}" suffix="15" theta="${15*0.393}" roller_type="${roller_type}"/>
+    </xacro:unless>
     <!-- transmission -->
     <transmission name="${prefix}_wheel_trans">

Commit message: Update transmission

File: urdf/common/mecanum_wheel.urdf.xacro (robot description, xacro)
@@ -114,10 +114,11 @@
       <xacro:roller prefix="${prefix}" suffix="15" theta="${15*0.393}" roller_type="${roller_type}"/>
     </xacro:unless>
-    <!-- transmission -->
+  </xacro:macro>
+  <xacro:macro name="wheel_transmission" params="prefix mechanical_reduction">
     <transmission name="${prefix}_wheel_trans">
       <type>transmission_interface/SimpleTransmission</type>
       <actuator name="${prefix}_wheel_motor">
         <hardwareInterface>hardware_interface/EffortJointInterface</hardwareInterface>
-        <mechanicalReduction>1</mechanicalReduction>
+        <mechanicalReduction>${mechanical_reduction}</mechanicalReduction>
       </actuator>
       <joint name="${prefix}_wheel_joint">

File: urdf/infantry/chassis.urdf.xacro (robot description, xacro)
@@ -44,4 +44,8 @@
                          wheel_z_offset="${wheel_offset_z}"
                          reflect="1" roller_type="${roller_type}"/>
+    <xacro:wheel_transmission prefix="front_left" mechanical_reduction="1"/>
+    <xacro:wheel_transmission prefix="front_right" mechanical_reduction="-1"/>
+    <xacro:wheel_transmission prefix="back_left" mechanical_reduction="1"/>
+    <xacro:wheel_transmission prefix="back_right" mechanical_reduction="-1"/>
   </xacro:macro>
 </robot>
