Commit message: Change name of sentry

File: urdf/common/mecanum_wheel.urdf.xacro (robot description, xacro)
@@ -90,5 +90,5 @@
             <origin xyz="${wheel_x_offset} ${wheel_y_offset} ${wheel_offset_z}" rpy="0 0 0"/>
             <!--      limit not work while type="continuous"-->
-            <limit effort="${wheel_joint_effort}" velocity="${wheel_joint_velocity}" lower="-1e16" upper="1e16"/>
+            <limit effort="${wheel_joint_effort}" velocity="${wheel_joint_velocity}" lower="-1e9" upper="1e9"/>
             <dynamics damping="0.0" friction="0.05"/>
             <parent link="${connected_to}"/>

File: urdf/sentry/chassis.transmission.urdf.xacro (robot description, xacro)
@@ -1,10 +1,10 @@
 <?xml version="1.0" encoding="utf-8"?>
 <robot>
-    <transmission name="trans_drive_joint">
+    <transmission name="trans_drive_wheel_joint">
         <type>transmission_interface/SimpleTransmission</type>
         <actuator name="drive_joint_motor">
             <mechanicalReduction>19.2032</mechanicalReduction>
         </actuator>
-        <joint name="drive_joint">
+        <joint name="drive_wheel_joint">
             <hardwareInterface>hardware_interface/EffortJointInterface</hardwareInterface>
         </joint>

File: urdf/sentry/chassis.urdf.xacro (robot description, xacro)
@@ -1,79 +1,79 @@
 <robot xmlns:xacro="http://www.ros.org/wiki/xacro">
-  <xacro:include filename="$(find rm_description)/urdf/sentry/driven_wheel.urdf.xacro"/>
-  <xacro:macro name="chassis" params="use_simulation">
-    <link name="base_link">
-      <inertial>
-        <mass value="8.250"/>
-        <origin xyz="0.0 0.051 -0.148"/>
-        <inertia ixx="3.838e-1" ixy="1.075e-2" ixz="1.397e-5" iyy="2.601e-1"
-                 iyz="7.528e-2" izz="2.369e-1"/>
-      </inertial>
-      <visual>
-        <origin xyz="0 0 0" rpy="0 0 0"/>
-        <geometry>
-          <mesh filename="package://rm_description/meshes/sentry/base_link.stl" scale="0.001 0.001 0.001"/>
-        </geometry>
-      </visual>
-      <collision>
-        <origin xyz="0 0 0" rpy="0 0 0"/>
-        <geometry>
-          <mesh filename="package://rm_description/meshes/sentry/base_link.stl" scale="0.001 0.001 0.001"/>
-        </geometry>
-      </collision>
-    </link>
-    <link name="link_drive_wheel">
-      <inertial>
-        <mass value="0.0839"/>
-        <origin xyz="0 0.01 0"/>
-        <inertia ixx="3.345e-5" ixy="0" ixz="0" iyy="-8.387e-5"
-                 iyz="-2.8558e-8" izz="3.347e-5"/>
-      </inertial>
-      <visual>
-        <origin xyz="0 0 0" rpy="0 0 0"/>
-        <geometry>
-          <mesh filename="package://rm_description/meshes/sentry/drive_wheel.stl" scale="0.001 0.001 0.001"/>
-        </geometry>
-      </visual>
-      <collision>
-        <origin xyz="0 0 0" rpy="0 0 0"/>
-        <geometry>
-          <mesh filename="package://rm_description/meshes/sentry/drive_wheel.stl" scale="0.001 0.001 0.001"/>
-        </geometry>
-      </collision>
-    </link>
-    <joint name="drive_joint" type="continuous">
-      <axis xyz="0 1 0"/>
-      <limit effort="1.2" velocity="34" lower="-${2*pi}" upper="${2*pi}"/>
-      <parent link="base_link"/>
-      <child link="link_drive_wheel"/>
-      <origin xyz="0 -0.0185 0" rpy="0 0 0"/>
-    </joint>
-    <xacro:if value="$(arg use_simulation)">
-      <xacro:driven_wheel num="1">
-        <origin rpy="${-pi/2} 0 0"/>
-        <axis xyz="0 1 0"/>
-        <origin xyz="-0.0977 0.0839 -0.013" rpy="0 0 0"/>
-      </xacro:driven_wheel>
-      <xacro:driven_wheel num="2">
-        <origin rpy="${-pi/2} 0 0"/>
-        <axis xyz="0 1 0"/>
-        <origin xyz="0.0977 0.0839 -0.013" rpy="0 0 0"/>
-      </xacro:driven_wheel>
-      <xacro:driven_wheel num="3">
-        <origin rpy="0 0 0"/>
-        <axis xyz="0 0 1"/>
-        <origin xyz="-0.0982 0.135 -0.0571" rpy="0 0 0"/>
-      </xacro:driven_wheel>
-      <xacro:driven_wheel num="4">
-        <origin rpy="0 0 0"/>
-        <axis xyz="0 0 1"/>
-        <origin xyz="0.0982 0.135 -0.0571" rpy="0 0 0"/>
-      </xacro:driven_wheel>
-      <xacro:driven_wheel num="5">
-        <origin rpy="0 0 0"/>
-        <axis xyz="0 0 1"/>
-        <origin xyz="0 -0.073 -0.0572" rpy="0 0 0"/>
-      </xacro:driven_wheel>
-    </xacro:if>
-  </xacro:macro>
+    <xacro:include filename="$(find rm_description)/urdf/sentry/driven_wheel.urdf.xacro"/>
+    <xacro:macro name="chassis" params="use_simulation">
+        <link name="base_link">
+            <inertial>
+                <mass value="8.250"/>
+                <origin xyz="0.0 0.051 -0.148"/>
+                <inertia ixx="3.838e-1" ixy="1.075e-2" ixz="1.397e-5" iyy="2.601e-1"
+                         iyz="7.528e-2" izz="2.369e-1"/>
+            </inertial>
+            <visual>
+                <origin xyz="0 0 0" rpy="0 0 0"/>
+                <geometry>
+                    <mesh filename="package://rm_description/meshes/sentry/base_link.stl" scale="0.001 0.001 0.001"/>
+                </geometry>
+            </visual>
+            <collision>
+                <origin xyz="0 0 0" rpy="0 0 0"/>
+                <geometry>
+                    <mesh filename="package://rm_description/meshes/sentry/base_link.stl" scale="0.001 0.001 0.001"/>
+                </geometry>
+            </collision>
+        </link>
+        <link name="drive_wheel_link">
+            <inertial>
+                <mass value="0.0839"/>
+                <origin xyz="0 0.01 0"/>
+                <inertia ixx="3.345e-5" ixy="0" ixz="0" iyy="-8.387e-5"
+                         iyz="-2.8558e-8" izz="3.347e-5"/>
+            </inertial>
+            <visual>
+                <origin xyz="0 0 0" rpy="0 0 0"/>
+                <geometry>
+                    <mesh filename="package://rm_description/meshes/sentry/drive_wheel.stl" scale="0.001 0.001 0.001"/>
+                </geometry>
+            </visual>
+            <collision>
+                <origin xyz="0 0 0" rpy="0 0 0"/>
+                <geometry>
+                    <mesh filename="package://rm_description/meshes/sentry/drive_wheel.stl" scale="0.001 0.001 0.001"/>
+                </geometry>
+            </collision>
+        </link>
+        <joint name="drive_wheel_joint" type="revolute">
+            <axis xyz="0 1 0"/>
+            <limit effort="1.2" velocity="34" lower="-1e9" upper="1e9"/>
+            <parent link="base_link"/>
+            <child link="drive_wheel_link"/>
+            <origin xyz="0 -0.0185 0" rpy="0 0 0"/>
+        </joint>
+        <xacro:if value="$(arg use_simulation)">
+            <xacro:driven_wheel num="1">
+                <origin rpy="${-pi/2} 0 0"/>
+                <axis xyz="0 1 0"/>
+                <origin xyz="-0.0977 0.0839 -0.013" rpy="0 0 0"/>
+            </xacro:driven_wheel>
+            <xacro:driven_wheel num="2">
+                <origin rpy="${-pi/2} 0 0"/>
+                <axis xyz="0 1 0"/>
+                <origin xyz="0.0977 0.0839 -0.013" rpy="0 0 0"/>
+            </xacro:driven_wheel>
+            <xacro:driven_wheel num="3">
+                <origin rpy="0 0 0"/>
+                <axis xyz="0 0 1"/>
+                <origin xyz="-0.0982 0.135 -0.0571" rpy="0 0 0"/>
+            </xacro:driven_wheel>
+            <xacro:driven_wheel num="4">
+                <origin rpy="0 0 0"/>
+                <axis xyz="0 0 1"/>
+                <origin xyz="0.0982 0.135 -0.0571" rpy="0 0 0"/>
+            </xacro:driven_wheel>
+            <xacro:driven_wheel num="5">
+                <origin rpy="0 0 0"/>
+                <axis xyz="0 0 1"/>
+                <origin xyz="0 -0.073 -0.0572" rpy="0 0 0"/>
+            </xacro:driven_wheel>
+        </xacro:if>
+    </xacro:macro>
 </robot>

Commit message: update

File: urdf/common/mecanum_wheel.urdf.xacro (robot description, xacro)
@@ -2,6 +2,6 @@
     <xacro:property name="wheel_radius" value="0.07625"/>
     <xacro:property name="roller_radius" value="0.009"/>
-    <xacro:property name="wheel_joint_effort" value="5"/>
-    <xacro:property name="wheel_joint_velocity" value="50"/>
+    <xacro:property name="wheel_joint_effort" value="10"/>
+    <xacro:property name="wheel_joint_velocity" value="70"/>
     <xacro:macro name="roller" params="prefix suffix theta roller_type">
         <!-- rotation math: roller_joint_axis -->
