Commit message: fix swerve stl error

File: urdf/common/swerve_drive.urdf.xacro (robot description, xacro)
@@ -1,5 +1,5 @@
 <robot xmlns:xacro="http://www.ros.org/wiki/xacro">
-    <xacro:macro name="swerve_drive" params="xyz rpy parent">
-        <link name="pivot">
+    <xacro:macro name="swerve_drive" params="prefix wheel_x_offset wheel_y_offset wheel_z_offset  connected_to">
+        <link name="${prefix}_pivot">
             <visual>
                 <origin xyz="0 0 0" rpy="0 0 0"/>
@@ -22,11 +22,11 @@
             </collision>
         </link>
-        <joint name="pivot_joint" type="continuous">
+        <joint name="${prefix}_pivot_joint" type="continuous">
             <axis xyz="0 0 1"/>
-            <origin xyz="${xyz}" rpy="${rpy}"/>
-            <parent link="${parent}"/>
-            <child link="pivot"/>
+            <origin xyz="${wheel_x_offset} ${wheel_y_offset} ${wheel_z_offset}" rpy="0 0 0"/>
+            <parent link="${connected_to}"/>
+            <child link="${prefix}_pivot"/>
         </joint>
-        <link name="wheel">
+        <link name="${prefix}_wheel">
             <visual>
                 <origin xyz="0 0 0" rpy="0 0 0"/>
@@ -49,9 +49,9 @@
             </collision>
         </link>
-        <joint name="wheel_joint" type="continuous">
+        <joint name="${prefix}_wheel_joint" type="continuous">
             <axis xyz="0 1 0"/>
             <origin xyz="0 -0.001 -0.094" rpy="0 0 0"/>
-            <parent link="pivot"/>
-            <child link="wheel"/>
+            <parent link="${prefix}_pivot"/>
+            <child link="${prefix}_wheel"/>
         </joint>
     </xacro:macro>

File: urdf/hero/hero.urdf.xacro (robot description, xacro)
@@ -10,8 +10,4 @@
     <xacro:chassis roller_type="$(arg roller_type)"/>
   </xacro:if>
-  <!--  <xacro:if value="$(arg load_shooter)">-->
-  <!--    <xacro:include filename="$(find rm_description)/urdf/sentry/shooter.urdf.xacro"/>-->
-  <!--    <xacro:include filename="$(find rm_description)/urdf/sentry/shooter.transmission.urdf.xacro"/>-->
-  <!--  </xacro:if>-->
   <xacro:if value="$(arg load_gimbal)">
     <xacro:include filename="$(find rm_description)/urdf/hero/gimbal.urdf.xacro"/>

Commit message: add swerve

File: urdf/common/swerve_drive.urdf.xacro (robot description, xacro)
@@ -56,3 +56,15 @@
         </joint>
     </xacro:macro>
+    <xacro:macro name="wheel_transmission" params="prefix swerve_reduction">
+        <transmission name="${prefix}_wheel_trans">
+            <type>transmission_interface/SimpleTransmission</type>
+            <actuator name="${prefix}_wheel_motor">
+                <hardwareInterface>hardware_interface/EffortJointInterface</hardwareInterface>
+                <mechanicalReduction>${mechanical_reduction}</mechanicalReduction>
+            </actuator>
+            <joint name="${prefix}_wheel_joint">
+                <hardwareInterface>hardware_interface/EffortJointInterface</hardwareInterface>
+            </joint>
+        </transmission>
+    </xacro:macro>
 </robot>

Commit message: Fix lots of stupid error about swerve

File: urdf/common/swerve_drive.urdf.xacro (robot description, xacro)
@@ -60,6 +60,5 @@
             <type>transmission_interface/SimpleTransmission</type>
             <actuator name="${prefix}_wheel_motor">
-                <hardwareInterface>hardware_interface/EffortJointInterface</hardwareInterface>
-                <mechanicalReduction>${mechanical_reduction}</mechanicalReduction>
+                <mechanicalReduction>${swerve_reduction}</mechanicalReduction>
             </actuator>
             <joint name="${prefix}_wheel_joint">

File: urdf/swerve/chassis.urdf.xacro (robot description, xacro)
@@ -7,39 +7,41 @@
     <xacro:property name="wheel_joint_damping" value="1.0"/>
     <xacro:property name="wheel_joint_friction" value="1.0"/>
-    <link name="base_link">
-        <inertial>
-            <mass value="19.31"/>
-            <origin xyz="-0.02282 0.002773 0.008173"/>
-            <inertia ixx="4.041e-1" ixy="7.617e-3" ixz="-1.317e-2" iyy="3.322e-1"
-                     iyz="7.985e-2" izz="1.8e-1"/>
-        </inertial>
-        <visual>
-            <origin xyz="0 0 0" rpy="0 0 0"/>
-            <geometry>
-                <mesh filename="package://rm_description/meshes/hero/base.stl" scale="0.001 .001 0.001"/>
-            </geometry>
-        </visual>
-        <collision>
-            <origin xyz="0 0 0" rpy="0 0 0"/>
-            <geometry>
-                <mesh filename="package://rm_description/meshes/hero/base.stl" scale="0.001 0.001 0.001"/>
-            </geometry>
-        </collision>
-    </link>
-    <xacro:swerve_drive prefix="left_front" connected_to="base_link"
-                        wheel_x_offset="${wheel_track/2}" wheel_y_offset="${wheel_base/2}"
-                        wheel_z_offset="${wheel_offset_z}"/>
-    <xacro:swerve_drive prefix="right_front" connected_to="base_link"
-                        wheel_x_offset="${wheel_track/2}" wheel_y_offset="${-wheel_base/2}"
-                        wheel_z_offset="${wheel_offset_z}"/>
-    <xacro:swerve_drive prefix="left_back" connected_to="base_link"
-                        wheel_x_offset="${-wheel_track/2}" wheel_y_offset="${wheel_base/2}"
-                        wheel_z_offset="${wheel_offset_z}"/>
-    <xacro:swerve_drive prefix="right_back" connected_to="base_link"
-                        wheel_x_offset="${-wheel_track/2}" wheel_y_offset="${-wheel_base/2}"
-                        wheel_z_offset="${wheel_offset_z}"/>
-            <xacro:wheel_transmission prefix="left_front" swerve_reduction="1"/>
-            <xacro:wheel_transmission prefix="right_front" swerve_reduction="-1"/>
-            <xacro:wheel_transmission prefix="left_back" swerve_reduction="1"/>
-            <xacro:wheel_transmission prefix="right_back" swerve_reduction="-1"/>
+    <xacro:macro name="chassis">
+        <link name="base_link">
+            <inertial>
+                <mass value="19.31"/>
+                <origin xyz="-0.02282 0.002773 0.008173"/>
+                <inertia ixx="4.041e-1" ixy="7.617e-3" ixz="-1.317e-2" iyy="3.322e-1"
+                         iyz="7.985e-2" izz="1.8e-1"/>
+            </inertial>
+            <visual>
+                <origin xyz="0 0 0" rpy="0 0 0"/>
+                <geometry>
+                    <mesh filename="package://rm_description/meshes/hero/base.stl" scale="0.001 .001 0.001"/>
+                </geometry>
+            </visual>
+            <collision>
+                <origin xyz="0 0 0" rpy="0 0 0"/>
+                <geometry>
+                    <mesh filename="package://rm_description/meshes/hero/base.stl" scale="0.001 0.001 0.001"/>
+                </geometry>
+            </collision>
+        </link>
+        <xacro:swerve_drive prefix="left_front" connected_to="base_link"
+                            wheel_x_offset="${wheel_track/2}" wheel_y_offset="${wheel_base/2}"
+                            wheel_z_offset="${wheel_offset_z}"/>
+        <xacro:swerve_drive prefix="right_front" connected_to="base_link"
+                            wheel_x_offset="${wheel_track/2}" wheel_y_offset="${-wheel_base/2}"
+                            wheel_z_offset="${wheel_offset_z}"/>
+        <xacro:swerve_drive prefix="left_back" connected_to="base_link"
+                            wheel_x_offset="${-wheel_track/2}" wheel_y_offset="${wheel_base/2}"
+                            wheel_z_offset="${wheel_offset_z}"/>
+        <xacro:swerve_drive prefix="right_back" connected_to="base_link"
+                            wheel_x_offset="${-wheel_track/2}" wheel_y_offset="${-wheel_base/2}"
+                            wheel_z_offset="${wheel_offset_z}"/>
+        <xacro:wheel_transmission prefix="left_front" swerve_reduction="1"/>
+        <xacro:wheel_transmission prefix="right_front" swerve_reduction="-1"/>
+        <xacro:wheel_transmission prefix="left_back" swerve_reduction="1"/>
+        <xacro:wheel_transmission prefix="right_back" swerve_reduction="-1"/>
+    </xacro:macro>
 </robot>

File: urdf/swerve/swerve.urdf.xacro (robot description, xacro)
@@ -2,23 +2,9 @@
 <robot xmlns:xacro="http://www.ros.org/wiki/xacro" name="swerve">
     <xacro:arg name="load_chassis" default="true"/>
-    <!--    <xacro:arg name="load_gimbal" default="true"/>-->
-    <!--    <xacro:arg name="load_shooter" default="true"/>-->
     <xacro:arg name="use_simulation" default="true"/>
-    <xacro:arg name="roller_type" default="realistic"/>
     <xacro:if value="$(arg load_chassis)">
         <xacro:include filename="$(find rm_description)/urdf/swerve/chassis.urdf.xacro"/>
-        <xacro:chassis roller_type="$(arg roller_type)"/>
+        <xacro:chassis/>
     </xacro:if>
-    <!--    <xacro:if value="$(arg load_gimbal)">-->
-    <!--        <xacro:include filename="$(find rm_description)/urdf/swerve/gimbal.urdf.xacro"/>-->
-    <!--        <xacro:include filename="$(find rm_description)/urdf/swerve/gimbal.transmission.urdf.xacro"/>-->
-    <!--        <xacro:include filename="$(find rm_description)/urdf/common/camera.urdf.xacro"/>-->
-    <!--        <xacro:camera_sensor xyz="0.127 0 -0.047" rpy="0 0 0" parent="pitch"-->
-    <!--                             camera_sim="$(arg use_simulation)"></xacro:camera_sensor>-->
-    <!--    </xacro:if>-->
-    <!--    <xacro:if value="$(arg load_shooter)">-->
-    <!--        <xacro:include filename="$(find rm_description)/urdf/hero/shooter.urdf.xacro"/>-->
-    <!--        &lt;!&ndash;    <xacro:include filename="$(find rm_description)/urdf/hero/shooter.transmission.urdf.xacro"/>&ndash;&gt;-->
-    <!--    </xacro:if>-->
     <xacro:if value="$(arg use_simulation)">
         <gazebo>

Commit message: Add pivot transmission

File: urdf/common/swerve_drive.urdf.xacro (robot description, xacro)
@@ -56,9 +56,18 @@
         </joint>
     </xacro:macro>
-    <xacro:macro name="wheel_transmission" params="prefix swerve_reduction">
+    <xacro:macro name="swerve_transmission" params="prefix wheel_reduction">
+        <transmission name="${prefix}_pivot_trans">
+            <type>transmission_interface/SimpleTransmission</type>
+            <actuator name="${prefix}_pivot_motor">
+                <mechanicalReduction>1</mechanicalReduction>
+            </actuator>
+            <joint name="${prefix}_pivot_joint">
+                <hardwareInterface>hardware_interface/EffortJointInterface</hardwareInterface>
+            </joint>
+        </transmission>
         <transmission name="${prefix}_wheel_trans">
             <type>transmission_interface/SimpleTransmission</type>
             <actuator name="${prefix}_wheel_motor">
-                <mechanicalReduction>${swerve_reduction}</mechanicalReduction>
+                <mechanicalReduction>${wheel_reduction}</mechanicalReduction>
             </actuator>
             <joint name="${prefix}_wheel_joint">

File: urdf/swerve/chassis.urdf.xacro (robot description, xacro)
@@ -38,8 +38,8 @@
                             wheel_x_offset="${-wheel_track/2}" wheel_y_offset="${-wheel_base/2}"
                             wheel_z_offset="${wheel_offset_z}"/>
-        <xacro:wheel_transmission prefix="left_front" swerve_reduction="1"/>
-        <xacro:wheel_transmission prefix="right_front" swerve_reduction="-1"/>
-        <xacro:wheel_transmission prefix="left_back" swerve_reduction="1"/>
-        <xacro:wheel_transmission prefix="right_back" swerve_reduction="-1"/>
+        <xacro:swerve_transmission prefix="left_front" wheel_reduction="1"/>
+        <xacro:swerve_transmission prefix="right_front" wheel_reduction="-1"/>
+        <xacro:swerve_transmission prefix="left_back" wheel_reduction="1"/>
+        <xacro:swerve_transmission prefix="right_back" wheel_reduction="-1"/>
     </xacro:macro>
 </robot>

Commit message: Change joint_handles_ from std::vector<hardware_interface::JointHandle *> to  std::vector<hardware_interface::JointHandle>

File: urdf/common/swerve_drive.urdf.xacro (robot description, xacro)
@@ -27,4 +27,6 @@
             <parent link="${connected_to}"/>
             <child link="${prefix}_pivot"/>
+            <dynamics damping="0.0" friction="0.1"/>
+            <limit effort="1.2" velocity="31" lower="-1e10" upper="1e10"/>
         </joint>
         <link name="${prefix}_wheel">
@@ -54,5 +56,14 @@
             <parent link="${prefix}_pivot"/>
             <child link="${prefix}_wheel"/>
+            <limit effort="3.0" velocity="50.0" lower="-1e10" upper="1e10"/>
+            <dynamics damping="0.0" friction="0.05"/>
         </joint>
+        <gazebo reference="${prefix}_wheel">
+            <mu1 value="2000.0"/>
+            <mu2 value="2000.0"/>
+            <kp value="1000000.0"/>
+            <kd value="100.0"/>
+            <material>Gazebo/Black</material>
+        </gazebo>
     </xacro:macro>
     <xacro:macro name="swerve_transmission" params="prefix wheel_reduction">

Commit message: Change collision of wheel to cylinder

File: urdf/common/swerve_drive.urdf.xacro (robot description, xacro)
@@ -44,8 +44,7 @@
             </inertial>
             <collision>
-                <origin xyz="0 0 0" rpy="0 0 0"/>
+                <origin xyz="0 0 0" rpy="${pi/2.} 0 0"/>
                 <geometry>
-                    <mesh filename="package://rm_description/meshes/common/swerve_wheel.stl"
-                          scale="0.001 0.001 0.001"/>
+                    <cylinder radius="0.055" length="0.04"/>
                 </geometry>
             </collision>

File: urdf/swerve/chassis.urdf.xacro (robot description, xacro)
@@ -2,6 +2,6 @@
     <xacro:include filename="$(find rm_description)/urdf/common/swerve_drive.urdf.xacro"/>
     <!-- https://upload.wikimedia.org/wikipedia/commons/5/52/Wheelbase_and_Track.png -->
-    <xacro:property name="wheel_track" value="0.500"/>
-    <xacro:property name="wheel_base" value="0.475"/>
+    <xacro:property name="wheel_track" value="0.4"/>
+    <xacro:property name="wheel_base" value="0.4"/>
     <xacro:property name="wheel_offset_z" value="-0.036"/>
     <xacro:macro name="chassis">

Commit message: Fix strange performance cause by lagre fiction

File: urdf/common/swerve_drive.urdf.xacro (robot description, xacro)
@@ -46,5 +46,5 @@
                 <origin xyz="0 0 0" rpy="${pi/2.} 0 0"/>
                 <geometry>
-                    <cylinder radius="0.055" length="0.04"/>
+                    <cylinder radius="0.055" length="0.001"/>
                 </geometry>
             </collision>
@@ -59,6 +59,6 @@
         </joint>
         <gazebo reference="${prefix}_wheel">
-            <mu1 value="2000.0"/>
-            <mu2 value="2000.0"/>
+            <mu1 value="20"/>
+            <mu2 value="20"/>
             <kp value="1000000.0"/>
             <kd value="100.0"/>

Commit message: Add pivot_offset in swerve_transmission

File: urdf/common/swerve_drive.urdf.xacro (robot description, xacro)
@@ -66,11 +66,12 @@
         </gazebo>
     </xacro:macro>
-    <xacro:macro name="swerve_transmission" params="prefix wheel_reduction">
+    <xacro:macro name="swerve_transmission" params="prefix wheel_reduction  pivot_offset">
         <transmission name="${prefix}_pivot_trans">
             <type>transmission_interface/SimpleTransmission</type>
             <actuator name="${prefix}_pivot_motor">
-                <mechanicalReduction>1</mechanicalReduction>
+                <mechanicalReduction>-1</mechanicalReduction>
             </actuator>
             <joint name="${prefix}_pivot_joint">
+                <offset>${pivot_offset}</offset>
                 <hardwareInterface>hardware_interface/EffortJointInterface</hardwareInterface>
             </joint>

File: urdf/swerve/chassis.urdf.xacro (robot description, xacro)
@@ -38,8 +38,8 @@
                             wheel_x_offset="${-wheel_track/2}" wheel_y_offset="${-wheel_base/2}"
                             wheel_z_offset="${wheel_offset_z}"/>
-        <xacro:swerve_transmission prefix="left_front" wheel_reduction="1"/>
-        <xacro:swerve_transmission prefix="right_front" wheel_reduction="-1"/>
-        <xacro:swerve_transmission prefix="left_back" wheel_reduction="1"/>
-        <xacro:swerve_transmission prefix="right_back" wheel_reduction="-1"/>
+        <xacro:swerve_transmission prefix="left_front" wheel_reduction="1" pivot_offset="2.3585"/>
+        <xacro:swerve_transmission prefix="right_front" wheel_reduction="-1" pivot_offset="2.332"/>
+        <xacro:swerve_transmission prefix="left_back" wheel_reduction="1" pivot_offset="3.911"/>
+        <xacro:swerve_transmission prefix="right_back" wheel_reduction="-1" pivot_offset="6.272"/>
     </xacro:macro>
 </robot>

Commit message: Change limit of swerve_drive

File: urdf/common/swerve_drive.urdf.xacro (robot description, xacro)
@@ -55,5 +55,5 @@
             <parent link="${prefix}_pivot"/>
             <child link="${prefix}_wheel"/>
-            <limit effort="3.0" velocity="50.0" lower="-1e10" upper="1e10"/>
+            <limit effort="2.2" velocity="68" lower="-1e10" upper="1e10"/>
             <dynamics damping="0.0" friction="0.05"/>
         </joint>
