Commit message: modify urdf of standard4

File: urdf/common/swerve_drive.urdf.xacro (robot description, xacro)
@@ -1,22 +1,44 @@
 <robot xmlns:xacro="http://www.ros.org/wiki/xacro">
-    <xacro:macro name="swerve_drive" params="prefix wheel_x_offset wheel_y_offset wheel_z_offset  connected_to">
+    <xacro:macro name="swerve_drive"
+                 params="prefix wheel_x_offset wheel_y_offset wheel_z_offset  connected_to reflect mirror">
         <link name="${prefix}_pivot">
             <visual>
                 <origin xyz="0 0 0" rpy="0 0 0"/>
                 <geometry>
-                    <mesh filename="package://rm_description/meshes/common/swerve_pivot.stl"
-                          scale="0.001 0.001 0.001"/>
+                    <xacro:if value="${reflect == 1}">
+                        <mesh filename="package://rm_description/meshes/common/right_front_swerve_pivot.stl"
+                              scale="0.001 0.001 0.001"/>
+                    </xacro:if>
+                    <xacro:if value="${reflect == -1}">
+                        <mesh filename="package://rm_description/meshes/common/left_front_swerve_pivot.stl"
+                              scale="0.001 0.001 0.001"/>
+                    </xacro:if>
                 </geometry>
             </visual>
             <inertial>
-                <mass value="2.819"/>
-                <origin xyz="0. 0.0 0.004" rpy="0 0 0"/>
-                <inertia ixx="3.904e-3" ixy="3.689e-6" ixz="-9.096e-6" iyy="3.847e-3" iyz="-9.129e-5" izz="1.952e-3"/>
+                <xacro:if value="${reflect == 1}">
+                    <mass value="3.725118"/>
+                    <origin xyz="0.951e-3 5.254e-3 -23.161e-3" rpy="0 0 0"/>
+                    <inertia ixx="1.645e-2" ixy="-13783.466e-9" ixz="2.345e-4" iyy="1.562e-2" iyz="2.132e-3"
+                             izz="3.256e-3"/>
+                </xacro:if>
+                <xacro:if value="${reflect == -1}">
+                    <mass value="3.725115"/>
+                    <origin xyz="0.156793 0.150588 0.030271" rpy="0 0 0"/>
+                    <inertia ixx="1.143e-1" ixy="-9.835e-2" ixz="-2.178e-2" iyy="1.207e-1" iyz="-2.289e-2"
+                             izz="2e-1"/>
+                </xacro:if>
             </inertial>
             <collision>
                 <origin xyz="0 0 0" rpy="0 0 0"/>
                 <geometry>
-                    <mesh filename="package://rm_description/meshes/common/swerve_pivot.stl"
-                          scale="0.001 0.001 0.001"/>
+                    <xacro:if value="${reflect == 1}">
+                        <mesh filename="package://rm_description/meshes/common/right_front_swerve_pivot.stl"
+                              scale="0.001 0.001 0.001"/>
+                    </xacro:if>
+                    <xacro:if value="${reflect == -1}">
+                        <mesh filename="package://rm_description/meshes/common/left_front_swerve_pivot.stl"
+                              scale="0.001 0.001 0.001"/>
+                    </xacro:if>
                 </geometry>
             </collision>
@@ -24,5 +46,10 @@
         <joint name="${prefix}_pivot_joint" type="continuous">
             <axis xyz="0 0 1"/>
-            <origin xyz="${wheel_x_offset} ${wheel_y_offset} ${wheel_z_offset}" rpy="0 0 0"/>
+            <xacro:if value="${mirror == 1}">
+                <origin xyz="${wheel_x_offset} ${wheel_y_offset} ${wheel_z_offset}" rpy="0 0 0"/>
+            </xacro:if>
+            <xacro:if value="${mirror == -1}">
+                <origin xyz="${wheel_x_offset} ${wheel_y_offset} ${wheel_z_offset}" rpy="0 0 ${pi}"/>
+            </xacro:if>
             <parent link="${connected_to}"/>
             <child link="${prefix}_pivot"/>
@@ -32,5 +59,5 @@
         <link name="${prefix}_wheel">
             <visual>
-                <origin xyz="0 0 0" rpy="0 0 0"/>
+                <origin xyz="0 0.0265 0" rpy="0 0 0"/>
                 <geometry>
                     <mesh filename="package://rm_description/meshes/common/swerve_wheel.stl"
@@ -39,12 +66,12 @@
             </visual>
             <inertial>
-                <mass value="0.213"/>
-                <origin xyz="0 -0.007 0.0" rpy="0 0 0"/>
-                <inertia ixx="2.012e-4" ixy="0" ixz="0" iyy="2.618e-4" iyz="8.07e-7" izz="2.002e-4"/>
+                <mass value="0.18791"/>
+                <origin xyz="6.908e-8 -7.298e-3 275e-6" rpy="0 0 0"/>
+                <inertia ixx="1.584e-4" ixy="0.199e-9" ixz="-0.173e-9" iyy="2.141e-4" iyz="768.622e-9" izz="1.575e-4"/>
             </inertial>
             <collision>
                 <origin xyz="0 0 0" rpy="${pi/2.} 0 0"/>
                 <geometry>
-                    <cylinder radius="0.055" length="0.001"/>
+                    <cylinder radius="0.05" length="0.053"/>
                 </geometry>
             </collision>
@@ -52,5 +79,5 @@
         <joint name="${prefix}_wheel_joint" type="continuous">
             <axis xyz="0 1 0"/>
-            <origin xyz="0 -0.001 -0.094" rpy="0 0 0"/>
+            <origin xyz="0 0 -0.112" rpy="0 0 0"/>
             <parent link="${prefix}_pivot"/>
             <child link="${prefix}_wheel"/>

File: urdf/standard4/chassis.urdf.xacro (robot description, xacro)
@@ -2,19 +2,20 @@
     <xacro:include filename="$(find rm_description)/urdf/common/swerve_drive.urdf.xacro"/>
     <!-- https://upload.wikimedia.org/wikipedia/commons/5/52/Wheelbase_and_Track.png -->
-    <xacro:property name="wheel_track" value="0.4"/>
-    <xacro:property name="wheel_base" value="0.4"/>
-    <xacro:property name="wheel_offset_z" value="-0.036"/>
+    <xacro:property name="wheel_track" value="0.35"/>
+    <xacro:property name="wheel_base" value="0.35"/>
+    <xacro:property name="wheel_offset_z" value="0.06"/>
     <xacro:macro name="chassis">
         <link name="base_link">
             <inertial>
-                <mass value="19.31"/>
-                <origin xyz="-0.02282 0.002773 0.008173"/>
-                <inertia ixx="4.041e-1" ixy="7.617e-3" ixz="-1.317e-2" iyy="3.322e-1"
-                         iyz="7.985e-2" izz="1.8e-1"/>
+                <mass value="35.539863"/>
+                <origin xyz="-0.032179 0.015648 0.0968"/>
+                <inertia ixx="1.519" ixy="4.205e-2" ixz="2.407e-1" iyy="1.668"
+                         iyz="8.007e-2" izz="1.891"/>
             </inertial>
             <visual>
                 <origin xyz="0 0 0" rpy="0 0 0"/>
                 <geometry>
-                    <mesh filename="package://rm_description/meshes/hero/base.stl" scale="0.001 .001 0.001"/>
+                    <mesh filename="package://rm_description/meshes/standard/standard4_base.stl"
+                          scale="0.001 .001 0.001"/>
                 </geometry>
             </visual>
@@ -22,5 +23,6 @@
                 <origin xyz="0 0 0" rpy="0 0 0"/>
                 <geometry>
-                    <mesh filename="package://rm_description/meshes/hero/base.stl" scale="0.001 0.001 0.001"/>
+                    <mesh filename="package://rm_description/meshes/standard/standard4_base.stl"
+                          scale="0.001 0.001 0.001"/>
                 </geometry>
             </collision>
@@ -28,14 +30,14 @@
         <xacro:swerve_drive prefix="left_front" connected_to="base_link"
                             wheel_x_offset="${wheel_track/2}" wheel_y_offset="${wheel_base/2}"
-                            wheel_z_offset="${wheel_offset_z}"/>
+                            wheel_z_offset="${wheel_offset_z}" reflect="-1" mirror="1"/>
         <xacro:swerve_drive prefix="right_front" connected_to="base_link"
                             wheel_x_offset="${wheel_track/2}" wheel_y_offset="${-wheel_base/2}"
-                            wheel_z_offset="${wheel_offset_z}"/>
+                            wheel_z_offset="${wheel_offset_z}" reflect="1" mirror="1"/>
         <xacro:swerve_drive prefix="left_back" connected_to="base_link"
                             wheel_x_offset="${-wheel_track/2}" wheel_y_offset="${wheel_base/2}"
-                            wheel_z_offset="${wheel_offset_z}"/>
+                            wheel_z_offset="${wheel_offset_z}" reflect="1" mirror="-1"/>
         <xacro:swerve_drive prefix="right_back" connected_to="base_link"
                             wheel_x_offset="${-wheel_track/2}" wheel_y_offset="${-wheel_base/2}"
-                            wheel_z_offset="${wheel_offset_z}"/>
+                            wheel_z_offset="${wheel_offset_z}" reflect="-1" mirror="-1"/>
         <xacro:swerve_transmission prefix="left_front" wheel_reduction="13.733" pivot_offset="0"/>
         <xacro:swerve_transmission prefix="right_front" wheel_reduction="-13.733" pivot_offset="1.861"/>
