Commit message: fix error

File: urdf/common/camera.urdf.xacro (robot description, xacro)
@@ -1,75 +1,73 @@
-<?xml version="1.0"?>
-<robot xmlns:xacro="http://www.ros.org/wiki/xacro" name="camera">
-    <xacro:property name="pi" value="3.1415926535897931"/>
-    <xacro:macro name="camera_sensor" params="xyz rpy parent">
-        <joint name="camera_sensor_joint" type="fixed">
-            <axis xyz="0 1 0" />
+<robot xmlns:xacro="http://www.ros.org/wiki/xacro">
+    <xacro:macro name="camera_sensor" params="xyz rpy parent camera_sim">
+        <joint name="camera_mount_joint" type="fixed">
+            <axis xyz="0 1 0"/>
             <origin xyz="${xyz}" rpy="${rpy}"/>
             <parent link="${parent}"/>
-            <child link="camera_link"/>
+            <child link="camera_mount"/>
         </joint>
-        <link name="camera_link">
+        <link name="camera_mount">
+            <visual>
+                <origin xyz="0 0 0" rpy="0 0 0"/>
+                <geometry>
+                    <mesh filename="package://rm_description/meshes/common/camera.stl" scale="0.001 0.001 0.001"/>
+                </geometry>
+            </visual>
+            <inertial>
+                <mass value="1.639"/>
+                <origin xyz="0.102 0 0.015" rpy="0 0 0"/>
+                <inertia ixx="3.98e-3" ixy="4.110e-6" ixz="-2.651e-3" iyy="2.723e-2" iyz="6.616e-6" izz="2.635e-2"/>
+            </inertial>
             <collision>
                 <origin xyz="0 0 0" rpy="0 0 0"/>
                 <geometry>
-                    <box size="0.02 0.08 0.05"/>
+                    <mesh filename="package://rm_description/meshes/common/camera.stl" scale="0.001 0.001 0.001"/>
                 </geometry>
             </collision>
-            <visual>
-                <origin xyz="0 0 0" rpy="0 0 0"/>
-                <geometry>
-                    <box size="0.02 0.08 0.05"/>
-                </geometry>
-                <material name="iRobot/Green"/>
-            </visual>
-            <inertial>
-                <mass value="0.0001" />
-                <origin xyz="0 0 0" rpy="0 0 ${pi}"/>
-                <inertia ixx="0.0000001" ixy="0" ixz="0" iyy="0.0000001" iyz="0" izz="0.0000001" />
-            </inertial>
         </link>
-        <link name="camera_sence"></link>
-        <joint name="camera_sence_joint" type="fixed">
-            <axis xyz="0 1 0" />
-            <origin xyz="${xyz}" rpy="${rpy}"/>
-            <parent link="camera_link"/>
-            <child link="camera_sence"/>
+        <joint name="camera_link_joint" type="fixed">
+            <origin xyz="0.026 0 -0.0145" rpy="1.57 0 1.57"/>
+            <parent link="camera_mount"/>
+            <child link="camera_link"/>
         </joint>
-        <gazebo reference="camera_link">
-            <sensor type="camera" name="camera">
-                <update_rate>30.0</update_rate>
-                <camera name="head">
-                    <horizontal_fov>1.3962634</horizontal_fov>
-                    <image>
-                        <width>800</width>
-                        <height>600</height>
-                        <format>R8G8B8</format>
-                    </image>
-                    <clip>
-                        <near>0.02</near>
-                        <far>300</far>
-                    </clip>
-                    <noise>
-                        <type>gaussian</type>
-                        <mean>0.0</mean>
-                        <stddev>0.007</stddev>
-                    </noise>
-                </camera>
-                <plugin name="camera_controller" filename="libgazebo_ros_camera.so">
-                    <alwaysOn>true</alwaysOn>
-                    <updateRate>0.0</updateRate>
-                    <cameraName>iRobot/camera</cameraName>
-                    <imageTopicName>image_raw</imageTopicName>
-                    <cameraInfoTopicName>camera_info</cameraInfoTopicName>
-                    <frameName>camera_link</frameName>
-                    <hackBaseline>0.07</hackBaseline>
-                    <distortionK1>0.0</distortionK1>
-                    <distortionK2>0.0</distortionK2>
-                    <distortionK3>0.0</distortionK3>
-                    <distortionT1>0.0</distortionT1>
-                    <distortionT2>0.0</distortionT2>
-                </plugin>
-            </sensor>
-        </gazebo>
+        <link name="camera_link"/>
+        <xacro:if value="${camera_sim}">
+            <gazebo reference="camera_link">
+                <sensor type="camera" name="camera">
+                    <update_rate>30.0</update_rate>
+                    <camera name="head">
+                        <horizontal_fov>1.3962634</horizontal_fov>
+                        <image>
+                            <width>800</width>
+                            <height>600</height>
+                            <format>R8G8B8</format>
+                        </image>
+                        <clip>
+                            <near>0.02</near>
+                            <far>300</far>
+                        </clip>
+                        <noise>
+                            <type>gaussian</type>
+                            <mean>0.0</mean>
+                            <stddev>0.007</stddev>
+                        </noise>
+                    </camera>
+                    <plugin name="camera_controller" filename="libgazebo_ros_camera.so">
+                        <alwaysOn>true</alwaysOn>
+                        <updateRate>0.0</updateRate>
+                        <cameraName>iRobot/camera</cameraName>
+                        <imageTopicName>image_raw</imageTopicName>
+                        <cameraInfoTopicName>camera_info</cameraInfoTopicName>
+                        <frameName>camera_link</frameName>
+                        <hackBaseline>0.07</hackBaseline>
+                        <distortionK1>0.0</distortionK1>
+                        <distortionK2>0.0</distortionK2>
+                        <distortionK3>0.0</distortionK3>
+                        <distortionT1>0.0</distortionT1>
+                        <distortionT2>0.0</distortionT2>
+                    </plugin>
+                </sensor>
+            </gazebo>
+        </xacro:if>
     </xacro:macro>
 </robot>

File: urdf/hero/gimbal.urdf.xacro (robot description, xacro)
@@ -35,8 +35,8 @@
     <link name="pitch">
         <inertial>
-            <mass value="1.65"/>
-            <origin xyz="0.080137 -0.002734 0.011093"/>
-            <inertia ixx="3.355e-3" ixy="2.3e-5" ixz="-1.069e-3" iyy="2.153e-2"
-                     iyz="-6.373e-5" izz="1.995e-2"/>
+            <mass value="1.63"/>
+            <origin xyz="0.102 -0.0 0.015"/>
+            <inertia ixx="3.980e-3" ixy="4.110e-6" ixz="-2.651e-3" iyy="2.723e-2"
+                     iyz="6.616e-6" izz=" 2.635e-2"/>
         </inertial>
         <visual>
@@ -65,29 +65,29 @@
         <axis xyz="0 1 0 "/>
     </joint>
-    <link name="camera">
-        <inertial>
-            <mass value="0.17671"/>
-            <origin xyz="0.022 0.0 0.0"/>
-            <inertia ixx="2.129e-5" ixy="7.329e-8" ixz="-1.11e-7" iyy="2.198e-4" iyz="-8.04e-7" izz="2.197e-4"/>
-        </inertial>
-        <visual>
-            <origin xyz=" 0 0 0 " rpy="0 -1.57 0"/>
-            <geometry>
-                <mesh filename="package://rm_description/meshes/common/camera.stl" scale="0.001 0.001 0.001"/>
-            </geometry>
-            <material name="Black"/>
-        </visual>
-        <collision>
-            <origin xyz="0 0 0" rpy="0 -1.57 0"/>
-            <geometry>
-                <mesh filename="package://rm_description/meshes/common/camera.stl" scale="0.001 0.001 0.001"/>
-            </geometry>
-        </collision>
-    </link>
-    <joint name="camera_joint" type="fixed">
-        <parent link="pitch"/>
-        <child link="camera"/>
-        <origin xyz="0.153 0.0 -0.052" rpy="1.57 0 1.57"/>
-        <axis xyz="0 0 1"/>
-    </joint>
+    <!--    <link name="camera">-->
+    <!--        <inertial>-->
+    <!--            <mass value="0.17671"/>-->
+    <!--            <origin xyz="0.022 0.0 0.0"/>-->
+    <!--            <inertia ixx="2.129e-5" ixy="7.329e-8" ixz="-1.11e-7" iyy="2.198e-4" iyz="-8.04e-7" izz="2.197e-4"/>-->
+    <!--        </inertial>-->
+    <!--        <visual>-->
+    <!--            <origin xyz=" 0 0 0 " rpy="0 -1.57 0"/>-->
+    <!--            <geometry>-->
+    <!--                <mesh filename="package://rm_description/meshes/common/camera.stl" scale="0.001 0.001 0.001"/>-->
+    <!--            </geometry>-->
+    <!--            <material name="Black"/>-->
+    <!--        </visual>-->
+    <!--        <collision>-->
+    <!--            <origin xyz="0 0 0" rpy="0 -1.57 0"/>-->
+    <!--            <geometry>-->
+    <!--                <mesh filename="package://rm_description/meshes/common/camera.stl" scale="0.001 0.001 0.001"/>-->
+    <!--            </geometry>-->
+    <!--        </collision>-->
+    <!--    </link>-->
+    <!--    <joint name="camera_joint" type="fixed">-->
+    <!--        <parent link="pitch"/>-->
+    <!--        <child link="camera"/>-->
+    <!--        <origin xyz="0.153 0.0 -0.052" rpy="1.57 0 1.57"/>-->
+    <!--        <axis xyz="0 0 1"/>-->
+    <!--    </joint>-->
 </robot>

File: urdf/hero/hero.urdf.xacro (robot description, xacro)
@@ -10,11 +10,18 @@
     <xacro:chassis roller_type="$(arg roller_type)"/>
   </xacro:if>
+  <xacro:if value="$(arg load_shooter)">
+    <xacro:include filename="$(find rm_description)/urdf/hero/shooter.urdf.xacro"/>
+    <xacro:include filename="$(find rm_description)/urdf/hero/shooter.transmission.urdf.xacro"/>
+  </xacro:if>
+  <!--  <xacro:if value="$(arg load_shooter)">-->
+  <!--    <xacro:include filename="$(find rm_description)/urdf/sentry/shooter.urdf.xacro"/>-->
+  <!--    <xacro:include filename="$(find rm_description)/urdf/sentry/shooter.transmission.urdf.xacro"/>-->
+  <!--  </xacro:if>-->
   <xacro:if value="$(arg load_gimbal)">
     <xacro:include filename="$(find rm_description)/urdf/hero/gimbal.urdf.xacro"/>
     <xacro:include filename="$(find rm_description)/urdf/hero/gimbal.transmission.urdf.xacro"/>
-  </xacro:if>
-  <xacro:if value="$(arg load_shooter)">
-    <xacro:include filename="$(find rm_description)/urdf/hero/shooter.urdf.xacro"/>
-    <xacro:include filename="$(find rm_description)/urdf/hero/shooter.transmission.urdf.xacro"/>
+    <xacro:include filename="$(find rm_description)/urdf/common/camera.urdf.xacro"/>
+    <xacro:camera_sensor xyz="0.127 0 -0.047" rpy="0 0 0" parent="pitch"
+                         camera_sim="$(arg use_simulation)"></xacro:camera_sensor>
   </xacro:if>
   <xacro:if value="$(arg use_simulation)">

File: urdf/hero/shooter.urdf.xacro (robot description, xacro)
@@ -1,41 +1,42 @@
 <robot xmlns:xacro="http://www.ros.org/wiki/xacro">
     <xacro:include filename="$(find rm_description)/urdf/common/friction.urdf.xacro"/>
-    <xacro:property name="wheel_offset_x" value="0.082"/>
-    <xacro:property name="wheel_offset_y" value="0.049"/>
-    <xacro:property name="wheel_offset_z" value="0.0"/>
-    <xacro:friction_wheel prefixs="left" connected_to="pitch"
-                          wheel_x_offset="${wheel_offset_x}" wheel_y_offset="${wheel_offset_y}"
-                          wheel_z_offset="${wheel_offset_z}"/>
-    <xacro:friction_wheel prefixs="right" connected_to="pitch"
-                          wheel_x_offset="${wheel_offset_x}"
-                          wheel_y_offset="${-wheel_offset_y}"
-                          wheel_z_offset="${wheel_offset_z}"/>
-    <link name="trigger">
-        <inertial>
-            <mass value="1.725"/>
-            <origin xyz="-0.03783 0.001 0.0162"/>
-            <inertia ixx="3.131e-3" ixy="-2.522e-4" ixz="7.492e-4" iyy="1.344e-2"
-                     iyz="6.02e-5" izz="1.265e-2"/>
-        </inertial>
-        <visual>
-            <origin xyz="0 0 0" rpy="0 0 0"/>
-            <geometry>
-                <mesh filename="package://rm_description/meshes/hero/trigger.stl" scale="0.001 0.001 0.001" />
-            </geometry>
-        </visual>
-        <collision>
-            <origin xyz="0 0 0" rpy="0 0 0"/>
-            <geometry>
-                <mesh filename="package://rm_description/meshes/hero/trigger.stl"  scale="0.001 0.001 0.001" />
-            </geometry>
-        </collision>
-    </link>
-    <joint name="trigger_joint" type="continuous">
-        <origin xyz="-0.173 0 0" rpy="0 0 0"/>
-        <dynamics damping="0.0" friction="0.01"/>
-        <limit effort="3.0" velocity="49.09" lower="-1e16" upper="1e16"/>
-        <parent link="base_link"/>
-        <child link="trigger"/>
-        <axis xyz="0 0 1 "/>
-    </joint>
+    <xacro:include filename="$(find rm_description)/urdf/hero/gimbal.urdf.xacro"/>
+    <!--    <xacro:property name="wheel_offset_x" value="0.082"/>-->
+    <!--    <xacro:property name="wheel_offset_y" value="0.049"/>-->
+    <!--    <xacro:property name="wheel_offset_z" value="0.0"/>-->
+    <!--    <xacro:friction_wheel prefixs="left" connected_to="pitch"-->
+    <!--                          wheel_x_offset="${wheel_offset_x}" wheel_y_offset="${wheel_offset_y}"-->
+    <!--                          wheel_z_offset="${wheel_offset_z}"/>-->
+    <!--    <xacro:friction_wheel prefixs="right" connected_to="pitch"-->
+    <!--                          wheel_x_offset="${wheel_offset_x}"-->
+    <!--                          wheel_y_offset="${-wheel_offset_y}"-->
+    <!--                          wheel_z_offset="${wheel_offset_z}"/>-->
+    <!--    <link name="trigger">-->
+    <!--        <inertial>-->
+    <!--            <mass value="1.725"/>-->
+    <!--            <origin xyz="-0.03783 0.001 0.0162"/>-->
+    <!--            <inertia ixx="3.131e-3" ixy="-2.522e-4" ixz="7.492e-4" iyy="1.344e-2"-->
+    <!--                     iyz="6.02e-5" izz="1.265e-2"/>-->
+    <!--        </inertial>-->
+    <!--        <visual>-->
+    <!--            <origin xyz="0 0 0" rpy="0 0 0"/>-->
+    <!--            <geometry>-->
+    <!--                <mesh filename="package://rm_description/meshes/hero/trigger.stl" scale="0.001 0.001 0.001" />-->
+    <!--            </geometry>-->
+    <!--        </visual>-->
+    <!--        <collision>-->
+    <!--            <origin xyz="0 0 0" rpy="0 0 0"/>-->
+    <!--            <geometry>-->
+    <!--                <mesh filename="package://rm_description/meshes/hero/trigger.stl"  scale="0.001 0.001 0.001" />-->
+    <!--            </geometry>-->
+    <!--        </collision>-->
+    <!--    </link>-->
+    <!--    <joint name="trigger_joint" type="continuous">-->
+    <!--        <origin xyz="-0.173 0 0" rpy="0 0 0"/>-->
+    <!--        <dynamics damping="0.0" friction="0.01"/>-->
+    <!--        <limit effort="3.0" velocity="49.09" lower="-1e16" upper="1e16"/>-->
+    <!--        <parent link="base_link"/>-->
+    <!--        <child link="trigger"/>-->
+    <!--        <axis xyz="0 0 1 "/>-->
+    <!--    </joint>-->
 </robot>

File: urdf/sentry/chassis.urdf.xacro (robot description, xacro)
@@ -4,8 +4,8 @@
     <link name="base_link">
       <inertial>
-        <mass value="7.41"/>
-        <origin xyz="0 0.055 -0.1747"/>
-        <inertia ixx="4.024e-1" ixy="7.617e-3" ixz="-1.318e-2" iyy="3.33e-1"
-                 iyz="7.959e-2" izz="1.802e-1"/>
+        <mass value="8.250"/>
+        <origin xyz="0.0 0.051 -0.148"/>
+        <inertia ixx="3.838e-1" ixy="1.075e-2" ixz="1.397e-5" iyy="2.601e-1"
+                 iyz="7.528e-2" izz="2.369e-1"/>
       </inertial>
       <visual>
@@ -25,6 +25,6 @@
       <inertial>
         <mass value="0.0839"/>
-        <origin xyz="0 0 0"/>
-        <inertia ixx="3.345e-5" ixy="0" ixz="0" iyy="4.185e-5"
+        <origin xyz="0 0.01 0"/>
+        <inertia ixx="3.345e-5" ixy="0" ixz="0" iyy="-8.387e-5"
                  iyz="-2.8558e-8" izz="3.347e-5"/>
       </inertial>
@@ -47,5 +47,5 @@
       <parent link="base_link"/>
       <child link="link_drive_wheel"/>
-      <origin xyz="0 0 0" rpy="0 0 0"/>
+      <origin xyz="0 -0.0185 0" rpy="0 0 0"/>
     </joint>
     <xacro:if value="$(arg use_simulation)">

File: urdf/sentry/gimbal.urdf.xacro (robot description, xacro)
@@ -1,5 +1,4 @@
 <?xml version="1.0" encoding="utf-8"?>
 <robot xmlns:xacro="http://www.ros.org/wiki/xacro">
-  <xacro:macro name="gimbal">
     <xacro:property name="threshold" value="0.1"/>
     <xacro:property name="pitch_lower_limit" value="0.241"/>
@@ -14,7 +13,7 @@
       <inertial>
         <mass value="0.225984"/>
-        <origin xyz="0.00336 0 -0.0494" rpy="0 0 0"/>
-        <inertia ixx="9.791e-4" ixy="6.37e-10" ixz="6.197e-5" iyy="1.507e-3"
-                 iyz="1.806e-9" izz="7.527e-4"/>
+        <origin xyz="-0.0516 -0.01431 -0.03823" rpy="0 0 0"/>
+        <inertia ixx="7.196e-3" ixy="1.102e-3" ixz="-2.150e-3" iyy="2.478e-2"
+                 iyz="-1.186e-3" izz="2.488e-2"/>
       </inertial>
       <collision>
@@ -30,5 +29,5 @@
       <child link="yaw"/>
       <axis xyz="0 0 1"/>
-      <origin xyz="0.00 0.0 -0.21"/>
+      <origin xyz="0.0 0.031 -0.2352"/>
       <dynamics damping="0" friction="0.1"/>
       <limit effort="1.2" velocity="34" lower="-${2*pi}" upper="${2*pi}"/>
@@ -36,8 +35,8 @@
     <link name="pitch">
       <inertial>
-        <mass value="1.155968"/>
-        <origin xyz="0.019 -0.045 0.022"/>
-        <inertia ixx="5.918e-3" ixy="1.6863e-6" ixz="2.4143e-6" iyy="2.048e-3"
-                 iyz="-1.348e-4" izz="7.506e-3"/>
+        <mass value="1.05"/>
+        <origin xyz="0.0 -0.022 -0.043"/>
+        <inertia ixx="5.350e-3" ixy="1.148e-3" ixz="-1.287e-5" iyy="1.055e-2"
+                 iyz="1.122e-3" izz="1.050e-2"/>
       </inertial>
       <visual>
@@ -58,5 +57,5 @@
       <child link="pitch"/>
       <axis xyz="0 1 0"/>
-      <origin xyz="0 0 -0.13"/>
+      <origin xyz="0 0 -0.0799"/>
       <dynamics damping="0" friction="0.1"/>
       <limit effort="1.2" velocity="13.82" lower="${pitch_lower_limit}" upper="${pitch_upper_limit}"/>
@@ -65,30 +64,29 @@
                          soft_upper_limit="${pitch_upper_limit-threshold}"/>
     </joint>
-    <link name="camera">
-      <inertial>
-        <mass value="0.17671"/>
-        <origin xyz="0.022 0.0 0.0"/>
-        <inertia ixx="2.129e-5" ixy="7.329e-8" ixz="-1.11e-7" iyy="2.198e-4" iyz="-8.04e-7" izz="2.197e-4"/>
-      </inertial>
-      <visual>
-        <origin xyz=" 0 0 0 " rpy="0 -1.57 0"/>
-        <geometry>
-          <mesh filename="package://rm_description/meshes/common/camera.stl" scale="0.001 0.001 0.001"/>
-        </geometry>
-        <material name="Black"/>
-      </visual>
-      <collision>
-        <origin xyz="0 0 0" rpy="0 -1.57 0"/>
-        <geometry>
-          <mesh filename="package://rm_description/meshes/common/camera.stl" scale="0.001 0.001 0.001"/>
-        </geometry>
-      </collision>
-    </link>
-    <joint name="camera_joint" type="fixed">
-      <parent link="pitch"/>
-      <child link="camera"/>
-      <origin xyz="0.086  0.0 -0.040" rpy="-1.57 0 -1.57"/>
-      <axis xyz="0 0 1"/>
-    </joint>
-  </xacro:macro>
+<!--    <link name="camera">-->
+<!--      <inertial>-->
+<!--        <mass value="0.17671"/>-->
+<!--        <origin xyz="0.022 0.0 0.0"/>-->
+<!--        <inertia ixx="2.129e-5" ixy="7.329e-8" ixz="-1.11e-7" iyy="2.198e-4" iyz="-8.04e-7" izz="2.197e-4"/>-->
+<!--      </inertial>-->
+<!--      <visual>-->
+<!--        <origin xyz=" 0 0 0 " rpy="0 -1.57 0"/>-->
+<!--        <geometry>-->
+<!--          <mesh filename="package://rm_description/meshes/common/camera.stl" scale="0.001 0.001 0.001"/>-->
+<!--        </geometry>-->
+<!--        <material name="Black"/>-->
+<!--      </visual>-->
+<!--      <collision>-->
+<!--        <origin xyz="0 0 0" rpy="0 -1.57 0"/>-->
+<!--        <geometry>-->
+<!--          <mesh filename="package://rm_description/meshes/common/camera.stl" scale="0.001 0.001 0.001"/>-->
+<!--        </geometry>-->
+<!--      </collision>-->
+<!--    </link>-->
+<!--    <joint name="camera_joint" type="fixed">-->
+<!--      <parent link="pitch"/>-->
+<!--      <child link="camera"/>-->
+<!--      <origin xyz="0.086  0.0 -0.040" rpy="-1.57 0 -1.57"/>-->
+<!--      <axis xyz="0 0 1"/>-->
+<!--    </joint>-->
 </robot>
