Commit message: fix error

File: urdf/sentry/sentry.urdf.xacro (robot description, xacro)
@@ -13,5 +13,7 @@
         <xacro:include filename="$(find rm_description)/urdf/sentry/gimbal.urdf.xacro"/>
         <xacro:include filename="$(find rm_description)/urdf/sentry/gimbal.transmission.urdf.xacro"/>
-        <xacro:gimbal/>
+        <xacro:include filename="$(find rm_description)/urdf/common/camera.urdf.xacro"/>
+        <xacro:camera_sensor xyz="0.127 0 -0.047" rpy="0 0 0" parent="pitch"
+                             camera_sim="$(arg use_simulation)"></xacro:camera_sensor>
     </xacro:if>
     <xacro:if value="$(arg load_shooter)">
@@ -28,2 +30,33 @@
     </xacro:if>
 </robot>
+        <!--<?xml version="1.0" encoding="utf-8"?>-->
+        <!--<robot name="sentry">-->
+        <!--    &lt;!&ndash;    <xacro:arg name="load_chassis" default="true"/>&ndash;&gt;-->
+        <!--    &lt;!&ndash;    <xacro:arg name="load_gimbal" default="true"/>&ndash;&gt;-->
+        <!--    &lt;!&ndash;    <xacro:arg name="load_shooter" default="true"/>&ndash;&gt;-->
+        <!--    &lt;!&ndash;    <xacro:arg name="use_simulation" default="true"/>&ndash;&gt;-->
+        <!--    &lt;!&ndash;    <xacro:if value="$(arg load_chassis)">&ndash;&gt;-->
+        <!--    &lt;!&ndash;        <xacro:include filename="$(find rm_description)/urdf/sentry/chassis.urdf.xacro"/>&ndash;&gt;-->
+        <!--    &lt;!&ndash;        <xacro:include filename="$(find rm_description)/urdf/sentry/chassis.transmission.urdf.xacro"/>&ndash;&gt;-->
+        <!--    &lt;!&ndash;        <xacro:chassis use_simulation="$(arg use_simulation)"/>&ndash;&gt;-->
+        <!--    &lt;!&ndash;    </xacro:if>&ndash;&gt;-->
+        <!--    &lt;!&ndash;    <xacro:if value="$(arg load_gimbal)">&ndash;&gt;-->
+        <!--    &lt;!&ndash;        <xacro:include filename="$(find rm_description)/urdf/sentry/gimbal.urdf.xacro"/>&ndash;&gt;-->
+        <!--    &lt;!&ndash;        <xacro:include filename="$(find rm_description)/urdf/sentry/gimbal.transmission.urdf.xacro"/>&ndash;&gt;-->
+        <!--    &lt;!&ndash;        <xacro:include filename="$(find rm_description)/urdf/common/camera.urdf.xacro"/>&ndash;&gt;-->
+        <!--    &lt;!&ndash;        <xacro:camera_sensor xyz="0.0857 0 -0.0396" rpy="0 0 0" parent="pitch"&ndash;&gt;-->
+        <!--    &lt;!&ndash;                             camera_sim="use_simulation"></xacro:camera_sensor>&ndash;&gt;-->
+        <!--    &lt;!&ndash;    </xacro:if>&ndash;&gt;-->
+        <!--    &lt;!&ndash;    <xacro:if value="$(arg load_shooter)">&ndash;&gt;-->
+        <!--    &lt;!&ndash;        <xacro:include filename="$(find rm_description)/urdf/sentry/shooter.urdf.xacro"/>&ndash;&gt;-->
+        <!--    &lt;!&ndash;        <xacro:include filename="$(find rm_description)/urdf/sentry/shooter.transmission.urdf.xacro"/>&ndash;&gt;-->
+        <!--    &lt;!&ndash;    </xacro:if>&ndash;&gt;-->
+        <!--    &lt;!&ndash;    <xacro:if value="$(arg use_simulation)">&ndash;&gt;-->
+        <!--    &lt;!&ndash;        <gazebo>&ndash;&gt;-->
+        <!--    &lt;!&ndash;            <plugin name="rm_ros_control" filename="librm_robot_hw_sim.so">&ndash;&gt;-->
+        <!--    &lt;!&ndash;                <robotNamespace>/</robotNamespace>&ndash;&gt;-->
+        <!--    &lt;!&ndash;                <robotSimType>rm_gazebo/RmRobotHWSim</robotSimType>&ndash;&gt;-->
+        <!--    &lt;!&ndash;            </plugin>&ndash;&gt;-->
+        <!--    &lt;!&ndash;        </gazebo>&ndash;&gt;-->
+        <!--    &lt;!&ndash;    </xacro:if>&ndash;&gt;-->
+        <!--</robot>-->

File: urdf/sentry/shooter.urdf.xacro (robot description, xacro)
@@ -1,11 +1,13 @@
 <robot xmlns:xacro="http://www.ros.org/wiki/xacro">
   <xacro:include filename="$(find rm_description)/urdf/common/friction.urdf.xacro"/>
-  <xacro:property name="wheel_offset_x" value="-0.03847"/>
-  <xacro:property name="wheel_offset_y" value="-0.06594"/>
-  <xacro:property name="wheel_offset_z" value="0.01132"/>
+  <xacro:property name="wheel_offset_x" value="0.0504"/>
+  <xacro:property name="wheel_offset_y" value="0.0365"/>
+  <xacro:property name="wheel_offset_z" value="0.01072"/>
   <xacro:friction_wheel prefixs="left" connected_to="pitch"
-                        wheel_x_offset="${-wheel_offset_x}" wheel_y_offset="${wheel_offset_y}" wheel_z_offset="${wheel_offset_z}"/>
+                        wheel_x_offset="${wheel_offset_x}" wheel_y_offset="${-wheel_offset_y}"
+                        wheel_z_offset="${wheel_offset_z}"/>
   <xacro:friction_wheel prefixs="right" connected_to="pitch"
-                        wheel_x_offset="${wheel_offset_x}" wheel_y_offset="${wheel_offset_y}" wheel_z_offset="${wheel_offset_z}"/>
+                        wheel_x_offset="${wheel_offset_x}" wheel_y_offset="${wheel_offset_y}"
+                        wheel_z_offset="${wheel_offset_z}"/>
   <link name="trigger">
     <inertial>

Commit message: add camera on standard

File: urdf/common/camera.urdf.xacro (robot description, xacro)
@@ -44,6 +44,6 @@
                         </image>
                         <clip>
-                            <near>0.02</near>
-                            <far>300</far>
+                            <near>0.05</near>
+                            <far>5</far>
                         </clip>
                         <noise>

File: urdf/engineer/hand.urdf.xacro (robot description, xacro)
@@ -133,5 +133,5 @@
             <origin xyz="0.032 0 0" rpy="0 0 0"/>
             <axis xyz="0 1 0"/>
-            <limit effort="588" lower="0.0" upper="0.02" velocity="3.772"/>
+            <limit effort="588" lower="0.0" upper="0.03" velocity="3.772"/>
         </joint>
         <joint name="left_finger_joint" type="prismatic">
@@ -140,5 +140,5 @@
             <origin xyz="0.032 0 0" rpy="0 0 0"/>
             <axis xyz="0 -1 0"/>
-            <limit effort="588" lower="0.0" upper="0.02" velocity="3.772"/>
+            <limit effort="588" lower="0.0" upper="0.03" velocity="3.772"/>
             <mimic joint="right_finger_joint"/>
         </joint>

File: urdf/standard/gimbal.urdf.xacro (robot description, xacro)
@@ -4,5 +4,4 @@
     <xacro:property name="pitch_lower_limit" value="-0.7"/>
     <xacro:property name="pitch_upper_limit" value="0.4"/>
-    <xacro:macro name="gimbal" params="simulation">
         <link name="yaw">
             <inertial>
@@ -65,68 +64,3 @@
             <axis xyz="0 1 0 "/>
         </joint>
-        <link name="camera_link">
-            <inertial>
-                <mass value="0.17671"/>
-                <origin xyz="0.022 0.0 0.0"/>
-                <inertia ixx="2.129e-5" ixy="7.329e-8" ixz="-1.11e-7" iyy="2.198e-4" iyz="-8.04e-7" izz="2.197e-4"/>
-            </inertial>
-            <visual>
-                <origin xyz=" 0 0 0 " rpy="0 -1.57 0"/>
-                <geometry>
-                    <mesh filename="package://rm_description/meshes/common/camera.stl" scale="0.001 0.001 0.001"/>
-                </geometry>
-                <material name="Black"/>
-            </visual>
-            <collision>
-                <origin xyz="0 0 0" rpy="0 -1.57 0"/>
-                <geometry>
-                    <mesh filename="package://rm_description/meshes/common/camera.stl" scale="0.001 0.001 0.001"/>
-                </geometry>
-            </collision>
-        </link>
-        <joint name="camera_joint" type="fixed">
-            <parent link="pitch"/>
-            <child link="camera_link"/>
-            <origin xyz="0.15 0.0 -0.03" rpy="-1.57 0 -1.57"/>
-            <axis xyz="0 0 1"/>
-        </joint>
-        <xacro:if value="${simulation}">
-            <!--            <gazebo reference="camera">-->
-            <!--                <sensor type="camera" name="camera_node">-->
-            <!--                    <update_rate>30.0</update_rate>-->
-            <!--                    <camera name="head">-->
-            <!--                        <horizontal_fov>1.3962634</horizontal_fov>-->
-            <!--                        <image>-->
-            <!--                            <width>1920</width>-->
-            <!--                            <height>1080</height>-->
-            <!--                            <format>R8G8B8</format>-->
-            <!--                        </image>-->
-            <!--                        <clip>-->
-            <!--                            <near>0.02</near>-->
-            <!--                            <far>300</far>-->
-            <!--                        </clip>-->
-            <!--                        <noise>-->
-            <!--                            <type>gaussian</type>-->
-            <!--                            <mean>0.0</mean>-->
-            <!--                            <stddev>0.007</stddev>-->
-            <!--                        </noise>-->
-            <!--                    </camera>-->
-            <!--                    <plugin name="gazebo_camera" filename="libgazebo_ros_camera.so">-->
-            <!--                        <alwaysOn>true</alwaysOn>-->
-            <!--                        <updateRate>0.0</updateRate>-->
-            <!--                        <cameraName>/camera</cameraName>-->
-            <!--                        <imageTopicName>image_raw</imageTopicName>-->
-            <!--                        <cameraInfoTopicName>camera_info</cameraInfoTopicName>-->
-            <!--                        <frameName>camera</frameName>-->
-            <!--                        <hackBaseline>0.07</hackBaseline>-->
-            <!--                        <distortionK1>0.0</distortionK1>-->
-            <!--                        <distortionK2>0.0</distortionK2>-->
-            <!--                        <distortionK3>0.0</distortionK3>-->
-            <!--                        <distortionT1>0.0</distortionT1>-->
-            <!--                        <distortionT2>0.0</distortionT2>-->
-            <!--                    </plugin>-->
-            <!--                </sensor>-->
-            <!--            </gazebo>-->
-        </xacro:if>
-    </xacro:macro>
 </robot>

File: urdf/standard/shooter.urdf.xacro (robot description, xacro)
@@ -1,5 +1,5 @@
 <robot xmlns:xacro="http://www.ros.org/wiki/xacro">
     <xacro:include filename="$(find rm_description)/urdf/common/friction.urdf.xacro"/>
-    <xacro:include filename="$(find rm_description)/urdf/standard/gimbal.urdf.xacro"/>
+<!--    <xacro:include filename="$(find rm_description)/urdf/standard/gimbal.urdf.xacro"/>-->
     <xacro:property name="wheel_offset_x" value="0.00884"/>
     <xacro:property name="wheel_offset_y" value="0.036564"/>

File: urdf/standard/standard.urdf.xacro (robot description, xacro)
@@ -16,5 +16,7 @@
         <xacro:include filename="$(find rm_description)/urdf/standard/gimbal.urdf.xacro"/>
         <xacro:include filename="$(find rm_description)/urdf/standard/gimbal.transmission.urdf.xacro"/>
-        <xacro:gimbal simulation="$(arg use_simulation)"/>
+        <xacro:include filename="$(find rm_description)/urdf/common/camera.urdf.xacro"/>
+        <xacro:camera_sensor xyz="0.127 0 -0.038" rpy="0 0 0" parent="pitch"
+                             camera_sim="$(arg use_simulation)"/>
     </xacro:if>
     <xacro:if value="$(arg load_shooter)">

Commit message: Rename camera link and camera optical frame

File: urdf/common/camera.urdf.xacro (robot description, xacro)
@@ -5,7 +5,7 @@
             <origin xyz="${xyz}" rpy="${rpy}"/>
             <parent link="${parent}"/>
-            <child link="camera_mount"/>
+            <child link="camera_link"/>
         </joint>
-        <link name="camera_mount">
+        <link name="camera_link">
             <visual>
                 <origin xyz="0 0 0" rpy="0 0 0"/>
@@ -15,7 +15,7 @@
             </visual>
             <inertial>
-                <mass value="1.639"/>
-                <origin xyz="0.102 0 0.015" rpy="0 0 0"/>
-                <inertia ixx="3.98e-3" ixy="4.110e-6" ixz="-2.651e-3" iyy="2.723e-2" iyz="6.616e-6" izz="2.635e-2"/>
+                <mass value="0.17671"/>
+                <origin xyz="0.022 0.0 0.0"/>
+                <inertia ixx="2.129e-5" ixy="7.329e-8" ixz="-1.11e-7" iyy="2.198e-4" iyz="-8.04e-7" izz="2.197e-4"/>
             </inertial>
             <collision>
@@ -26,12 +26,12 @@
             </collision>
         </link>
-        <joint name="camera_link_joint" type="fixed">
+        <joint name="camera_optical_frame_joint" type="fixed">
             <origin xyz="0.026 0 -0.0145" rpy="1.57 0 1.57"/>
-            <parent link="camera_mount"/>
-            <child link="camera_link"/>
+            <parent link="camera_link"/>
+            <child link="camera_optical_frame"/>
         </joint>
-        <link name="camera_link"/>
+        <link name="camera_optical_frame"/>
         <xacro:if value="${camera_sim}">
-            <gazebo reference="camera_mount">
+            <gazebo reference="camera_link">
                 <sensor type="camera" name="camera">
                     <update_rate>30.0</update_rate>
@@ -39,6 +39,6 @@
                         <horizontal_fov>1.3962634</horizontal_fov>
                         <image>
-                            <width>800</width>
-                            <height>600</height>
+                            <width>1920</width>
+                            <height>1080</height>
                             <format>R8G8B8</format>
                         </image>

Commit message: Fix camera pose

File: urdf/common/camera.urdf.xacro (robot description, xacro)
@@ -27,5 +27,5 @@
         </link>
         <joint name="camera_optical_frame_joint" type="fixed">
-            <origin xyz="0.026 0 -0.0145" rpy="1.57 0 1.57"/>
+            <origin xyz="0.026 0 -0.0145" rpy="-1.57 0 -1.57"/>
             <parent link="camera_link"/>
             <child link="camera_optical_frame"/>
@@ -59,5 +59,5 @@
                         <imageTopicName>image_raw</imageTopicName>
                         <cameraInfoTopicName>camera_info</cameraInfoTopicName>
-                        <frameName>camera_link</frameName>
+                        <frameName>camera_optical_frame</frameName>
                         <hackBaseline>0.07</hackBaseline>
                         <distortionK1>0.0</distortionK1>

File: urdf/standard/standard.urdf.xacro (robot description, xacro)
@@ -17,5 +17,5 @@
         <xacro:include filename="$(find rm_description)/urdf/standard/gimbal.transmission.urdf.xacro"/>
         <xacro:include filename="$(find rm_description)/urdf/common/camera.urdf.xacro"/>
-        <xacro:camera_sensor xyz="0.127 0 -0.038" rpy="-1.57 0 -1.57" parent="pitch"
+        <xacro:camera_sensor xyz="0.127 0 -0.038" rpy="0 0 0" parent="pitch"
                              camera_sim="$(arg use_simulation)"/>
     </xacro:if>

Commit message: Separate camera_link and camera_optical_frame in urdf

File: urdf/common/camera.urdf.xacro (robot description, xacro)
@@ -26,7 +26,9 @@
             </collision>
         </link>
+    </xacro:macro>
+    <xacro:macro name="camera_optical_frame" params="xyz rpy parent camera_sim">
         <joint name="camera_optical_frame_joint" type="fixed">
-            <origin xyz="0.026 0 -0.0145" rpy="-1.57 0 -1.57"/>
-            <parent link="camera_link"/>
+            <origin xyz="${xyz}" rpy="${rpy}"/>
+            <parent link="${parent}"/>
             <child link="camera_optical_frame"/>
         </joint>

File: urdf/hero/hero.urdf.xacro (robot description, xacro)
@@ -19,4 +19,6 @@
     <xacro:camera_sensor xyz="0.127 0 -0.038" rpy="3.14 0 0" parent="pitch"
                          camera_sim="$(arg use_simulation)"/>
+    <xacro:camera_optical_frame xyz="0.2527 0.0071 -0.0984" rpy="1.5486 -0.0025 1.600" parent="pitch"
+                                camera_sim="$(arg use_simulation)"/>
   </xacro:if>
   <xacro:if value="$(arg load_shooter)">

File: urdf/sentry/sentry.urdf.xacro (robot description, xacro)
@@ -14,6 +14,8 @@
         <xacro:include filename="$(find rm_description)/urdf/sentry/gimbal.transmission.urdf.xacro"/>
         <xacro:include filename="$(find rm_description)/urdf/common/camera.urdf.xacro"/>
-        <xacro:camera_sensor xyz="0.127 0 -0.047" rpy="3.14 0 0" parent="pitch"
+        <xacro:camera_sensor xyz="0.127 0 -0.047" rpy="0 0 0" parent="pitch"
                              camera_sim="$(arg use_simulation)"/>
+        <xacro:camera_optical_frame xyz="0.153 0 -0.0615" rpy="1.57 0 1.57" parent="pitch"
+                                    camera_sim="$(arg use_simulation)"/>
     </xacro:if>
     <xacro:if value="$(arg load_shooter)">

File: urdf/standard3/standard3.urdf.xacro (robot description, xacro)
@@ -19,4 +19,6 @@
         <xacro:camera_sensor xyz="0.127 0 -0.038" rpy="0 0 0" parent="pitch"
                              camera_sim="$(arg use_simulation)"/>
+        <xacro:camera_optical_frame xyz="0.153 0 -0.0525" rpy="-1.57 0 -1.57" parent="pitch"
+                                    camera_sim="$(arg use_simulation)"/>
     </xacro:if>
     <xacro:if value="$(arg load_shooter)">

File: urdf/standard4/standard4.urdf.xacro (robot description, xacro)
@@ -18,4 +18,6 @@
         <xacro:camera_sensor xyz="0.127 0 -0.038" rpy="0 0 0" parent="pitch"
                              camera_sim="$(arg use_simulation)"/>
+        <xacro:camera_optical_frame xyz="0.153 0 -0.0525" rpy="-1.57 0 -1.57" parent="pitch"
+                                    camera_sim="$(arg use_simulation)"/>
     </xacro:if>
     <xacro:if value="$(arg load_shooter)">

File: urdf/standard5/standard5.urdf.xacro (robot description, xacro)
@@ -19,4 +19,6 @@
         <xacro:camera_sensor xyz="0.127 0 -0.038" rpy="0 0 0" parent="pitch"
                              camera_sim="$(arg use_simulation)"/>
+        <xacro:camera_optical_frame xyz="0.153 0 -0.0525" rpy="-1.57 0 -1.57" parent="pitch"
+                                    camera_sim="$(arg use_simulation)"/>
     </xacro:if>
     <xacro:if value="$(arg load_shooter)">
