Commit message: Update camera frame

File: urdf/common/camera.urdf.xacro (robot description, xacro)
@@ -1,11 +1,11 @@
 <robot xmlns:xacro="http://www.ros.org/wiki/xacro">
-    <xacro:macro name="camera_sensor" params="xyz rpy parent camera_sim">
-        <joint name="camera_mount_joint" type="fixed">
+    <xacro:macro name="camera_sensor" params="xyz rpy frame_id parent camera_sim">
+        <joint name="${frame_id}_joint" type="fixed">
             <axis xyz="0 1 0"/>
             <origin xyz="${xyz}" rpy="${rpy}"/>
             <parent link="${parent}"/>
-            <child link="camera_link"/>
+            <child link="${frame_id}"/>
         </joint>
-        <link name="camera_link">
+        <link name="${frame_id}">
             <visual>
                 <origin xyz="0 0 0" rpy="0 0 0"/>
@@ -27,11 +27,11 @@
         </link>
     </xacro:macro>
-    <xacro:macro name="camera_optical_frame" params="xyz rpy parent camera_sim">
-        <joint name="camera_optical_frame_joint" type="fixed">
+    <xacro:macro name="camera_optical_frame" params="xyz rpy frame_id parent camera_sim">
+        <joint name="${frame_id}_joint" type="fixed">
             <origin xyz="${xyz}" rpy="${rpy}"/>
             <parent link="${parent}"/>
-            <child link="camera_optical_frame"/>
+            <child link="${frame_id}"/>
         </joint>
-        <link name="camera_optical_frame"/>
+        <link name="${frame_id}"/>
         <xacro:if value="${camera_sim}">
             <gazebo reference="camera_link">

File: urdf/sentry/sentry.urdf.xacro (robot description, xacro)
@@ -4,4 +4,8 @@
     <xacro:arg name="load_gimbal" default="true"/>
     <xacro:arg name="load_shooter" default="true"/>
+    <xacro:arg name="upper_camera_link" default="upper_camera_link"/>
+    <xacro:arg name="upper_camera_optical_frame" default="upper_camera_optical_frame"/>
+    <xacro:arg name="lower_camera_link" default="lower_camera_link"/>
+    <xacro:arg name="lower_camera_optical_frame" default="lower_camera_optical_frame"/>
     <xacro:arg name="use_simulation" default="true"/>
     <xacro:if value="$(arg load_chassis)">
@@ -13,16 +17,18 @@
         <xacro:include filename="$(find rm_description)/urdf/sentry/lower_gimbal.urdf.xacro"/>
         <xacro:include filename="$(find rm_description)/urdf/sentry/lower_gimbal.transmission.urdf.xacro"/>
-<!--        <xacro:include filename="$(find rm_description)/urdf/common/camera.urdf.xacro"/>-->
-        <!--        <xacro:camera_sensor xyz="0.127 0 -0.047" rpy="0 0 0" parent="lower_pitch"-->
-        <!--                             camera_sim="$(arg use_simulation)"/>-->
-        <!--        <xacro:camera_optical_frame xyz="0.153 0 -0.0615" rpy="${-pi/2} 0 ${-pi/2}" parent="lower_pitch"-->
-        <!--                                    camera_sim="$(arg use_simulation)"/>-->
+        <xacro:include filename="$(find rm_description)/urdf/common/camera.urdf.xacro"/>
+        <xacro:camera_sensor xyz="0.127 0 -0.047" rpy="0 0 0" frame_id="$(arg lower_camera_link)" parent="lower_pitch"
+                             camera_sim="$(arg use_simulation)"/>
+        <xacro:camera_optical_frame xyz="0.153 0 -0.0615" rpy="${pi/2} 0 ${pi/2}"
+                                    frame_id="$(arg lower_camera_optical_frame)"
+                                    parent="lower_pitch" camera_sim="$(arg use_simulation)"/>
         <xacro:include filename="$(find rm_description)/urdf/sentry/upper_gimbal.urdf.xacro"/>
         <xacro:include filename="$(find rm_description)/urdf/sentry/upper_gimbal.transmission.urdf.xacro"/>
-        <!--        <xacro:include filename="$(find rm_description)/urdf/common/camera.urdf.xacro"/>-->
-        <!--        <xacro:camera_sensor xyz="0.127 0 -0.047" rpy="0 0 0" parent="upper_pitch"-->
-        <!--                             camera_sim="$(arg use_simulation)"/>-->
-        <!--        <xacro:camera_optical_frame xyz="0.153 0 -0.0615" rpy="${-pi/2} 0 ${-pi/2}" parent="upper_pitch"-->
-        <!--                                    camera_sim="$(arg use_simulation)"/>-->
+        <xacro:include filename="$(find rm_description)/urdf/common/camera.urdf.xacro"/>
+        <xacro:camera_sensor xyz="0.127 0 -0.047" rpy="0 0 0" frame_id="$(arg upper_camera_link)" parent="upper_pitch"
+                             camera_sim="$(arg use_simulation)"/>
+        <xacro:camera_optical_frame xyz="0.153 0 -0.0615" rpy="${-pi/2} 0 ${-pi/2}"
+                                    frame_id="$(arg upper_camera_optical_frame)"
+                                    parent="upper_pitch" camera_sim="$(arg use_simulation)"/>
     </xacro:if>
     <xacro:if value="$(arg load_shooter)">

File: urdf/standard3/standard3.urdf.xacro (robot description, xacro)
@@ -4,4 +4,6 @@
     <xacro:arg name="load_gimbal" default="true"/>
     <xacro:arg name="load_shooter" default="true"/>
+    <xacro:arg name="camera_link" default="camera_link"/>
+    <xacro:arg name="camera_optical_frame" default="camera_optical_frame"/>
     <xacro:arg name="use_simulation" default="true"/>
     <xacro:arg name="roller_type" default="realistic"/>
@@ -17,7 +19,8 @@
         <xacro:include filename="$(find rm_description)/urdf/standard3/gimbal.transmission.urdf.xacro"/>
         <xacro:include filename="$(find rm_description)/urdf/common/camera.urdf.xacro"/>
-        <xacro:camera_sensor xyz="0.127 0 -0.038" rpy="0 0 0" parent="pitch"
+        <xacro:camera_sensor xyz="0.127 0 -0.038" rpy="0 0 0" frame_id="$(arg camera_link)" parent="pitch"
                              camera_sim="$(arg use_simulation)"/>
-        <xacro:camera_optical_frame xyz="0.089 -0.004 -0.053" rpy="1.593 0.0 1.567" parent="pitch"
+        <xacro:camera_optical_frame xyz="0.089 -0.004 -0.053" rpy="1.593 0.0 1.567"
+                                    frame_id="$(arg camera_optical_frame)" parent="pitch"
                                     camera_sim="$(arg use_simulation)"/>
     </xacro:if>

File: urdf/standard4/standard4.urdf.xacro (robot description, xacro)
@@ -4,4 +4,6 @@
     <xacro:arg name="load_gimbal" default="true"/>
     <xacro:arg name="load_shooter" default="true"/>
+    <xacro:arg name="camera_link" default="camera_link"/>
+    <xacro:arg name="camera_optical_frame" default="camera_optical_frame"/>
     <xacro:arg name="use_simulation" default="true"/>
     <xacro:if value="$(arg load_chassis)">
@@ -16,7 +18,8 @@
         <xacro:include filename="$(find rm_description)/urdf/standard4/gimbal.transmission.urdf.xacro"/>
         <xacro:include filename="$(find rm_description)/urdf/common/camera.urdf.xacro"/>
-        <xacro:camera_sensor xyz="0.127 0 -0.038" rpy="0 0 0" parent="pitch"
+        <xacro:camera_sensor xyz="0.127 0 -0.038" rpy="0 0 0" frame_id="$(arg camera_link)" parent="pitch"
                              camera_sim="$(arg use_simulation)"/>
-        <xacro:camera_optical_frame xyz="0.089 -0.004 -0.083" rpy="1.593 0.0 1.567" parent="pitch"
+        <xacro:camera_optical_frame xyz="0.089 -0.004 -0.083" rpy="1.593 0.0 1.567"
+                                    frame_id="$(arg camera_optical_frame)" parent="pitch"
                                     camera_sim="$(arg use_simulation)"/>
     </xacro:if>

File: urdf/standard5/standard5.urdf.xacro (robot description, xacro)
@@ -4,4 +4,6 @@
     <xacro:arg name="load_gimbal" default="true"/>
     <xacro:arg name="load_shooter" default="true"/>
+    <xacro:arg name="camera_link" default="camera_link"/>
+    <xacro:arg name="camera_optical_frame" default="camera_optical_frame"/>
     <xacro:arg name="use_simulation" default="true"/>
     <xacro:arg name="roller_type" default="realistic"/>
@@ -17,7 +19,8 @@
         <xacro:include filename="$(find rm_description)/urdf/standard5/gimbal.transmission.urdf.xacro"/>
         <xacro:include filename="$(find rm_description)/urdf/common/camera.urdf.xacro"/>
-        <xacro:camera_sensor xyz="0.127 0 -0.038" rpy="0 0 0" parent="pitch"
+        <xacro:camera_sensor xyz="0.127 0 -0.038" rpy="0 0 0" frame_id="$(arg camera_link)" parent="pitch"
                              camera_sim="$(arg use_simulation)"/>
-        <xacro:camera_optical_frame xyz="0.089 -0.004 -0.083" rpy="1.593 0.0 1.567" parent="pitch"
+        <xacro:camera_optical_frame xyz="0.089 -0.004 -0.083" rpy="1.593 0.0 1.567"
+                                    frame_id="$(arg camera_optical_frame)" parent="pitch"
                                     camera_sim="$(arg use_simulation)"/>
     </xacro:if>
