Commit message: Rename lidar_link_name to lidar_name, rename imu_link_name to imu_name.

File: urdf/auto/auto.urdf.xacro (robot description, xacro)
@@ -10,8 +10,8 @@
         <xacro:chassis roller_type="$(arg roller_type)"/>
         <xacro:include filename="$(find rm_description)/urdf/common/imu.urdf.xacro"/>
-        <xacro:IMU connected_to="base_link" imu_link_name="base_imu" simulation="true"
+        <xacro:IMU connected_to="base_link" imu_name="base_imu" simulation="true"
                    xyz="0.065 0.12 0.07"/>
         <xacro:include filename="$(find rm_description)/urdf/common/lidar2d.urdf.xacro"/>
-        <xacro:lidar2d connected_to="base_link" lidar_link_name="base_scan" simulation="true"
+        <xacro:lidar2d connected_to="base_link" lidar_name="base_scan" simulation="true"
                        xyz="0.2 0 0.2"/>
     </xacro:if>

File: urdf/common/imu.urdf.xacro (robot description, xacro)
@@ -3,8 +3,7 @@
 <!-- Documentation can be found at http://wiki.ros.org/hector_gazebo_plugins -->
 <robot xmlns:xacro="http://www.ros.org/wiki/xacro" name="imu">
-    <xacro:macro name="IMU" params="connected_to imu_link_name simulation xyz:='0 0 0' rpy:='0 0 0' ">
-        <xacro:property name="imu_base_link" value="${base_link}"/>
+    <xacro:macro name="IMU" params="connected_to imu_name simulation xyz:='0 0 0' rpy:='0 0 0' ">
         <xacro:property name="imu_update_rate" value="200"/>
-        <xacro:property name="imu_calibration_service_name" value="${imu_link_name}/calibrate"/>
+        <xacro:property name="imu_calibration_service_name" value="${imu_name}/calibrate"/>
         <xacro:property name="acceleration_offset" value="0.0 0.0 0.0"/>
         <xacro:property name="acceleration_drift" value="0.0 0.0 0.0"/>
@@ -20,11 +19,11 @@
         <xacro:property name="heading_gaussian_noise" value="0.3"/>
         <!-- Imu is fixed to the base link -->
-        <joint name="${imu_link_name}_joint" type="fixed">
+        <joint name="${imu_name}_joint" type="fixed">
             <origin xyz="${xyz}" rpy="${rpy}"/>
             <parent link="${connected_to}"/>
-            <child link="${imu_link_name}"/>
+            <child link="${imu_name}"/>
         </joint>
         <!-- Imu link -->
-        <link name="${imu_link_name}">
+        <link name="${imu_name}">
             <inertial>
                 <mass value="0.001"/>
@@ -42,8 +41,8 @@
             </material>
         </link>
-        <gazebo reference="${imu_link_name}">
+        <gazebo reference="${imu_name}">
             <material>Gazebo/Orange</material>
         </gazebo>
-        <gazebo reference="${imu_link_name}_joint">
+        <gazebo reference="${imu_name}_joint">
             <disableFixedJointLumping>true</disableFixedJointLumping>
         </gazebo>
@@ -52,7 +51,7 @@
                 <plugin name="smb_imu_plugin" filename="libhector_gazebo_ros_imu.so">
                     <updateRate>${imu_update_rate}</updateRate>
-                    <bodyName>${imu_link_name}</bodyName>
-                    <frameId>${imu_link_name}</frameId>
-                    <topicName>${imu_link_name}</topicName>
+                    <bodyName>${imu_name}</bodyName>
+                    <frameId>${imu_name}</frameId>
+                    <topicName>${imu_name}</topicName>
                     <serviceName>${imu_calibration_service_name}</serviceName>
                     <accelOffset>${acceleration_offset}</accelOffset>

File: urdf/common/lidar2d.urdf.xacro (robot description, xacro)
@@ -1,13 +1,13 @@
 <?xml version="1.0"?>
 <robot xmlns:xacro="http://www.ros.org/wiki/xacro" name="lidar2d">
-    <xacro:macro name="lidar2d" params="connected_to lidar_link_name simulation xyz:='0 0 0' rpy:='0 0 0' ">
+    <xacro:macro name="lidar2d" params="connected_to lidar_name simulation xyz:='0 0 0' rpy:='0 0 0' ">
         <!-- Lidar is fixed to the connected_to link -->
-        <joint name="${lidar_link_name}_joint" type="fixed">
+        <joint name="${lidar_name}_joint" type="fixed">
             <origin xyz="${xyz}" rpy="${rpy}"/>
             <parent link="${connected_to}"/>
-            <child link="${lidar_link_name}"/>
+            <child link="${lidar_name}"/>
         </joint>
         <!-- Lidar link -->
-        <link name="${lidar_link_name}">
+        <link name="${lidar_name}">
             <inertial>
                 <mass value="0.114"/>
@@ -32,5 +32,5 @@
         </link>
         <xacro:if value="${simulation}">
-            <gazebo reference="${lidar_link_name}">
+            <gazebo reference="${lidar_name}">
                 <material>Gazebo/FlatBlack</material>
                 <sensor type="ray" name="lds_lfcd_sensor">

File: urdf/standard/standard.urdf.xacro (robot description, xacro)
@@ -10,5 +10,5 @@
         <xacro:chassis roller_type="$(arg roller_type)"/>
         <xacro:include filename="$(find rm_description)/urdf/common/imu.urdf.xacro"/>
-        <xacro:IMU connected_to="base_link" imu_link_name="base_imu" simulation="true"
+        <xacro:IMU connected_to="base_link" imu_name="base_imu" simulation="true"
                    xyz="0.065 0.12 0.07"/>
     </xacro:if>
