Commit message: Remove track

File: urdf/sentry/chassis.transmission.urdf.xacro (robot description, xacro)
@@ -3,5 +3,5 @@
 <transmission name="trans_drive_joint">
     <type>transmission_interface/SimpleTransmission</type>
-    <actuator name="pitch_drive_joint">
+    <actuator name="drive_joint_motor">
         <hardwareInterface>hardware_interface/EffortJointInterface</hardwareInterface>
         <mechanicalReduction>1</mechanicalReduction>

File: urdf/sentry/chassis.urdf.xacro (robot description, xacro)
@@ -2,26 +2,4 @@
   <xacro:include filename="$(find rm_description)/urdf/sentry/driven_wheel.urdf.xacro"/>
   <xacro:macro name="chassis">
-    <!-- link -->
-    <link name="world"/>
-    <link name="link_track">
-      <inertial>
-        <mass value="29.08"/>
-        <origin xyz="0 0 0"/>
-        <inertia ixx="8.676e-2" ixy="0" ixz="0" iyy="2.432"
-                 iyz="0" izz="2.501"/>
-      </inertial>
-      <visual>
-        <origin xyz="0 0 0" rpy="0 0 0"/>
-        <geometry>
-          <mesh filename="package://rm_description/meshes/sentry/track.stl" scale="0.001 0.001 0.001"/>
-        </geometry>
-      </visual>
-      <collision>
-        <origin xyz="0 0 0" rpy="0 0 0"/>
-        <geometry>
-          <mesh filename="package://rm_description/meshes/sentry/track.stl" scale="0.001 0.001 0.001"/>
-        </geometry>
-      </collision>
-    </link>
     <link name="base_link">
       <inertial>
@@ -64,17 +42,4 @@
       </collision>
     </link>
-    <!-- joint -->
-    <joint name="track_joint" type="fixed">
-      <parent link="world"/>
-      <child link="link_track"/>
-      <origin xyz="0 0 0.5" rpy="0 0 0"/>
-    </joint>
-    <joint name="base_joint" type="prismatic">
-      <axis xyz="1 0 0"/>
-      <limit effort="1.2" velocity="34" lower="-${2*pi}" upper="${2*pi}"/>
-      <parent link="link_track"/>
-      <child link="base_link"/>
-      <origin xyz="0 -0.053 0.060" rpy="0 0 0"/>
-    </joint>
     <joint name="drive_joint" type="continuous">
       <axis xyz="0 1 0"/>

File: urdf/sentry/driven_wheel.urdf.xacro (robot description, xacro)
@@ -18,5 +18,6 @@
       </inertial>
       <collision>
-        <origin xyz="0 0 0" rpy="0 0 0"/>
+<!--        <origin xyz="0 0 0" rpy="0 0 0"/>-->
+        <xacro:insert_block name="pose"/>
         <geometry>
           <mesh filename="package://rm_description/meshes/sentry/driven_wheel.stl"

File: urdf/sentry/sentry.urdf.xacro (robot description, xacro)
@@ -4,6 +4,5 @@
     <xacro:arg name="load_gimbal" default="true"/>
     <xacro:arg name="load_shooter" default="true"/>
-    <xacro:arg name="load_gazebo" default="true"/>
-    <xacro:arg name="use_rm_gazebo" default="false"/>
+    <xacro:arg name="use_simulation" default="true"/>
     <xacro:if value="$(arg load_chassis)">
         <xacro:include filename="$(find rm_description)/urdf/sentry/chassis.urdf.xacro"/>
@@ -20,22 +19,11 @@
         <xacro:include filename="$(find rm_description)/urdf/sentry/shooter.transmission.urdf.xacro"/>
     </xacro:if>
-    <xacro:if value="$(arg load_gazebo)">
-        <xacro:if value="$(arg use_rm_gazebo)">
-            <gazebo>
-                <plugin name="rm_ros_control" filename="librm_robot_hw_sim.so">
-                    <robotNamespace>/</robotNamespace>
-                    <robotSimType>rm_gazebo/RmRobotHWSim</robotSimType>
-                </plugin>
-            </gazebo>
-        </xacro:if>
-        <xacro:unless value="$(arg use_rm_gazebo)">
-            <gazebo>
-                <plugin name="gazebo_ros_control" filename="libgazebo_ros_control.so">
-                    <robotNamespace>/mugator_manip</robotNamespace>
-                    <robotSimType>gazebo_ros_control/DefaultRobotHWSim</robotSimType>
-                    <legacyModeNS>true</legacyModeNS>
-                </plugin>
-            </gazebo>
-        </xacro:unless>
+    <xacro:if value="$(arg use_simulation)">
+        <gazebo>
+            <plugin name="rm_ros_control" filename="librm_robot_hw_sim.so">
+                <robotNamespace>/</robotNamespace>
+                <robotSimType>rm_gazebo/RmRobotHWSim</robotSimType>
+            </plugin>
+        </gazebo>
     </xacro:if>
 </robot>
