Commit message: Update shooter mechanicalReduction and pitch id

File: urdf/sentry/gimbal.urdf.xacro (robot description, xacro)
@@ -57,5 +57,5 @@
         <origin xyz="0 0 -0.1"/>
         <dynamics damping="0" friction="0.1"/>
-        <limit effort="${wheel_joint_effort}" velocity="${wheel_joint_velocity}" lower="0" upper="${pi/2}"/>
+        <limit effort="1.2" velocity="13.82" lower="0" upper="${pi/2}"/>
       </joint>
   </xacro:macro>

File: urdf/sentry/shooter.transmission.urdf.xacro (robot description, xacro)
@@ -5,5 +5,5 @@
         <actuator name="trigger_joint_motor">
             <hardwareInterface>hardware_interface/EffortJointInterface</hardwareInterface>
-            <mechanicalReduction>-1</mechanicalReduction>
+            <mechanicalReduction>1</mechanicalReduction>
         </actuator>
         <joint name="trigger_joint">
@@ -15,5 +15,5 @@
         <actuator name="left_friction_wheel_joint_motor">
             <hardwareInterface>hardware_interface/EffortJointInterface</hardwareInterface>
-            <mechanicalReduction>1</mechanicalReduction>
+            <mechanicalReduction>-1</mechanicalReduction>
         </actuator>
         <joint name="left_friction_wheel_joint">
@@ -25,5 +25,5 @@
         <actuator name="right_friction_wheel_joint_motor">
             <hardwareInterface>hardware_interface/EffortJointInterface</hardwareInterface>
-            <mechanicalReduction>1</mechanicalReduction>
+            <mechanicalReduction>-1</mechanicalReduction>
         </actuator>
         <joint name="right_friction_wheel_joint">

File: urdf/sentry/shooter.urdf.xacro (robot description, xacro)
@@ -31,5 +31,5 @@
     <origin xyz="0.0797 -0.0169 -0.2355" rpy="0 0 0"/>
     <dynamics damping="0.0" friction="0.01"/>
-    <limit effort="3.0" velocity="49.09" lower="-1e16" upper="1e16"/>
+    <limit effort="1.0" velocity="43.54" lower="-1e16" upper="1e16"/>
     <parent link="base_link"/>
     <child link="trigger"/>

Commit message: Add safety_controller in sentry

File: urdf/sentry/gimbal.urdf.xacro (robot description, xacro)
@@ -2,4 +2,7 @@
 <robot xmlns:xacro="http://www.ros.org/wiki/xacro">
   <xacro:macro name="gimbal">
+    <xacro:property name="threshold" value="0.1"/>
+    <xacro:property name="pitch_lower_limit" value="-0.716"/>
+    <xacro:property name="pitch_upper_limit" value="0.487"/>
     <link name="link_yaw">
       <visual>
@@ -57,5 +60,8 @@
         <origin xyz="0 0 -0.1"/>
         <dynamics damping="0" friction="0.1"/>
-        <limit effort="1.2" velocity="13.82" lower="0" upper="${pi/2}"/>
+        <limit effort="1.2" velocity="13.82" lower="${pitch_lower_limit}" upper="${pitch_upper_limit}"/>
+        <safety_controller k_position="100" k_velocity="0.1"
+                           soft_lower_limit="${pitch_lower_limit+threshold}"
+                           soft_upper_limit="${pitch_upper_limit-threshold}"/>
       </joint>
   </xacro:macro>

Commit message: pitch name change

File: urdf/sentry/gimbal.urdf.xacro (robot description, xacro)
@@ -2,5 +2,5 @@
 <robot xmlns:xacro="http://www.ros.org/wiki/xacro">
   <xacro:macro name="gimbal">
-    <link name="link_yaw">
+    <link name="yaw">
       <visual>
         <geometry>
@@ -25,5 +25,5 @@
     <joint name="yaw_joint" type="continuous">
       <parent link="base_link"/>
-      <child link="link_yaw"/>
+      <child link="yaw"/>
       <axis xyz="0 0 1"/>
       <origin xyz="0.0007 0.053 -0.31"/>
@@ -31,5 +31,5 @@
       <limit effort="1.2" velocity="34" lower="-${2*pi}" upper="${2*pi}"/>
     </joint>
-      <link name="link_pitch">
+      <link name="pitch">
         <inertial>
           <mass value="1.155968"/>
@@ -52,6 +52,6 @@
       </link>
       <joint name="pitch_joint" type="revolute">
-        <parent link="link_yaw"/>
-        <child link="link_pitch"/>
+        <parent link="yaw"/>
+        <child link="pitch"/>
         <axis xyz="1 0 0"/>
         <origin xyz="0 0 -0.1"/>

File: urdf/sentry/shooter.urdf.xacro (robot description, xacro)
@@ -4,7 +4,7 @@
   <xacro:property name="wheel_offset_y" value="-0.06594"/>
   <xacro:property name="wheel_offset_z" value="0.01132"/>
-  <xacro:friction_wheel prefixs="left" connected_to="link_pitch"
+  <xacro:friction_wheel prefixs="left" connected_to="pitch"
                         wheel_x_offset="${-wheel_offset_x}" wheel_y_offset="${wheel_offset_y}" wheel_z_offset="${wheel_offset_z}"/>
-  <xacro:friction_wheel prefixs="right" connected_to="link_pitch"
+  <xacro:friction_wheel prefixs="right" connected_to="pitch"
                         wheel_x_offset="${wheel_offset_x}" wheel_y_offset="${wheel_offset_y}" wheel_z_offset="${wheel_offset_z}"/>
   <link name="trigger">

Commit message: pitch name change

File: urdf/sentry/gimbal.urdf.xacro (robot description, xacro)
@@ -5,5 +5,5 @@
     <xacro:property name="pitch_lower_limit" value="0"/>
     <xacro:property name="pitch_upper_limit" value="0.767"/>
-    <link name="link_yaw">
+    <link name="yaw">
       <visual>
         <geometry>
@@ -28,5 +28,5 @@
     <joint name="yaw_joint" type="continuous">
       <parent link="base_link"/>
-      <child link="link_yaw"/>
+      <child link="yaw"/>
       <axis xyz="0 0 1"/>
       <origin xyz="0.0007 0.053 -0.31"/>
@@ -34,5 +34,5 @@
       <limit effort="1.2" velocity="34" lower="-${2*pi}" upper="${2*pi}"/>
     </joint>
-      <link name="link_pitch">
+      <link name="pitch">
         <inertial>
           <mass value="1.155968"/>
@@ -55,6 +55,6 @@
       </link>
       <joint name="pitch_joint" type="revolute">
-        <parent link="link_yaw"/>
-        <child link="link_pitch"/>
+        <parent link="yaw"/>
+        <child link="pitch"/>
         <axis xyz="1 0 0"/>
         <origin xyz="0 0 -0.1"/>

Commit message: Update sentry gimbal parameter

File: urdf/sentry/gimbal.urdf.xacro (robot description, xacro)
@@ -3,6 +3,6 @@
   <xacro:macro name="gimbal">
     <xacro:property name="threshold" value="0.1"/>
-    <xacro:property name="pitch_lower_limit" value="0"/>
-    <xacro:property name="pitch_upper_limit" value="0.767"/>
+    <xacro:property name="pitch_lower_limit" value="-0.537"/>
+    <xacro:property name="pitch_upper_limit" value="0.443"/>
     <link name="yaw">
       <visual>

Commit message: Add limit in gimbal and update parameter

File: urdf/sentry/gimbal.urdf.xacro (robot description, xacro)
@@ -3,6 +3,6 @@
   <xacro:macro name="gimbal">
     <xacro:property name="threshold" value="0.1"/>
-    <xacro:property name="pitch_lower_limit" value="0.192"/>
-    <xacro:property name="pitch_upper_limit" value="0.872"/>
+    <xacro:property name="pitch_lower_limit" value="0.241"/>
+    <xacro:property name="pitch_upper_limit" value="0.885"/>
     <link name="yaw">
       <visual>
@@ -34,35 +34,35 @@
       <limit effort="1.2" velocity="34" lower="-${2*pi}" upper="${2*pi}"/>
     </joint>
-      <link name="pitch">
-        <inertial>
-          <mass value="1.155968"/>
-          <origin xyz="0.019 -0.045 0.022"/>
-          <inertia ixx="5.918e-3" ixy="1.6863e-6" ixz="2.4143e-6" iyy="2.048e-3"
-                   iyz="-1.348e-4" izz="7.506e-3"/>
-        </inertial>
-        <visual>
-          <origin xyz="0 0 0" rpy="0 0 0"/>
-          <geometry>
-            <mesh filename="package://rm_description/meshes/sentry/pitch.stl" scale="0.001 0.001 0.001"/>
-          </geometry>
-        </visual>
-        <collision>
-          <origin xyz="0 0 0" rpy="0 0 0"/>
-          <geometry>
-            <mesh filename="package://rm_description/meshes/sentry/pitch.stl" scale="0.001 0.001 0.001"/>
-          </geometry>
-        </collision>
-      </link>
-      <joint name="pitch_joint" type="revolute">
-        <parent link="yaw"/>
-        <child link="pitch"/>
-        <axis xyz="0 1 0"/>
-        <origin xyz="0 0 -0.13"/>
-        <dynamics damping="0" friction="0.1"/>
-        <limit effort="1.2" velocity="13.82" lower="${pitch_lower_limit}" upper="${pitch_upper_limit}"/>
-<!--        <safety_controller k_position="100" k_velocity="0.1"
-                           soft_lower_limit="${pitch_lower_limit+threshold}"
-                           soft_upper_limit="${pitch_upper_limit-threshold}"/>-->
-      </joint>
+    <link name="pitch">
+      <inertial>
+        <mass value="1.155968"/>
+        <origin xyz="0.019 -0.045 0.022"/>
+        <inertia ixx="5.918e-3" ixy="1.6863e-6" ixz="2.4143e-6" iyy="2.048e-3"
+                 iyz="-1.348e-4" izz="7.506e-3"/>
+      </inertial>
+      <visual>
+        <origin xyz="0 0 0" rpy="0 0 0"/>
+        <geometry>
+          <mesh filename="package://rm_description/meshes/sentry/pitch.stl" scale="0.001 0.001 0.001"/>
+        </geometry>
+      </visual>
+      <collision>
+        <origin xyz="0 0 0" rpy="0 0 0"/>
+        <geometry>
+          <mesh filename="package://rm_description/meshes/sentry/pitch.stl" scale="0.001 0.001 0.001"/>
+        </geometry>
+      </collision>
+    </link>
+    <joint name="pitch_joint" type="revolute">
+      <parent link="yaw"/>
+      <child link="pitch"/>
+      <axis xyz="0 1 0"/>
+      <origin xyz="0 0 -0.13"/>
+      <dynamics damping="0" friction="0.1"/>
+      <limit effort="1.2" velocity="13.82" lower="${pitch_lower_limit}" upper="${pitch_upper_limit}"/>
+      <safety_controller k_position="100" k_velocity="0.1"
+                         soft_lower_limit="${pitch_lower_limit+threshold}"
+                         soft_upper_limit="${pitch_upper_limit-threshold}"/>
+    </joint>
   </xacro:macro>
 </robot>

Commit message: Update sentry gimbal urdf

File: urdf/sentry/gimbal.urdf.xacro (robot description, xacro)
@@ -57,11 +57,11 @@
         <parent link="yaw"/>
         <child link="pitch"/>
-        <axis xyz="0 1 0"/>
-        <origin xyz="0 0 -0.13"/>
+        <axis xyz="1 0 0"/>
+        <origin xyz="0 0 -0.1"/>
         <dynamics damping="0" friction="0.1"/>
         <limit effort="1.2" velocity="13.82" lower="${pitch_lower_limit}" upper="${pitch_upper_limit}"/>
-<!--        <safety_controller k_position="100" k_velocity="0.1"
-                           soft_lower_limit="${pitch_lower_limit+threshold}"
-                           soft_upper_limit="${pitch_upper_limit-threshold}"/>-->
+        <!--        <safety_controller k_position="100" k_velocity="0.1"
+                                   soft_lower_limit="${pitch_lower_limit+threshold}"
+                                   soft_upper_limit="${pitch_upper_limit-threshold}"/>-->
       </joint>
   </xacro:macro>
