Commit message: set sentry offset

File: urdf/sentry/gimbal.transmission.urdf.xacro (robot description, xacro)
@@ -8,5 +8,5 @@
         </actuator>
         <joint name="yaw_joint">
-            <offset>1.09</offset>
+            <offset>-5.477</offset>
             <hardwareInterface>hardware_interface/EffortJointInterface</hardwareInterface>
         </joint>
@@ -19,5 +19,5 @@
         </actuator>
         <joint name="pitch_joint">
-            <offset>-2.46</offset>
+            <offset>-5.417</offset>
             <hardwareInterface>hardware_interface/EffortJointInterface</hardwareInterface>
         </joint>

File: urdf/sentry/gimbal.urdf.xacro (robot description, xacro)
@@ -3,6 +3,6 @@
   <xacro:macro name="gimbal">
     <xacro:property name="threshold" value="0.1"/>
-    <xacro:property name="pitch_lower_limit" value="-0.716"/>
-    <xacro:property name="pitch_upper_limit" value="0.487"/>
+    <xacro:property name="pitch_lower_limit" value="0"/>
+    <xacro:property name="pitch_upper_limit" value="0.767"/>
     <link name="link_yaw">
       <visual>

Commit message: Update sentry config

File: urdf/sentry/gimbal.transmission.urdf.xacro (robot description, xacro)
@@ -8,5 +8,5 @@
         </actuator>
         <joint name="yaw_joint">
-            <offset>-5.477</offset>
+            <offset>-0.746</offset>
             <hardwareInterface>hardware_interface/EffortJointInterface</hardwareInterface>
         </joint>

File: urdf/sentry/gimbal.urdf.xacro (robot description, xacro)
@@ -30,5 +30,5 @@
       <child link="yaw"/>
       <axis xyz="0 0 1"/>
-      <origin xyz="0.0007 0.053 -0.31"/>
+      <origin xyz="0.00 0.0 -0.21"/>
       <dynamics damping="0" friction="0.1"/>
       <limit effort="1.2" velocity="34" lower="-${2*pi}" upper="${2*pi}"/>
@@ -57,11 +57,11 @@
         <parent link="yaw"/>
         <child link="pitch"/>
-        <axis xyz="1 0 0"/>
-        <origin xyz="0 0 -0.1"/>
+        <axis xyz="0 1 0"/>
+        <origin xyz="0 0 -0.13"/>
         <dynamics damping="0" friction="0.1"/>
         <limit effort="1.2" velocity="13.82" lower="${pitch_lower_limit}" upper="${pitch_upper_limit}"/>
-        <safety_controller k_position="100" k_velocity="0.1"
+<!--        <safety_controller k_position="100" k_velocity="0.1"
                            soft_lower_limit="${pitch_lower_limit+threshold}"
-                           soft_upper_limit="${pitch_upper_limit-threshold}"/>
+                           soft_upper_limit="${pitch_upper_limit-threshold}"/>-->
       </joint>
   </xacro:macro>

Commit message: Update sentry parameter and shooter launch

File: urdf/sentry/gimbal.transmission.urdf.xacro (robot description, xacro)
@@ -8,5 +8,5 @@
         </actuator>
         <joint name="yaw_joint">
-            <offset>-5.469</offset>
+            <offset>-3.881</offset>
             <hardwareInterface>hardware_interface/EffortJointInterface</hardwareInterface>
         </joint>
@@ -19,5 +19,5 @@
         </actuator>
         <joint name="pitch_joint">
-            <offset>-5.839</offset>
+            <offset>-5.213</offset>
             <hardwareInterface>hardware_interface/EffortJointInterface</hardwareInterface>
         </joint>

File: urdf/sentry/gimbal.urdf.xacro (robot description, xacro)
@@ -3,6 +3,6 @@
   <xacro:macro name="gimbal">
     <xacro:property name="threshold" value="0.1"/>
-    <xacro:property name="pitch_lower_limit" value="-0.537"/>
-    <xacro:property name="pitch_upper_limit" value="0.443"/>
+    <xacro:property name="pitch_lower_limit" value="0.192"/>
+    <xacro:property name="pitch_upper_limit" value="0.872"/>
     <link name="yaw">
       <visual>

Commit message: fix sentry gimbal but not finish

File: urdf/sentry/gimbal.transmission.urdf.xacro (robot description, xacro)
@@ -8,5 +8,5 @@
         </actuator>
         <joint name="yaw_joint">
-            <offset>-5.469</offset>
+            <offset>-3.909</offset>
             <hardwareInterface>hardware_interface/EffortJointInterface</hardwareInterface>
         </joint>
@@ -19,5 +19,5 @@
         </actuator>
         <joint name="pitch_joint">
-            <offset>-5.839</offset>
+            <offset>-5.211</offset>
             <hardwareInterface>hardware_interface/EffortJointInterface</hardwareInterface>
         </joint>

File: urdf/sentry/gimbal.urdf.xacro (robot description, xacro)
@@ -3,6 +3,6 @@
   <xacro:macro name="gimbal">
     <xacro:property name="threshold" value="0.1"/>
-    <xacro:property name="pitch_lower_limit" value="-0.537"/>
-    <xacro:property name="pitch_upper_limit" value="0.443"/>
+    <xacro:property name="pitch_lower_limit" value="0.241"/>
+    <xacro:property name="pitch_upper_limit" value="0.885"/>
     <link name="yaw">
       <visual>

Commit message: Update standard camare_optical_frame

File: urdf/sentry/gimbal.transmission.urdf.xacro (robot description, xacro)
@@ -7,5 +7,5 @@
         </actuator>
         <joint name="yaw_joint">
-            <offset>0.784</offset>
+            <offset>-3.211</offset>
             <hardwareInterface>hardware_interface/EffortJointInterface</hardwareInterface>
         </joint>

File: urdf/sentry/gimbal.urdf.xacro (robot description, xacro)
@@ -1,92 +1,97 @@
 <?xml version="1.0" encoding="utf-8"?>
 <robot xmlns:xacro="http://www.ros.org/wiki/xacro">
-    <xacro:property name="threshold" value="0.1"/>
-    <xacro:property name="pitch_lower_limit" value="0.241"/>
-    <xacro:property name="pitch_upper_limit" value="0.885"/>
-    <link name="yaw">
-      <visual>
-        <geometry>
-          <mesh filename="package://rm_description/meshes/sentry/yaw.stl"
-                scale="0.001 0.001 0.001"/>
-        </geometry>
-      </visual>
-      <inertial>
-        <mass value="0.225984"/>
-        <origin xyz="-0.0516 -0.01431 -0.03823" rpy="0 0 0"/>
-        <inertia ixx="7.196e-3" ixy="1.102e-3" ixz="-2.150e-3" iyy="2.478e-2"
-                 iyz="-1.186e-3" izz="2.488e-2"/>
-      </inertial>
-      <collision>
-        <origin xyz="0 0 0" rpy="0 0 0"/>
-        <geometry>
-          <mesh filename="package://rm_description/meshes/sentry/yaw.stl"
-                scale="0.001 0.001 0.001"/>
-        </geometry>
-      </collision>
-    </link>
-    <joint name="yaw_joint" type="continuous">
-      <parent link="base_link"/>
-      <child link="yaw"/>
-      <axis xyz="0 0 1"/>
-      <origin xyz="0.0 0.031 -0.2352"/>
-      <dynamics damping="0" friction="0.1"/>
-      <limit effort="1.2" velocity="34" lower="-${2*pi}" upper="${2*pi}"/>
-    </joint>
-    <link name="pitch">
-      <inertial>
-        <mass value="1.05"/>
-        <origin xyz="0.0 -0.022 -0.043"/>
-        <inertia ixx="5.350e-3" ixy="1.148e-3" ixz="-1.287e-5" iyy="1.055e-2"
-                 iyz="1.122e-3" izz="1.050e-2"/>
-      </inertial>
-      <visual>
-        <origin xyz="0 0 0" rpy="0 0 0"/>
-        <geometry>
-          <mesh filename="package://rm_description/meshes/sentry/pitch.stl" scale="0.001 0.001 0.001"/>
-        </geometry>
-      </visual>
-      <collision>
-        <origin xyz="0 0 0" rpy="0 0 0"/>
-        <geometry>
-          <mesh filename="package://rm_description/meshes/sentry/pitch.stl" scale="0.001 0.001 0.001"/>
-        </geometry>
-      </collision>
-    </link>
-    <joint name="pitch_joint" type="revolute">
-      <parent link="yaw"/>
-      <child link="pitch"/>
-      <axis xyz="0 1 0"/>
-      <origin xyz="0 0 -0.0799"/>
-      <dynamics damping="0" friction="0.1"/>
-      <limit effort="1.2" velocity="13.82" lower="${pitch_lower_limit}" upper="${pitch_upper_limit}"/>
-      <safety_controller k_position="100" k_velocity="0.1"
-                         soft_lower_limit="${pitch_lower_limit+threshold}"
-                         soft_upper_limit="${pitch_upper_limit-threshold}"/>
-    </joint>
-<!--    <link name="camera">-->
-<!--      <inertial>-->
-<!--        <mass value="0.17671"/>-->
-<!--        <origin xyz="0.022 0.0 0.0"/>-->
-<!--        <inertia ixx="2.129e-5" ixy="7.329e-8" ixz="-1.11e-7" iyy="2.198e-4" iyz="-8.04e-7" izz="2.197e-4"/>-->
-<!--      </inertial>-->
-<!--      <visual>-->
-<!--        <origin xyz=" 0 0 0 " rpy="0 -1.57 0"/>-->
-<!--        <geometry>-->
-<!--          <mesh filename="package://rm_description/meshes/common/camera.stl" scale="0.001 0.001 0.001"/>-->
-<!--        </geometry>-->
-<!--        <material name="Black"/>-->
-<!--      </visual>-->
-<!--      <collision>-->
-<!--        <origin xyz="0 0 0" rpy="0 -1.57 0"/>-->
-<!--        <geometry>-->
-<!--          <mesh filename="package://rm_description/meshes/common/camera.stl" scale="0.001 0.001 0.001"/>-->
-<!--        </geometry>-->
-<!--      </collision>-->
-<!--    </link>-->
-<!--    <joint name="camera_joint" type="fixed">-->
-<!--      <parent link="pitch"/>-->
-<!--      <child link="camera"/>-->
-<!--      <origin xyz="0.086  0.0 -0.040" rpy="-1.57 0 -1.57"/>-->
-<!--      <axis xyz="0 0 1"/>-->
-<!--    </joint>-->
+  <xacro:property name="threshold" value="0.1"/>
+  <xacro:property name="yaw_lower_limit" value="-3.0"/>
+  <xacro:property name="yaw_upper_limit" value="-0.2"/>
+  <xacro:property name="pitch_lower_limit" value="0.241"/>
+  <xacro:property name="pitch_upper_limit" value="0.885"/>
+  <link name="yaw">
+    <visual>
+      <geometry>
+        <mesh filename="package://rm_description/meshes/sentry/yaw.stl"
+              scale="0.001 0.001 0.001"/>
+      </geometry>
+    </visual>
+    <inertial>
+      <mass value="0.225984"/>
+      <origin xyz="-0.0516 -0.01431 -0.03823" rpy="0 0 0"/>
+      <inertia ixx="7.196e-3" ixy="1.102e-3" ixz="-2.150e-3" iyy="2.478e-2"
+               iyz="-1.186e-3" izz="2.488e-2"/>
+    </inertial>
+    <collision>
+      <origin xyz="0 0 0" rpy="0 0 0"/>
+      <geometry>
+        <mesh filename="package://rm_description/meshes/sentry/yaw.stl"
+              scale="0.001 0.001 0.001"/>
+      </geometry>
+    </collision>
+  </link>
+  <joint name="yaw_joint" type="revolute">
+    <parent link="base_link"/>
+    <child link="yaw"/>
+    <axis xyz="0 0 1"/>
+    <origin xyz="0.0 0.031 -0.2352"/>
+    <dynamics damping="0" friction="0.1"/>
+    <limit effort="1.2" velocity="34" lower="${yaw_lower_limit}" upper="${yaw_upper_limit}"/>
+    <safety_controller k_position="100" k_velocity="0.1"
+                       soft_lower_limit="${yaw_lower_limit+threshold}"
+                       soft_upper_limit="${yaw_upper_limit-threshold}"/>
+  </joint>
+  <link name="pitch">
+    <inertial>
+      <mass value="1.05"/>
+      <origin xyz="0.0 -0.022 -0.043"/>
+      <inertia ixx="5.350e-3" ixy="1.148e-3" ixz="-1.287e-5" iyy="1.055e-2"
+               iyz="1.122e-3" izz="1.050e-2"/>
+    </inertial>
+    <visual>
+      <origin xyz="0 0 0" rpy="0 0 0"/>
+      <geometry>
+        <mesh filename="package://rm_description/meshes/sentry/pitch.stl" scale="0.001 0.001 0.001"/>
+      </geometry>
+    </visual>
+    <collision>
+      <origin xyz="0 0 0" rpy="0 0 0"/>
+      <geometry>
+        <mesh filename="package://rm_description/meshes/sentry/pitch.stl" scale="0.001 0.001 0.001"/>
+      </geometry>
+    </collision>
+  </link>
+  <joint name="pitch_joint" type="revolute">
+    <parent link="yaw"/>
+    <child link="pitch"/>
+    <axis xyz="0 1 0"/>
+    <origin xyz="0 0 -0.0799"/>
+    <dynamics damping="0" friction="0.1"/>
+    <limit effort="1.2" velocity="13.82" lower="${pitch_lower_limit}" upper="${pitch_upper_limit}"/>
+    <safety_controller k_position="100" k_velocity="0.1"
+                       soft_lower_limit="${pitch_lower_limit+threshold}"
+                       soft_upper_limit="${pitch_upper_limit-threshold}"/>
+  </joint>
+  <!--    <link name="camera">-->
+  <!--      <inertial>-->
+  <!--        <mass value="0.17671"/>-->
+  <!--        <origin xyz="0.022 0.0 0.0"/>-->
+  <!--        <inertia ixx="2.129e-5" ixy="7.329e-8" ixz="-1.11e-7" iyy="2.198e-4" iyz="-8.04e-7" izz="2.197e-4"/>-->
+  <!--      </inertial>-->
+  <!--      <visual>-->
+  <!--        <origin xyz=" 0 0 0 " rpy="0 -1.57 0"/>-->
+  <!--        <geometry>-->
+  <!--          <mesh filename="package://rm_description/meshes/common/camera.stl" scale="0.001 0.001 0.001"/>-->
+  <!--        </geometry>-->
+  <!--        <material name="Black"/>-->
+  <!--      </visual>-->
+  <!--      <collision>-->
+  <!--        <origin xyz="0 0 0" rpy="0 -1.57 0"/>-->
+  <!--        <geometry>-->
+  <!--          <mesh filename="package://rm_description/meshes/common/camera.stl" scale="0.001 0.001 0.001"/>-->
+  <!--        </geometry>-->
+  <!--      </collision>-->
+  <!--    </link>-->
+  <!--    <joint name="camera_joint" type="fixed">-->
+  <!--      <parent link="pitch"/>-->
+  <!--      <child link="camera"/>-->
+  <!--      <origin xyz="0.086  0.0 -0.040" rpy="-1.57 0 -1.57"/>-->
+  <!--      <axis xyz="0 0 1"/>-->
+  <!--    </joint>-->
 </robot>

File: urdf/standard3/standard3.urdf.xacro (robot description, xacro)
@@ -19,5 +19,5 @@
         <xacro:camera_sensor xyz="0.127 0 -0.038" rpy="0 0 0" parent="pitch"
                              camera_sim="$(arg use_simulation)"/>
-        <xacro:camera_optical_frame xyz="0.153 0 -0.0525" rpy="${-pi/2} 0 ${-pi/2}" parent="pitch"
+        <xacro:camera_optical_frame xyz="0.153 0 -0.0525" rpy="${pi/2} 0 ${pi/2}" parent="pitch"
                                     camera_sim="$(arg use_simulation)"/>
     </xacro:if>

File: urdf/standard4/standard4.urdf.xacro (robot description, xacro)
@@ -18,5 +18,5 @@
         <xacro:camera_sensor xyz="0.127 0 -0.038" rpy="0 0 0" parent="pitch"
                              camera_sim="$(arg use_simulation)"/>
-        <xacro:camera_optical_frame xyz="0.153 0 -0.0525" rpy="${-pi/2} 0 ${-pi/2}" parent="pitch"
+        <xacro:camera_optical_frame xyz="0.153 0 -0.0525" rpy="${pi/2} 0 ${pi/2}" parent="pitch"
                                     camera_sim="$(arg use_simulation)"/>
     </xacro:if>
