Commit message: fix error of sentry urdf

File: urdf/sentry/lower_shooter.urdf.xacro (robot description, xacro)
@@ -31,5 +31,5 @@
   </link>
   <joint name="lower_trigger_joint" type="continuous">
-    <origin xyz="0 0.15 0.136" rpy="0 0 0"/>
+    <origin xyz="0 0.15 -0.136" rpy="0 0 0"/>
     <dynamics damping="0.0" friction="0.01"/>
     <limit effort="1.0" velocity="43.54" lower="-1e16" upper="1e16"/>

File: urdf/sentry/upper_shooter.urdf.xacro (robot description, xacro)
@@ -34,5 +34,5 @@
         <dynamics damping="0.0" friction="0.01"/>
         <limit effort="1.0" velocity="43.54" lower="-1e16" upper="1e16"/>
-        <parent link="base_link"/>
+        <parent link="upper_pitch"/>
         <child link="upper_trigger"/>
         <axis xyz="0 0 1 "/>
