Commit message: Update offset and reduction and limit

File: urdf/sentry/lower_gimbal.transmission.urdf.xacro (robot description, xacro)
@@ -4,8 +4,8 @@
         <type>transmission_interface/SimpleTransmission</type>
         <actuator name="lower_yaw_joint_motor">
-            <mechanicalReduction>1</mechanicalReduction>
+            <mechanicalReduction>-1</mechanicalReduction>
         </actuator>
         <joint name="lower_yaw_joint">
-            <offset>-1.523</offset>
+            <offset>2.736</offset>
             <hardwareInterface>hardware_interface/EffortJointInterface</hardwareInterface>
         </joint>
@@ -17,5 +17,5 @@
         </actuator>
         <joint name="lower_pitch_joint">
-            <offset>-5.211</offset>
+            <offset>0.97</offset>
             <hardwareInterface>hardware_interface/EffortJointInterface</hardwareInterface>
         </joint>

File: urdf/sentry/lower_gimbal.urdf.xacro (robot description, xacro)
@@ -3,7 +3,7 @@
   <xacro:property name="threshold" value="0.1"/>
   <xacro:property name="yaw_lower_limit" value="-3.0"/>
-  <xacro:property name="yaw_upper_limit" value="-0.2"/>
-  <xacro:property name="pitch_lower_limit" value="0.241"/>
-  <xacro:property name="pitch_upper_limit" value="0.885"/>
+  <xacro:property name="yaw_upper_limit" value="1.885"/>
+  <xacro:property name="pitch_lower_limit" value="0.009"/>
+  <xacro:property name="pitch_upper_limit" value="0.917"/>
   <link name="lower_yaw">
     <visual>

File: urdf/sentry/lower_shooter.transmission.urdf.xacro (robot description, xacro)
@@ -13,5 +13,5 @@
         <type>transmission_interface/SimpleTransmission</type>
         <actuator name="lower_left_friction_wheel_joint_motor">
-            <mechanicalReduction>-1</mechanicalReduction>
+            <mechanicalReduction>1</mechanicalReduction>
         </actuator>
         <joint name="lower_left_friction_wheel_joint">
@@ -22,5 +22,5 @@
         <type>transmission_interface/SimpleTransmission</type>
         <actuator name="lower_right_friction_wheel_joint_motor">
-            <mechanicalReduction>-1</mechanicalReduction>
+            <mechanicalReduction>1</mechanicalReduction>
         </actuator>
         <joint name="lower_right_friction_wheel_joint">

File: urdf/sentry/lower_shooter.urdf.xacro (robot description, xacro)
@@ -34,5 +34,5 @@
     <dynamics damping="0.0" friction="0.01"/>
     <limit effort="1.0" velocity="43.54" lower="-1e16" upper="1e16"/>
-    <parent link="base_link"/>
+    <parent link="lower_pitch"/>
     <child link="lower_trigger"/>
     <axis xyz="0 0 1 "/>

File: urdf/sentry/sentry.urdf.xacro (robot description, xacro)
@@ -2,8 +2,6 @@
 <robot xmlns:xacro="http://www.ros.org/wiki/xacro" name="sentry">
     <xacro:arg name="load_chassis" default="true"/>
-    <xacro:arg name="load_upper_gimbal" default="true"/>
-    <xacro:arg name="load_lower_gimbal" default="true"/>
-    <xacro:arg name="load_upper_shooter" default="true"/>
-    <xacro:arg name="load_lower_shooter" default="true"/>
+    <xacro:arg name="load_gimbal" default="true"/>
+    <xacro:arg name="load_shooter" default="true"/>
     <xacro:arg name="use_simulation" default="true"/>
     <xacro:if value="$(arg load_chassis)">
@@ -12,17 +10,15 @@
         <xacro:chassis use_simulation="$(arg use_simulation)"/>
     </xacro:if>
-    <xacro:if value="$(arg load_lower_gimbal)">
-        <xacro:include filename="lower_gimbal.urdf.xacro"/>
-        <xacro:include filename="lower_gimbal.transmission.urdf.xacro"/>
-        <xacro:include filename="$(find rm_description)/urdf/common/camera.urdf.xacro"/>
+    <xacro:if value="$(arg load_gimbal)">
+        <xacro:include filename="$(find rm_description)/urdf/sentry/lower_gimbal.urdf.xacro"/>
+        <xacro:include filename="$(find rm_description)/urdf/sentry/lower_gimbal.transmission.urdf.xacro"/>
+<!--        <xacro:include filename="$(find rm_description)/urdf/common/camera.urdf.xacro"/>-->
         <!--        <xacro:camera_sensor xyz="0.127 0 -0.047" rpy="0 0 0" parent="lower_pitch"-->
         <!--                             camera_sim="$(arg use_simulation)"/>-->
         <!--        <xacro:camera_optical_frame xyz="0.153 0 -0.0615" rpy="${-pi/2} 0 ${-pi/2}" parent="lower_pitch"-->
         <!--                                    camera_sim="$(arg use_simulation)"/>-->
-    </xacro:if>
-    <xacro:if value="$(arg load_upper_gimbal)">
-        <xacro:include filename="upper_gimbal.urdf.xacro"/>
-        <xacro:include filename="upper_gimbal.transmission.urdf.xacro"/>
-        <xacro:include filename="$(find rm_description)/urdf/common/camera.urdf.xacro"/>
+        <xacro:include filename="$(find rm_description)/urdf/sentry/upper_gimbal.urdf.xacro"/>
+        <xacro:include filename="$(find rm_description)/urdf/sentry/upper_gimbal.transmission.urdf.xacro"/>
+        <!--        <xacro:include filename="$(find rm_description)/urdf/common/camera.urdf.xacro"/>-->
         <!--        <xacro:camera_sensor xyz="0.127 0 -0.047" rpy="0 0 0" parent="upper_pitch"-->
         <!--                             camera_sim="$(arg use_simulation)"/>-->
@@ -30,9 +26,7 @@
         <!--                                    camera_sim="$(arg use_simulation)"/>-->
     </xacro:if>
-    <xacro:if value="$(arg load_upper_shooter)">
+    <xacro:if value="$(arg load_shooter)">
         <xacro:include filename="$(find rm_description)/urdf/sentry/upper_shooter.urdf.xacro"/>
         <xacro:include filename="$(find rm_description)/urdf/sentry/upper_shooter.transmission.urdf.xacro"/>
-    </xacro:if>
-    <xacro:if value="$(arg load_lower_shooter)">
         <xacro:include filename="$(find rm_description)/urdf/sentry/lower_shooter.urdf.xacro"/>
         <xacro:include filename="$(find rm_description)/urdf/sentry/lower_shooter.transmission.urdf.xacro"/>

File: urdf/sentry/upper_gimbal.transmission.urdf.xacro (robot description, xacro)
@@ -7,5 +7,5 @@
         </actuator>
         <joint name="upper_yaw_joint">
-            <offset>-3.211</offset>
+            <offset>2.165</offset>
             <hardwareInterface>hardware_interface/EffortJointInterface</hardwareInterface>
         </joint>
@@ -17,5 +17,5 @@
         </actuator>
         <joint name="upper_pitch_joint">
-            <offset>-5.211</offset>
+            <offset>0.485</offset>
             <hardwareInterface>hardware_interface/EffortJointInterface</hardwareInterface>
         </joint>

File: urdf/sentry/upper_gimbal.urdf.xacro (robot description, xacro)
@@ -2,8 +2,8 @@
 <robot xmlns:xacro="http://www.ros.org/wiki/xacro">
     <xacro:property name="threshold" value="0.1"/>
-    <xacro:property name="yaw_lower_limit" value="-3.0"/>
-    <xacro:property name="yaw_upper_limit" value="-0.2"/>
-    <xacro:property name="pitch_lower_limit" value="0.241"/>
-    <xacro:property name="pitch_upper_limit" value="0.885"/>
+    <xacro:property name="yaw_lower_limit" value="-3.764"/>
+    <xacro:property name="yaw_upper_limit" value="2.1"/>
+    <xacro:property name="pitch_lower_limit" value="-0.6"/>
+    <xacro:property name="pitch_upper_limit" value="0.6"/>
     <link name="upper_yaw">
         <visual>
@@ -33,5 +33,5 @@
         <origin xyz="0 0 83.4e-3"/>
         <dynamics damping="0" friction="0.1"/>
-        <limit effort="1.2" velocity="34" lower="${yaw_lower_limit}" upper="${yaw_upper_limit}"/>
+        <limit effort="1.2" velocity="13.82" lower="${yaw_lower_limit}" upper="${yaw_upper_limit}"/>
         <safety_controller k_position="100" k_velocity="0.1"
                            soft_lower_limit="${yaw_lower_limit+threshold}"

File: urdf/sentry/upper_shooter.transmission.urdf.xacro (robot description, xacro)
@@ -13,5 +13,5 @@
         <type>transmission_interface/SimpleTransmission</type>
         <actuator name="upper_left_friction_wheel_joint_motor">
-            <mechanicalReduction>-1</mechanicalReduction>
+            <mechanicalReduction>1</mechanicalReduction>
         </actuator>
         <joint name="upper_left_friction_wheel_joint">
@@ -22,5 +22,5 @@
         <type>transmission_interface/SimpleTransmission</type>
         <actuator name="upper_right_friction_wheel_joint_motor">
-            <mechanicalReduction>-1</mechanicalReduction>
+            <mechanicalReduction>1</mechanicalReduction>
         </actuator>
         <joint name="upper_right_friction_wheel_joint">

Commit message: Update offset and limit

File: urdf/sentry/lower_gimbal.transmission.urdf.xacro (robot description, xacro)
@@ -7,5 +7,5 @@
         </actuator>
         <joint name="lower_yaw_joint">
-            <offset>2.736</offset>
+            <offset>2.011</offset>
             <hardwareInterface>hardware_interface/EffortJointInterface</hardwareInterface>
         </joint>
@@ -17,5 +17,5 @@
         </actuator>
         <joint name="lower_pitch_joint">
-            <offset>0.97</offset>
+            <offset>1.151</offset>
             <hardwareInterface>hardware_interface/EffortJointInterface</hardwareInterface>
         </joint>

File: urdf/sentry/lower_gimbal.urdf.xacro (robot description, xacro)
@@ -2,8 +2,8 @@
 <robot xmlns:xacro="http://www.ros.org/wiki/xacro">
   <xacro:property name="threshold" value="0.1"/>
-  <xacro:property name="yaw_lower_limit" value="-3.0"/>
-  <xacro:property name="yaw_upper_limit" value="1.885"/>
-  <xacro:property name="pitch_lower_limit" value="0.009"/>
-  <xacro:property name="pitch_upper_limit" value="0.917"/>
+  <xacro:property name="yaw_lower_limit" value="-2.461"/>
+  <xacro:property name="yaw_upper_limit" value="1.998"/>
+  <xacro:property name="pitch_lower_limit" value="0.112"/>
+  <xacro:property name="pitch_upper_limit" value="1.157"/>
   <link name="lower_yaw">
     <visual>

File: urdf/sentry/lower_shooter.transmission.urdf.xacro (robot description, xacro)
@@ -13,5 +13,5 @@
         <type>transmission_interface/SimpleTransmission</type>
         <actuator name="lower_left_friction_wheel_joint_motor">
-            <mechanicalReduction>1</mechanicalReduction>
+            <mechanicalReduction>-1</mechanicalReduction>
         </actuator>
         <joint name="lower_left_friction_wheel_joint">
@@ -22,5 +22,5 @@
         <type>transmission_interface/SimpleTransmission</type>
         <actuator name="lower_right_friction_wheel_joint_motor">
-            <mechanicalReduction>1</mechanicalReduction>
+            <mechanicalReduction>-1</mechanicalReduction>
         </actuator>
         <joint name="lower_right_friction_wheel_joint">

File: urdf/sentry/upper_gimbal.transmission.urdf.xacro (robot description, xacro)
@@ -7,5 +7,5 @@
         </actuator>
         <joint name="upper_yaw_joint">
-            <offset>2.165</offset>
+            <offset>3.021</offset>
             <hardwareInterface>hardware_interface/EffortJointInterface</hardwareInterface>
         </joint>
@@ -17,5 +17,5 @@
         </actuator>
         <joint name="upper_pitch_joint">
-            <offset>0.485</offset>
+            <offset>0.498</offset>
             <hardwareInterface>hardware_interface/EffortJointInterface</hardwareInterface>
         </joint>

File: urdf/sentry/upper_gimbal.urdf.xacro (robot description, xacro)
@@ -2,8 +2,8 @@
 <robot xmlns:xacro="http://www.ros.org/wiki/xacro">
     <xacro:property name="threshold" value="0.1"/>
-    <xacro:property name="yaw_lower_limit" value="-3.764"/>
-    <xacro:property name="yaw_upper_limit" value="2.1"/>
-    <xacro:property name="pitch_lower_limit" value="-0.6"/>
-    <xacro:property name="pitch_upper_limit" value="0.6"/>
+    <xacro:property name="yaw_lower_limit" value="-2.949"/>
+    <xacro:property name="yaw_upper_limit" value="3.027"/>
+    <xacro:property name="pitch_lower_limit" value="-0.843"/>
+    <xacro:property name="pitch_upper_limit" value="0.472"/>
     <link name="upper_yaw">
         <visual>

File: urdf/sentry/upper_shooter.transmission.urdf.xacro (robot description, xacro)
@@ -13,5 +13,5 @@
         <type>transmission_interface/SimpleTransmission</type>
         <actuator name="upper_left_friction_wheel_joint_motor">
-            <mechanicalReduction>1</mechanicalReduction>
+            <mechanicalReduction>-1</mechanicalReduction>
         </actuator>
         <joint name="upper_left_friction_wheel_joint">
@@ -22,5 +22,5 @@
         <type>transmission_interface/SimpleTransmission</type>
         <actuator name="upper_right_friction_wheel_joint_motor">
-            <mechanicalReduction>1</mechanicalReduction>
+            <mechanicalReduction>-1</mechanicalReduction>
         </actuator>
         <joint name="upper_right_friction_wheel_joint">
