Commit message: Update to load the driven wheel only when running the simulation

File: urdf/sentry/chassis.urdf.xacro (robot description, xacro)
@@ -1,5 +1,5 @@
 <robot xmlns:xacro="http://www.ros.org/wiki/xacro">
   <xacro:include filename="$(find rm_description)/urdf/sentry/driven_wheel.urdf.xacro"/>
-  <xacro:macro name="chassis">
+  <xacro:macro name="chassis" params="use_simulation">
     <link name="base_link">
       <inertial>
@@ -49,29 +49,31 @@
       <origin xyz="0 0 0" rpy="0 0 0"/>
     </joint>
-    <xacro:driven_wheel num="1">
-      <origin rpy="0 0 0"/>
-      <axis xyz="0 1 0"/>
-      <origin xyz="-0.1 0.118 -0.015" rpy="0 0 0"/>
-    </xacro:driven_wheel>
-    <xacro:driven_wheel num="2">
-      <origin rpy="0 0 0"/>
-      <axis xyz="0 1 0"/>
-      <origin xyz="0.1 0.118 -0.015" rpy="0 0 0"/>
-    </xacro:driven_wheel>
-    <xacro:driven_wheel num="3">
-      <origin rpy="${pi/2} 0 0"/>
-      <axis xyz="0 0 1"/>
-      <origin xyz="-0.1 0.158 -0.0635" rpy="0 0 0"/>
-    </xacro:driven_wheel>
-    <xacro:driven_wheel num="4">
-      <origin rpy="${pi/2} 0 0"/>
-      <axis xyz="0 0 1"/>
-      <origin xyz="0.1 0.158 -0.0635" rpy="0 0 0"/>
-    </xacro:driven_wheel>
-    <xacro:driven_wheel num="5">
-      <origin rpy="${pi/2} 0 0"/>
-      <axis xyz="0 0 1"/>
-      <origin xyz="0 -0.052 -0.0635" rpy="0 0 0"/>
-    </xacro:driven_wheel>
+    <xacro:if value="$(arg use_simulation)">
+      <xacro:driven_wheel num="1">
+        <origin rpy="0 0 0"/>
+        <axis xyz="0 1 0"/>
+        <origin xyz="-0.1 0.118 -0.015" rpy="0 0 0"/>
+      </xacro:driven_wheel>
+      <xacro:driven_wheel num="2">
+        <origin rpy="0 0 0"/>
+        <axis xyz="0 1 0"/>
+        <origin xyz="0.1 0.118 -0.015" rpy="0 0 0"/>
+      </xacro:driven_wheel>
+      <xacro:driven_wheel num="3">
+        <origin rpy="${pi/2} 0 0"/>
+        <axis xyz="0 0 1"/>
+        <origin xyz="-0.1 0.158 -0.0635" rpy="0 0 0"/>
+      </xacro:driven_wheel>
+      <xacro:driven_wheel num="4">
+        <origin rpy="${pi/2} 0 0"/>
+        <axis xyz="0 0 1"/>
+        <origin xyz="0.1 0.158 -0.0635" rpy="0 0 0"/>
+      </xacro:driven_wheel>
+      <xacro:driven_wheel num="5">
+        <origin rpy="${pi/2} 0 0"/>
+        <axis xyz="0 0 1"/>
+        <origin xyz="0 -0.052 -0.0635" rpy="0 0 0"/>
+      </xacro:driven_wheel>
+    </xacro:if>
   </xacro:macro>
 </robot>

File: urdf/sentry/driven_wheel.urdf.xacro (robot description, xacro)
@@ -2,15 +2,15 @@
   <xacro:property name="wheel_joint_effort" value="5"/>
   <xacro:property name="wheel_joint_velocity" value="50"/>
-  <xacro:macro name="driven_wheel" params="num *pose *axis *origin">
-    <link name="link_driven_wheel${num}">
-      <visual>
-        <xacro:insert_block name="pose"/>
-        <geometry>
-          <mesh filename="package://rm_description/meshes/sentry/driven_wheel.stl"
-                scale="0.001 0.001 0.001"/>
-        </geometry>
-      </visual>
-      <inertial>
-        <mass value="9.665e-3"/>
+  <xacro:macro name="driven_wheel" params="num *pose *axis *origin ">
+      <link name="link_driven_wheel${num}">
+          <visual>
+              <xacro:insert_block name="pose"/>
+              <geometry>
+                  <mesh filename="package://rm_description/meshes/sentry/driven_wheel.stl"
+                        scale="0.001 0.001 0.001"/>
+              </geometry>
+          </visual>
+          <inertial>
+              <mass value="9.665e-3"/>
         <origin xyz="0 0 0" rpy="0 0 0"/>
         <inertia ixx="7.0766e-7" ixy="0" ixz="0" iyy="1.0067e-6"

File: urdf/sentry/sentry.urdf.xacro (robot description, xacro)
@@ -8,5 +8,5 @@
         <xacro:include filename="$(find rm_description)/urdf/sentry/chassis.urdf.xacro"/>
         <xacro:include filename="$(find rm_description)/urdf/sentry/chassis.transmission.urdf.xacro"/>
-        <xacro:chassis/>
+        <xacro:chassis use_simulation="$(arg use_simulation)"/>
     </xacro:if>
     <xacro:if value="$(arg load_gimbal)">

Commit message: fix driven_wheel

File: urdf/sentry/chassis.urdf.xacro (robot description, xacro)
@@ -51,27 +51,27 @@
     <xacro:if value="$(arg use_simulation)">
       <xacro:driven_wheel num="1">
-        <origin rpy="0 0 0"/>
+        <origin rpy="${-pi/2} 0 0"/>
         <axis xyz="0 1 0"/>
-        <origin xyz="-0.1 0.118 -0.015" rpy="0 0 0"/>
+        <origin xyz="-0.0977 0.0839 -0.013" rpy="0 0 0"/>
       </xacro:driven_wheel>
       <xacro:driven_wheel num="2">
-        <origin rpy="0 0 0"/>
+        <origin rpy="${-pi/2} 0 0"/>
         <axis xyz="0 1 0"/>
-        <origin xyz="0.1 0.118 -0.015" rpy="0 0 0"/>
+        <origin xyz="0.0977 0.0839 -0.013" rpy="0 0 0"/>
       </xacro:driven_wheel>
       <xacro:driven_wheel num="3">
-        <origin rpy="${pi/2} 0 0"/>
+        <origin rpy="0 0 0"/>
         <axis xyz="0 0 1"/>
-        <origin xyz="-0.1 0.158 -0.0635" rpy="0 0 0"/>
+        <origin xyz="-0.0982 0.135 -0.0571" rpy="0 0 0"/>
       </xacro:driven_wheel>
       <xacro:driven_wheel num="4">
-        <origin rpy="${pi/2} 0 0"/>
+        <origin rpy="0 0 0"/>
         <axis xyz="0 0 1"/>
-        <origin xyz="0.1 0.158 -0.0635" rpy="0 0 0"/>
+        <origin xyz="0.0982 0.135 -0.0571" rpy="0 0 0"/>
       </xacro:driven_wheel>
       <xacro:driven_wheel num="5">
-        <origin rpy="${pi/2} 0 0"/>
+        <origin rpy="0 0 0"/>
         <axis xyz="0 0 1"/>
-        <origin xyz="0 -0.052 -0.0635" rpy="0 0 0"/>
+        <origin xyz="0 -0.073 -0.0572" rpy="0 0 0"/>
       </xacro:driven_wheel>
     </xacro:if>

Commit message: Add cover joint on sentry

File: urdf/sentry/chassis.urdf.xacro (robot description, xacro)
@@ -77,3 +77,28 @@
         </xacro:if>
     </xacro:macro>
+    <link name="cover">
+    <inertial>
+        <mass value="0.118"/>
+        <origin xyz="-0.037 -0.003 0.0"/>
+        <inertia ixx="6.240e-4" ixy="7.325e-4" ixz="1.839e-5" iyy="1.083e-3" iyz="-1.166e-5" izz="1.602e-3"/>
+    </inertial>
+    </link>
+    <joint name="cover_joint" type="revolute">
+        <axis xyz="1 0 0"/>
+        <origin xyz="-0.27 0.201 0.125"/>
+        <limit effort="1" velocity="30" lower="-3.14" upper="3.14"/>
+        <dynamics damping="0.0" friction="0.1"/>
+        <parent link="pitch"/>
+        <child link="cover"/>
+    </joint>
+    <transmission name="trans_cover_joint">
+        <type>transmission_interface/SimpleTransmission</type>
+        <actuator name="cover_joint_motor">
+            <mechanicalReduction>1</mechanicalReduction>
+        </actuator>
+        <joint name="cover_joint">
+            <offset>0</offset>
+            <hardwareInterface>hardware_interface/EffortJointInterface</hardwareInterface>
+        </joint>
+    </transmission>
 </robot>

Commit message: conplete chassis and gimbal of sentry

File: urdf/sentry/chassis.urdf.xacro (robot description, xacro)
@@ -4,8 +4,8 @@
         <link name="base_link">
             <inertial>
-                <mass value="8.250"/>
-                <origin xyz="0.0 0.051 -0.148"/>
-                <inertia ixx="3.838e-1" ixy="1.075e-2" ixz="1.397e-5" iyy="2.601e-1"
-                         iyz="7.528e-2" izz="2.369e-1"/>
+                <mass value="6982.046e-3"/>
+                <origin xyz="2.335e-3 21.529e-3 -63.905e-3"/>
+                <inertia ixx="1.984e-1" ixy="1.366e-3" ixz="2.748e-3" iyy="1.284e-1"
+                         iyz="3.820e-3" izz="1.524e-1"/>
             </inertial>
             <visual>
@@ -24,8 +24,8 @@
         <link name="drive_wheel_link">
             <inertial>
-                <mass value="0.0839"/>
-                <origin xyz="0 0.01 0"/>
-                <inertia ixx="3.345e-5" ixy="0" ixz="0" iyy="-8.387e-5"
-                         iyz="-2.8558e-8" izz="3.347e-5"/>
+                <mass value="65.448e-3"/>
+                <origin xyz="0.027e-3 29.066e-3 0.001e-3"/>
+                <inertia ixx="74809.989e-9" ixy="-10.328e-9" ixz="-0.001e-9" iyy="32620.511e-9"
+                         iyz="-2.066e-9" izz="74795.135e-9"/>
             </inertial>
             <visual>
@@ -47,5 +47,5 @@
             <parent link="base_link"/>
             <child link="drive_wheel_link"/>
-            <origin xyz="0 -0.0185 0" rpy="0 0 0"/>
+            <origin xyz="0 -63.36e-3 5e-3" rpy="0 0 0"/>
         </joint>
         <xacro:if value="$(arg use_simulation)">
@@ -77,28 +77,28 @@
         </xacro:if>
     </xacro:macro>
-    <link name="cover">
-    <inertial>
-        <mass value="0.118"/>
-        <origin xyz="-0.037 -0.003 0.0"/>
-        <inertia ixx="6.240e-4" ixy="7.325e-4" ixz="1.839e-5" iyy="1.083e-3" iyz="-1.166e-5" izz="1.602e-3"/>
-    </inertial>
-    </link>
-    <joint name="cover_joint" type="revolute">
-        <axis xyz="1 0 0"/>
-        <origin xyz="-0.27 0.201 0.125"/>
-        <limit effort="1" velocity="30" lower="-3.14" upper="3.14"/>
-        <dynamics damping="0.0" friction="0.1"/>
-        <parent link="pitch"/>
-        <child link="cover"/>
-    </joint>
-    <transmission name="trans_cover_joint">
-        <type>transmission_interface/SimpleTransmission</type>
-        <actuator name="cover_joint_motor">
-            <mechanicalReduction>1</mechanicalReduction>
-        </actuator>
-        <joint name="cover_joint">
-            <offset>0</offset>
-            <hardwareInterface>hardware_interface/EffortJointInterface</hardwareInterface>
-        </joint>
-    </transmission>
+    <!--    <link name="cover">-->
+    <!--    <inertial>-->
+    <!--        <mass value="0.118"/>-->
+    <!--        <origin xyz="-0.037 -0.003 0.0"/>-->
+    <!--        <inertia ixx="6.240e-4" ixy="7.325e-4" ixz="1.839e-5" iyy="1.083e-3" iyz="-1.166e-5" izz="1.602e-3"/>-->
+    <!--    </inertial>-->
+    <!--    </link>-->
+    <!--    <joint name="cover_joint" type="revolute">-->
+    <!--        <axis xyz="1 0 0"/>-->
+    <!--        <origin xyz="-0.27 0.201 0.125"/>-->
+    <!--        <limit effort="1" velocity="30" lower="-3.14" upper="3.14"/>-->
+    <!--        <dynamics damping="0.0" friction="0.1"/>-->
+    <!--        <parent link="pitch"/>-->
+    <!--        <child link="cover"/>-->
+    <!--    </joint>-->
+    <!--    <transmission name="trans_cover_joint">-->
+    <!--        <type>transmission_interface/SimpleTransmission</type>-->
+    <!--        <actuator name="cover_joint_motor">-->
+    <!--            <mechanicalReduction>1</mechanicalReduction>-->
+    <!--        </actuator>-->
+    <!--        <joint name="cover_joint">-->
+    <!--            <offset>0</offset>-->
+    <!--            <hardwareInterface>hardware_interface/EffortJointInterface</hardwareInterface>-->
+    <!--        </joint>-->
+    <!--    </transmission>-->
 </robot>

File: urdf/sentry/gimbal.transmission.urdf.xacro (robot description, xacro)
@@ -1,20 +1,40 @@
 <?xml version="1.0" encoding="utf-8"?>
 <robot>
-    <transmission name="trans_yaw_joint">
+    <transmission name="trans_upper_yaw_joint">
         <type>transmission_interface/SimpleTransmission</type>
-        <actuator name="yaw_joint_motor">
+        <actuator name="upper_yaw_joint_motor">
             <mechanicalReduction>1</mechanicalReduction>
         </actuator>
-        <joint name="yaw_joint">
+        <joint name="upper_yaw_joint">
             <offset>-3.211</offset>
             <hardwareInterface>hardware_interface/EffortJointInterface</hardwareInterface>
         </joint>
     </transmission>
-    <transmission name="trans_pitch_joint">
+    <transmission name="trans_upper_pitch_joint">
         <type>transmission_interface/SimpleTransmission</type>
-        <actuator name="pitch_joint_motor">
+        <actuator name="upper_pitch_joint_motor">
             <mechanicalReduction>1</mechanicalReduction>
         </actuator>
-        <joint name="pitch_joint">
+        <joint name="upper_pitch_joint">
+            <offset>-5.211</offset>
+            <hardwareInterface>hardware_interface/EffortJointInterface</hardwareInterface>
+        </joint>
+    </transmission>
+    <transmission name="trans_lower_yaw_joint">
+        <type>transmission_interface/SimpleTransmission</type>
+        <actuator name="lower_yaw_joint_motor">
+            <mechanicalReduction>1</mechanicalReduction>
+        </actuator>
+        <joint name="lower_yaw_joint">
+            <offset>-3.211</offset>
+            <hardwareInterface>hardware_interface/EffortJointInterface</hardwareInterface>
+        </joint>
+    </transmission>
+    <transmission name="trans_lower_pitch_joint">
+        <type>transmission_interface/SimpleTransmission</type>
+        <actuator name="lower_pitch_joint_motor">
+            <mechanicalReduction>1</mechanicalReduction>
+        </actuator>
+        <joint name="lower_pitch_joint">
             <offset>-5.211</offset>
             <hardwareInterface>hardware_interface/EffortJointInterface</hardwareInterface>

File: urdf/sentry/gimbal.urdf.xacro (robot description, xacro)
@@ -6,30 +6,30 @@
   <xacro:property name="pitch_lower_limit" value="0.241"/>
   <xacro:property name="pitch_upper_limit" value="0.885"/>
-  <link name="yaw">
+  <link name="upper_yaw">
     <visual>
       <geometry>
-        <mesh filename="package://rm_description/meshes/sentry/yaw.stl"
+        <mesh filename="package://rm_description/meshes/sentry/upper_yaw.stl"
               scale="0.001 0.001 0.001"/>
       </geometry>
     </visual>
     <inertial>
-      <mass value="0.225984"/>
-      <origin xyz="-0.0516 -0.01431 -0.03823" rpy="0 0 0"/>
-      <inertia ixx="7.196e-3" ixy="1.102e-3" ixz="-2.150e-3" iyy="2.478e-2"
-               iyz="-1.186e-3" izz="2.488e-2"/>
+      <mass value="934.339e-3"/>
+      <origin xyz="-0.08e-3 -61.185e-3 90.777e-3" rpy="0 0 0"/>
+      <inertia ixx="1.880e-2" ixy="-6662.219e-9" ixz="7064.827e-9" iyy="1.083e-2"
+               iyz="7.150e-3" izz="9.057e-3"/>
     </inertial>
     <collision>
       <origin xyz="0 0 0" rpy="0 0 0"/>
       <geometry>
-        <mesh filename="package://rm_description/meshes/sentry/yaw.stl"
+        <mesh filename="package://rm_description/meshes/sentry/upper_yaw.stl"
               scale="0.001 0.001 0.001"/>
       </geometry>
     </collision>
   </link>
-  <joint name="yaw_joint" type="revolute">
+  <joint name="upper_yaw_joint" type="revolute">
     <parent link="base_link"/>
-    <child link="yaw"/>
+    <child link="upper_yaw"/>
     <axis xyz="0 0 1"/>
-    <origin xyz="0.0 0.031 -0.2352"/>
+    <origin xyz="0 0 83.4e-3"/>
     <dynamics damping="0" friction="0.1"/>
     <limit effort="1.2" velocity="34" lower="${yaw_lower_limit}" upper="${yaw_upper_limit}"/>
@@ -38,15 +38,15 @@
                        soft_upper_limit="${yaw_upper_limit-threshold}"/>
   </joint>
-  <link name="pitch">
+  <link name="upper_pitch">
     <inertial>
-      <mass value="1.05"/>
-      <origin xyz="0.0 -0.022 -0.043"/>
-      <inertia ixx="5.350e-3" ixy="1.148e-3" ixz="-1.287e-5" iyy="1.055e-2"
-               iyz="1.122e-3" izz="1.050e-2"/>
+      <mass value="1227.797e-3"/>
+      <origin xyz="15.667e-3 -0.268e-3 27.267e-3"/>
+      <inertia ixx="4.484e-3" ixy="813.964e-9" ixz="2.786e-4" iyy="6.599e-3"
+               iyz="-6822.846e-9" izz="5.343E-3"/>
     </inertial>
     <visual>
       <origin xyz="0 0 0" rpy="0 0 0"/>
       <geometry>
-        <mesh filename="package://rm_description/meshes/sentry/pitch.stl" scale="0.001 0.001 0.001"/>
+        <mesh filename="package://rm_description/meshes/sentry/upper_pitch.stl" scale="0.001 0.001 0.001"/>
       </geometry>
     </visual>
@@ -54,13 +54,13 @@
       <origin xyz="0 0 0" rpy="0 0 0"/>
       <geometry>
-        <mesh filename="package://rm_description/meshes/sentry/pitch.stl" scale="0.001 0.001 0.001"/>
+        <mesh filename="package://rm_description/meshes/sentry/upper_pitch.stl" scale="0.001 0.001 0.001"/>
       </geometry>
     </collision>
   </link>
-  <joint name="pitch_joint" type="revolute">
-    <parent link="yaw"/>
-    <child link="pitch"/>
+  <joint name="upper_pitch_joint" type="revolute">
+    <parent link="upper_yaw"/>
+    <child link="upper_pitch"/>
     <axis xyz="0 1 0"/>
-    <origin xyz="0 0 -0.0799"/>
+    <origin xyz="0 0 0.125"/>
     <dynamics damping="0" friction="0.1"/>
     <limit effort="1.2" velocity="13.82" lower="${pitch_lower_limit}" upper="${pitch_upper_limit}"/>
@@ -69,29 +69,92 @@
                        soft_upper_limit="${pitch_upper_limit-threshold}"/>
   </joint>
-  <!--    <link name="camera">-->
-  <!--      <inertial>-->
-  <!--        <mass value="0.17671"/>-->
-  <!--        <origin xyz="0.022 0.0 0.0"/>-->
-  <!--        <inertia ixx="2.129e-5" ixy="7.329e-8" ixz="-1.11e-7" iyy="2.198e-4" iyz="-8.04e-7" izz="2.197e-4"/>-->
-  <!--      </inertial>-->
-  <!--      <visual>-->
-  <!--        <origin xyz=" 0 0 0 " rpy="0 -1.57 0"/>-->
-  <!--        <geometry>-->
-  <!--          <mesh filename="package://rm_description/meshes/common/camera.stl" scale="0.001 0.001 0.001"/>-->
-  <!--        </geometry>-->
-  <!--        <material name="Black"/>-->
-  <!--      </visual>-->
-  <!--      <collision>-->
-  <!--        <origin xyz="0 0 0" rpy="0 -1.57 0"/>-->
-  <!--        <geometry>-->
-  <!--          <mesh filename="package://rm_description/meshes/common/camera.stl" scale="0.001 0.001 0.001"/>-->
-  <!--        </geometry>-->
-  <!--      </collision>-->
-  <!--    </link>-->
-  <!--    <joint name="camera_joint" type="fixed">-->
-  <!--      <parent link="pitch"/>-->
-  <!--      <child link="camera"/>-->
-  <!--      <origin xyz="0.086  0.0 -0.040" rpy="-1.57 0 -1.57"/>-->
-  <!--      <axis xyz="0 0 1"/>-->
-  <!--    </joint>-->
+  <link name="lower_yaw">
+    <visual>
+      <geometry>
+        <mesh filename="package://rm_description/meshes/sentry/lower_yaw.stl"
+              scale="0.001 0.001 0.001"/>
+      </geometry>
+    </visual>
+    <inertial>
+      <mass value="1.84153"/>
+      <origin xyz="-48.613e-3 -7.311e-3 -40.711e-3" rpy="0 0 0"/>
+      <inertia ixx="9.308e-3" ixy="1.131e-3" ixz="-2.237e-3" iyy="2.582e-2"
+               iyz="-5.566e-4" izz="2.598e-2"/>
+    </inertial>
+    <collision>
+      <origin xyz="0 0 0" rpy="0 0 0"/>
+      <geometry>
+        <mesh filename="package://rm_description/meshes/sentry/lower_yaw.stl"
+              scale="0.001 0.001 0.001"/>
+      </geometry>
+    </collision>
+  </link>
+  <joint name="lower_yaw_joint" type="revolute">
+    <parent link="base_link"/>
+    <child link="lower_yaw"/>
+    <axis xyz="0 0 1"/>
+    <origin xyz="2.261e-3 31.206e-3 -235.253e-3"/>
+    <dynamics damping="0" friction="0.1"/>
+    <limit effort="1.2" velocity="34" lower="${yaw_lower_limit}" upper="${yaw_upper_limit}"/>
+    <safety_controller k_position="100" k_velocity="0.1"
+                       soft_lower_limit="${yaw_lower_limit+threshold}"
+                       soft_upper_limit="${yaw_upper_limit-threshold}"/>
+  </joint>
+  <link name="lower_pitch">
+    <inertial>
+      <mass value="725.237e-3"/>
+      <origin xyz="4.587e-3 2.933e-3 17.233e-3"/>
+      <inertia ixx="2.408e-3" ixy="7.760e-5" ixz="-8.109e-5" iyy="1.183e-3"
+               iyz="-1.337e-4" izz="2.824e-3"/>
+    </inertial>
+    <visual>
+      <origin xyz="0 0 0" rpy="0 0 0"/>
+      <geometry>
+        <mesh filename="package://rm_description/meshes/sentry/lower_pitch.stl" scale="0.001 0.001 0.001"/>
+      </geometry>
+    </visual>
+    <collision>
+      <origin xyz="0 0 0" rpy="0 0 0"/>
+      <geometry>
+        <mesh filename="package://rm_description/meshes/sentry/lower_pitch.stl" scale="0.001 0.001 0.001"/>
+      </geometry>
+    </collision>
+  </link>
+  <joint name="lower_pitch_joint" type="revolute">
+    <parent link="lower_yaw"/>
+    <child link="lower_pitch"/>
+    <axis xyz="0 1 0"/>
+    <origin xyz="0 0 -0.1"/>
+    <dynamics damping="0" friction="0.1"/>
+    <limit effort="1.2" velocity="13.82" lower="${pitch_lower_limit}" upper="${pitch_upper_limit}"/>
+    <safety_controller k_position="100" k_velocity="0.1"
+                       soft_lower_limit="${pitch_lower_limit+threshold}"
+                       soft_upper_limit="${pitch_upper_limit-threshold}"/>
+  </joint>
+  <!--  <link name="upper_camera">-->
+  <!--    <inertial>-->
+  <!--          <mass value="0.17671"/>-->
+  <!--          <origin xyz="0.022 0.0 0.0"/>-->
+  <!--          <inertia ixx="2.129e-5" ixy="7.329e-8" ixz="-1.11e-7" iyy="2.198e-4" iyz="-8.04e-7" izz="2.197e-4"/>-->
+  <!--        </inertial>-->
+  <!--        <visual>-->
+  <!--          <origin xyz=" 0 0 0 " rpy="0 -1.57 0"/>-->
+  <!--          <geometry>-->
+  <!--            <mesh filename="package://rm_description/meshes/common/camera.stl" scale="0.001 0.001 0.001"/>-->
+  <!--          </geometry>-->
+  <!--          <material name="Black"/>-->
+  <!--        </visual>-->
+  <!--        <collision>-->
+  <!--          <origin xyz="0 0 0" rpy="0 -1.57 0"/>-->
+  <!--          <geometry>-->
+  <!--            <mesh filename="package://rm_description/meshes/common/camera.stl" scale="0.001 0.001 0.001"/>-->
+  <!--          </geometry>-->
+  <!--        </collision>-->
+  <!--      </link>-->
+  <!--      <joint name="camera_joint" type="fixed">-->
+  <!--        <parent link="pitch"/>-->
+  <!--        <child link="camera"/>-->
+  <!--        <origin xyz="0.086  0.0 -0.040" rpy="-1.57 0 -1.57"/>-->
+  <!--        <axis xyz="0 0 1"/>-->
+  <!--      </joint>-->
 </robot>
