Commit message: add driven wheel to sentry urdf

File: urdf/sentry/chassis.urdf.xacro (robot description, xacro)
@@ -1,4 +1,6 @@
 <robot xmlns:xacro="http://www.ros.org/wiki/xacro">
-    <xacro:include filename="$(find rm_description)/urdf/sentry/driven_wheel.urdf.xacro"/>
+    <xacro:include filename="driven_wheel1.urdf.xacro"/>
+    <xacro:include filename="driven_wheel2.urdf.xacro"/>
+    <xacro:include filename="driven_wheel3.urdf.xacro"/>
     <xacro:macro name="chassis" params="use_simulation">
         <link name="base_link">
@@ -50,29 +52,34 @@
         </joint>
         <xacro:if value="$(arg use_simulation)">
-            <xacro:driven_wheel num="1">
+            <xacro:driven_wheel1 num="1">
                 <origin rpy="${-pi/2} 0 0"/>
                 <axis xyz="0 1 0"/>
                 <origin xyz="-0.0977 0.0839 -0.013" rpy="0 0 0"/>
-            </xacro:driven_wheel>
-            <xacro:driven_wheel num="2">
+            </xacro:driven_wheel1>
+            <xacro:driven_wheel1 num="2">
                 <origin rpy="${-pi/2} 0 0"/>
                 <axis xyz="0 1 0"/>
                 <origin xyz="0.0977 0.0839 -0.013" rpy="0 0 0"/>
-            </xacro:driven_wheel>
-            <xacro:driven_wheel num="3">
+            </xacro:driven_wheel1>
+            <xacro:driven_wheel2 num="3">
                 <origin rpy="0 0 0"/>
                 <axis xyz="0 0 1"/>
-                <origin xyz="-0.0982 0.135 -0.0571" rpy="0 0 0"/>
-            </xacro:driven_wheel>
-            <xacro:driven_wheel num="4">
+                <origin xyz="0.11 0.098 -0.05486" rpy="0 0 0"/>
+            </xacro:driven_wheel2>
+            <xacro:driven_wheel2 num="4">
                 <origin rpy="0 0 0"/>
                 <axis xyz="0 0 1"/>
-                <origin xyz="0.0982 0.135 -0.0571" rpy="0 0 0"/>
-            </xacro:driven_wheel>
-            <xacro:driven_wheel num="5">
+                <origin xyz="-0.11 0.098 -0.05486" rpy="0 0 0"/>
+            </xacro:driven_wheel2>
+            <xacro:driven_wheel3 num="5">
                 <origin rpy="0 0 0"/>
                 <axis xyz="0 0 1"/>
-                <origin xyz="0 -0.073 -0.0572" rpy="0 0 0"/>
-            </xacro:driven_wheel>
+                <origin xyz="-0.07 -0.1 -0.05527" rpy="0 0 0"/>
+            </xacro:driven_wheel3>
+            <xacro:driven_wheel3 num="6">
+                <origin rpy="0 0 0"/>
+                <axis xyz="0 0 1"/>
+                <origin xyz="0.07 -0.1 0.05527" rpy="0 0 0"/>
+            </xacro:driven_wheel3>
         </xacro:if>
     </xacro:macro>

File: urdf/sentry/driven_wheel1.urdf.xacro (robot description, xacro)
@@ -2,28 +2,28 @@
   <xacro:property name="wheel_joint_effort" value="5"/>
   <xacro:property name="wheel_joint_velocity" value="50"/>
-  <xacro:macro name="driven_wheel" params="num *pose *axis *origin ">
+  <xacro:macro name="driven_wheel1" params="num *pose *axis *origin ">
       <link name="link_driven_wheel${num}">
           <visual>
               <xacro:insert_block name="pose"/>
               <geometry>
-                  <mesh filename="package://rm_description/meshes/sentry/driven_wheel.stl"
+                  <mesh filename="package://rm_description/meshes/sentry/driven_wheel1.stl"
                         scale="0.001 0.001 0.001"/>
               </geometry>
           </visual>
           <inertial>
-              <mass value="9.665e-3"/>
-        <origin xyz="0 0 0" rpy="0 0 0"/>
-        <inertia ixx="7.0766e-7" ixy="0" ixz="0" iyy="1.0067e-6"
-                 iyz="0" izz="7.0766e-7"/>
-      </inertial>
-      <collision>
-<!--        <origin xyz="0 0 0" rpy="0 0 0"/>-->
-        <xacro:insert_block name="pose"/>
-        <geometry>
-          <mesh filename="package://rm_description/meshes/sentry/driven_wheel.stl"
-                scale="0.001 0.001 0.001"/>
-        </geometry>
-      </collision>
-    </link>
+              <mass value="11.136e-3"/>
+              <origin xyz="0 0 0" rpy="0 0 0"/>
+              <inertia ixx="2319.294e-9" ixy="-0.016e-9" ixz="-2.80e-9" iyy="2720.243e-9"
+                       iyz="-7.716e-9" izz="1014.719e-9"/>
+          </inertial>
+          <collision>
+              <!--        <origin xyz="0 0 0" rpy="0 0 0"/>-->
+              <xacro:insert_block name="pose"/>
+              <geometry>
+                  <mesh filename="package://rm_description/meshes/sentry/driven_wheel1.stl"
+                        scale="0.001 0.001 0.001"/>
+              </geometry>
+          </collision>
+      </link>
     <joint name="joint_wheel${num}" type="continuous">
       <parent link="base_link"/>

Commit message: Delete cover joint in sentry

File: urdf/sentry/chassis.urdf.xacro (robot description, xacro)
@@ -84,28 +84,3 @@
         </xacro:if>
     </xacro:macro>
-    <!--    <link name="cover">-->
-    <!--    <inertial>-->
-    <!--        <mass value="0.118"/>-->
-    <!--        <origin xyz="-0.037 -0.003 0.0"/>-->
-    <!--        <inertia ixx="6.240e-4" ixy="7.325e-4" ixz="1.839e-5" iyy="1.083e-3" iyz="-1.166e-5" izz="1.602e-3"/>-->
-    <!--    </inertial>-->
-    <!--    </link>-->
-    <!--    <joint name="cover_joint" type="revolute">-->
-    <!--        <axis xyz="1 0 0"/>-->
-    <!--        <origin xyz="-0.27 0.201 0.125"/>-->
-    <!--        <limit effort="1" velocity="30" lower="-3.14" upper="3.14"/>-->
-    <!--        <dynamics damping="0.0" friction="0.1"/>-->
-    <!--        <parent link="pitch"/>-->
-    <!--        <child link="cover"/>-->
-    <!--    </joint>-->
-    <!--    <transmission name="trans_cover_joint">-->
-    <!--        <type>transmission_interface/SimpleTransmission</type>-->
-    <!--        <actuator name="cover_joint_motor">-->
-    <!--            <mechanicalReduction>1</mechanicalReduction>-->
-    <!--        </actuator>-->
-    <!--        <joint name="cover_joint">-->
-    <!--            <offset>0</offset>-->
-    <!--            <hardwareInterface>hardware_interface/EffortJointInterface</hardwareInterface>-->
-    <!--        </joint>-->
-    <!--    </transmission>-->
 </robot>
