Commit message: complete shooter of sentry,except camera.

File: urdf/sentry/lower_gimbal.urdf.xacro (robot description, xacro)
@@ -6,67 +6,4 @@
   <xacro:property name="pitch_lower_limit" value="0.241"/>
   <xacro:property name="pitch_upper_limit" value="0.885"/>
-  <link name="upper_yaw">
-    <visual>
-      <geometry>
-        <mesh filename="package://rm_description/meshes/sentry/upper_yaw.stl"
-              scale="0.001 0.001 0.001"/>
-      </geometry>
-    </visual>
-    <inertial>
-      <mass value="934.339e-3"/>
-      <origin xyz="-0.08e-3 -61.185e-3 90.777e-3" rpy="0 0 0"/>
-      <inertia ixx="1.880e-2" ixy="-6662.219e-9" ixz="7064.827e-9" iyy="1.083e-2"
-               iyz="7.150e-3" izz="9.057e-3"/>
-    </inertial>
-    <collision>
-      <origin xyz="0 0 0" rpy="0 0 0"/>
-      <geometry>
-        <mesh filename="package://rm_description/meshes/sentry/upper_yaw.stl"
-              scale="0.001 0.001 0.001"/>
-      </geometry>
-    </collision>
-  </link>
-  <joint name="upper_yaw_joint" type="revolute">
-    <parent link="base_link"/>
-    <child link="upper_yaw"/>
-    <axis xyz="0 0 1"/>
-    <origin xyz="0 0 83.4e-3"/>
-    <dynamics damping="0" friction="0.1"/>
-    <limit effort="1.2" velocity="34" lower="${yaw_lower_limit}" upper="${yaw_upper_limit}"/>
-    <safety_controller k_position="100" k_velocity="0.1"
-                       soft_lower_limit="${yaw_lower_limit+threshold}"
-                       soft_upper_limit="${yaw_upper_limit-threshold}"/>
-  </joint>
-  <link name="upper_pitch">
-    <inertial>
-      <mass value="1227.797e-3"/>
-      <origin xyz="15.667e-3 -0.268e-3 27.267e-3"/>
-      <inertia ixx="4.484e-3" ixy="813.964e-9" ixz="2.786e-4" iyy="6.599e-3"
-               iyz="-6822.846e-9" izz="5.343E-3"/>
-    </inertial>
-    <visual>
-      <origin xyz="0 0 0" rpy="0 0 0"/>
-      <geometry>
-        <mesh filename="package://rm_description/meshes/sentry/upper_pitch.stl" scale="0.001 0.001 0.001"/>
-      </geometry>
-    </visual>
-    <collision>
-      <origin xyz="0 0 0" rpy="0 0 0"/>
-      <geometry>
-        <mesh filename="package://rm_description/meshes/sentry/upper_pitch.stl" scale="0.001 0.001 0.001"/>
-      </geometry>
-    </collision>
-  </link>
-  <joint name="upper_pitch_joint" type="revolute">
-    <parent link="upper_yaw"/>
-    <child link="upper_pitch"/>
-    <axis xyz="0 1 0"/>
-    <origin xyz="0 0 0.125"/>
-    <dynamics damping="0" friction="0.1"/>
-    <limit effort="1.2" velocity="13.82" lower="${pitch_lower_limit}" upper="${pitch_upper_limit}"/>
-    <safety_controller k_position="100" k_velocity="0.1"
-                       soft_lower_limit="${pitch_lower_limit+threshold}"
-                       soft_upper_limit="${pitch_upper_limit-threshold}"/>
-  </joint>
   <link name="lower_yaw">
     <visual>

File: urdf/sentry/lower_shooter.urdf.xacro (robot description, xacro)
@@ -4,21 +4,21 @@
   <xacro:property name="wheel_offset_y" value="0.0365"/>
   <xacro:property name="wheel_offset_z" value="0.01072"/>
-  <xacro:friction_wheel prefixs="left" connected_to="pitch"
+  <xacro:friction_wheel prefixs="lower_left" connected_to="lower_pitch"
                         wheel_x_offset="${wheel_offset_x}" wheel_y_offset="${-wheel_offset_y}"
                         wheel_z_offset="${wheel_offset_z}"/>
-  <xacro:friction_wheel prefixs="right" connected_to="pitch"
+  <xacro:friction_wheel prefixs="lower_right" connected_to="lower_pitch"
                         wheel_x_offset="${wheel_offset_x}" wheel_y_offset="${wheel_offset_y}"
                         wheel_z_offset="${wheel_offset_z}"/>
-  <link name="trigger">
+  <link name="lower_trigger">
     <inertial>
-      <mass value="0.216"/>
-      <origin xyz="0 0 -0.023"/>
-      <inertia ixx="2.568e-4" ixy="1.465e-6" ixz="4.224e-7" iyy="2.534e-4"
-               iyz="1.169e-6" izz="1.627e-4"/>
+      <mass value="0.25496"/>
+      <origin xyz="0.282e-3 0.011e-3 18.873e-3"/>
+      <inertia ixx="2.844e-4" ixy="-432.025e-9" ixz="-882.662e-9" iyy="2.858e-4"
+               iyz="-19.177e-9" izz="2.347e-4"/>
     </inertial>
     <visual>
       <origin xyz="0 0 0" rpy="0 0 0"/>
       <geometry>
-        <mesh filename="package://rm_description/meshes/sentry/trigger.stl" scale="0.001 0.001 0.001" />
+        <mesh filename="package://rm_description/meshes/sentry/lower_trigger.stl" scale="0.001 0.001 0.001"/>
       </geometry>
     </visual>
@@ -26,14 +26,14 @@
       <origin xyz="0 0 0" rpy="0 0 0"/>
       <geometry>
-        <mesh filename="package://rm_description/meshes/hero/trigger.stl"  scale="0.001 0.001 0.001" />
+        <mesh filename="package://rm_description/meshes/sentry/lower_trigger.stl" scale="0.001 0.001 0.001"/>
       </geometry>
     </collision>
   </link>
-  <joint name="trigger_joint" type="continuous">
-    <origin xyz="0.0797 -0.0169 -0.2355" rpy="0 0 0"/>
+  <joint name="lower_trigger_joint" type="continuous">
+    <origin xyz="0 0.15 0.136" rpy="0 0 0"/>
     <dynamics damping="0.0" friction="0.01"/>
     <limit effort="1.0" velocity="43.54" lower="-1e16" upper="1e16"/>
     <parent link="base_link"/>
-    <child link="trigger"/>
+    <child link="lower_trigger"/>
     <axis xyz="0 0 1 "/>
   </joint>

File: urdf/sentry/sentry.urdf.xacro (robot description, xacro)
@@ -2,6 +2,8 @@
 <robot xmlns:xacro="http://www.ros.org/wiki/xacro" name="sentry">
     <xacro:arg name="load_chassis" default="true"/>
-    <xacro:arg name="load_gimbal" default="true"/>
-    <xacro:arg name="load_shooter" default="true"/>
+    <xacro:arg name="load_upper_gimbal" default="true"/>
+    <xacro:arg name="load_lower_gimbal" default="true"/>
+    <xacro:arg name="load_upper_shooter" default="true"/>
+    <xacro:arg name="load_lower_shooter" default="true"/>
     <xacro:arg name="use_simulation" default="true"/>
     <xacro:if value="$(arg load_chassis)">
@@ -10,16 +12,29 @@
         <xacro:chassis use_simulation="$(arg use_simulation)"/>
     </xacro:if>
-    <xacro:if value="$(arg load_gimbal)">
-        <xacro:include filename="$(find rm_description)/urdf/sentry/gimbal.urdf.xacro"/>
-        <xacro:include filename="$(find rm_description)/urdf/sentry/gimbal.transmission.urdf.xacro"/>
+    <xacro:if value="$(arg load_lower_gimbal)">
+        <xacro:include filename="lower_gimbal.urdf.xacro"/>
+        <xacro:include filename="lower_gimbal.transmission.urdf.xacro"/>
         <xacro:include filename="$(find rm_description)/urdf/common/camera.urdf.xacro"/>
-        <xacro:camera_sensor xyz="0.127 0 -0.047" rpy="0 0 0" parent="pitch"
-                             camera_sim="$(arg use_simulation)"/>
-        <xacro:camera_optical_frame xyz="0.153 0 -0.0615" rpy="${-pi/2} 0 ${-pi/2}" parent="pitch"
-                                    camera_sim="$(arg use_simulation)"/>
+        <!--        <xacro:camera_sensor xyz="0.127 0 -0.047" rpy="0 0 0" parent="lower_pitch"-->
+        <!--                             camera_sim="$(arg use_simulation)"/>-->
+        <!--        <xacro:camera_optical_frame xyz="0.153 0 -0.0615" rpy="${-pi/2} 0 ${-pi/2}" parent="lower_pitch"-->
+        <!--                                    camera_sim="$(arg use_simulation)"/>-->
     </xacro:if>
-    <xacro:if value="$(arg load_shooter)">
-        <xacro:include filename="$(find rm_description)/urdf/sentry/shooter.urdf.xacro"/>
-        <xacro:include filename="$(find rm_description)/urdf/sentry/shooter.transmission.urdf.xacro"/>
+    <xacro:if value="$(arg load_upper_gimbal)">
+        <xacro:include filename="upper_gimbal.urdf.xacro"/>
+        <xacro:include filename="upper_gimbal.transmission.urdf.xacro"/>
+        <xacro:include filename="$(find rm_description)/urdf/common/camera.urdf.xacro"/>
+        <!--        <xacro:camera_sensor xyz="0.127 0 -0.047" rpy="0 0 0" parent="upper_pitch"-->
+        <!--                             camera_sim="$(arg use_simulation)"/>-->
+        <!--        <xacro:camera_optical_frame xyz="0.153 0 -0.0615" rpy="${-pi/2} 0 ${-pi/2}" parent="upper_pitch"-->
+        <!--                                    camera_sim="$(arg use_simulation)"/>-->
+    </xacro:if>
+    <xacro:if value="$(arg load_upper_shooter)">
+        <xacro:include filename="$(find rm_description)/urdf/sentry/upper_shooter.urdf.xacro"/>
+        <xacro:include filename="$(find rm_description)/urdf/sentry/upper_shooter.transmission.urdf.xacro"/>
+    </xacro:if>
+    <xacro:if value="$(arg load_lower_shooter)">
+        <xacro:include filename="$(find rm_description)/urdf/sentry/lower_shooter.urdf.xacro"/>
+        <xacro:include filename="$(find rm_description)/urdf/sentry/lower_shooter.transmission.urdf.xacro"/>
     </xacro:if>
     <xacro:if value="$(arg use_simulation)">

File: urdf/sentry/upper_gimbal.transmission.urdf.xacro (robot description, xacro)
@@ -21,23 +21,3 @@
         </joint>
     </transmission>
-    <transmission name="trans_lower_yaw_joint">
-        <type>transmission_interface/SimpleTransmission</type>
-        <actuator name="lower_yaw_joint_motor">
-            <mechanicalReduction>1</mechanicalReduction>
-        </actuator>
-        <joint name="lower_yaw_joint">
-            <offset>-3.211</offset>
-            <hardwareInterface>hardware_interface/EffortJointInterface</hardwareInterface>
-        </joint>
-    </transmission>
-    <transmission name="trans_lower_pitch_joint">
-        <type>transmission_interface/SimpleTransmission</type>
-        <actuator name="lower_pitch_joint_motor">
-            <mechanicalReduction>1</mechanicalReduction>
-        </actuator>
-        <joint name="lower_pitch_joint">
-            <offset>-5.211</offset>
-            <hardwareInterface>hardware_interface/EffortJointInterface</hardwareInterface>
-        </joint>
-    </transmission>
 </robot>

File: urdf/sentry/upper_shooter.transmission.urdf.xacro (robot description, xacro)
@@ -1,28 +1,28 @@
 <?xml version="1.0" encoding="utf-8"?>
 <robot>
-    <transmission name="trans_trigger_joint">
+    <transmission name="trans_upper_trigger_joint">
         <type>transmission_interface/SimpleTransmission</type>
-        <actuator name="trigger_joint_motor">
+        <actuator name="upper_trigger_joint_motor">
             <mechanicalReduction>1</mechanicalReduction>
         </actuator>
-        <joint name="trigger_joint">
+        <joint name="upper_trigger_joint">
             <hardwareInterface>hardware_interface/EffortJointInterface</hardwareInterface>
         </joint>
     </transmission>
-    <transmission name="trans_left_friction_wheel_joint_joint">
+    <transmission name="trans_upper_left_friction_wheel_joint_joint">
         <type>transmission_interface/SimpleTransmission</type>
-        <actuator name="left_friction_wheel_joint_motor">
+        <actuator name="upper_left_friction_wheel_joint_motor">
             <mechanicalReduction>-1</mechanicalReduction>
         </actuator>
-        <joint name="left_friction_wheel_joint">
+        <joint name="upper_left_friction_wheel_joint">
             <hardwareInterface>hardware_interface/EffortJointInterface</hardwareInterface>
         </joint>
     </transmission>
-    <transmission name="trans_right_friction_wheel_joint_joint">
+    <transmission name="trans_upper_right_friction_wheel_joint_joint">
         <type>transmission_interface/SimpleTransmission</type>
-        <actuator name="right_friction_wheel_joint_motor">
+        <actuator name="upper_right_friction_wheel_joint_motor">
             <mechanicalReduction>-1</mechanicalReduction>
         </actuator>
-        <joint name="right_friction_wheel_joint">
+        <joint name="upper_right_friction_wheel_joint">
             <hardwareInterface>hardware_interface/EffortJointInterface</hardwareInterface>
         </joint>

Commit message: Update sentry pitch limit

File: urdf/sentry/lower_gimbal.urdf.xacro (robot description, xacro)
@@ -1,9 +1,9 @@
 <?xml version="1.0" encoding="utf-8"?>
 <robot xmlns:xacro="http://www.ros.org/wiki/xacro">
-  <xacro:property name="threshold" value="0.1"/>
+  <xacro:property name="threshold" value="0.03"/>
   <xacro:property name="yaw_lower_limit" value="-2.461"/>
   <xacro:property name="yaw_upper_limit" value="1.998"/>
-  <xacro:property name="pitch_lower_limit" value="0.112"/>
-  <xacro:property name="pitch_upper_limit" value="1.157"/>
+  <xacro:property name="pitch_lower_limit" value="0.129"/>
+  <xacro:property name="pitch_upper_limit" value="1.175"/>
   <link name="lower_yaw">
     <visual>

File: urdf/sentry/upper_gimbal.urdf.xacro (robot description, xacro)
@@ -1,5 +1,5 @@
 <?xml version="1.0" encoding="utf-8"?>
 <robot xmlns:xacro="http://www.ros.org/wiki/xacro">
-    <xacro:property name="threshold" value="0.1"/>
+    <xacro:property name="threshold" value="0.03"/>
     <xacro:property name="yaw_lower_limit" value="-2.949"/>
     <xacro:property name="yaw_upper_limit" value="3.027"/>
