Commit message: Update upper yaw limit

File: urdf/sentry/upper_gimbal.urdf.xacro (robot description, xacro)
@@ -2,6 +2,6 @@
 <robot xmlns:xacro="http://www.ros.org/wiki/xacro">
     <xacro:property name="threshold" value="0.03"/>
-    <xacro:property name="yaw_lower_limit" value="-2.949"/>
-    <xacro:property name="yaw_upper_limit" value="3.027"/>
+    <xacro:property name="yaw_lower_limit" value="-2.90"/>
+    <xacro:property name="yaw_upper_limit" value="2.97"/>
     <xacro:property name="pitch_lower_limit" value="-0.843"/>
     <xacro:property name="pitch_upper_limit" value="0.472"/>
