Commit message: Fix imu topic name in gazebo

File: urdf/balance/balance.urdf.xacro (robot description, xacro)
@@ -28,5 +28,5 @@
         <topic>__default_topic__</topic>
         <plugin filename="libgazebo_ros_imu_sensor.so" name="imu_plugin">
-          <topicName>imu</topicName>
+          <topicName>base_imu</topicName>
           <bodyName>imu_link</bodyName>
           <updateRateHZ>1000.0</updateRateHZ>

File: urdf/balance/rubber_wheel.urdf.xacro (robot description, xacro)
@@ -2,5 +2,5 @@
     <xacro:property name="wheel_radius" value="0.06"/>
     <xacro:property name="wheel_width" value="0.032"/>
-    <xacro:property name="wheel_joint_effort" value="1"/>
+    <xacro:property name="wheel_joint_effort" value="3"/>
     <xacro:property name="wheel_joint_velocity" value="50"/>
     <xacro:macro name="rubber_wheel"
