Commit message: Added 3d model of Balanced Infantry and some parameter

File: urdf/balance/chassis.urdf.xacro (robot description, xacro)
@@ -1,16 +1,14 @@
 <robot xmlns:xacro="http://www.ros.org/wiki/xacro">
-    <xacro:include filename="$(find rm_description)/urdf/common/rubber_wheel.urdf.xacro"/>
+    <xacro:include filename="$(find rm_description)/urdf/balance/rubber_wheel.urdf.xacro"/>
     <!-- https://upload.wikimedia.org/wikipedia/commons/5/52/Wheelbase_and_Track.png -->
-    <xacro:property name="wheel_base" value="0.475"/>
-    <xacro:property name="wheel_offset_z" value="-0.036"/>
-    <xacro:property name="wheel_joint_damping" value="1.0"/>
-    <xacro:property name="wheel_joint_friction" value="1.0"/>
+    <xacro:property name="wheel_base" value="0.405"/>
+    <xacro:property name="wheel_offset_z" value="-0.085"/>
     <xacro:macro name="chassis">
         <link name="base_link">
             <inertial>
-                <mass value="17.23"/>
-                <origin xyz="0 0 0"/>
-                <inertia ixx="2.708e+5" ixy="14.57" ixz="-3.207e+3" iyy="3.585e+5"
-                         iyz="-3.192e+3" izz="2.504e+5"/>
+                <mass value="17.21"/>
+                <origin xyz="-0.006488 0.006497 0.062596"/>
+                <inertia ixx="0.2744" ixy="-2.342e-5" ixz="2.162e-3" iyy="0.2444"
+                         iyz="-2.346e-3" izz="0.1928"/>
             </inertial>
             <visual>
@@ -21,7 +19,8 @@
             </visual>
             <collision>
-                <origin xyz="0 0 0" rpy="0 0 0"/>
+                <origin xyz="0 0 -0.067" rpy="0 0 0"/>
                 <geometry>
-                    <mesh filename="package://rm_description/meshes/balance/base.stl" scale="0.001 0.001 0.001"/>
+                    <!--                    <mesh filename="package://rm_description/meshes/balance/base.stl" scale="0.001 0.001 0.001"/>-->
+                    <box size="0.35 0.22 0.03"/>
                 </geometry>
             </collision>

File: urdf/balance/rubber_wheel.urdf.xacro (robot description, xacro)
@@ -1,4 +1,5 @@
 <robot xmlns:xacro="http://www.ros.org/wiki/xacro">
-    <xacro:property name="wheel_radius" value="0.07625"/>
+    <xacro:property name="wheel_radius" value="0.06"/>
+    <xacro:property name="wheel_width" value="0.032"/>
     <xacro:property name="wheel_joint_effort" value="5"/>
     <xacro:property name="wheel_joint_velocity" value="50"/>
@@ -9,11 +10,29 @@
             <visual>
                 <geometry>
-                    <mesh filename="package://rm_description/meshes/common/rubber_wheel.stl"
-                          scale="0.001 0.001 0.001"/>
+                    <xacro:if value="${prefix=='left'}">
+                        <mesh filename="package://rm_description/meshes/balance/left_rubber_wheel.stl"
+                              scale="0.001 0.001 0.001"/>
+                    </xacro:if>
+                    <xacro:if value="${prefix=='right'}">
+                        <mesh filename="package://rm_description/meshes/balance/right_rubber_wheel.stl"
+                              scale="0.001 0.001 0.001"/>
+                    </xacro:if>
                 </geometry>
             </visual>
+            <collision>
+                <origin rpy="1.57 0 0" xyz="0 0 0"/>
+                <geometry>
+                    <cylinder length="0.032" radius="0.06"/>
+                </geometry>
+            </collision>
             <inertial>
                 <mass value="0.23"/>
-                <inertia ixx="5.647e+2" ixy="0.0" ixz="0.0" iyy="3.048e+2" iyz="0.0" izz="3.048e+2"/>
+                <xacro:if value="${prefix=='left'}">
+                    <origin xyz="0 0.00419 0"/>
+                </xacro:if>
+                <xacro:if value="${prefix=='right'}">
+                    <origin xyz="0 -0.00419 0"/>
+                </xacro:if>
+                <inertia ixx="3.048e-4" ixy="0.0" ixz="0.0" iyy="5.647e-4" iyz="0.0" izz="3.048e-4"/>
             </inertial>
         </link>

Commit message: Add balance.yaml

File: urdf/balance/chassis.urdf.xacro (robot description, xacro)
@@ -28,8 +28,8 @@
         <xacro:rubber_wheel prefix="left" connected_to="base_link"
                             wheel_x_offset="0" wheel_y_offset="${wheel_base/2}"
-                            wheel_z_offset="${wheel_offset_z}" mechanical_reduction="0.166"/>
+                            wheel_z_offset="${wheel_offset_z}" mechanical_reduction="-0.166"/>
         <xacro:rubber_wheel prefix="right" connected_to="base_link"
                             wheel_x_offset="0" wheel_y_offset="${-wheel_base/2}"
-                            wheel_z_offset="${wheel_offset_z}" mechanical_reduction="-0.166"/>
+                            wheel_z_offset="${wheel_offset_z}" mechanical_reduction="0.166"/>
     </xacro:macro>
 </robot>

File: urdf/balance/rubber_wheel.urdf.xacro (robot description, xacro)
@@ -2,5 +2,5 @@
     <xacro:property name="wheel_radius" value="0.06"/>
     <xacro:property name="wheel_width" value="0.032"/>
-    <xacro:property name="wheel_joint_effort" value="3"/>
+    <xacro:property name="wheel_joint_effort" value="1"/>
     <xacro:property name="wheel_joint_velocity" value="50"/>
     <xacro:macro name="rubber_wheel"

Commit message: Use test edition parameter of balance

File: urdf/balance/chassis.urdf.xacro (robot description, xacro)
@@ -3,15 +3,15 @@
     <!-- https://upload.wikimedia.org/wikipedia/commons/5/52/Wheelbase_and_Track.png -->
     <xacro:property name="wheel_base" value="0.405"/>
-    <xacro:property name="wheel_offset_z" value="-0.085"/>
+    <xacro:property name="wheel_z_offset" value="0"/>
     <xacro:macro name="chassis">
         <link name="base_link">
             <inertial>
-                <mass value="17.21"/>
-                <origin xyz="-0.006488 0.006497 0.062596"/>
-                <inertia ixx="0.2744" ixy="-2.342e-5" ixz="2.162e-3" iyy="0.2444"
-                         iyz="-2.346e-3" izz="0.1928"/>
+                <mass value="4.595"/>
+                <origin xyz="-0.000190 -0.000075 0.110987"/>
+                <inertia ixx="0.126" ixy="-1.806e-6" ixz="1.142e-4" iyy="5.337e-2"
+                         iyz="1.133e-4" izz="8.685e-2"/>
             </inertial>
             <visual>
-                <origin xyz="0 0 0" rpy="0 0 0"/>
+                <origin xyz="0 0 0.085" rpy="0 0 0"/>
                 <geometry>
                     <mesh filename="package://rm_description/meshes/balance/base.stl" scale="0.001 0.001 0.001"/>
@@ -19,5 +19,5 @@
             </visual>
             <collision>
-                <origin xyz="0 0 -0.067" rpy="0 0 0"/>
+                <origin xyz="0 0 0.018" rpy="0 0 0"/>
                 <geometry>
                     <!--                    <mesh filename="package://rm_description/meshes/balance/base.stl" scale="0.001 0.001 0.001"/>-->
@@ -28,8 +28,8 @@
         <xacro:rubber_wheel prefix="left" connected_to="base_link"
                             wheel_x_offset="0" wheel_y_offset="${wheel_base/2}"
-                            wheel_z_offset="${wheel_offset_z}" mechanical_reduction="-0.166"/>
+                            wheel_z_offset="${wheel_z_offset}" mechanical_reduction="-0.166"/>
         <xacro:rubber_wheel prefix="right" connected_to="base_link"
                             wheel_x_offset="0" wheel_y_offset="${-wheel_base/2}"
-                            wheel_z_offset="${wheel_offset_z}" mechanical_reduction="0.166"/>
+                            wheel_z_offset="${wheel_z_offset}" mechanical_reduction="0.166"/>
     </xacro:macro>
 </robot>

File: urdf/balance/rubber_wheel.urdf.xacro (robot description, xacro)
@@ -2,5 +2,5 @@
     <xacro:property name="wheel_radius" value="0.06"/>
     <xacro:property name="wheel_width" value="0.032"/>
-    <xacro:property name="wheel_joint_effort" value="3"/>
+    <xacro:property name="wheel_joint_effort" value="1.0"/>
     <xacro:property name="wheel_joint_velocity" value="50"/>
     <xacro:macro name="rubber_wheel"
@@ -40,5 +40,5 @@
         <joint name="${prefix}_wheel_joint" type="revolute">
             <axis xyz="0 1 0"/>
-            <origin xyz="${wheel_x_offset} ${wheel_y_offset} ${wheel_offset_z}" rpy="0 0 0"/>
+            <origin xyz="${wheel_x_offset} ${wheel_y_offset} ${wheel_z_offset}" rpy="0 0 0"/>
             <!--      limit not work while type="continuous"-->
             <limit effort="${wheel_joint_effort}" velocity="${wheel_joint_velocity}" lower="-1e16" upper="1e16"/>
