Commit message: Add DoubleActuatorTransmission to engineer arm

File: urdf/balance/rubber_wheel.urdf.xacro (robot description, xacro)
@@ -2,5 +2,5 @@
     <xacro:property name="wheel_radius" value="0.06"/>
     <xacro:property name="wheel_width" value="0.032"/>
-    <xacro:property name="wheel_joint_effort" value="5"/>
+    <xacro:property name="wheel_joint_effort" value="3"/>
     <xacro:property name="wheel_joint_velocity" value="50"/>
     <xacro:macro name="rubber_wheel"

File: urdf/engineer/arm.transmission.xacro (robot description, xacro)
@@ -13,14 +13,4 @@
             </joint>
         </transmission>
-        <transmission name="trans_joint2">
-            <type>transmission_interface/SimpleTransmission</type>
-            <actuator name="joint2_motor">
-                <mechanicalReduction>-3</mechanicalReduction>
-            </actuator>
-            <joint name="joint2">
-                <hardwareInterface>hardware_interface/EffortJointInterface</hardwareInterface>
-                <offset>-3.1904</offset>
-            </joint>
-        </transmission>
         <transmission name="trans_joint3">
             <type>transmission_interface/SimpleTransmission</type>
@@ -34,4 +24,20 @@
         </transmission>
         <xacro:unless value="${simulation}">
+            <transmission name="trans_joint2">
+                <type>transmission_interface/DoubleActuatorTransmission</type>
+                <actuator name="joint2_left_motor">
+                    <role>actuator1</role>
+                    <mechanicalReduction>3</mechanicalReduction>
+                </actuator>
+                <actuator name="joint2_right_motor">
+                    <role>actuator2</role>
+                    <mechanicalReduction>-3</mechanicalReduction>
+                </actuator>
+                <joint name="joint2">
+                    <offset>0</offset>
+                    <mechanicalReduction>1</mechanicalReduction>
+                    <hardwareInterface>hardware_interface/EffortJointInterface</hardwareInterface>
+                </joint>
+            </transmission>
             <transmission name="trans_wrist">
                 <type>transmission_interface/DifferentialTransmission</type>
@@ -61,4 +67,14 @@
         </xacro:unless>
         <xacro:if value="${simulation}">
+            <transmission name="trans_joint2">
+                <type>transmission_interface/SimpleTransmission</type>
+                <actuator name="joint2_motor">
+                    <mechanicalReduction>-3</mechanicalReduction>
+                </actuator>
+                <joint name="joint2">
+                    <hardwareInterface>hardware_interface/EffortJointInterface</hardwareInterface>
+                    <offset>0</offset>
+                </joint>
+            </transmission>
             <transmission name="trans_joint4">
                 <type>transmission_interface/SimpleTransmission</type>
@@ -66,5 +82,4 @@
                     <hardwareInterface>hardware_interface/EffortJointInterface</hardwareInterface>
                     <mechanicalReduction>1</mechanicalReduction>
-                    <offset>0</offset>
                 </actuator>
                 <joint name="joint4">
@@ -77,5 +92,4 @@
                     <hardwareInterface>hardware_interface/EffortJointInterface</hardwareInterface>
                     <mechanicalReduction>1</mechanicalReduction>
-                    <offset>0</offset>
                 </actuator>
                 <joint name="joint5">

Commit message: romove redundant hardwareInterface

File: urdf/balance/rubber_wheel.urdf.xacro (robot description, xacro)
@@ -55,5 +55,4 @@
             </actuator>
             <joint name="${prefix}_wheel_joint">
-                <hardwareInterface>hardware_interface/EffortJointInterface</hardwareInterface>
             </joint>
         </transmission>

File: urdf/hero/gimbal.transmission.urdf.xacro (robot description, xacro)
@@ -4,5 +4,4 @@
         <type>transmission_interface/SimpleTransmission</type>
         <actuator name="yaw_joint_motor">
-            <hardwareInterface>hardware_interface/EffortJointInterface</hardwareInterface>
             <mechanicalReduction>1</mechanicalReduction>
         </actuator>
@@ -15,5 +14,4 @@
         <type>transmission_interface/SimpleTransmission</type>
         <actuator name="pitch_joint_motor">
-            <hardwareInterface>hardware_interface/EffortJointInterface</hardwareInterface>
             <mechanicalReduction>1</mechanicalReduction>
         </actuator>

File: urdf/hero/shooter.transmission.urdf.xacro (robot description, xacro)
@@ -4,5 +4,4 @@
         <type>transmission_interface/SimpleTransmission</type>
         <actuator name="trigger_joint_motor">
-            <hardwareInterface>hardware_interface/EffortJointInterface</hardwareInterface>
             <mechanicalReduction>-1</mechanicalReduction>
         </actuator>
@@ -14,5 +13,4 @@
         <type>transmission_interface/SimpleTransmission</type>
         <actuator name="left_friction_wheel_joint_motor">
-            <hardwareInterface>hardware_interface/EffortJointInterface</hardwareInterface>
             <mechanicalReduction>1</mechanicalReduction>
         </actuator>
@@ -24,5 +22,4 @@
         <type>transmission_interface/SimpleTransmission</type>
         <actuator name="right_friction_wheel_joint_motor">
-            <hardwareInterface>hardware_interface/EffortJointInterface</hardwareInterface>
             <mechanicalReduction>1</mechanicalReduction>
         </actuator>

File: urdf/sentry/chassis.transmission.urdf.xacro (robot description, xacro)
@@ -1,13 +1,12 @@
 <?xml version="1.0" encoding="utf-8"?>
 <robot>
-<transmission name="trans_drive_joint">
-    <type>transmission_interface/SimpleTransmission</type>
-    <actuator name="drive_joint_motor">
-        <hardwareInterface>hardware_interface/EffortJointInterface</hardwareInterface>
-        <mechanicalReduction>1</mechanicalReduction>
-    </actuator>
-    <joint name="drive_joint">
-        <hardwareInterface>hardware_interface/EffortJointInterface</hardwareInterface>
-    </joint>
-</transmission>
+    <transmission name="trans_drive_joint">
+        <type>transmission_interface/SimpleTransmission</type>
+        <actuator name="drive_joint_motor">
+            <mechanicalReduction>1</mechanicalReduction>
+        </actuator>
+        <joint name="drive_joint">
+            <hardwareInterface>hardware_interface/EffortJointInterface</hardwareInterface>
+        </joint>
+    </transmission>
 </robot>

File: urdf/sentry/gimbal.transmission.urdf.xacro (robot description, xacro)
@@ -4,5 +4,4 @@
         <type>transmission_interface/SimpleTransmission</type>
         <actuator name="yaw_joint_motor">
-            <hardwareInterface>hardware_interface/EffortJointInterface</hardwareInterface>
             <mechanicalReduction>1</mechanicalReduction>
         </actuator>
@@ -15,5 +14,4 @@
         <type>transmission_interface/SimpleTransmission</type>
         <actuator name="pitch_joint_motor">
-            <hardwareInterface>hardware_interface/EffortJointInterface</hardwareInterface>
             <mechanicalReduction>1</mechanicalReduction>
         </actuator>

File: urdf/sentry/shooter.transmission.urdf.xacro (robot description, xacro)
@@ -4,5 +4,4 @@
         <type>transmission_interface/SimpleTransmission</type>
         <actuator name="trigger_joint_motor">
-            <hardwareInterface>hardware_interface/EffortJointInterface</hardwareInterface>
             <mechanicalReduction>1</mechanicalReduction>
         </actuator>
@@ -14,5 +13,4 @@
         <type>transmission_interface/SimpleTransmission</type>
         <actuator name="left_friction_wheel_joint_motor">
-            <hardwareInterface>hardware_interface/EffortJointInterface</hardwareInterface>
             <mechanicalReduction>-1</mechanicalReduction>
         </actuator>
@@ -24,5 +22,4 @@
         <type>transmission_interface/SimpleTransmission</type>
         <actuator name="right_friction_wheel_joint_motor">
-            <hardwareInterface>hardware_interface/EffortJointInterface</hardwareInterface>
             <mechanicalReduction>-1</mechanicalReduction>
         </actuator>

File: urdf/standard/gimbal.transmission.urdf.xacro (robot description, xacro)
@@ -4,5 +4,4 @@
         <type>transmission_interface/SimpleTransmission</type>
         <actuator name="yaw_joint_motor">
-            <hardwareInterface>hardware_interface/EffortJointInterface</hardwareInterface>
             <mechanicalReduction>1</mechanicalReduction>
         </actuator>
@@ -15,5 +14,4 @@
         <type>transmission_interface/SimpleTransmission</type>
         <actuator name="pitch_joint_motor">
-            <hardwareInterface>hardware_interface/EffortJointInterface</hardwareInterface>
             <mechanicalReduction>-1</mechanicalReduction>
         </actuator>

File: urdf/standard/shooter.transmission.urdf.xacro (robot description, xacro)
@@ -4,5 +4,4 @@
         <type>transmission_interface/SimpleTransmission</type>
         <actuator name="trigger_joint_motor">
-            <hardwareInterface>hardware_interface/EffortJointInterface</hardwareInterface>
             <mechanicalReduction>1</mechanicalReduction>
         </actuator>
@@ -14,5 +13,4 @@
         <type>transmission_interface/SimpleTransmission</type>
         <actuator name="left_friction_wheel_joint_motor">
-            <hardwareInterface>hardware_interface/EffortJointInterface</hardwareInterface>
             <mechanicalReduction>-1</mechanicalReduction>
         </actuator>
@@ -24,5 +22,4 @@
         <type>transmission_interface/SimpleTransmission</type>
         <actuator name="right_friction_wheel_joint_motor">
-            <hardwareInterface>hardware_interface/EffortJointInterface</hardwareInterface>
             <mechanicalReduction>-1</mechanicalReduction>
         </actuator>
