Commit message: Update hero shooter, gimabal config parameter and urdf

File: urdf/hero/gimbal.transmission.urdf.xacro (robot description, xacro)
@@ -8,5 +8,5 @@
         </actuator>
         <joint name="yaw_joint">
-            <offset>1.09</offset>
+            <offset>-2.160</offset>
             <hardwareInterface>hardware_interface/EffortJointInterface</hardwareInterface>
         </joint>
@@ -16,8 +16,8 @@
         <actuator name="pitch_joint_motor">
             <hardwareInterface>hardware_interface/EffortJointInterface</hardwareInterface>
-            <mechanicalReduction>1</mechanicalReduction>
+            <mechanicalReduction>-1</mechanicalReduction>
         </actuator>
         <joint name="pitch_joint">
-            <offset>-2.46</offset>
+            <offset>0.902</offset>
             <hardwareInterface>hardware_interface/EffortJointInterface</hardwareInterface>
         </joint>

File: urdf/hero/shooter.urdf.xacro (robot description, xacro)
@@ -4,16 +4,17 @@
     <xacro:property name="wheel_offset_y" value="0.049"/>
     <xacro:property name="wheel_offset_z" value="0.0"/>
-    <xacro:property name="wheel_and_wheel_offset_x" value="0.08"/>
+    <xacro:property name="wheel_and_wheel_offset_x" value="0.06"/>
     <xacro:friction_wheel prefixs="left_follow" connected_to="pitch"
+                          wheel_x_offset="${wheel_offset_x+wheel_and_wheel_offset_x}" wheel_y_offset="${wheel_offset_y}"
+                          wheel_z_offset="${wheel_offset_z}"/>
+    <xacro:friction_wheel prefixs="right_follow" connected_to="pitch"
+                          wheel_x_offset="${wheel_offset_x+wheel_and_wheel_offset_x}"
+                          wheel_y_offset="${-wheel_offset_y}"
+                          wheel_z_offset="${wheel_offset_z}"/>
+    <xacro:friction_wheel prefixs="left_back" connected_to="pitch"
                           wheel_x_offset="${wheel_offset_x}" wheel_y_offset="${wheel_offset_y}"
                           wheel_z_offset="${wheel_offset_z}"/>
-    <xacro:friction_wheel prefixs="right_follow" connected_to="pitch"
-                          wheel_x_offset="${wheel_offset_x}" wheel_y_offset="${-wheel_offset_y}"
-                          wheel_z_offset="${wheel_offset_z}"/>
-    <xacro:friction_wheel prefixs="left_back" connected_to="pitch"
-                          wheel_x_offset="${wheel_offset_x+wheel_and_wheel_offset_x}" wheel_y_offset="${wheel_offset_y}"
-                          wheel_z_offset="${wheel_offset_z}"/>
     <xacro:friction_wheel prefixs="right_back" connected_to="pitch"
-                          wheel_x_offset="${wheel_offset_x+wheel_and_wheel_offset_x}"
+                          wheel_x_offset="${wheel_offset_x}"
                           wheel_y_offset="${-wheel_offset_y}"
                           wheel_z_offset="${wheel_offset_z}"/>
