Commit message: simplify base.stl
Former-commit-id: 818f7dbbc56cf3d5d6dbcfc91b75cad694cbcff9
Former-commit-id: 045f926265b07919a3b88eafc40777f5c0e48c3d

File: urdf/hero/chassis.urdf.xacro (robot description, xacro)
@@ -22,8 +22,8 @@
     </visual>
     <collision>
-      <!--      <origin xyz="0 0 0" rpy="0 0 0"/>-->
-      <!--      <geometry>-->
-      <!--        <mesh filename="package://rm_description/meshes/hero/base.stl" scale="0.001 0.001 0.001"/>-->
-      <!--      </geometry>-->
+      <origin xyz="0 0 0" rpy="0 0 0"/>
+      <geometry>
+        <mesh filename="package://rm_description/meshes/hero/base.stl" scale="0.001 0.001 0.001"/>
+      </geometry>
     </collision>
   </link>

Commit message: Add argd to xacro for dynamic loading chassis, gimbal, shooter and gazebo

File: urdf/hero/chassis.urdf.xacro (robot description, xacro)
@@ -1,3 +1,3 @@
-<robot xmlns:xacro="http://www.ros.org/wiki/xacro" name="hero">
+<robot xmlns:xacro="http://www.ros.org/wiki/xacro">
   <xacro:include filename="$(find rm_description)/urdf/common/mecanum_wheel.urdf.xacro"/>
   <!-- https://upload.wikimedia.org/wikipedia/commons/5/52/Wheelbase_and_Track.png -->
@@ -7,47 +7,41 @@
   <xacro:property name="wheel_joint_damping" value="1.0"/>
   <xacro:property name="wheel_joint_friction" value="1.0"/>
-  <link name="base_link">
-    <inertial>
-      <mass value="10"/>
-      <origin xyz="0 0 0"/>
-      <inertia ixx="1.013" ixy="1.818e-3" ixz="5.843e-2" iyy="1.516"
-               iyz="3.179e-2" izz="2.208"/>
-    </inertial>
-    <visual>
-      <origin xyz="0 0 0" rpy="0 0 0"/>
-      <geometry>
-        <mesh filename="package://rm_description/meshes/hero/base.stl" scale="0.001 0.001 0.001"/>
-      </geometry>
-      <material name="DarkGrey"/>
-    </visual>
-    <collision>
-      <origin xyz="0 0 0" rpy="0 0 0"/>
-      <geometry>
-        <mesh filename="package://rm_description/meshes/hero/base.stl" scale="0.001 0.001 0.001"/>
-      </geometry>
-    </collision>
-  </link>
-  <xacro:mecanum_wheel prefix="front_left" parent="base_link"
-                       wheel_x_offset="${wheel_track/2}" wheel_y_offset="${wheel_base/2}"
-                       wheel_z_offset="${wheel_offset_z}"
-                       reflect="1"/>
-  <xacro:mecanum_wheel prefix="front_right" parent="base_link"
-                       wheel_x_offset="${wheel_track/2}" wheel_y_offset="${-wheel_base/2}"
-                       wheel_z_offset="${wheel_offset_z}"
-                       reflect="-1"/>
-  <xacro:mecanum_wheel prefix="back_left" parent="base_link"
-                       wheel_x_offset="${-wheel_track/2}" wheel_y_offset="${wheel_base/2}"
-                       wheel_z_offset="${wheel_offset_z}"
-                       reflect="-1"/>
-  <xacro:mecanum_wheel prefix="back_right" parent="base_link"
-                       wheel_x_offset="${-wheel_track/2}" wheel_y_offset="${-wheel_base/2}"
-                       wheel_z_offset="${wheel_offset_z}"
-                       reflect="1"/>
-  <!-- Gazebo plugin for ROS Control -->
-  <gazebo>
-    <plugin name="rm_ros_control" filename="librm_robot_hw_sim.so">
-      <robotNamespace>/</robotNamespace>
-      <robotSimType>rm_gazebo/RmRobotHWSim</robotSimType>
-    </plugin>
-  </gazebo>
+  <xacro:macro name="chassis" params="roller_type">
+    <link name="base_link">
+      <inertial>
+        <mass value="10"/>
+        <origin xyz="0 0 0"/>
+        <inertia ixx="1.013" ixy="1.818e-3" ixz="5.843e-2" iyy="1.516"
+                 iyz="3.179e-2" izz="2.208"/>
+      </inertial>
+      <visual>
+        <origin xyz="0 0 0" rpy="0 0 0"/>
+        <geometry>
+          <mesh filename="package://rm_description/meshes/hero/base.stl" scale="0.001 0.001 0.001"/>
+        </geometry>
+      </visual>
+      <collision>
+        <origin xyz="0 0 0" rpy="0 0 0"/>
+        <geometry>
+          <mesh filename="package://rm_description/meshes/hero/base.stl" scale="0.001 0.001 0.001"/>
+        </geometry>
+      </collision>
+    </link>
+    <xacro:mecanum_wheel prefix="front_left" connected_to="base_link"
+                         wheel_x_offset="${wheel_track/2}" wheel_y_offset="${wheel_base/2}"
+                         wheel_z_offset="${wheel_offset_z}"
+                         reflect="1" roller_type="${roller_type}"/>
+    <xacro:mecanum_wheel prefix="front_right" connected_to="base_link"
+                         wheel_x_offset="${wheel_track/2}" wheel_y_offset="${-wheel_base/2}"
+                         wheel_z_offset="${wheel_offset_z}"
+                         reflect="-1" roller_type="${roller_type}"/>
+    <xacro:mecanum_wheel prefix="back_left" connected_to="base_link"
+                         wheel_x_offset="${-wheel_track/2}" wheel_y_offset="${wheel_base/2}"
+                         wheel_z_offset="${wheel_offset_z}"
+                         reflect="-1" roller_type="${roller_type}"/>
+    <xacro:mecanum_wheel prefix="back_right" connected_to="base_link"
+                         wheel_x_offset="${-wheel_track/2}" wheel_y_offset="${-wheel_base/2}"
+                         wheel_z_offset="${wheel_offset_z}"
+                         reflect="1" roller_type="${roller_type}"/>
+  </xacro:macro>
 </robot>

Commit message: chnge hero urdf

File: urdf/hero/chassis.urdf.xacro (robot description, xacro)
@@ -10,13 +10,13 @@
     <link name="base_link">
       <inertial>
-        <mass value="10"/>
-        <origin xyz="0 0 0"/>
-        <inertia ixx="1.013" ixy="1.818e-3" ixz="5.843e-2" iyy="1.516"
-                 iyz="3.179e-2" izz="2.208"/>
+        <mass value="19.93"/>
+        <origin xyz="-0.02282 0.002773 0.008173"/>
+        <inertia ixx="5.96e-1" ixy="6.075e-3" ixz="4.655e-2" iyy="9.41e-1"
+                 iyz="-3.105e-3" izz="1.381e+0"/>
       </inertial>
       <visual>
         <origin xyz="0 0 0" rpy="0 0 0"/>
         <geometry>
-          <mesh filename="package://rm_description/meshes/hero/base.stl" scale="0.001 0.001 0.001"/>
+          <mesh filename="package://rm_description/meshes/hero/base.stl" scale="0.001 .001 0.001"/>
         </geometry>
       </visual>

File: urdf/hero/gimbal.urdf.xacro (robot description, xacro)
@@ -6,13 +6,13 @@
     <link name="yaw">
         <inertial>
-            <mass value="0.592087"/>
-            <origin xyz="0 0 0.013702"/>
-            <inertia ixx="9.726e-4" ixy="0." ixz="0." iyy="8.809e-4"
-                     iyz="0" izz="1.58e-3"/>
+            <mass value="9.19417"/>
+            <origin xyz="0.042103 0.001062 0.132315"/>
+            <inertia ixx="2.820e-1" ixy="-1.017e-5" ixz="-3.986e-2" iyy="3.396e-1"
+                     iyz="1.293e-3" izz="7.004e-2"/>
         </inertial>
         <visual>
             <origin xyz="0 0 0" rpy="0 0 0"/>
             <geometry>
-                <mesh filename="package://rm_description/meshes/hero/yaw_arm.stl" scale="0.001 0.001 0.001"/>
+                <mesh filename="package://rm_description/meshes/hero/yaw.stl" scale="0.001 0.001 0.001" />
             </geometry>
         </visual>
@@ -20,5 +20,5 @@
             <origin xyz="0 0 0" rpy="0 0 0"/>
             <geometry>
-                <mesh filename="package://rm_description/meshes/hero/yaw_arm.stl" scale="0.001 0.001 0.001"/>
+                <mesh filename="package://rm_description/meshes/hero/yaw.stl"  scale="0.001 0.001 0.001" />
             </geometry>
         </collision>
@@ -27,4 +27,5 @@
         <origin xyz="0 0 0.1"
                 rpy="0 0 0"/>
+        <dynamics damping="0.0" friction="0.5"/>
         <parent link="base_link"/>
         <child link="yaw"/>
@@ -33,13 +34,13 @@
     <link name="pitch">
         <inertial>
-            <mass value="1.538674"/>
-            <origin xyz="0.080443 -0.002306 0.010242"/>
-            <inertia ixx="4.18e-3" ixy="-2.3e-5" ixz="-1.212e-3" iyy="2.369e-2"
-                     iyz="-6.373e-5" izz="2.286e-2"/>
+            <mass value="1.956376"/>
+            <origin xyz="0.080443 -0.002306 0.294343"/>
+            <inertia ixx="1.148e-2" ixy="1.569e-3" ixz="2.374e-3" iyy="2.472e-2"
+                     iyz="-8.276e-4" izz="2.189e-2"/>
         </inertial>
         <visual>
             <origin xyz="0 0 0" rpy="0 0 0"/>
             <geometry>
-                <mesh filename="package://rm_description/meshes/hero/pitch.stl" scale="0.001 0.001 0.001"/>
+                <mesh filename="package://rm_description/meshes/hero/pitch.stl" scale="0.001 0.001 0.001" />
             </geometry>
         </visual>
@@ -52,10 +53,11 @@
     </link>
     <joint name="pitch_joint" type="revolute">
-        <origin xyz="0 0 0.2841" rpy="0 0 0"/>
-        <limit effort="3000" velocity="1000" lower="${lower_limit}" upper="${upper_limit}"/>
-        <safety_controller k_velocity="10"
-                           k_position="15"
-                           soft_lower_limit="${lower_limit+threshold}"
-                           soft_upper_limit="${upper_limit-threshold}"/>
+        <origin xyz="0 0 0.284" rpy="0 0 0"/>
+        <dynamics damping="0.0" friction="0.1"/>
+        <limit effort="1.2" velocity="13.82" lower="${lower_limit}" upper="${upper_limit}"/>
+        <!--        <safety_controller k_velocity="10"-->
+        <!--                           k_position="15"-->
+        <!--                           soft_lower_limit="${lower_limit+threshold}"-->
+        <!--                           soft_upper_limit="${upper_limit-threshold}"/>-->
         <parent link="yaw"/>
         <child link="pitch"/>

File: urdf/hero/hero.urdf.xacro (robot description, xacro)
@@ -4,5 +4,5 @@
   <xacro:arg name="load_gimbal" default="true"/>
   <xacro:arg name="load_shooter" default="true"/>
-  <xacro:arg name="use_simulation" default="true"/>
+  <xacro:arg name="load_gazebo" default="true"/>
   <xacro:arg name="use_rm_gazebo" default="false"/>
   <xacro:arg name="roller_type" default="realistic"/>
@@ -13,8 +13,11 @@
   <xacro:if value="$(arg load_gimbal)">
     <xacro:include filename="$(find rm_description)/urdf/hero/gimbal.urdf.xacro"/>
+    <xacro:include filename="$(find rm_description)/urdf/hero/gimbal.transmission.urdf.xacro"/>
   </xacro:if>
   <xacro:if value="$(arg load_shooter)">
+    <xacro:include filename="$(find rm_description)/urdf/hero/shooter.urdf.xacro"/>
+    <xacro:include filename="$(find rm_description)/urdf/hero/shooter.transmission.urdf.xacro"/>
   </xacro:if>
-  <xacro:if value="$(arg use_simulation)">
+  <xacro:if value="$(arg load_gazebo)">
     <xacro:if value="$(arg use_rm_gazebo)">
       <gazebo>

File: urdf/standard/gimbal.urdf.xacro (robot description, xacro)
@@ -28,5 +28,4 @@
                 rpy="0 0 0"/>
         <dynamics damping="0.0" friction="0.5"/>
-        <limit effort="1.2" velocity="13.82" lower="${lower_limit}" upper="${upper_limit}"/>
         <parent link="base_link"/>
         <child link="yaw"/>

Commit message: change inertia and stl

File: urdf/hero/chassis.urdf.xacro (robot description, xacro)
@@ -10,5 +10,5 @@
     <link name="base_link">
       <inertial>
-        <mass value="19.93"/>
+        <mass value="19.31"/>
         <origin xyz="-0.02282 0.002773 0.008173"/>
         <inertia ixx="5.96e-1" ixy="6.075e-3" ixz="4.655e-2" iyy="9.41e-1"

File: urdf/hero/gimbal.urdf.xacro (robot description, xacro)
@@ -6,8 +6,8 @@
     <link name="yaw">
         <inertial>
-            <mass value="9.19417"/>
+            <mass value="4.367"/>
             <origin xyz="0.042103 0.001062 0.132315"/>
-            <inertia ixx="2.820e-1" ixy="-1.017e-5" ixz="-3.986e-2" iyy="3.396e-1"
-                     iyz="1.293e-3" izz="7.004e-2"/>
+            <inertia ixx="7.943e-2" ixy="-4.889e-5" ixz="-5.618e-3" iyy="8.143e-2"
+                     iyz="-4.14e-5" izz="7.76e-3"/>
         </inertial>
         <visual>
@@ -25,5 +25,5 @@
     </link>
     <joint name="yaw_joint" type="continuous">
-        <origin xyz="0 0 0.1"
+        <origin xyz="0 0 0.124"
                 rpy="0 0 0"/>
         <dynamics damping="0.0" friction="0.1"/>
@@ -35,8 +35,8 @@
     <link name="pitch">
         <inertial>
-            <mass value="1.956376"/>
-            <origin xyz="0.080443 -0.002306 0.294343"/>
-            <inertia ixx="1.148e-2" ixy="1.569e-3" ixz="2.374e-3" iyy="2.472e-2"
-                     iyz="-8.276e-4" izz="2.189e-2"/>
+            <mass value="1.65"/>
+            <origin xyz="0.080137 -0.002734 0.011093"/>
+            <inertia ixx="3.355e-3" ixy="2.3e-5" ixz="-1.069e-3" iyy="2.153e-2"
+                     iyz="-6.373e-5" izz="1.995e-2"/>
         </inertial>
         <visual>
@@ -54,5 +54,5 @@
     </link>
     <joint name="pitch_joint" type="revolute">
-        <origin xyz="0 0 0.284" rpy="0 0 0"/>
+        <origin xyz="0 0 0.360" rpy="0 0 0"/>
         <dynamics damping="0.0" friction="0.1"/>
         <limit effort="1.2" velocity="13.82" lower="${lower_limit}" upper="${upper_limit}"/>

File: urdf/hero/shooter.urdf.xacro (robot description, xacro)
@@ -10,8 +10,8 @@
     <link name="trigger">
         <inertial>
-            <mass value="0.295177"/>
-            <origin xyz="-0.00842 0.0 0.00605"/>
-            <inertia ixx="2.255e-4" ixy="2.5698e-7" ixz="2.3929e-6" iyy="2.233e-4"
-                     iyz="5.22e-7" izz="2.643e-4"/>
+            <mass value="1.725"/>
+            <origin xyz="-0.03783 0.001 0.0162"/>
+            <inertia ixx="3.131e-3" ixy="-2.522e-4" ixz="7.492e-4" iyy="1.344e-2"
+                     iyz="6.02e-5" izz="1.265e-2"/>
         </inertial>
         <visual>
@@ -29,5 +29,5 @@
     </link>
     <joint name="trigger_joint" type="continuous">
-        <origin xyz="-0.064 0 0" rpy="0 0 0"/>
+        <origin xyz="-0.173 0 0" rpy="0 0 0"/>
         <dynamics damping="0.0" friction="0.01"/>
         <limit effort="3.0" velocity="49.09" lower="-1e16" upper="1e16"/>

Commit message: add sentry setting

File: urdf/hero/chassis.urdf.xacro (robot description, xacro)
@@ -12,6 +12,6 @@
         <mass value="19.31"/>
         <origin xyz="-0.02282 0.002773 0.008173"/>
-        <inertia ixx="5.96e-1" ixy="6.075e-3" ixz="4.655e-2" iyy="9.41e-1"
-                 iyz="-3.105e-3" izz="1.381e+0"/>
+        <inertia ixx="4.041e-1" ixy="7.617e-3" ixz="-1.317e-2" iyy="3.322e-1"
+                 iyz="7.985e-2" izz="1.8e-1"/>
       </inertial>
       <visual>

Commit message: Change chassis joints name of hero

File: urdf/hero/chassis.urdf.xacro (robot description, xacro)
@@ -1,51 +1,51 @@
 <robot xmlns:xacro="http://www.ros.org/wiki/xacro">
-  <xacro:include filename="$(find rm_description)/urdf/common/mecanum_wheel.urdf.xacro"/>
-  <!-- https://upload.wikimedia.org/wikipedia/commons/5/52/Wheelbase_and_Track.png -->
-  <xacro:property name="wheel_track" value="0.500"/>
-  <xacro:property name="wheel_base" value="0.475"/>
-  <xacro:property name="wheel_offset_z" value="-0.036"/>
-  <xacro:property name="wheel_joint_damping" value="1.0"/>
-  <xacro:property name="wheel_joint_friction" value="1.0"/>
-  <xacro:macro name="chassis" params="roller_type">
-    <link name="base_link">
-      <inertial>
-        <mass value="19.31"/>
-        <origin xyz="-0.02282 0.002773 0.008173"/>
-        <inertia ixx="4.041e-1" ixy="7.617e-3" ixz="-1.317e-2" iyy="3.322e-1"
-                 iyz="7.985e-2" izz="1.8e-1"/>
-      </inertial>
-      <visual>
-        <origin xyz="0 0 0" rpy="0 0 0"/>
-        <geometry>
-          <mesh filename="package://rm_description/meshes/hero/base.stl" scale="0.001 .001 0.001"/>
-        </geometry>
-      </visual>
-      <collision>
-        <origin xyz="0 0 0" rpy="0 0 0"/>
-        <geometry>
-          <mesh filename="package://rm_description/meshes/hero/base.stl" scale="0.001 0.001 0.001"/>
-        </geometry>
-      </collision>
-    </link>
-    <xacro:mecanum_wheel prefix="front_left" connected_to="base_link"
-                         wheel_x_offset="${wheel_track/2}" wheel_y_offset="${wheel_base/2}"
-                         wheel_z_offset="${wheel_offset_z}"
-                         reflect="1" roller_type="${roller_type}"/>
-    <xacro:mecanum_wheel prefix="front_right" connected_to="base_link"
-                         wheel_x_offset="${wheel_track/2}" wheel_y_offset="${-wheel_base/2}"
-                         wheel_z_offset="${wheel_offset_z}"
-                         reflect="-1" roller_type="${roller_type}"/>
-    <xacro:mecanum_wheel prefix="back_left" connected_to="base_link"
-                         wheel_x_offset="${-wheel_track/2}" wheel_y_offset="${wheel_base/2}"
-                         wheel_z_offset="${wheel_offset_z}"
-                         reflect="-1" roller_type="${roller_type}"/>
-    <xacro:mecanum_wheel prefix="back_right" connected_to="base_link"
-                         wheel_x_offset="${-wheel_track/2}" wheel_y_offset="${-wheel_base/2}"
-                         wheel_z_offset="${wheel_offset_z}"
-                         reflect="1" roller_type="${roller_type}"/>
-    <xacro:wheel_transmission prefix="front_left" mechanical_reduction="1"/>
-    <xacro:wheel_transmission prefix="front_right" mechanical_reduction="-1"/>
-    <xacro:wheel_transmission prefix="back_left" mechanical_reduction="1"/>
-    <xacro:wheel_transmission prefix="back_right" mechanical_reduction="-1"/>
-  </xacro:macro>
+    <xacro:include filename="$(find rm_description)/urdf/common/mecanum_wheel.urdf.xacro"/>
+    <!-- https://upload.wikimedia.org/wikipedia/commons/5/52/Wheelbase_and_Track.png -->
+    <xacro:property name="wheel_track" value="0.500"/>
+    <xacro:property name="wheel_base" value="0.475"/>
+    <xacro:property name="wheel_offset_z" value="-0.036"/>
+    <xacro:property name="wheel_joint_damping" value="1.0"/>
+    <xacro:property name="wheel_joint_friction" value="1.0"/>
+    <xacro:macro name="chassis" params="roller_type">
+        <link name="base_link">
+            <inertial>
+                <mass value="19.31"/>
+                <origin xyz="-0.02282 0.002773 0.008173"/>
+                <inertia ixx="4.041e-1" ixy="7.617e-3" ixz="-1.317e-2" iyy="3.322e-1"
+                         iyz="7.985e-2" izz="1.8e-1"/>
+            </inertial>
+            <visual>
+                <origin xyz="0 0 0" rpy="0 0 0"/>
+                <geometry>
+                    <mesh filename="package://rm_description/meshes/hero/base.stl" scale="0.001 .001 0.001"/>
+                </geometry>
+            </visual>
+            <collision>
+                <origin xyz="0 0 0" rpy="0 0 0"/>
+                <geometry>
+                    <mesh filename="package://rm_description/meshes/hero/base.stl" scale="0.001 0.001 0.001"/>
+                </geometry>
+            </collision>
+        </link>
+        <xacro:mecanum_wheel prefix="left_front" connected_to="base_link"
+                             wheel_x_offset="${wheel_track/2}" wheel_y_offset="${wheel_base/2}"
+                             wheel_z_offset="${wheel_offset_z}"
+                             reflect="1" roller_type="${roller_type}"/>
+        <xacro:mecanum_wheel prefix="right_front" connected_to="base_link"
+                             wheel_x_offset="${wheel_track/2}" wheel_y_offset="${-wheel_base/2}"
+                             wheel_z_offset="${wheel_offset_z}"
+                             reflect="-1" roller_type="${roller_type}"/>
+        <xacro:mecanum_wheel prefix="left_back" connected_to="base_link"
+                             wheel_x_offset="${-wheel_track/2}" wheel_y_offset="${wheel_base/2}"
+                             wheel_z_offset="${wheel_offset_z}"
+                             reflect="-1" roller_type="${roller_type}"/>
+        <xacro:mecanum_wheel prefix="right_back" connected_to="base_link"
+                             wheel_x_offset="${-wheel_track/2}" wheel_y_offset="${-wheel_base/2}"
+                             wheel_z_offset="${wheel_offset_z}"
+                             reflect="1" roller_type="${roller_type}"/>
+        <xacro:wheel_transmission prefix="left_front" mechanical_reduction="1"/>
+        <xacro:wheel_transmission prefix="right_front" mechanical_reduction="-1"/>
+        <xacro:wheel_transmission prefix="left_back" mechanical_reduction="1"/>
+        <xacro:wheel_transmission prefix="right_back" mechanical_reduction="-1"/>
+    </xacro:macro>
 </robot>

Commit message: Delete wheel_joint_damping and wheel_joint_friction of chassis

File: urdf/hero/chassis.urdf.xacro (robot description, xacro)
@@ -5,6 +5,4 @@
     <xacro:property name="wheel_base" value="0.475"/>
     <xacro:property name="wheel_offset_z" value="-0.036"/>
-    <xacro:property name="wheel_joint_damping" value="1.0"/>
-    <xacro:property name="wheel_joint_friction" value="1.0"/>
     <xacro:macro name="chassis" params="roller_type">
         <link name="base_link">

File: urdf/standard/chassis.urdf.xacro (robot description, xacro)
@@ -5,6 +5,4 @@
     <xacro:property name="wheel_base" value="0.395"/>
     <xacro:property name="wheel_offset_z" value="0.0"/>
-    <xacro:property name="wheel_joint_damping" value="1.0"/>
-    <xacro:property name="wheel_joint_friction" value="1.0"/>
     <xacro:macro name="chassis" params="roller_type">
         <link name="base_link">

File: urdf/swerve/chassis.urdf.xacro (robot description, xacro)
@@ -5,6 +5,4 @@
     <xacro:property name="wheel_base" value="0.475"/>
     <xacro:property name="wheel_offset_z" value="-0.036"/>
-    <xacro:property name="wheel_joint_damping" value="1.0"/>
-    <xacro:property name="wheel_joint_friction" value="1.0"/>
     <xacro:macro name="chassis">
         <link name="base_link">
