Commit message: add imu and cover link

File: urdf/hero/chassis.urdf.xacro (robot description, xacro)
@@ -26,4 +26,41 @@
             </collision>
         </link>
+        <link name="cover">
+            <inertial>
+                <mass value="0.118"/>
+                <origin xyz="-0.037 -0.003 0.0"/>
+                <inertia ixx="6.240e-4" ixy="7.325e-4" ixz="1.839e-5" iyy="1.083e-3" iyz="-1.166e-5" izz="1.602e-3"/>
+            </inertial>
+            <visual>
+                <origin xyz="0 0 0" rpy="0 0 0"/>
+                <geometry>
+                    <mesh filename="package://rm_description/meshes/hero/cover.stl" scale="0.001 0.001 0.001"/>
+                </geometry>
+            </visual>
+            <collision>
+                <origin xyz="0.033 0.0 -0.0" rpy="0 0.0 0"/>
+                <geometry>
+                    <mesh filename="package://rm_description/meshes/hero/cover.stl" scale="0.001 0.001 0.001"/>
+                </geometry>
+            </collision>
+        </link>
+        <joint name="cover_joint" type="revolute">
+            <axis xyz="1 0 0"/>
+            <origin xyz="-0.27 0.201 0.125"/>
+            <limit effort="1" velocity="30" lower="-3.14" upper="3.14"/>
+            <dynamics damping="0.0" friction="0.1"/>
+            <parent link="pitch"/>
+            <child link="cover"/>
+        </joint>
+        <transmission name="trans_cover_joint">
+            <type>transmission_interface/SimpleTransmission</type>
+            <actuator name="cover_joint_motor">
+                <mechanicalReduction>1</mechanicalReduction>
+            </actuator>
+            <joint name="cover_joint">
+                <offset>0</offset>
+                <hardwareInterface>hardware_interface/EffortJointInterface</hardwareInterface>
+            </joint>
+        </transmission>
         <xacro:mecanum_wheel prefix="left_front" connected_to="base_link"
                              wheel_x_offset="${wheel_track/2}" wheel_y_offset="${wheel_base/2}"

File: urdf/hero/hero.urdf.xacro (robot description, xacro)
@@ -13,4 +13,7 @@
     <xacro:include filename="$(find rm_description)/urdf/hero/gimbal.urdf.xacro"/>
     <xacro:include filename="$(find rm_description)/urdf/hero/gimbal.transmission.urdf.xacro"/>
+    <xacro:include filename="$(find rm_description)/urdf/common/imu.urdf.xacro"/>
+    <xacro:IMU connected_to="yaw" imu_name="base_imu" simulation="true"
+               xyz="0.024 -0.014 0.088" rpy="${pi} ${-pi/2} 0"/>
     <xacro:include filename="$(find rm_description)/urdf/common/camera.urdf.xacro"/>
     <xacro:camera_sensor xyz="0.127 0 -0.038" rpy="3.14 0 0" parent="pitch"

File: urdf/standard/gimbal.transmission.urdf.xacro (robot description, xacro)
@@ -21,3 +21,13 @@
         </joint>
     </transmission>
+    <transmission name="trans_cover_joint">
+        <type>transmission_interface/SimpleTransmission</type>
+        <actuator name="cover_joint_motor">
+            <mechanicalReduction>1</mechanicalReduction>
+        </actuator>
+        <joint name="cover_joint">
+            <offset>0</offset>
+            <hardwareInterface>hardware_interface/EffortJointInterface</hardwareInterface>
+        </joint>
+    </transmission>
 </robot>

File: urdf/standard/gimbal.urdf.xacro (robot description, xacro)
@@ -64,3 +64,30 @@
             <axis xyz="0 1 0 "/>
         </joint>
+    <link name="cover">
+        <inertial>
+            <mass value="0.149"/>
+            <origin xyz="-0.008 -0.005 0.019"/>
+            <inertia ixx="2.366e-3" ixy="-2.372e-4" ixz="-7.983e-4" iyy="2.959e-3" iyz="-2.826e-4" izz="9.090e-4"/>
+        </inertial>
+        <visual>
+            <origin xyz="0 0 0" rpy="0 0 0"/>
+            <geometry>
+                <mesh filename="package://rm_description/meshes/standard/cover.stl" scale="0.001 0.001 0.001"/>
+            </geometry>
+        </visual>
+        <collision>
+            <origin xyz="0.033 0.0 -0.0" rpy="0 0.0 0"/>
+            <geometry>
+                <mesh filename="package://rm_description/meshes/standard/cover.stl" scale="0.001 0.001 0.001"/>
+            </geometry>
+        </collision>
+    </link>
+    <joint name="cover_joint" type="revolute">
+        <axis xyz="0 0 1"/>
+        <origin xyz="0.037 0.042 0.122"/>
+        <limit effort="0.1" velocity="30" lower="-3.14" upper="3.14"/>
+        <dynamics damping="0.0" friction="0.1"/>
+        <parent link="pitch"/>
+        <child link="cover"/>
+    </joint>
 </robot>

File: urdf/standard/standard.urdf.xacro (robot description, xacro)
@@ -9,11 +9,11 @@
         <xacro:include filename="$(find rm_description)/urdf/standard/chassis.urdf.xacro"/>
         <xacro:chassis roller_type="$(arg roller_type)"/>
-        <xacro:include filename="$(find rm_description)/urdf/common/imu.urdf.xacro"/>
-        <xacro:IMU connected_to="base_link" imu_name="base_imu" simulation="true"
-                   xyz="0.065 0.12 0.07"/>
     </xacro:if>
     <xacro:if value="$(arg load_gimbal)">
         <xacro:include filename="$(find rm_description)/urdf/standard/gimbal.urdf.xacro"/>
         <xacro:include filename="$(find rm_description)/urdf/standard/gimbal.transmission.urdf.xacro"/>
+        <xacro:include filename="$(find rm_description)/urdf/common/imu.urdf.xacro"/>
+        <xacro:IMU connected_to="yaw" imu_name="base_imu" simulation="true"
+                   xyz="-0.068 0.064 0.077" rpy="${pi} ${-pi/2} 0"/>
         <xacro:include filename="$(find rm_description)/urdf/common/camera.urdf.xacro"/>
         <xacro:camera_sensor xyz="0.127 0 -0.038" rpy="0 0 0" parent="pitch"
