Commit message: Add hero four friction wheel urdf

File: urdf/hero/shooter.transmission.urdf.xacro (robot description, xacro)
@@ -11,21 +11,41 @@
         </joint>
     </transmission>
-    <transmission name="trans_left_friction_wheel_joint_joint">
+    <transmission name="trans_left_follow_friction_wheel_joint_joint">
         <type>transmission_interface/SimpleTransmission</type>
-        <actuator name="left_friction_wheel_joint_motor">
+        <actuator name="left_follow_friction_wheel_joint_motor">
             <hardwareInterface>hardware_interface/EffortJointInterface</hardwareInterface>
             <mechanicalReduction>1</mechanicalReduction>
         </actuator>
-        <joint name="left_friction_wheel_joint">
+        <joint name="left_follow_friction_wheel_joint">
             <hardwareInterface>hardware_interface/EffortJointInterface</hardwareInterface>
         </joint>
     </transmission>
-    <transmission name="trans_right_friction_wheel_joint_joint">
+    <transmission name="trans_right_follow_friction_wheel_joint_joint">
         <type>transmission_interface/SimpleTransmission</type>
-        <actuator name="right_friction_wheel_joint_motor">
+        <actuator name="right_follow_friction_wheel_joint_motor">
             <hardwareInterface>hardware_interface/EffortJointInterface</hardwareInterface>
             <mechanicalReduction>1</mechanicalReduction>
         </actuator>
-        <joint name="right_friction_wheel_joint">
+        <joint name="right_follow_friction_wheel_joint">
+            <hardwareInterface>hardware_interface/EffortJointInterface</hardwareInterface>
+        </joint>
+    </transmission>
+    <transmission name="trans_left_back_friction_wheel_joint_joint">
+        <type>transmission_interface/SimpleTransmission</type>
+        <actuator name="left_back_friction_wheel_joint_motor">
+            <hardwareInterface>hardware_interface/EffortJointInterface</hardwareInterface>
+            <mechanicalReduction>1</mechanicalReduction>
+        </actuator>
+        <joint name="left_back_friction_wheel_joint">
+            <hardwareInterface>hardware_interface/EffortJointInterface</hardwareInterface>
+        </joint>
+    </transmission>
+    <transmission name="trans_right_back_friction_wheel_joint_joint">
+        <type>transmission_interface/SimpleTransmission</type>
+        <actuator name="right_back_friction_wheel_joint_motor">
+            <hardwareInterface>hardware_interface/EffortJointInterface</hardwareInterface>
+            <mechanicalReduction>1</mechanicalReduction>
+        </actuator>
+        <joint name="right_back_friction_wheel_joint">
             <hardwareInterface>hardware_interface/EffortJointInterface</hardwareInterface>
         </joint>

File: urdf/hero/shooter.urdf.xacro (robot description, xacro)
@@ -4,8 +4,18 @@
     <xacro:property name="wheel_offset_y" value="0.049"/>
     <xacro:property name="wheel_offset_z" value="0.0"/>
-    <xacro:friction_wheel prefixs="left" connected_to="pitch"
-                          wheel_x_offset="${wheel_offset_x}" wheel_y_offset="${wheel_offset_y}" wheel_z_offset="${wheel_offset_z}"/>
-    <xacro:friction_wheel prefixs="right" connected_to="pitch"
-                          wheel_x_offset="${wheel_offset_x}" wheel_y_offset="${-wheel_offset_y}" wheel_z_offset="${wheel_offset_z}"/>
+    <xacro:property name="wheel_and_wheel_offset_x" value="0.0"/>
+    <xacro:friction_wheel prefixs="left_follow" connected_to="pitch"
+                          wheel_x_offset="${wheel_offset_x}" wheel_y_offset="${wheel_offset_y}"
+                          wheel_z_offset="${wheel_offset_z}"/>
+    <xacro:friction_wheel prefixs="right_follow" connected_to="pitch"
+                          wheel_x_offset="${wheel_offset_x}" wheel_y_offset="${-wheel_offset_y}"
+                          wheel_z_offset="${wheel_offset_z}"/>
+    <xacro:friction_wheel prefixs="left_back" connected_to="pitch"
+                          wheel_x_offset="${wheel_offset_x+wheel_and_wheel_offset_x}" wheel_y_offset="${wheel_offset_y}"
+                          wheel_z_offset="${wheel_offset_z}"/>
+    <xacro:friction_wheel prefixs="right_back" connected_to="pitch"
+                          wheel_x_offset="${wheel_offset_x+wheel_and_wheel_offset_x}"
+                          wheel_y_offset="${-wheel_offset_y}"
+                          wheel_z_offset="${wheel_offset_z}"/>
     <link name="trigger">
         <inertial>

Commit message: Fix front spelling mistakes in hero.yaml and urdf

File: urdf/hero/shooter.transmission.urdf.xacro (robot description, xacro)
@@ -11,21 +11,21 @@
         </joint>
     </transmission>
-    <transmission name="trans_left_follow_friction_wheel_joint_joint">
+    <transmission name="trans_left_front_friction_wheel_joint_joint">
         <type>transmission_interface/SimpleTransmission</type>
-        <actuator name="left_follow_friction_wheel_joint_motor">
+        <actuator name="left_front_friction_wheel_joint_motor">
             <hardwareInterface>hardware_interface/EffortJointInterface</hardwareInterface>
             <mechanicalReduction>1</mechanicalReduction>
         </actuator>
-        <joint name="left_follow_friction_wheel_joint">
+        <joint name="left_front_friction_wheel_joint">
             <hardwareInterface>hardware_interface/EffortJointInterface</hardwareInterface>
         </joint>
     </transmission>
-    <transmission name="trans_right_follow_friction_wheel_joint_joint">
+    <transmission name="trans_right_front_friction_wheel_joint_joint">
         <type>transmission_interface/SimpleTransmission</type>
-        <actuator name="right_follow_friction_wheel_joint_motor">
+        <actuator name="right_front_friction_wheel_joint_motor">
             <hardwareInterface>hardware_interface/EffortJointInterface</hardwareInterface>
             <mechanicalReduction>1</mechanicalReduction>
         </actuator>
-        <joint name="right_follow_friction_wheel_joint">
+        <joint name="right_front_friction_wheel_joint">
             <hardwareInterface>hardware_interface/EffortJointInterface</hardwareInterface>
         </joint>

File: urdf/hero/shooter.urdf.xacro (robot description, xacro)
@@ -4,9 +4,9 @@
     <xacro:property name="wheel_offset_y" value="0.049"/>
     <xacro:property name="wheel_offset_z" value="0.0"/>
-    <xacro:property name="wheel_and_wheel_offset_x" value="0.06"/>
-    <xacro:friction_wheel prefixs="left_follow" connected_to="pitch"
+    <xacro:property name="wheel_and_wheel_offset_x" value="0.07"/>
+    <xacro:friction_wheel prefixs="left_front" connected_to="pitch"
                           wheel_x_offset="${wheel_offset_x+wheel_and_wheel_offset_x}" wheel_y_offset="${wheel_offset_y}"
                           wheel_z_offset="${wheel_offset_z}"/>
-    <xacro:friction_wheel prefixs="right_follow" connected_to="pitch"
+    <xacro:friction_wheel prefixs="right_front" connected_to="pitch"
                           wheel_x_offset="${wheel_offset_x+wheel_and_wheel_offset_x}"
                           wheel_y_offset="${-wheel_offset_y}"

Commit message: Update hero shooter urdf and friction wheel number

File: urdf/hero/shooter.transmission.urdf.xacro (robot description, xacro)
@@ -11,24 +11,24 @@
         </joint>
     </transmission>
-    <transmission name="trans_left_front_friction_wheel_joint_joint">
-        <type>transmission_interface/SimpleTransmission</type>
-        <actuator name="left_front_friction_wheel_joint_motor">
-            <hardwareInterface>hardware_interface/EffortJointInterface</hardwareInterface>
-            <mechanicalReduction>1</mechanicalReduction>
-        </actuator>
-        <joint name="left_front_friction_wheel_joint">
-            <hardwareInterface>hardware_interface/EffortJointInterface</hardwareInterface>
-        </joint>
-    </transmission>
-    <transmission name="trans_right_front_friction_wheel_joint_joint">
-        <type>transmission_interface/SimpleTransmission</type>
-        <actuator name="right_front_friction_wheel_joint_motor">
-            <hardwareInterface>hardware_interface/EffortJointInterface</hardwareInterface>
-            <mechanicalReduction>1</mechanicalReduction>
-        </actuator>
-        <joint name="right_front_friction_wheel_joint">
-            <hardwareInterface>hardware_interface/EffortJointInterface</hardwareInterface>
-        </joint>
-    </transmission>
+    <!--    <transmission name="trans_left_front_friction_wheel_joint_joint">-->
+    <!--        <type>transmission_interface/SimpleTransmission</type>-->
+    <!--        <actuator name="left_front_friction_wheel_joint_motor">-->
+    <!--            <hardwareInterface>hardware_interface/EffortJointInterface</hardwareInterface>-->
+    <!--            <mechanicalReduction>1</mechanicalReduction>-->
+    <!--        </actuator>-->
+    <!--        <joint name="left_front_friction_wheel_joint">-->
+    <!--            <hardwareInterface>hardware_interface/EffortJointInterface</hardwareInterface>-->
+    <!--        </joint>-->
+    <!--    </transmission>-->
+    <!--    <transmission name="trans_right_front_friction_wheel_joint_joint">-->
+    <!--        <type>transmission_interface/SimpleTransmission</type>-->
+    <!--        <actuator name="right_front_friction_wheel_joint_motor">-->
+    <!--            <hardwareInterface>hardware_interface/EffortJointInterface</hardwareInterface>-->
+    <!--            <mechanicalReduction>1</mechanicalReduction>-->
+    <!--        </actuator>-->
+    <!--        <joint name="right_front_friction_wheel_joint">-->
+    <!--            <hardwareInterface>hardware_interface/EffortJointInterface</hardwareInterface>-->
+    <!--        </joint>-->
+    <!--    </transmission>-->
     <transmission name="trans_left_back_friction_wheel_joint_joint">
         <type>transmission_interface/SimpleTransmission</type>

File: urdf/hero/shooter.urdf.xacro (robot description, xacro)
@@ -5,11 +5,11 @@
     <xacro:property name="wheel_offset_z" value="0.0"/>
     <xacro:property name="wheel_and_wheel_offset_x" value="0.07"/>
-    <xacro:friction_wheel prefixs="left_front" connected_to="pitch"
-                          wheel_x_offset="${wheel_offset_x+wheel_and_wheel_offset_x}" wheel_y_offset="${wheel_offset_y}"
-                          wheel_z_offset="${wheel_offset_z}"/>
-    <xacro:friction_wheel prefixs="right_front" connected_to="pitch"
-                          wheel_x_offset="${wheel_offset_x+wheel_and_wheel_offset_x}"
-                          wheel_y_offset="${-wheel_offset_y}"
-                          wheel_z_offset="${wheel_offset_z}"/>
+    <!--    <xacro:friction_wheel prefixs="left_front" connected_to="pitch"-->
+    <!--                          wheel_x_offset="${wheel_offset_x+wheel_and_wheel_offset_x}" wheel_y_offset="${wheel_offset_y}"-->
+    <!--                          wheel_z_offset="${wheel_offset_z}"/>-->
+    <!--    <xacro:friction_wheel prefixs="right_front" connected_to="pitch"-->
+    <!--                          wheel_x_offset="${wheel_offset_x+wheel_and_wheel_offset_x}"-->
+    <!--                          wheel_y_offset="${-wheel_offset_y}"-->
+    <!--                          wheel_z_offset="${wheel_offset_z}"/>-->
     <xacro:friction_wheel prefixs="left_back" connected_to="pitch"
                           wheel_x_offset="${wheel_offset_x}" wheel_y_offset="${wheel_offset_y}"

Commit message: Delete shooter Hero.cpp and update urdf

File: urdf/hero/shooter.transmission.urdf.xacro (robot description, xacro)
@@ -11,41 +11,21 @@
         </joint>
     </transmission>
-    <!--    <transmission name="trans_left_front_friction_wheel_joint_joint">-->
-    <!--        <type>transmission_interface/SimpleTransmission</type>-->
-    <!--        <actuator name="left_front_friction_wheel_joint_motor">-->
-    <!--            <hardwareInterface>hardware_interface/EffortJointInterface</hardwareInterface>-->
-    <!--            <mechanicalReduction>1</mechanicalReduction>-->
-    <!--        </actuator>-->
-    <!--        <joint name="left_front_friction_wheel_joint">-->
-    <!--            <hardwareInterface>hardware_interface/EffortJointInterface</hardwareInterface>-->
-    <!--        </joint>-->
-    <!--    </transmission>-->
-    <!--    <transmission name="trans_right_front_friction_wheel_joint_joint">-->
-    <!--        <type>transmission_interface/SimpleTransmission</type>-->
-    <!--        <actuator name="right_front_friction_wheel_joint_motor">-->
-    <!--            <hardwareInterface>hardware_interface/EffortJointInterface</hardwareInterface>-->
-    <!--            <mechanicalReduction>1</mechanicalReduction>-->
-    <!--        </actuator>-->
-    <!--        <joint name="right_front_friction_wheel_joint">-->
-    <!--            <hardwareInterface>hardware_interface/EffortJointInterface</hardwareInterface>-->
-    <!--        </joint>-->
-    <!--    </transmission>-->
-    <transmission name="trans_left_back_friction_wheel_joint_joint">
+    <transmission name="trans_left_friction_wheel_joint_joint">
         <type>transmission_interface/SimpleTransmission</type>
-        <actuator name="left_back_friction_wheel_joint_motor">
+        <actuator name="left_friction_wheel_joint_motor">
             <hardwareInterface>hardware_interface/EffortJointInterface</hardwareInterface>
             <mechanicalReduction>1</mechanicalReduction>
         </actuator>
-        <joint name="left_back_friction_wheel_joint">
+        <joint name="left_friction_wheel_joint">
             <hardwareInterface>hardware_interface/EffortJointInterface</hardwareInterface>
         </joint>
     </transmission>
-    <transmission name="trans_right_back_friction_wheel_joint_joint">
+    <transmission name="trans_right_friction_wheel_joint_joint">
         <type>transmission_interface/SimpleTransmission</type>
-        <actuator name="right_back_friction_wheel_joint_motor">
+        <actuator name="right_friction_wheel_joint_motor">
             <hardwareInterface>hardware_interface/EffortJointInterface</hardwareInterface>
             <mechanicalReduction>1</mechanicalReduction>
         </actuator>
-        <joint name="right_back_friction_wheel_joint">
+        <joint name="right_friction_wheel_joint">
             <hardwareInterface>hardware_interface/EffortJointInterface</hardwareInterface>
         </joint>

File: urdf/hero/shooter.urdf.xacro (robot description, xacro)
@@ -4,16 +4,8 @@
     <xacro:property name="wheel_offset_y" value="0.049"/>
     <xacro:property name="wheel_offset_z" value="0.0"/>
-    <xacro:property name="wheel_and_wheel_offset_x" value="0.07"/>
-    <!--    <xacro:friction_wheel prefixs="left_front" connected_to="pitch"-->
-    <!--                          wheel_x_offset="${wheel_offset_x+wheel_and_wheel_offset_x}" wheel_y_offset="${wheel_offset_y}"-->
-    <!--                          wheel_z_offset="${wheel_offset_z}"/>-->
-    <!--    <xacro:friction_wheel prefixs="right_front" connected_to="pitch"-->
-    <!--                          wheel_x_offset="${wheel_offset_x+wheel_and_wheel_offset_x}"-->
-    <!--                          wheel_y_offset="${-wheel_offset_y}"-->
-    <!--                          wheel_z_offset="${wheel_offset_z}"/>-->
-    <xacro:friction_wheel prefixs="left_back" connected_to="pitch"
+    <xacro:friction_wheel prefixs="left" connected_to="pitch"
                           wheel_x_offset="${wheel_offset_x}" wheel_y_offset="${wheel_offset_y}"
                           wheel_z_offset="${wheel_offset_z}"/>
-    <xacro:friction_wheel prefixs="right_back" connected_to="pitch"
+    <xacro:friction_wheel prefixs="right" connected_to="pitch"
                           wheel_x_offset="${wheel_offset_x}"
                           wheel_y_offset="${-wheel_offset_y}"

Commit message: Add magazine joint in standard and hero urdf

File: urdf/hero/shooter.transmission.urdf.xacro (robot description, xacro)
@@ -28,3 +28,12 @@
         </joint>
     </transmission>
+    <transmission name="trans_magazine_joint">
+        <type>transmission_interface/SimpleTransmission</type>
+        <actuator name="magazine_joint_motor">
+            <mechanicalReduction>1</mechanicalReduction>
+        </actuator>
+        <joint name="magazine_joint">
+            <hardwareInterface>hardware_interface/EffortJointInterface</hardwareInterface>
+        </joint>
+    </transmission>
 </robot>

File: urdf/hero/shooter.urdf.xacro (robot description, xacro)
@@ -38,3 +38,19 @@
         <axis xyz="0 0 1 "/>
     </joint>
+    <link name="magazine">
+        <inertial>
+            <mass value="0.295177"/>
+            <origin xyz="-0.00842 0.0 0.00605"/>
+            <inertia ixx="2.255e-4" ixy="2.5698e-7" ixz="2.3929e-6" iyy="2.233e-4"
+                     iyz="5.22e-7" izz="2.643e-4"/>
+        </inertial>
+    </link>
+    <joint name="magazine_joint" type="continuous">
+        <origin xyz="-0.1 0.04 0.08" rpy="0 0 0"/>
+        <dynamics damping="0.0" friction="0.01"/>
+        <limit effort="1.0" velocity="43.54" lower="-1e16" upper="1e16"/>
+        <parent link="base_link"/>
+        <child link="magazine"/>
+        <axis xyz="0 0 1 "/>
+    </joint>
 </robot>

File: urdf/standard/shooter.transmission.urdf.xacro (robot description, xacro)
@@ -28,3 +28,12 @@
         </joint>
     </transmission>
+    <transmission name="trans_magazine_joint">
+        <type>transmission_interface/SimpleTransmission</type>
+        <actuator name="magazine_joint_motor">
+            <mechanicalReduction>1</mechanicalReduction>
+        </actuator>
+        <joint name="magazine_joint">
+            <hardwareInterface>hardware_interface/EffortJointInterface</hardwareInterface>
+        </joint>
+    </transmission>
 </robot>

File: urdf/standard/shooter.urdf.xacro (robot description, xacro)
@@ -39,3 +39,19 @@
         <axis xyz="0 0 1 "/>
     </joint>
+    <link name="magazine">
+        <inertial>
+            <mass value="0.295177"/>
+            <origin xyz="-0.00842 0.0 0.00605"/>
+            <inertia ixx="2.255e-4" ixy="2.5698e-7" ixz="2.3929e-6" iyy="2.233e-4"
+                     iyz="5.22e-7" izz="2.643e-4"/>
+        </inertial>
+    </link>
+    <joint name="magazine_joint" type="continuous">
+        <origin xyz="-0.1 0.04 0.08" rpy="0 0 0"/>
+        <dynamics damping="0.0" friction="0.01"/>
+        <limit effort="1.0" velocity="43.54" lower="-1e16" upper="1e16"/>
+        <parent link="pitch"/>
+        <child link="magazine"/>
+        <axis xyz="0 0 1 "/>
+    </joint>
 </robot>

Commit message: Delete useless joint and transmission

File: urdf/hero/shooter.transmission.urdf.xacro (robot description, xacro)
@@ -28,12 +28,3 @@
         </joint>
     </transmission>
-    <transmission name="trans_magazine_joint">
-        <type>transmission_interface/SimpleTransmission</type>
-        <actuator name="magazine_joint_motor">
-            <mechanicalReduction>1</mechanicalReduction>
-        </actuator>
-        <joint name="magazine_joint">
-            <hardwareInterface>hardware_interface/EffortJointInterface</hardwareInterface>
-        </joint>
-    </transmission>
 </robot>

File: urdf/hero/shooter.urdf.xacro (robot description, xacro)
@@ -38,19 +38,3 @@
         <axis xyz="0 0 1 "/>
     </joint>
-    <link name="magazine">
-        <inertial>
-            <mass value="0.295177"/>
-            <origin xyz="-0.00842 0.0 0.00605"/>
-            <inertia ixx="2.255e-4" ixy="2.5698e-7" ixz="2.3929e-6" iyy="2.233e-4"
-                     iyz="5.22e-7" izz="2.643e-4"/>
-        </inertial>
-    </link>
-    <joint name="magazine_joint" type="continuous">
-        <origin xyz="-0.1 0.04 0.08" rpy="0 0 0"/>
-        <dynamics damping="0.0" friction="0.01"/>
-        <limit effort="1.0" velocity="43.54" lower="-1e16" upper="1e16"/>
-        <parent link="base_link"/>
-        <child link="magazine"/>
-        <axis xyz="0 0 1 "/>
-    </joint>
 </robot>

File: urdf/standard/gimbal.urdf.xacro (robot description, xacro)
@@ -86,5 +86,5 @@
         <axis xyz="0 0 1"/>
         <origin xyz="0.037 0.042 0.122"/>
-        <limit effort="0.1" velocity="30" lower="-3.14" upper="3.14"/>
+        <limit effort="1.0" velocity="30" lower="-3.14" upper="3.14"/>
         <dynamics damping="0.0" friction="0.1"/>
         <parent link="pitch"/>

File: urdf/standard/shooter.transmission.urdf.xacro (robot description, xacro)
@@ -28,12 +28,3 @@
         </joint>
     </transmission>
-    <transmission name="trans_magazine_joint">
-        <type>transmission_interface/SimpleTransmission</type>
-        <actuator name="magazine_joint_motor">
-            <mechanicalReduction>1</mechanicalReduction>
-        </actuator>
-        <joint name="magazine_joint">
-            <hardwareInterface>hardware_interface/EffortJointInterface</hardwareInterface>
-        </joint>
-    </transmission>
 </robot>

File: urdf/standard/shooter.urdf.xacro (robot description, xacro)
@@ -39,19 +39,3 @@
         <axis xyz="0 0 1 "/>
     </joint>
-    <link name="magazine">
-        <inertial>
-            <mass value="0.295177"/>
-            <origin xyz="-0.00842 0.0 0.00605"/>
-            <inertia ixx="2.255e-4" ixy="2.5698e-7" ixz="2.3929e-6" iyy="2.233e-4"
-                     iyz="5.22e-7" izz="2.643e-4"/>
-        </inertial>
-    </link>
-    <joint name="magazine_joint" type="continuous">
-        <origin xyz="-0.1 0.04 0.08" rpy="0 0 0"/>
-        <dynamics damping="0.0" friction="0.01"/>
-        <limit effort="1.0" velocity="43.54" lower="-1e16" upper="1e16"/>
-        <parent link="pitch"/>
-        <child link="magazine"/>
-        <axis xyz="0 0 1 "/>
-    </joint>
 </robot>

Commit message: Update hero trigger urdf "mechanicalReduction"

File: urdf/hero/shooter.transmission.urdf.xacro (robot description, xacro)
@@ -4,5 +4,5 @@
         <type>transmission_interface/SimpleTransmission</type>
         <actuator name="trigger_joint_motor">
-            <mechanicalReduction>-26.851</mechanicalReduction>
+            <mechanicalReduction>-19.2032</mechanicalReduction>
         </actuator>
         <joint name="trigger_joint">

File: urdf/hero/shooter.urdf.xacro (robot description, xacro)
@@ -33,5 +33,5 @@
         <origin xyz="-0.064 0 0" rpy="0 0 0"/>
         <dynamics damping="0.0" friction="0.01"/>
-        <limit effort="7.0" velocity="43.54" lower="-1e16" upper="1e16"/>
+        <limit effort="5.0" velocity="50" lower="-1e16" upper="1e16"/>
         <parent link="base_link"/>
         <child link="trigger"/>
