Commit message: Update hero shooter urdf and hero.yaml

File: urdf/hero/shooter.urdf.xacro (robot description, xacro)
@@ -4,5 +4,5 @@
     <xacro:property name="wheel_offset_y" value="0.049"/>
     <xacro:property name="wheel_offset_z" value="0.0"/>
-    <xacro:property name="wheel_and_wheel_offset_x" value="0.0"/>
+    <xacro:property name="wheel_and_wheel_offset_x" value="0.08"/>
     <xacro:friction_wheel prefixs="left_follow" connected_to="pitch"
                           wheel_x_offset="${wheel_offset_x}" wheel_y_offset="${wheel_offset_y}"

Commit message: Change hero trigger joint effort to 5

File: urdf/hero/shooter.urdf.xacro (robot description, xacro)
@@ -34,5 +34,5 @@
         <origin xyz="-0.064 0 0" rpy="0 0 0"/>
         <dynamics damping="0.0" friction="0.01"/>
-        <limit effort="1.0" velocity="43.54" lower="-1e16" upper="1e16"/>
+        <limit effort="5.0" velocity="43.54" lower="-1e16" upper="1e16"/>
         <parent link="base_link"/>
         <child link="trigger"/>

Commit message: Update shooter urdf of hero

File: urdf/hero/shooter.urdf.xacro (robot description, xacro)
@@ -33,5 +33,5 @@
         <origin xyz="-0.064 0 0" rpy="0 0 0"/>
         <dynamics damping="0.0" friction="0.01"/>
-        <limit effort="5.0" velocity="43.54" lower="-1e16" upper="1e16"/>
+        <limit effort="7.0" velocity="43.54" lower="-1e16" upper="1e16"/>
         <parent link="base_link"/>
         <child link="trigger"/>

Commit message: Update trigger's reduction ratio.

File: urdf/hero/shooter.urdf.xacro (robot description, xacro)
@@ -33,5 +33,5 @@
         <origin xyz="-0.064 0 0" rpy="0 0 0"/>
         <dynamics damping="0.0" friction="0.01"/>
-        <limit effort="5.0" velocity="50" lower="-1e16" upper="1e16"/>
+        <limit effort="6.99" velocity="35.758" lower="-1e16" upper="1e16"/>
         <parent link="base_link"/>
         <child link="trigger"/>
