Commit message: add infantry

File: urdf/hero/gimbal.urdf.xacro (robot description, xacro)
@@ -58,7 +58,7 @@
         <inertial>
             <mass value="1.538674"/>
-            <origin xyz="0.049138 -0.002939 0.348926"/>
-            <inertia ixx="1.93e-1" ixy="6.188e-5" ixz="-2.95e-2" iyy="2.016e-1"
-                     iyz="1.256e-3" izz="1.021e-2"/>
+            <origin xyz="0.080443 -0.002306 0.010242"/>
+            <inertia ixx="4.18e-3" ixy="-2.3e-5" ixz="-1.212e-3" iyy="2.369e-2"
+                     iyz="-6.373e-5" izz="2.286e-2"/>
         </inertial>
         <visual>
@@ -77,8 +77,8 @@
     <joint name="pitch_joint"  type="revolute">
         <origin xyz="0 0 0.2841"  rpy="0 0 0" />
-        <limit effort="30" velocity="10" lower="-0.436323" upper="0.7853982"/>
+        <limit effort="3000" velocity="1000" lower="-0.436323" upper="0.7853982"/>
         <parent link="yaw_base_link" />
         <child link="pitch_link" />
-        <axis xyz="1 0 0 " />
+        <axis xyz="0 1 0 " />
     </joint>
     <!-- transmission -->

Commit message: add shooter

File: urdf/hero/gimbal.urdf.xacro (robot description, xacro)
@@ -27,30 +27,4 @@
         <axis xyz="0 0 1" />
     </joint>
-    <link name="yaw_base_link">
-        <inertial>
-            <mass value="4.17874"/>
-            <origin xyz="-0.012411 -0.01295 0.120327"/>
-            <inertia ixx="7.425e-2" ixy="-4.926e-5" ixz="4.741e-3" iyy="7.597e-2"
-                     iyz="7.286e-5" izz="7.357e-3"/>
-        </inertial>
-        <visual>
-            <origin xyz="0 0 0" rpy="0 0 0"/>
-            <geometry>
-                <mesh filename="package://rm_description/meshes/hero/yaw_arm.stl" scale="0.001 0.001 0.001" />
-            </geometry>
-        </visual>
-        <collision>
-            <origin xyz="0 0 0" rpy="0 0 0"/>
-            <geometry>
-                <mesh filename="package://rm_description/meshes/hero/yaw_arm.stl"  scale="0.001 0.001 0.001" />
-            </geometry>
-        </collision>
-    </link>
-    <joint name="yaw_arm_joint"  type="continuous">
-        <origin xyz="0 0 0"  rpy="0 0 0" />
-        <parent link="yaw_link" />
-        <child link="yaw_base_link" />
-        <axis xyz="0 0 1" />
-    </joint>
     <link name="pitch_link">
         <inertial>
@@ -76,28 +50,8 @@
         <origin xyz="0 0 0.2841"  rpy="0 0 0" />
         <limit effort="3000" velocity="1000" lower="-0.436323" upper="0.7853982"/>
-        <parent link="yaw_base_link" />
+        <safety_controller k_velocity="10" k_position="15" soft_lower_limit="" soft_upper_limit="0.5" />
+        <parent link="yaw_link" />
         <child link="pitch_link" />
         <axis xyz="0 1 0 " />
     </joint>
-    <!-- transmission -->
-    <transmission name="trans_yaw_arm_joint">
-        <type>transmission_interface/SimpleTransmission</type>
-        <actuator name="yaw_arm_joint_motor">
-            <hardwareInterface>hardware_interface/EffortJointInterface</hardwareInterface>
-            <mechanicalReduction>1</mechanicalReduction>
-        </actuator>
-        <joint name="yaw_arm_joint">
-            <hardwareInterface>hardware_interface/EffortJointInterface</hardwareInterface>
-        </joint>
-    </transmission>
-    <transmission name="trans_pitch_joint">
-        <type>transmission_interface/SimpleTransmission</type>
-        <actuator name="pitch_joint_motor">
-            <hardwareInterface>hardware_interface/EffortJointInterface</hardwareInterface>
-            <mechanicalReduction>1</mechanicalReduction>
-        </actuator>
-        <joint name="pitch_joint">
-            <hardwareInterface>hardware_interface/EffortJointInterface</hardwareInterface>
-        </joint>
-    </transmission>
 </robot>

File: urdf/standard/chassis.urdf.xacro (robot description, xacro)
@@ -11,6 +11,6 @@
       <inertial>
         <mass value="10"/>
-        <origin xyz="-0.025857  0  0.054312"/>
-        <inertia ixx="2.247e-1" ixy="-1.139e-5" ixz="2.983e-2" iyy="3.747e-1"
+        <origin xyz="-0.025077  0  0.055047"/>
+        <inertia ixx="2.247e-1" ixy="-1.139e-5" ixz="2.983e-2" iyy="3.771e-1"
                  iyz="3.3454e-6" izz="4.803e-1"/>
       </inertial>

File: urdf/standard/gimbal.urdf.xacro (robot description, xacro)
@@ -1,4 +1,8 @@
-<robot>
-    <link name="yaw_link">
+<?xml version="1.0" encoding="utf-8"?>
+<robot xmlns:xacro="http://www.ros.org/wiki/xacro">
+    <xacro:property name="threshold" value="0.01"/>
+    <xacro:property name="lower_limit" value="-0.436323"/>
+    <xacro:property name="upper_limit" value="0.7853982"/>
+    <link name="yaw">
         <inertial>
             <mass value="0.592087"/>
@@ -10,5 +14,5 @@
             <origin xyz="0 0 0" rpy="0 0 0"/>
             <geometry>
-                <mesh filename="package://rm_description/meshes/standard/yaw_base.stl" scale="0.001 0.001 0.001"/>
+                <mesh filename="package://rm_description/meshes/standard/yaw.stl" scale="0.001 0.001 0.001" />
             </geometry>
         </visual>
@@ -16,26 +20,26 @@
             <origin xyz="0 0 0" rpy="0 0 0"/>
             <geometry>
-                <mesh filename="package://rm_description/meshes/standard/yaw_base.stl" scale="0.001 0.001 0.001"/>
+                <mesh filename="package://rm_description/meshes/standard/yaw.stl"  scale="0.001 0.001 0.001" />
             </geometry>
         </collision>
     </link>
-    <joint name="yaw_joint"  type="fixed">
-        <origin xyz="0 0 0.0466"
+    <joint name="yaw_joint"  type="continuous">
+        <origin xyz="0 0 0.0696"
                 rpy="0 0 0" />
         <parent link="base_link" />
-        <child link="yaw_link" />
+        <child link="yaw" />
         <axis xyz="0 0 1" />
     </joint>
-    <link name="yaw_base_link">
+    <link name="pitch">
         <inertial>
-            <mass value="4.17874"/>
-            <origin xyz="-0.00282 0 0.06328"/>
-            <inertia ixx="2.401e-2" ixy="-1.449e-4" ixz="7.408e-4" iyy="2.166e-2"
-                     iyz="-1.47e-4" izz="5.707e-3"/>
+            <mass value="1.538674"/>
+            <origin xyz="0.009047 -0.00307 0.019014"/>
+            <inertia ixx="1.148e-2" ixy="1.569e-3" ixz="2.374e-3" iyy="2.472e-2"
+                     iyz="-8.276e-4" izz="2.189e-2"/>
         </inertial>
         <visual>
             <origin xyz="0 0 0" rpy="0 0 0"/>
             <geometry>
-                <mesh filename="package://rm_description/meshes/standard/yaw_arm.stl" scale="0.001 0.001 0.001"/>
+                <mesh filename="package://rm_description/meshes/standard/pitch.stl" scale="0.001 0.001 0.001" />
             </geometry>
         </visual>
@@ -43,31 +47,5 @@
             <origin xyz="0 0 0" rpy="0 0 0"/>
             <geometry>
-                <mesh filename="package://rm_description/meshes/standard/yaw_arm.stl" scale="0.001 0.001 0.001"/>
-            </geometry>
-        </collision>
-    </link>
-    <joint name="yaw_arm_joint"  type="continuous">
-        <origin xyz="0 0 0.023"  rpy="0 0 0" />
-        <parent link="yaw_link" />
-        <child link="yaw_base_link" />
-        <axis xyz="0 0 1" />
-    </joint>
-    <link name="pitch_link">
-        <inertial>
-            <mass value="1.538674"/>
-            <origin xyz="0.009047 -0.00307 0.019014"/>
-            <inertia ixx="1.217e-2" ixy="1.677e-3" ixz="3.224e-3" iyy="2.570e-2"
-                     iyz="-8.223e-4" izz="2.342e-2"/>
-        </inertial>
-        <visual>
-            <origin xyz="0 0 0" rpy="0 0 0"/>
-            <geometry>
-                <mesh filename="package://rm_description/meshes/standard/pitch.stl" scale="0.001 0.001 0.001"/>
-            </geometry>
-        </visual>
-        <collision>
-            <origin xyz="0 0 0" rpy="0 0 0"/>
-            <geometry>
-                <mesh filename="package://rm_description/meshes/standard/pitch.stl" scale="0.001 0.001 0.001"/>
+                <mesh filename="package://rm_description/meshes/standard/pitch.stl"  scale="0.001 0.001 0.001" />
             </geometry>
         </collision>
@@ -75,29 +53,12 @@
     <joint name="pitch_joint"  type="revolute">
         <origin xyz="0 0 0.189"  rpy="0 0 0" />
-        <limit effort="3000" velocity="1000" lower="-0.436323" upper="0.7853982"/>
-        <parent link="yaw_base_link" />
-        <child link="pitch_link" />
+        <limit effort="3000" velocity="1000" lower="${lower_limit}" upper="${upper_limit}"/>
+        <safety_controller k_velocity="10"
+                k_position="15"
+                soft_lower_limit="${lower_limit+threshold}"
+                soft_upper_limit="${upper_limit-threshold}" />
+        <parent link="yaw" />
+        <child link="pitch" />
         <axis xyz="0 1 0 " />
     </joint>
-    <!-- transmission -->
-    <transmission name="trans_yaw_arm_joint">
-        <type>transmission_interface/SimpleTransmission</type>
-        <actuator name="yaw_arm_joint_motor">
-            <hardwareInterface>hardware_interface/EffortJointInterface</hardwareInterface>
-            <mechanicalReduction>1</mechanicalReduction>
-        </actuator>
-        <joint name="yaw_arm_joint">
-            <hardwareInterface>hardware_interface/EffortJointInterface</hardwareInterface>
-        </joint>
-    </transmission>
-    <transmission name="trans_pitch_joint">
-        <type>transmission_interface/SimpleTransmission</type>
-        <actuator name="pitch_joint_motor">
-            <hardwareInterface>hardware_interface/EffortJointInterface</hardwareInterface>
-            <mechanicalReduction>1</mechanicalReduction>
-        </actuator>
-        <joint name="pitch_joint">
-            <hardwareInterface>hardware_interface/EffortJointInterface</hardwareInterface>
-        </joint>
-    </transmission>
 </robot>

File: urdf/standard/standard.urdf.xacro (robot description, xacro)
@@ -15,4 +15,5 @@
   </xacro:if>
   <xacro:if value="$(arg load_shooter)">
+    <xacro:include filename="$(find rm_description)/urdf/standard/shooter.urdf.xacro"/>
   </xacro:if>
   <xacro:if value="$(arg load_gazebo)">

Commit message: Update gimbal.urdf.xacro and something else

File: urdf/hero/gimbal.urdf.xacro (robot description, xacro)
@@ -1,4 +1,8 @@
-<robot>
-    <link name="yaw_link">
+<?xml version="1.0" encoding="utf-8"?>
+<robot xmlns:xacro="http://www.ros.org/wiki/xacro">
+    <xacro:property name="threshold" value="0.01"/>
+    <xacro:property name="lower_limit" value="-0.436323"/>
+    <xacro:property name="upper_limit" value="0.7853982"/>
+    <link name="yaw">
         <inertial>
             <mass value="0.592087"/>
@@ -10,5 +14,5 @@
             <origin xyz="0 0 0" rpy="0 0 0"/>
             <geometry>
-                <mesh filename="package://rm_description/meshes/hero/yaw_base.stl" scale="0.001 0.001 0.001" />
+                <mesh filename="package://rm_description/meshes/hero/yaw_arm.stl" scale="0.001 0.001 0.001"/>
             </geometry>
         </visual>
@@ -16,16 +20,16 @@
             <origin xyz="0 0 0" rpy="0 0 0"/>
             <geometry>
-                <mesh filename="package://rm_description/meshes/hero/yaw_base.stl"  scale="0.001 0.001 0.001" />
+                <mesh filename="package://rm_description/meshes/hero/yaw_arm.stl" scale="0.001 0.001 0.001"/>
             </geometry>
         </collision>
     </link>
-    <joint name="yaw_joint"  type="fixed">
+    <joint name="yaw_joint" type="continuous">
         <origin xyz="0 0 0.1"
-                rpy="0 0 0" />
-        <parent link="base_link" />
-        <child link="yaw_link" />
-        <axis xyz="0 0 1" />
+                rpy="0 0 0"/>
+        <parent link="base_link"/>
+        <child link="yaw"/>
+        <axis xyz="0 0 1"/>
     </joint>
-    <link name="pitch_link">
+    <link name="pitch">
         <inertial>
             <mass value="1.538674"/>
@@ -37,5 +41,5 @@
             <origin xyz="0 0 0" rpy="0 0 0"/>
             <geometry>
-                <mesh filename="package://rm_description/meshes/hero/pitch.stl" scale="0.001 0.001 0.001" />
+                <mesh filename="package://rm_description/meshes/hero/pitch.stl" scale="0.001 0.001 0.001"/>
             </geometry>
         </visual>
@@ -43,15 +47,18 @@
             <origin xyz="0 0 0" rpy="0 0 0"/>
             <geometry>
-                <mesh filename="package://rm_description/meshes/hero/pitch.stl"  scale="0.001 0.001 0.001" />
+                <mesh filename="package://rm_description/meshes/hero/pitch.stl" scale="0.001 0.001 0.001"/>
             </geometry>
         </collision>
     </link>
-    <joint name="pitch_joint"  type="revolute">
-        <origin xyz="0 0 0.2841"  rpy="0 0 0" />
-        <limit effort="3000" velocity="1000" lower="-0.436323" upper="0.7853982"/>
-        <safety_controller k_velocity="10" k_position="15" soft_lower_limit="" soft_upper_limit="0.5" />
-        <parent link="yaw_link" />
-        <child link="pitch_link" />
-        <axis xyz="0 1 0 " />
+    <joint name="pitch_joint" type="revolute">
+        <origin xyz="0 0 0.2841" rpy="0 0 0"/>
+        <limit effort="3000" velocity="1000" lower="${lower_limit}" upper="${upper_limit}"/>
+        <safety_controller k_velocity="10"
+                           k_position="15"
+                           soft_lower_limit="${lower_limit+threshold}"
+                           soft_upper_limit="${upper_limit-threshold}"/>
+        <parent link="yaw"/>
+        <child link="pitch"/>
+        <axis xyz="0 1 0 "/>
     </joint>
 </robot>

Commit message: change pitch height

File: urdf/hero/gimbal.urdf.xacro (robot description, xacro)
@@ -54,5 +54,5 @@
     </link>
     <joint name="pitch_joint" type="revolute">
-        <origin xyz="0 0 0.360" rpy="0 0 0"/>
+        <origin xyz="0 0 0.384" rpy="0 0 0"/>
         <dynamics damping="0.0" friction="0.1"/>
         <limit effort="1.2" velocity="13.82" lower="${lower_limit}" upper="${upper_limit}"/>

Commit message: Update pitch limit

File: urdf/hero/gimbal.urdf.xacro (robot description, xacro)
@@ -2,6 +2,6 @@
 <robot xmlns:xacro="http://www.ros.org/wiki/xacro">
     <xacro:property name="threshold" value="0.01"/>
-    <xacro:property name="lower_limit" value="-0.436323"/>
-    <xacro:property name="upper_limit" value="0.7853982"/>
+    <xacro:property name="pitch_lower_limit" value="-0.4"/>
+    <xacro:property name="pitch_upper_limit" value="0.7"/>
     <link name="yaw">
         <inertial>
@@ -24,9 +24,9 @@
         </collision>
     </link>
-    <joint name="yaw_joint" type="continuous">
+    <joint name="yaw_joint" type="revolute">
         <origin xyz="0 0 0.124"
                 rpy="0 0 0"/>
         <dynamics damping="0.0" friction="0.1"/>
-        <limit effort="1.2" velocity="13.82" lower="${lower_limit}" upper="${upper_limit}"/>
+        <limit effort="1.2" velocity="13.82" lower="-1e10" upper="1e10"/>
         <parent link="base_link"/>
         <child link="yaw"/>
@@ -56,9 +56,9 @@
         <origin xyz="0 0 0.384" rpy="0 0 0"/>
         <dynamics damping="0.0" friction="0.1"/>
-        <limit effort="1.2" velocity="13.82" lower="${lower_limit}" upper="${upper_limit}"/>
+        <limit effort="1.2" velocity="13.82" lower="${pitch_lower_limit}" upper="${pitch_upper_limit}"/>
         <!--        <safety_controller k_velocity="10"-->
         <!--                           k_position="15"-->
-        <!--                           soft_lower_limit="${lower_limit+threshold}"-->
-        <!--                           soft_upper_limit="${upper_limit-threshold}"/>-->
+        <!--                           soft_lower_limit="${pitch_lower_limit+threshold}"-->
+        <!--                           soft_upper_limit="${pitch_upper_limit-threshold}"/>-->
         <parent link="yaw"/>
         <child link="pitch"/>

File: urdf/standard/gimbal.urdf.xacro (robot description, xacro)
@@ -2,6 +2,6 @@
 <robot xmlns:xacro="http://www.ros.org/wiki/xacro">
     <xacro:property name="threshold" value="0.1"/>
-    <xacro:property name="pitch_lower_limit" value="-0.482"/>
-    <xacro:property name="pitch_upper_limit" value="0.257"/>
+    <xacro:property name="pitch_lower_limit" value="-0.716"/>
+    <xacro:property name="pitch_upper_limit" value="0.487"/>
     <link name="yaw">
         <inertial>

Commit message: Update hero parameter

File: urdf/hero/gimbal.urdf.xacro (robot description, xacro)
@@ -2,6 +2,6 @@
 <robot xmlns:xacro="http://www.ros.org/wiki/xacro">
     <xacro:property name="threshold" value="0.01"/>
-    <xacro:property name="pitch_lower_limit" value="-0.4"/>
-    <xacro:property name="pitch_upper_limit" value="0.7"/>
+    <xacro:property name="pitch_lower_limit" value="-1.282"/>
+    <xacro:property name="pitch_upper_limit" value="0.405"/>
     <link name="yaw">
         <inertial>

Commit message: Delete static_transform of camera and add camera link and joint

File: urdf/hero/gimbal.urdf.xacro (robot description, xacro)
@@ -65,3 +65,29 @@
         <axis xyz="0 1 0 "/>
     </joint>
+    <link name="camera">
+        <inertial>
+            <mass value="0.17671"/>
+            <origin xyz="0.022 0.0 0.0"/>
+            <inertia ixx="2.129e-5" ixy="7.329e-8" ixz="-1.11e-7" iyy="2.198e-4" iyz="-8.04e-7" izz="2.197e-4"/>
+        </inertial>
+        <visual>
+            <origin xyz=" 0 0 0 " rpy="0 -1.57 0"/>
+            <geometry>
+                <mesh filename="package://rm_description/meshes/common/camera.stl" scale="0.001 0.001 0.001"/>
+            </geometry>
+            <material name="Black"/>
+        </visual>
+        <collision>
+            <origin xyz="0 0 0" rpy="0 -1.57 0"/>
+            <geometry>
+                <mesh filename="package://rm_description/meshes/common/camera.stl" scale="0.001 0.001 0.001"/>
+            </geometry>
+        </collision>
+    </link>
+    <joint name="camera_joint" type="fixed">
+        <parent link="pitch"/>
+        <child link="camera"/>
+        <origin xyz="0.12 0.0 -0.05" rpy="-1.57 0 -1.57"/>
+        <axis xyz="0 0 1"/>
+    </joint>
 </robot>

File: urdf/sentry/gimbal.urdf.xacro (robot description, xacro)
@@ -65,4 +65,30 @@
                          soft_upper_limit="${pitch_upper_limit-threshold}"/>
     </joint>
+    <link name="camera">
+      <inertial>
+        <mass value="0.17671"/>
+        <origin xyz="0.022 0.0 0.0"/>
+        <inertia ixx="2.129e-5" ixy="7.329e-8" ixz="-1.11e-7" iyy="2.198e-4" iyz="-8.04e-7" izz="2.197e-4"/>
+      </inertial>
+      <visual>
+        <origin xyz=" 0 0 0 " rpy="0 -1.57 0"/>
+        <geometry>
+          <mesh filename="package://rm_description/meshes/common/camera.stl" scale="0.001 0.001 0.001"/>
+        </geometry>
+        <material name="Black"/>
+      </visual>
+      <collision>
+        <origin xyz="0 0 0" rpy="0 -1.57 0"/>
+        <geometry>
+          <mesh filename="package://rm_description/meshes/common/camera.stl" scale="0.001 0.001 0.001"/>
+        </geometry>
+      </collision>
+    </link>
+    <joint name="camera_joint" type="fixed">
+      <parent link="pitch"/>
+      <child link="camera"/>
+      <origin xyz="0.086  0.0 -0.040" rpy="-1.57 0 -1.57"/>
+      <axis xyz="0 0 1"/>
+    </joint>
   </xacro:macro>
 </robot>

File: urdf/standard/gimbal.urdf.xacro (robot description, xacro)
@@ -72,5 +72,5 @@
             </inertial>
             <visual>
-                <origin xyz=" 0 0 0 " rpy="0 0 0"/>
+                <origin xyz=" 0 0 0 " rpy="0 -1.57 0"/>
                 <geometry>
                     <mesh filename="package://rm_description/meshes/common/camera.stl" scale="0.001 0.001 0.001"/>
@@ -79,5 +79,5 @@
             </visual>
             <collision>
-                <origin xyz="0.02 0.0 0.0" rpy="0 0 0"/>
+                <origin xyz="0.02 0.0 0.0" rpy="0 -1.57 0"/>
                 <geometry>
                     <mesh filename="package://rm_description/meshes/common/camera.stl" scale="0.001 0.001 0.001"/>
@@ -88,5 +88,5 @@
             <parent link="pitch"/>
             <child link="camera"/>
-            <origin xyz="0.064 0.0 -0.043" rpy="0 0 0"/>
+            <origin xyz="0.064 0.0 -0.043" rpy="-1.57 0 -1.57"/>
             <axis xyz="0 0 1"/>
         </joint>

Commit message: Update camera position in hero

File: urdf/hero/gimbal.urdf.xacro (robot description, xacro)
@@ -88,5 +88,5 @@
         <parent link="pitch"/>
         <child link="camera"/>
-        <origin xyz="0.12 0.0 -0.05" rpy="-1.57 0 -1.57"/>
+        <origin xyz="0.153 0.0 -0.052" rpy="-1.57 0 -1.57"/>
         <axis xyz="0 0 1"/>
     </joint>

Commit message: Update camera tf in hero

File: urdf/hero/gimbal.urdf.xacro (robot description, xacro)
@@ -88,5 +88,5 @@
         <parent link="pitch"/>
         <child link="camera"/>
-        <origin xyz="0.153 0.0 -0.052" rpy="-1.57 0 -1.57"/>
+        <origin xyz="0.153 0.0 -0.052" rpy="1.57 0 1.57"/>
         <axis xyz="0 0 1"/>
     </joint>

Commit message: Update hero gimbal urdf soft_limit

File: urdf/hero/gimbal.urdf.xacro (robot description, xacro)
@@ -2,6 +2,6 @@
 <robot xmlns:xacro="http://www.ros.org/wiki/xacro">
     <xacro:property name="threshold" value="0.01"/>
-    <xacro:property name="pitch_lower_limit" value="-1.282"/>
-    <xacro:property name="pitch_upper_limit" value="0.405"/>
+    <xacro:property name="pitch_lower_limit" value="-0.980"/>
+    <xacro:property name="pitch_upper_limit" value="0.198"/>
     <link name="yaw">
         <inertial>
@@ -57,8 +57,8 @@
         <dynamics damping="0.0" friction="0.1"/>
         <limit effort="1.2" velocity="13.82" lower="${pitch_lower_limit}" upper="${pitch_upper_limit}"/>
-        <!--        <safety_controller k_velocity="10"-->
-        <!--                           k_position="15"-->
-        <!--                           soft_lower_limit="${pitch_lower_limit+threshold}"-->
-        <!--                           soft_upper_limit="${pitch_upper_limit-threshold}"/>-->
+        <safety_controller k_velocity="0.1"
+                           k_position="100"
+                           soft_lower_limit="${pitch_lower_limit+threshold}"
+                           soft_upper_limit="${pitch_upper_limit-threshold}"/>
         <parent link="yaw"/>
         <child link="pitch"/>

Commit message: Update hero gimbal soft_limit and shooter parameter

File: urdf/hero/gimbal.urdf.xacro (robot description, xacro)
@@ -3,5 +3,5 @@
     <xacro:property name="threshold" value="0.01"/>
     <xacro:property name="pitch_lower_limit" value="-0.980"/>
-    <xacro:property name="pitch_upper_limit" value="0.198"/>
+    <xacro:property name="pitch_upper_limit" value="0.320"/>
     <link name="yaw">
         <inertial>

Commit message: Update parameter of hero

File: urdf/hero/gimbal.urdf.xacro (robot description, xacro)
@@ -1,7 +1,7 @@
 <?xml version="1.0" encoding="utf-8"?>
 <robot xmlns:xacro="http://www.ros.org/wiki/xacro">
-    <xacro:property name="threshold" value="0.01"/>
-    <xacro:property name="pitch_lower_limit" value="-0.980"/>
-    <xacro:property name="pitch_upper_limit" value="0.320"/>
+    <xacro:property name="threshold" value="0.1"/>
+    <xacro:property name="pitch_lower_limit" value="-1.39"/>
+    <xacro:property name="pitch_upper_limit" value="0.31"/>
     <link name="yaw">
         <inertial>
