Commit message: update hero intertial and  xyz  parameter

File: urdf/hero/gimbal.urdf.xacro (robot description, xacro)
@@ -6,8 +6,8 @@
     <link name="yaw">
         <inertial>
-            <mass value="4.367"/>
-            <origin xyz="0.042103 0.001062 0.132315"/>
-            <inertia ixx="7.943e-2" ixy="-4.889e-5" ixz="-5.618e-3" iyy="8.143e-2"
-                     iyz="-4.14e-5" izz="7.76e-3"/>
+            <mass value="3.941"/>
+            <origin xyz="-0.052 -0.057 0.152"/>
+            <inertia ixx="1.250e-1" ixy="-1.357e-2" ixz="3.487e-2" iyy="1.218e-1"
+                     iyz="3.775e-2" izz="3.242e-2"/>
         </inertial>
         <visual>
@@ -25,5 +25,5 @@
     </link>
     <joint name="yaw_joint" type="revolute">
-        <origin xyz="0 0 0.124"
+        <origin xyz="0 0 0.129"
                 rpy="0 0 0"/>
         <dynamics damping="0.0" friction="0.1"/>
@@ -35,8 +35,8 @@
     <link name="pitch">
         <inertial>
-            <mass value="1.63"/>
-            <origin xyz="0.102 -0.0 0.015"/>
-            <inertia ixx="3.980e-3" ixy="4.110e-6" ixz="-2.651e-3" iyy="2.723e-2"
-                     iyz="6.616e-6" izz=" 2.635e-2"/>
+            <mass value="1.125"/>
+            <origin xyz="0.104 0.0 0.024"/>
+            <inertia ixx="2.658e-3" ixy="4.995e-6" ixz="-3.326e-3" iyy="2.084e-2"
+                     iyz="6.020e-6" izz="1.948e-2"/>
         </inertial>
         <visual>
@@ -54,5 +54,5 @@
     </link>
     <joint name="pitch_joint" type="revolute">
-        <origin xyz="0 0 0.384" rpy="0 0 0"/>
+        <origin xyz="-0.06  0 0.191 " rpy="0 0 0"/>
         <dynamics damping="0.0" friction="0.1"/>
         <limit effort="1.2" velocity="13.82" lower="${pitch_lower_limit}" upper="${pitch_upper_limit}"/>
@@ -65,29 +65,3 @@
         <axis xyz="0 1 0 "/>
     </joint>
-    <!--    <link name="camera">-->
-    <!--        <inertial>-->
-    <!--            <mass value="0.17671"/>-->
-    <!--            <origin xyz="0.022 0.0 0.0"/>-->
-    <!--            <inertia ixx="2.129e-5" ixy="7.329e-8" ixz="-1.11e-7" iyy="2.198e-4" iyz="-8.04e-7" izz="2.197e-4"/>-->
-    <!--        </inertial>-->
-    <!--        <visual>-->
-    <!--            <origin xyz=" 0 0 0 " rpy="0 -1.57 0"/>-->
-    <!--            <geometry>-->
-    <!--                <mesh filename="package://rm_description/meshes/common/camera.stl" scale="0.001 0.001 0.001"/>-->
-    <!--            </geometry>-->
-    <!--            <material name="Black"/>-->
-    <!--        </visual>-->
-    <!--        <collision>-->
-    <!--            <origin xyz="0 0 0" rpy="0 -1.57 0"/>-->
-    <!--            <geometry>-->
-    <!--                <mesh filename="package://rm_description/meshes/common/camera.stl" scale="0.001 0.001 0.001"/>-->
-    <!--            </geometry>-->
-    <!--        </collision>-->
-    <!--    </link>-->
-    <!--    <joint name="camera_joint" type="fixed">-->
-    <!--        <parent link="pitch"/>-->
-    <!--        <child link="camera"/>-->
-    <!--        <origin xyz="0.153 0.0 -0.052" rpy="1.57 0 1.57"/>-->
-    <!--        <axis xyz="0 0 1"/>-->
-    <!--    </joint>-->
 </robot>

File: urdf/hero/hero.urdf.xacro (robot description, xacro)
@@ -14,5 +14,5 @@
     <xacro:include filename="$(find rm_description)/urdf/hero/gimbal.transmission.urdf.xacro"/>
     <xacro:include filename="$(find rm_description)/urdf/common/camera.urdf.xacro"/>
-    <xacro:camera_sensor xyz="0.127 0 -0.075" rpy="0 0 0" parent="pitch"
+    <xacro:camera_sensor xyz="0.127 0 -0.038" rpy="0 0 0" parent="pitch"
                          camera_sim="$(arg use_simulation)"/>
   </xacro:if>

File: urdf/hero/shooter.urdf.xacro (robot description, xacro)
@@ -2,6 +2,6 @@
     <xacro:include filename="$(find rm_description)/urdf/common/friction.urdf.xacro"/>
     <xacro:include filename="$(find rm_description)/urdf/standard/gimbal.urdf.xacro"/>
-    <xacro:property name="wheel_offset_x" value="0.00884"/>
-    <xacro:property name="wheel_offset_y" value="0.036564"/>
+    <xacro:property name="wheel_offset_x" value="0.084"/>
+    <xacro:property name="wheel_offset_y" value="0.049"/>
     <xacro:property name="wheel_offset_z" value="0.0"/>
     <xacro:friction_wheel prefixs="left" connected_to="pitch"

Commit message: Update parameter

File: urdf/hero/gimbal.urdf.xacro (robot description, xacro)
@@ -1,5 +1,5 @@
 <?xml version="1.0" encoding="utf-8"?>
 <robot xmlns:xacro="http://www.ros.org/wiki/xacro">
-    <xacro:property name="threshold" value="0.1"/>
+    <xacro:property name="threshold" value="0.05"/>
     <xacro:property name="pitch_lower_limit" value="-1.39"/>
     <xacro:property name="pitch_upper_limit" value="0.31"/>

Commit message: Update hero pitch limit

File: urdf/hero/gimbal.urdf.xacro (robot description, xacro)
@@ -3,5 +3,5 @@
     <xacro:property name="threshold" value="0.05"/>
     <xacro:property name="pitch_lower_limit" value="-1.39"/>
-    <xacro:property name="pitch_upper_limit" value="0.31"/>
+    <xacro:property name="pitch_upper_limit" value="0.35"/>
     <link name="yaw">
         <inertial>
@@ -14,5 +14,5 @@
             <origin xyz="0 0 0" rpy="0 0 0"/>
             <geometry>
-                <mesh filename="package://rm_description/meshes/hero/yaw.stl" scale="0.001 0.001 0.001" />
+                <mesh filename="package://rm_description/meshes/hero/yaw.stl" scale="0.001 0.001 0.001"/>
             </geometry>
         </visual>
@@ -20,5 +20,5 @@
             <origin xyz="0 0 0" rpy="0 0 0"/>
             <geometry>
-                <mesh filename="package://rm_description/meshes/hero/yaw.stl"  scale="0.001 0.001 0.001" />
+                <mesh filename="package://rm_description/meshes/hero/yaw.stl" scale="0.001 0.001 0.001"/>
             </geometry>
         </collision>
@@ -43,5 +43,5 @@
             <origin xyz="0 0 0" rpy="0 0 0"/>
             <geometry>
-                <mesh filename="package://rm_description/meshes/hero/pitch.stl" scale="0.001 0.001 0.001" />
+                <mesh filename="package://rm_description/meshes/hero/pitch.stl" scale="0.001 0.001 0.001"/>
             </geometry>
         </visual>

Commit message: Update gimbal limit

File: urdf/hero/gimbal.urdf.xacro (robot description, xacro)
@@ -2,6 +2,6 @@
 <robot xmlns:xacro="http://www.ros.org/wiki/xacro">
     <xacro:property name="threshold" value="0.05"/>
-    <xacro:property name="pitch_lower_limit" value="-1.39"/>
-    <xacro:property name="pitch_upper_limit" value="0.35"/>
+    <xacro:property name="pitch_lower_limit" value="-1.4"/>
+    <xacro:property name="pitch_upper_limit" value="0.4"/>
     <link name="yaw">
         <inertial>

File: urdf/standard/gimbal.urdf.xacro (robot description, xacro)
@@ -3,5 +3,5 @@
     <xacro:property name="threshold" value="0.1"/>
     <xacro:property name="pitch_lower_limit" value="-0.7"/>
-    <xacro:property name="pitch_upper_limit" value="0.4"/>
+    <xacro:property name="pitch_upper_limit" value="0.45"/>
         <link name="yaw">
             <inertial>
