Commit message: rmua_description stl commit

File: urdf/rmua/chassis.urdf.xacro (robot description, xacro)
@@ -2,4 +2,5 @@
     <xacro:include filename="$(find rm_description)/urdf/common/mecanum_wheel.urdf.xacro"/>
     <!-- https://upload.wikimedia.org/wikipedia/commons/5/52/Wheelbase_and_Track.png -->
+    <xacro:property name="wheel_offset_z" value="0.0269"/>
     <xacro:macro name="chassis" params="roller_type">
         <link name="base_link">
@@ -25,17 +26,17 @@
         <xacro:mecanum_wheel prefix="left_front" connected_to="base_link"
                              wheel_x_offset="-0.2165" wheel_y_offset="0.1990"
-                             wheel_z_offset="0.0269"
+                             wheel_z_offset="${wheel_offset_z}"
                              reflect="1" roller_type="${roller_type}"/>
         <xacro:mecanum_wheel prefix="right_front" connected_to="base_link"
                              wheel_x_offset="0.2165" wheel_y_offset="0.1990"
-                             wheel_z_offset="0.0269"
+                             wheel_z_offset="${wheel_offset_z}"
                              reflect="-1" roller_type="${roller_type}"/>
         <xacro:mecanum_wheel prefix="left_back" connected_to="base_link"
                              wheel_x_offset="-0.1601" wheel_y_offset="-0.1986"
-                             wheel_z_offset="0.0265"
+                             wheel_z_offset="${wheel_offset_z}"
                              reflect="-1" roller_type="${roller_type}"/>
         <xacro:mecanum_wheel prefix="right_back" connected_to="base_link"
                              wheel_x_offset="0.1601" wheel_y_offset="-0.1986"
-                             wheel_z_offset="0.0265"
+                             wheel_z_offset="${wheel_offset_z}"
                              reflect="1" roller_type="${roller_type}"/>
         <xacro:wheel_transmission prefix="left_front" mechanical_reduction="19.2032"/>

Commit message: rmua_description hassis urdf commit

File: urdf/rmua/chassis.urdf.xacro (robot description, xacro)
@@ -2,12 +2,12 @@
     <xacro:include filename="$(find rm_description)/urdf/common/mecanum_wheel.urdf.xacro"/>
     <!-- https://upload.wikimedia.org/wikipedia/commons/5/52/Wheelbase_and_Track.png -->
-    <xacro:property name="wheel_offset_z" value="0.0269"/>
+    <xacro:property name="wheel_offset_z" value="-0.0269"/>
     <xacro:macro name="chassis" params="roller_type">
         <link name="base_link">
             <inertial>
                 <mass value="13.80"/>
-                <origin xyz="0.0309 0.0007  0.0219"/>
-                <inertia ixx="5.443e-4" ixy="3.212e-6" ixz="3.283e-6" iyy="3.205e-4"
-                         iyz="1.262e-5" izz="7.634e-4"/>
+                <origin xyz="0.031 -0.0007  0.0219"/>
+                <inertia ixx="3.205e-1" ixy="-3.253e-3" ixz="8.127e-4" iyy="4.709e-1"
+                         iyz="3.283e-3" izz="6.980e-1"/>
             </inertial>
             <visual>
@@ -25,17 +25,17 @@
         </link>
         <xacro:mecanum_wheel prefix="left_front" connected_to="base_link"
-                             wheel_x_offset="-0.2165" wheel_y_offset="0.1990"
+                             wheel_x_offset="0.2165" wheel_y_offset="0.1990"
                              wheel_z_offset="${wheel_offset_z}"
                              reflect="1" roller_type="${roller_type}"/>
         <xacro:mecanum_wheel prefix="right_front" connected_to="base_link"
-                             wheel_x_offset="0.2165" wheel_y_offset="0.1990"
+                             wheel_x_offset="0.2165" wheel_y_offset="-0.1990"
                              wheel_z_offset="${wheel_offset_z}"
                              reflect="-1" roller_type="${roller_type}"/>
         <xacro:mecanum_wheel prefix="left_back" connected_to="base_link"
-                             wheel_x_offset="-0.1601" wheel_y_offset="-0.1986"
+                             wheel_x_offset="-0.1601" wheel_y_offset="0.1990"
                              wheel_z_offset="${wheel_offset_z}"
                              reflect="-1" roller_type="${roller_type}"/>
         <xacro:mecanum_wheel prefix="right_back" connected_to="base_link"
-                             wheel_x_offset="0.1601" wheel_y_offset="-0.1986"
+                             wheel_x_offset="-0.1601" wheel_y_offset="-0.1990"
                              wheel_z_offset="${wheel_offset_z}"
                              reflect="1" roller_type="${roller_type}"/>

File: urdf/rmua/rmua.urdf.xacro (robot description, xacro)
@@ -1,4 +1,4 @@
 <?xml version="1.0"?>
-<robot xmlns:xacro="http://www.ros.org/wiki/xacro" name="standard3">
+<robot xmlns:xacro="http://www.ros.org/wiki/xacro" name="rmua">
     <xacro:arg name="load_chassis" default="true"/>
     <xacro:arg name="load_gimbal" default="true"/>

Commit message: rmua_description chassis'collission urdf commit

File: urdf/rmua/chassis.urdf.xacro (robot description, xacro)
@@ -20,5 +20,5 @@
                 <origin xyz="0 0 0" rpy="0 0 0"/>
                 <geometry>
-                    <box size="0.580 0.500 0.050"/>
+                    <mesh filename="package://rm_description/meshes/rmua/base.stl" scale="0.001 0.001 0.001"/>
                 </geometry>
             </collision>

File: urdf/rmua/rmua.urdf.xacro (robot description, xacro)
@@ -9,16 +9,13 @@
         <xacro:include filename="$(find rm_description)/urdf/rmua/chassis.urdf.xacro"/>
         <xacro:chassis roller_type="$(arg roller_type)"/>
-        <xacro:include filename="$(find rm_description)/urdf/common/imu.urdf.xacro"/>
-        <xacro:IMU connected_to="base_link" imu_name="base_imu" simulation="true"
-                   xyz="0.0 -0.165 0.0" rpy="0 0 ${pi}"/>
     </xacro:if>
     <xacro:if value="$(arg load_gimbal)">
         <xacro:include filename="$(find rm_description)/urdf/rmua/gimbal.urdf.xacro"/>
         <xacro:include filename="$(find rm_description)/urdf/rmua/gimbal.transmission.urdf.xacro"/>
-        <xacro:include filename="$(find rm_description)/urdf/common/camera.urdf.xacro"/>
-        <xacro:camera_sensor xyz="0.127 0 -0.038" rpy="0 0 0" parent="pitch"
-                             camera_sim="$(arg use_simulation)"/>
-        <xacro:camera_optical_frame xyz="0.153 0 -0.0525" rpy="${pi/2} 0 ${pi/2}" parent="pitch"
-                                    camera_sim="$(arg use_simulation)"/>
+<!--        <xacro:include filename="$(find rm_description)/urdf/common/camera.urdf.xacro"/>-->
+<!--        <xacro:camera_sensor xyz="0.127 0 -0.038" rpy="0 0 0" parent="pitch"-->
+<!--                             camera_sim="$(arg use_simulation)"/>-->
+<!--        <xacro:camera_optical_frame xyz="0.153 0 -0.0525" rpy="${pi/2} 0 ${pi/2}" parent="pitch"-->
+<!--                                    camera_sim="$(arg use_simulation)"/>-->
     </xacro:if>
     <xacro:if value="$(arg load_shooter)">

Commit message: rmua_description rmua urdf commit

File: urdf/rmua/chassis.urdf.xacro (robot description, xacro)
@@ -2,5 +2,5 @@
     <xacro:include filename="$(find rm_description)/urdf/common/mecanum_wheel.urdf.xacro"/>
     <!-- https://upload.wikimedia.org/wikipedia/commons/5/52/Wheelbase_and_Track.png -->
-    <xacro:property name="wheel_offset_z" value="-0.0269"/>
+    <xacro:property name="wheel_offset_z" value="-0.0266"/>
     <xacro:macro name="chassis" params="roller_type">
         <link name="base_link">
@@ -25,17 +25,17 @@
         </link>
         <xacro:mecanum_wheel prefix="left_front" connected_to="base_link"
-                             wheel_x_offset="0.2165" wheel_y_offset="0.1990"
+                             wheel_x_offset="0.172" wheel_y_offset="0.199"
                              wheel_z_offset="${wheel_offset_z}"
                              reflect="1" roller_type="${roller_type}"/>
         <xacro:mecanum_wheel prefix="right_front" connected_to="base_link"
-                             wheel_x_offset="0.2165" wheel_y_offset="-0.1990"
+                             wheel_x_offset="0.172" wheel_y_offset="-0.199"
                              wheel_z_offset="${wheel_offset_z}"
                              reflect="-1" roller_type="${roller_type}"/>
         <xacro:mecanum_wheel prefix="left_back" connected_to="base_link"
-                             wheel_x_offset="-0.1601" wheel_y_offset="0.1990"
+                             wheel_x_offset="-0.205" wheel_y_offset="0.1990"
                              wheel_z_offset="${wheel_offset_z}"
                              reflect="-1" roller_type="${roller_type}"/>
         <xacro:mecanum_wheel prefix="right_back" connected_to="base_link"
-                             wheel_x_offset="-0.1601" wheel_y_offset="-0.1990"
+                             wheel_x_offset="-0.205" wheel_y_offset="-0.1990"
                              wheel_z_offset="${wheel_offset_z}"
                              reflect="1" roller_type="${roller_type}"/>
