Commit message: fix error of yaw position

File: urdf/rmua/gimbal.urdf.xacro (robot description, xacro)
@@ -25,5 +25,5 @@
     </link>
     <joint name="yaw_joint" type="revolute">
-        <origin xyz="0 0 89.5e-3"
+        <origin xyz="44.5e-3 0 89.5e-3"
                 rpy="0 0 0"/>
         <dynamics damping="0.0" friction="0.1"/>

Commit message: rmua_description rmua gimbal urdf commit

File: urdf/rmua/gimbal.urdf.xacro (robot description, xacro)
@@ -25,5 +25,5 @@
     </link>
     <joint name="yaw_joint" type="revolute">
-        <origin xyz="44.5e-3 0 89.5e-3"
+        <origin xyz="0 0 89.5e-3"
                 rpy="0 0 0"/>
         <dynamics damping="0.0" friction="0.1"/>
