Commit message: Add multiple cycle encoder support to cheetah

File: test/test_motor.xacro (robot description, xacro)
@@ -13,8 +13,11 @@
     <origin xyz="0 0 0.25"/>
   </joint>
-  <joint name="joint_mit_cheetah" type="continuous">
+  <joint name="joint_mit_cheetah" type="revolute">
+    <axis xyz="0 1 0"/>
+    <origin xyz="0.250 0 0"/>
+    <limit effort="30" velocity="10" lower="-2.268" upper="2.268"/>
+    <dynamics damping="0.0" friction="0.5"/>
     <parent link="link_mit_cheetah"/>
     <child link="link_end"/>
-    <origin xyz="0 0 0.25"/>
   </joint>
   <transmission name="joint_3508_trans">
@@ -32,7 +35,8 @@
     <joint name="joint_mit_cheetah">
       <hardwareInterface>hardware_interface/EffortJointInterface</hardwareInterface>
+      <offset>1.759</offset>
     </joint>
     <actuator name="act_mit_cheetah">
-      <mechanicalReduction>1</mechanicalReduction>
+      <mechanicalReduction>-3</mechanicalReduction>
       <hardwareInterface>hardware_interface/EffortJointInterface</hardwareInterface>
     </actuator>

Commit message: add GripperActionController

File: test/test_motor.xacro (robot description, xacro)
@@ -2,6 +2,8 @@
   <link name="world"/>
   <link name="link_3508"/>
-  <link name="link_mit_cheetah"/>
-  <link name="link_end"/>
+  <link name="link_mit_cheetah0"/>
+  <link name="link_mit_cheetah1"/>
+  <link name="link_mit_cheetah2"/>
+<!--  <link name="link_end"/>-->
   <joint name="fixed" type="fixed">
     <parent link="world"/>
@@ -10,15 +12,31 @@
   <joint name="joint_3508" type="continuous">
     <parent link="link_3508"/>
-    <child link="link_mit_cheetah"/>
+    <child link="link_mit_cheetah0"/>
     <origin xyz="0 0 0.25"/>
   </joint>
-  <joint name="joint_mit_cheetah" type="revolute">
+  <joint name="joint_mit_cheetah0" type="revolute">
     <axis xyz="0 1 0"/>
     <origin xyz="0.250 0 0"/>
     <limit effort="30" velocity="10" lower="-2.268" upper="2.268"/>
     <dynamics damping="0.0" friction="0.5"/>
-    <parent link="link_mit_cheetah"/>
-    <child link="link_end"/>
+    <parent link="link_mit_cheetah0"/>
+    <child link="link_mit_cheetah1"/>
   </joint>
+  <joint name="joint_mit_cheetah1" type="revolute">
+    <axis xyz="0 1 0"/>
+    <origin xyz="0.250 0 0"/>
+    <limit effort="30" velocity="10" lower="-2.268" upper="2.268"/>
+    <dynamics damping="0.0" friction="0.5"/>
+    <parent link="link_mit_cheetah1"/>
+    <child link="link_mit_cheetah2"/>
+  </joint>
+<!--  <joint name="joint_mit_cheetah2" type="revolute">-->
+<!--    <axis xyz="0 1 0"/>-->
+<!--    <origin xyz="0.250 0 0"/>-->
+<!--    <limit effort="30" velocity="10" lower="-2.268" upper="2.268"/>-->
+<!--    <dynamics damping="0.0" friction="0.5"/>-->
+<!--    <parent link="link_mit_cheetah2"/>-->
+<!--    <child link="link_end"/>-->
+<!--  </joint>-->
   <transmission name="joint_3508_trans">
     <type>transmission_interface/SimpleTransmission</type>
@@ -27,18 +45,55 @@
     </joint>
     <actuator name="act_3508">
-      <mechanicalReduction>1</mechanicalReduction>
+      <mechanicalReduction>4712.25</mechanicalReduction>
       <hardwareInterface>hardware_interface/EffortJointInterface</hardwareInterface>
     </actuator>
   </transmission>
-  <transmission name="joint_mit_cheetah_trans">
+  <transmission name="joint_mit_cheetah_trans0">
     <type>transmission_interface/SimpleTransmission</type>
-    <joint name="joint_mit_cheetah">
+    <joint name="joint_mit_cheetah0">
       <hardwareInterface>hardware_interface/EffortJointInterface</hardwareInterface>
-      <offset>0</offset>
+      <offset>1.759</offset>
     </joint>
-    <actuator name="act_mit_cheetah">
-      <mechanicalReduction>0.1666</mechanicalReduction>
+    <actuator name="act_mit_cheetah0">
+      <mechanicalReduction>-3</mechanicalReduction>
       <hardwareInterface>hardware_interface/EffortJointInterface</hardwareInterface>
     </actuator>
   </transmission>
+  <transmission name="joint_mit_cheetah_trans1">
+    <type>transmission_interface/SimpleTransmission</type>
+    <joint name="joint_mit_cheetah1">
+      <hardwareInterface>hardware_interface/EffortJointInterface</hardwareInterface>
+      <offset>1.759</offset>
+    </joint>
+    <actuator name="act_mit_cheetah1">
+      <mechanicalReduction>-3</mechanicalReduction>
+      <hardwareInterface>hardware_interface/EffortJointInterface</hardwareInterface>
+    </actuator>
+  </transmission>
+<!--  <transmission name="joint_mit_cheetah_trans2">-->
+<!--    <type>transmission_interface/SimpleTransmission</type>-->
+<!--    <joint name="joint_mit_cheetah2">-->
+<!--      <hardwareInterface>hardware_interface/EffortJointInterface</hardwareInterface>-->
+<!--      <offset>1.759</offset>-->
+<!--    </joint>-->
+<!--    <actuator name="act_mit_cheetah2">-->
+<!--      <mechanicalReduction>-3</mechanicalReduction>-->
+<!--      <hardwareInterface>hardware_interface/EffortJointInterface</hardwareInterface>-->
+<!--    </actuator>-->
+<!--  </transmission>-->
+  <!--  <transmission name="joint_mit_cheetah_trans1">-->
+<!--    <type>transmission_interface/DoubleActuatorTransmission</type>-->
+<!--    <joint name="joint_mit_cheetah1">-->
+<!--      <hardwareInterface>hardware_interface/EffortJointInterface</hardwareInterface>-->
+<!--      <offset>0</offset>-->
+<!--    </joint>-->
+<!--    <actuator name="act_mit_cheetah2_1">-->
+<!--      <role>actuator1</role>-->
+<!--      <mechanicalReduction>-3</mechanicalReduction>-->
+<!--    </actuator>-->
+<!--    <actuator name="act_mit_cheetah2_2">-->
+<!--      <role>actuator2</role>-->
+<!--      <mechanicalReduction>-3</mechanicalReduction>-->
+<!--    </actuator>-->
+<!--  </transmission>-->
 </robot>

Commit message: add GripperActionController

File: test/test_motor.xacro (robot description, xacro)
@@ -2,6 +2,8 @@
   <link name="world"/>
   <link name="link_3508"/>
-  <link name="link_mit_cheetah"/>
-  <link name="link_end"/>
+  <link name="link_mit_cheetah0"/>
+  <link name="link_mit_cheetah1"/>
+  <link name="link_mit_cheetah2"/>
+<!--  <link name="link_end"/>-->
   <joint name="fixed" type="fixed">
     <parent link="world"/>
@@ -10,14 +12,22 @@
   <joint name="joint_3508" type="continuous">
     <parent link="link_3508"/>
-    <child link="link_mit_cheetah"/>
+    <child link="link_mit_cheetah0"/>
     <origin xyz="0 0 0.25"/>
   </joint>
-  <joint name="joint_mit_cheetah" type="revolute">
+  <joint name="joint_mit_cheetah0" type="revolute">
     <axis xyz="0 1 0"/>
     <origin xyz="0.250 0 0"/>
     <limit effort="30" velocity="10" lower="-2.268" upper="2.268"/>
     <dynamics damping="0.0" friction="0.5"/>
-    <parent link="link_mit_cheetah"/>
-    <child link="link_end"/>
+    <parent link="link_mit_cheetah0"/>
+    <child link="link_mit_cheetah1"/>
+  </joint>
+  <joint name="joint_mit_cheetah1" type="revolute">
+    <axis xyz="0 1 0"/>
+    <origin xyz="0.250 0 0"/>
+    <limit effort="30" velocity="10" lower="-2.268" upper="2.268"/>
+    <dynamics damping="0.0" friction="0.5"/>
+    <parent link="link_mit_cheetah1"/>
+    <child link="link_mit_cheetah2"/>
   </joint>
   <transmission name="joint_3508_trans">
@@ -31,14 +41,29 @@
     </actuator>
   </transmission>
-  <transmission name="joint_mit_cheetah_trans">
+  <transmission name="joint_mit_cheetah_trans0">
     <type>transmission_interface/SimpleTransmission</type>
-    <joint name="joint_mit_cheetah">
+    <joint name="joint_mit_cheetah0">
       <hardwareInterface>hardware_interface/EffortJointInterface</hardwareInterface>
       <offset>1.759</offset>
     </joint>
-    <actuator name="act_mit_cheetah">
+    <actuator name="act_mit_cheetah0">
       <mechanicalReduction>-3</mechanicalReduction>
       <hardwareInterface>hardware_interface/EffortJointInterface</hardwareInterface>
     </actuator>
   </transmission>
+  <transmission name="joint_mit_cheetah_trans1">
+    <type>transmission_interface/DoubleActuatorTransmission</type>
+    <joint name="joint_mit_cheetah1">
+      <hardwareInterface>hardware_interface/EffortJointInterface</hardwareInterface>
+      <offset>0</offset>
+    </joint>
+    <actuator name="act_mit_cheetah2_1">
+      <role>actuator1</role>
+      <mechanicalReduction>-3</mechanicalReduction>
+    </actuator>
+    <actuator name="act_mit_cheetah2_2">
+      <role>actuator2</role>
+      <mechanicalReduction>-3</mechanicalReduction>
+    </actuator>
+  </transmission>
 </robot>

Commit message: test motor

File: test/test_motor.xacro (robot description, xacro)
@@ -31,12 +31,4 @@
     <child link="link_mit_cheetah2"/>
   </joint>
-<!--  <joint name="joint_mit_cheetah2" type="revolute">-->
-<!--    <axis xyz="0 1 0"/>-->
-<!--    <origin xyz="0.250 0 0"/>-->
-<!--    <limit effort="30" velocity="10" lower="-2.268" upper="2.268"/>-->
-<!--    <dynamics damping="0.0" friction="0.5"/>-->
-<!--    <parent link="link_mit_cheetah2"/>-->
-<!--    <child link="link_end"/>-->
-<!--  </joint>-->
   <transmission name="joint_3508_trans">
     <type>transmission_interface/SimpleTransmission</type>
@@ -45,5 +37,5 @@
     </joint>
     <actuator name="act_3508">
-      <mechanicalReduction>4712.25</mechanicalReduction>
+      <mechanicalReduction>1</mechanicalReduction>
       <hardwareInterface>hardware_interface/EffortJointInterface</hardwareInterface>
     </actuator>
@@ -61,39 +53,17 @@
   </transmission>
   <transmission name="joint_mit_cheetah_trans1">
-    <type>transmission_interface/SimpleTransmission</type>
+    <type>transmission_interface/DoubleActuatorTransmission</type>
     <joint name="joint_mit_cheetah1">
       <hardwareInterface>hardware_interface/EffortJointInterface</hardwareInterface>
-      <offset>1.759</offset>
+      <offset>0</offset>
     </joint>
-    <actuator name="act_mit_cheetah1">
+    <actuator name="act_mit_cheetah2_1">
+      <role>actuator1</role>
       <mechanicalReduction>-3</mechanicalReduction>
-      <hardwareInterface>hardware_interface/EffortJointInterface</hardwareInterface>
+    </actuator>
+    <actuator name="act_mit_cheetah2_2">
+      <role>actuator2</role>
+      <mechanicalReduction>-3</mechanicalReduction>
     </actuator>
   </transmission>
-<!--  <transmission name="joint_mit_cheetah_trans2">-->
-<!--    <type>transmission_interface/SimpleTransmission</type>-->
-<!--    <joint name="joint_mit_cheetah2">-->
-<!--      <hardwareInterface>hardware_interface/EffortJointInterface</hardwareInterface>-->
-<!--      <offset>1.759</offset>-->
-<!--    </joint>-->
-<!--    <actuator name="act_mit_cheetah2">-->
-<!--      <mechanicalReduction>-3</mechanicalReduction>-->
-<!--      <hardwareInterface>hardware_interface/EffortJointInterface</hardwareInterface>-->
-<!--    </actuator>-->
-<!--  </transmission>-->
-  <!--  <transmission name="joint_mit_cheetah_trans1">-->
-<!--    <type>transmission_interface/DoubleActuatorTransmission</type>-->
-<!--    <joint name="joint_mit_cheetah1">-->
-<!--      <hardwareInterface>hardware_interface/EffortJointInterface</hardwareInterface>-->
-<!--      <offset>0</offset>-->
-<!--    </joint>-->
-<!--    <actuator name="act_mit_cheetah2_1">-->
-<!--      <role>actuator1</role>-->
-<!--      <mechanicalReduction>-3</mechanicalReduction>-->
-<!--    </actuator>-->
-<!--    <actuator name="act_mit_cheetah2_2">-->
-<!--      <role>actuator2</role>-->
-<!--      <mechanicalReduction>-3</mechanicalReduction>-->
-<!--    </actuator>-->
-<!--  </transmission>-->
 </robot>

Commit message: one motor test

File: test/test_motor.xacro (robot description, xacro)
@@ -1,69 +1,21 @@
-<robot name="test_robot">
-  <link name="world"/>
+<?xml version="1.0" encoding="utf-8"?>
+<robot xmlns:xacro="http://www.ros.org/wiki/xacro" name="test">
   <link name="link_3508"/>
   <link name="link_mit_cheetah0"/>
-  <link name="link_mit_cheetah1"/>
-  <link name="link_mit_cheetah2"/>
-<!--  <link name="link_end"/>-->
-  <joint name="fixed" type="fixed">
-    <parent link="world"/>
-    <child link="link_3508"/>
-  </joint>
-  <joint name="joint_3508" type="continuous">
+  <joint name="joint_3508" type="prismatic">
     <parent link="link_3508"/>
     <child link="link_mit_cheetah0"/>
+    <limit effort="1.2" velocity="13.82" lower="-1e10" upper="1e10"/>
     <origin xyz="0 0 0.25"/>
-  </joint>
-  <joint name="joint_mit_cheetah0" type="revolute">
-    <axis xyz="0 1 0"/>
-    <origin xyz="0.250 0 0"/>
-    <limit effort="30" velocity="10" lower="-2.268" upper="2.268"/>
-    <dynamics damping="0.0" friction="0.5"/>
-    <parent link="link_mit_cheetah0"/>
-    <child link="link_mit_cheetah1"/>
-  </joint>
-  <joint name="joint_mit_cheetah1" type="revolute">
-    <axis xyz="0 1 0"/>
-    <origin xyz="0.250 0 0"/>
-    <limit effort="30" velocity="10" lower="-2.268" upper="2.268"/>
-    <dynamics damping="0.0" friction="0.5"/>
-    <parent link="link_mit_cheetah1"/>
-    <child link="link_mit_cheetah2"/>
   </joint>
   <transmission name="joint_3508_trans">
     <type>transmission_interface/SimpleTransmission</type>
+    <actuator name="act_3508">
+      <mechanicalReduction>72.1</mechanicalReduction>
+    </actuator>
     <joint name="joint_3508">
       <hardwareInterface>hardware_interface/EffortJointInterface</hardwareInterface>
+      <offset>-0.004</offset>
     </joint>
-    <actuator name="act_3508">
-      <mechanicalReduction>1</mechanicalReduction>
-      <hardwareInterface>hardware_interface/EffortJointInterface</hardwareInterface>
-    </actuator>
-  </transmission>
-  <transmission name="joint_mit_cheetah_trans0">
-    <type>transmission_interface/SimpleTransmission</type>
-    <joint name="joint_mit_cheetah0">
-      <hardwareInterface>hardware_interface/EffortJointInterface</hardwareInterface>
-      <offset>1.759</offset>
-    </joint>
-    <actuator name="act_mit_cheetah0">
-      <mechanicalReduction>-3</mechanicalReduction>
-      <hardwareInterface>hardware_interface/EffortJointInterface</hardwareInterface>
-    </actuator>
-  </transmission>
-  <transmission name="joint_mit_cheetah_trans1">
-    <type>transmission_interface/DoubleActuatorTransmission</type>
-    <joint name="joint_mit_cheetah1">
-      <hardwareInterface>hardware_interface/EffortJointInterface</hardwareInterface>
-      <offset>0</offset>
-    </joint>
-    <actuator name="act_mit_cheetah2_1">
-      <role>actuator1</role>
-      <mechanicalReduction>-3</mechanicalReduction>
-    </actuator>
-    <actuator name="act_mit_cheetah2_2">
-      <role>actuator2</role>
-      <mechanicalReduction>-3</mechanicalReduction>
-    </actuator>
   </transmission>
 </robot>

Commit message: update chassis platform

File: test/test_motor.xacro (robot description, xacro)
@@ -6,5 +6,5 @@
     <parent link="link_3508"/>
     <child link="link_mit_cheetah0"/>
-    <limit effort="1.2" velocity="13.82" lower="-1e10" upper="1e10"/>
+    <limit effort="70" velocity="13.82" lower="-1e10" upper="1e10"/>
     <origin xyz="0 0 0.25"/>
   </joint>

Commit message: Update test files

File: test/test_motor.xacro (robot description, xacro)
@@ -1,21 +1,21 @@
 <?xml version="1.0" encoding="utf-8"?>
-<robot xmlns:xacro="http://www.ros.org/wiki/xacro" name="test">
-  <link name="link_3508"/>
-  <link name="link_mit_cheetah0"/>
-  <joint name="joint_3508" type="prismatic">
-    <parent link="link_3508"/>
-    <child link="link_mit_cheetah0"/>
-    <limit effort="70" velocity="13.82" lower="-1e10" upper="1e10"/>
-    <origin xyz="0 0 0.25"/>
-  </joint>
-  <transmission name="joint_3508_trans">
-    <type>transmission_interface/SimpleTransmission</type>
-    <actuator name="act_3508">
-      <mechanicalReduction>72.1</mechanicalReduction>
-    </actuator>
-    <joint name="joint_3508">
-      <hardwareInterface>hardware_interface/EffortJointInterface</hardwareInterface>
-      <offset>-0.004</offset>
+<robot name="test">
+    <link name="base_link"/>
+    <link name="mit_link"/>
+    <joint name="mit_joint" type="revolute">
+        <parent link="base_link"/>
+        <child link="mit_link"/>
+        <limit effort="30" velocity="50" lower="-1e10" upper="1e10"/>
+        <origin xyz="0 0 0.25"/>
     </joint>
-  </transmission>
+    <transmission name="mit_joint_trans">
+        <type>transmission_interface/SimpleTransmission</type>
+        <actuator name="mit_joint_motor">
+            <mechanicalReduction>1.0</mechanicalReduction>
+        </actuator>
+        <joint name="mit_joint">
+            <hardwareInterface>hardware_interface/EffortJointInterface</hardwareInterface>
+            <offset>-0.004</offset>
+        </joint>
+    </transmission>
 </robot>
