Commit message: Add TODO

File: urdf/engineer/arm.urdf.xacro (robot description, xacro)
@@ -37,7 +37,5 @@
       <collision>
         <origin xyz="0 0 0" rpy="0 0 0"/>
-        <geometry>
-          <mesh filename="package://rm_description/meshes/engineer/link1_collision.stl" scale="0.001 0.001 0.001"/>
-        </geometry>
+        <!--TODO: add collision-->
       </collision>
     </link>

Commit message: Change wrong value

File: urdf/engineer/arm.urdf.xacro (robot description, xacro)
@@ -76,5 +76,5 @@
         <origin xyz="0.100 0 0"/>
         <geometry>
-          <box size="0.248.78 0.089 0.0895"/>
+          <box size="0.2488 0.089 0.0895"/>
         </geometry>
       </collision>

Commit message: Set limit

File: urdf/engineer/arm.urdf.xacro (robot description, xacro)
@@ -36,6 +36,8 @@
       </visual>
       <collision>
-        <origin xyz="0 0 0" rpy="0 0 0"/>
-        <!--TODO: add collision-->
+        <origin xyz="-0.02 0 0.05" rpy="0 0 0"/>
+        <geometry>
+          <box size="0.200 0.182 0.100"/>
+        </geometry>
       </collision>
     </link>
@@ -74,7 +76,7 @@
       </visual>
       <collision>
-        <origin xyz="0.100 0 0"/>
+        <origin xyz="0.090 0 0"/>
         <geometry>
-          <box size="0.2488 0.089 0.0895"/>
+          <box size="0.245 0.089 0.0895"/>
         </geometry>
       </collision>
@@ -125,5 +127,5 @@
       <origin xyz="0 0 0.019"/>
       <!--      limit not work while type="continuous"-->
-      <limit effort="20" velocity="999" lower="-1e16" upper="1e16"/>
+      <limit effort="20" velocity="25" lower="-${3*pi}" upper="${3*pi}"/>
       <dynamics damping="0.0" friction="0.1"/>
       <parent link="link0"/>
@@ -133,5 +135,5 @@
       <axis xyz="0 1 0"/>
       <origin xyz="0.11341 0 0.1380"/>
-      <limit effort="60" velocity="10" lower="-1e16" upper="1e16"/>
+      <limit effort="60" velocity="10" lower="-${pi}" upper="${0.44*pi}"/>
       <dynamics damping="0.0" friction="0.2"/>
       <parent link="link1"/>
@@ -141,5 +143,5 @@
       <axis xyz="0 1 0"/>
       <origin xyz="0.250 0 0"/>
-      <limit effort="30" velocity="10" lower="-1e16" upper="1e16"/>
+      <limit effort="30" velocity="10" lower="-${0.722*pi}" upper="${0.722*pi}"/>
       <dynamics damping="0.0" friction="0.1"/>
       <parent link="link2"/>
@@ -149,5 +151,5 @@
       <axis xyz="0 1 0"/>
       <origin xyz="0.180 0 0"/>
-      <limit effort="1.2" velocity="50" lower="-1e16" upper="1e16"/>
+      <limit effort="1.2" velocity="34" lower="-${0.55*pi}" upper="${0.55*pi}"/>
       <dynamics damping="0.0" friction="0.05"/>
       <parent link="link3"/>
@@ -157,5 +159,5 @@
       <axis xyz="1 0 0"/>
       <origin xyz="0 0 0"/>
-      <limit effort="1.2" velocity="50" lower="-1e16" upper="1e16"/>
+      <limit effort="1.2" velocity="34" lower="-${2*pi}" upper="${2*pi}"/>
       <dynamics damping="0.0" friction="0.05"/>
       <parent link="link4"/>

Commit message: Limit joint0 angle

File: urdf/engineer/arm.urdf.xacro (robot description, xacro)
@@ -127,5 +127,5 @@
       <origin xyz="0 0 0.019"/>
       <!--      limit not work while type="continuous"-->
-      <limit effort="20" velocity="25" lower="-${3*pi}" upper="${3*pi}"/>
+      <limit effort="20" velocity="25" lower="-${pi}" upper="${pi}"/>
       <dynamics damping="0.0" friction="0.1"/>
       <parent link="link0"/>

Commit message: Add transmission and fixed arm

File: urdf/engineer/arm.urdf.xacro (robot description, xacro)
@@ -1,4 +1,4 @@
 <robot xmlns:xacro="http://www.ros.org/wiki/xacro">
-  <xacro:macro name="arm" params="fix">
+  <xacro:macro name="arm" params="connected_to">
     <!--  link  -->
     <link name="link0">
@@ -123,4 +123,9 @@
     </link>
     <!--  joint  -->
+    <joint name="joint0" type="fixed">
+      <origin xyz="0 0 0.35"/>
+      <parent link="${connected_to}"/>
+      <child link="link0"/>
+    </joint>
     <joint name="joint1" type="revolute">
       <axis xyz="0 0 1"/>
@@ -136,5 +141,5 @@
       <origin xyz="0.11341 0 0.1380"/>
       <limit effort="60" velocity="10" lower="-${pi}" upper="${0.44*pi}"/>
-      <dynamics damping="0.0" friction="0.2"/>
+      <dynamics damping="0.0" friction="0.8"/>
       <parent link="link1"/>
       <child link="link2"/>
@@ -144,5 +149,5 @@
       <origin xyz="0.250 0 0"/>
       <limit effort="30" velocity="10" lower="-${0.722*pi}" upper="${0.722*pi}"/>
-      <dynamics damping="0.0" friction="0.1"/>
+      <dynamics damping="0.0" friction="0.5"/>
       <parent link="link2"/>
       <child link="link3"/>
@@ -164,4 +169,60 @@
       <child link="link5"/>
     </joint>
+    <!-- transmission -->
+    <transmission name="joint1_trans">
+      <type>transmission_interface/SimpleTransmission</type>
+      <actuator name="joint1_motor">
+        <hardwareInterface>hardware_interface/EffortJointInterface</hardwareInterface>
+        <mechanicalReduction>1</mechanicalReduction>
+        <offset>0</offset>
+      </actuator>
+      <joint name="joint1">
+        <hardwareInterface>hardware_interface/EffortJointInterface</hardwareInterface>
+      </joint>
+    </transmission>
+    <transmission name="joint2_trans">
+      <type>transmission_interface/SimpleTransmission</type>
+      <actuator name="joint2_motor">
+        <hardwareInterface>hardware_interface/EffortJointInterface</hardwareInterface>
+        <mechanicalReduction>1</mechanicalReduction>
+        <offset>0</offset>
+      </actuator>
+      <joint name="joint2">
+        <hardwareInterface>hardware_interface/EffortJointInterface</hardwareInterface>
+      </joint>
+    </transmission>
+    <transmission name="joint3_trans">
+      <type>transmission_interface/SimpleTransmission</type>
+      <actuator name="joint3_motor">
+        <hardwareInterface>hardware_interface/EffortJointInterface</hardwareInterface>
+        <mechanicalReduction>1</mechanicalReduction>
+        <offset>0</offset>
+      </actuator>
+      <joint name="joint3">
+        <hardwareInterface>hardware_interface/EffortJointInterface</hardwareInterface>
+      </joint>
+    </transmission>
+    <transmission name="joint4_trans">
+      <type>transmission_interface/SimpleTransmission</type>
+      <actuator name="joint4_motor">
+        <hardwareInterface>hardware_interface/EffortJointInterface</hardwareInterface>
+        <mechanicalReduction>1</mechanicalReduction>
+        <offset>0</offset>
+      </actuator>
+      <joint name="joint4">
+        <hardwareInterface>hardware_interface/EffortJointInterface</hardwareInterface>
+      </joint>
+    </transmission>
+    <transmission name="joint5_trans">
+      <type>transmission_interface/SimpleTransmission</type>
+      <actuator name="joint5_motor">
+        <hardwareInterface>hardware_interface/EffortJointInterface</hardwareInterface>
+        <mechanicalReduction>1</mechanicalReduction>
+        <offset>0</offset>
+      </actuator>
+      <joint name="joint5">
+        <hardwareInterface>hardware_interface/EffortJointInterface</hardwareInterface>
+      </joint>
+    </transmission>
   </xacro:macro>
 </robot>

File: urdf/engineer/engineer.urdf.xacro (robot description, xacro)
@@ -6,5 +6,5 @@
   <xacro:arg name="use_rm_gazebo" default="false"/>
   <xacro:arg name="roller_type" default="realistic"/>
-  <xacro:arg name="fix_arm" default="false"/>
+  <xacro:arg name="fixed_arm" default="true"/>
   <xacro:if value="$(arg load_chassis)">
     <xacro:include filename="$(find rm_description)/urdf/hero/chassis.urdf.xacro"/>
@@ -13,5 +13,8 @@
   <xacro:if value="$(arg load_arm)">
     <xacro:include filename="$(find rm_description)/urdf/engineer/arm.urdf.xacro"/>
-    <xacro:arm fix="$(arg fix_arm)"/>
+    <xacro:if value="$(arg fixed_arm)">
+      <link name="world"/>
+      <xacro:arm connected_to="world"/>
+    </xacro:if>
   </xacro:if>
   <xacro:if value="$(arg load_gazebo)">

Commit message: Set right collision origin of link5

File: urdf/engineer/arm.urdf.xacro (robot description, xacro)
@@ -116,5 +116,5 @@
       </visual>
       <collision>
-        <origin xyz="0 0 0" rpy="0 0 0"/>
+        <origin xyz="0.015 0 0" rpy="0 0 0"/>
         <geometry>
           <box size="0.057 0.0513 0.0513"/>

Commit message: Simplify arm.urdf.xacro

File: urdf/engineer/arm.urdf.xacro (robot description, xacro)
@@ -6,6 +6,5 @@
         <mass value="0.293"/>
         <origin xyz="0 0 0.00608"/>
-        <inertia ixx="2.916e-4" ixy="0" ixz="869.776e-9" iyy="2.9134e-4"
-                 iyz="0." izz="5.507e-4"/>
+        <inertia ixx="2.916e-4" ixy="0" ixz="869.776e-9" iyy="2.9134e-4" iyz="0." izz="5.507e-4"/>
       </inertial>
       <visual>
@@ -26,6 +25,5 @@
         <mass value="2.775151"/>
         <origin xyz="0.00286 0.00018 0.05209"/>
-        <inertia ixx="1.962e-2" ixy="4573.477e-9" ixz="-3.727e-3" iyy="2.223e-2"
-                 iyz="-2536.137e-9" izz="1.949e-2"/>
+        <inertia ixx="1.962e-2" ixy="4573.477e-9" ixz="-3.727e-3" iyy="2.223e-2" iyz="-2536.137e-9" izz="1.949e-2"/>
       </inertial>
       <visual>
@@ -46,6 +44,5 @@
         <mass value="1.372"/>
         <origin xyz="0.07668 -0.001679 0"/>
-        <inertia ixx="2.04e-3" ixy="1.959e-4" ixz="-235.828e-9" iyy="1.496e-2"
-                 iyz="0." izz="1.564e-2"/>
+        <inertia ixx="2.04e-3" ixy="1.959e-4" ixz="-235.828e-9" iyy="1.496e-2" iyz="0." izz="1.564e-2"/>
       </inertial>
       <visual>
@@ -66,6 +63,5 @@
         <mass value="0.697"/>
         <origin xyz="0.079837 -0.00581 0.000299"/>
-        <inertia ixx="8.905e-4" ixy="6.123e-5" ixz="-3.193e-5" iyy="6.036e-3"
-                 iyz="1936.328e-9" izz="6.588e-3"/>
+        <inertia ixx="8.905e-4" ixy="6.123e-5" ixz="-3.193e-5" iyy="6.036e-3" iyz="1936.328e-9" izz="6.588e-3"/>
       </inertial>
       <visual>
@@ -86,6 +82,5 @@
         <mass value="0.367"/>
         <origin xyz="0 0 0"/>
-        <inertia ixx="2.803e-4" ixy="0.15e-9" ixz="0" iyy="19.296e-5"
-                 iyz="0." izz="2.798e-4"/>
+        <inertia ixx="2.803e-4" ixy="0.15e-9" ixz="0" iyy="19.296e-5" iyz="0." izz="2.798e-4"/>
       </inertial>
       <visual>
@@ -106,6 +101,5 @@
         <mass value="0.257"/>
         <origin xyz="0.02803 0.00084 -0.00089"/>
-        <inertia ixx="6.485e-5" ixy="-754.967e-9" ixz="-793.024e-9" iyy="2.477e-4"
-                 iyz="0." izz="2.477e-4"/>
+        <inertia ixx="6.485e-5" ixy="-754.967e-9" ixz="-793.024e-9" iyy="2.477e-4" iyz="0." izz="2.477e-4"/>
       </inertial>
       <visual>

Commit message: Add transmission

File: urdf/engineer/arm.urdf.xacro (robot description, xacro)
@@ -1,2 +1,3 @@
+<?xml version="1.0" encoding="utf-8"?>
 <robot xmlns:xacro="http://www.ros.org/wiki/xacro">
   <xacro:macro name="arm" params="connected_to">
@@ -164,5 +165,5 @@
     </joint>
     <!-- transmission -->
-    <transmission name="joint1_trans">
+    <transmission name="trans_joint1">
       <type>transmission_interface/SimpleTransmission</type>
       <actuator name="joint1_motor">
@@ -175,5 +176,5 @@
       </joint>
     </transmission>
-    <transmission name="joint2_trans">
+    <transmission name="trans_joint2">
       <type>transmission_interface/SimpleTransmission</type>
       <actuator name="joint2_motor">
@@ -186,5 +187,5 @@
       </joint>
     </transmission>
-    <transmission name="joint3_trans">
+    <transmission name="trans_joint3">
       <type>transmission_interface/SimpleTransmission</type>
       <actuator name="joint3_motor">
@@ -197,5 +198,5 @@
       </joint>
     </transmission>
-    <transmission name="joint4_trans">
+    <transmission name="trans_joint4">
       <type>transmission_interface/SimpleTransmission</type>
       <actuator name="joint4_motor">
@@ -208,5 +209,5 @@
       </joint>
     </transmission>
-    <transmission name="joint5_trans">
+    <transmission name="trans_joint5">
       <type>transmission_interface/SimpleTransmission</type>
       <actuator name="joint5_motor">

File: urdf/engineer/hand.urdf.xacro (robot description, xacro)
@@ -77,4 +77,24 @@
       <mimic joint="right_finger_joint"/>
     </joint>
+    <transmission name="trans_right_finger_joint">
+      <type>transmission_interface/SimpleTransmission</type>
+      <joint name="right_finger_joint">
+        <hardwareInterface>hardware_interface/EffortJointInterface</hardwareInterface>
+      </joint>
+      <actuator name="right_finger_motor">
+        <hardwareInterface>hardware_interface/EffortJointInterface</hardwareInterface>
+        <mechanicalReduction>1</mechanicalReduction>
+      </actuator>
+    </transmission>
+    <transmission name="trans_left_finger_joint">
+      <type>transmission_interface/SimpleTransmission</type>
+      <joint name="left_finger_joint">
+        <hardwareInterface>hardware_interface/EffortJointInterface</hardwareInterface>
+      </joint>
+      <actuator name="left_finger_motor">
+        <hardwareInterface>hardware_interface/EffortJointInterface</hardwareInterface>
+        <mechanicalReduction>1</mechanicalReduction>
+      </actuator>
+    </transmission>
   </xacro:macro>
 </robot>

Commit message: Set limit of hand

File: urdf/engineer/arm.urdf.xacro (robot description, xacro)
@@ -73,7 +73,7 @@
       </visual>
       <collision>
-        <origin xyz="0.090 0 0"/>
-        <geometry>
-          <box size="0.245 0.089 0.0895"/>
+        <origin xyz="0.060 0 0"/>
+        <geometry>
+          <box size="0.200 0.08 0.07"/>
         </geometry>
       </collision>

File: urdf/engineer/hand.urdf.xacro (robot description, xacro)
@@ -17,5 +17,5 @@
         <origin xyz="0.020 0.02 0" rpy="0 0 0"/>
         <geometry>
-          <box size="0.06 0.230 0.06"/>
+          <box size="0.04 0.230 0.06"/>
         </geometry>
       </collision>
@@ -67,5 +67,5 @@
       <origin xyz="0.032 0 0" rpy="0 0 0"/>
       <axis xyz="0 1 0"/>
-      <limit effort="20" lower="0.0" upper="0.02" velocity="0.5"/>
+      <limit effort="588" lower="0.0" upper="0.02" velocity="3.772"/>
     </joint>
     <joint name="left_finger_joint" type="prismatic">
@@ -74,5 +74,5 @@
       <origin xyz="0.032 0 0" rpy="0 0 0"/>
       <axis xyz="0 -1 0"/>
-      <limit effort="20" lower="0.0" upper="0.02" velocity="0.5"/>
+      <limit effort="588" lower="0.0" upper="0.02" velocity="3.772"/>
       <mimic joint="right_finger_joint"/>
     </joint>

Commit message: Separate arm transmission

File: urdf/engineer/arm.urdf.xacro (robot description, xacro)
@@ -164,60 +164,8 @@
       <child link="link5"/>
     </joint>
-    <!-- transmission -->
-    <transmission name="trans_joint1">
-      <type>transmission_interface/SimpleTransmission</type>
-      <actuator name="joint1_motor">
-        <hardwareInterface>hardware_interface/EffortJointInterface</hardwareInterface>
-        <mechanicalReduction>1</mechanicalReduction>
-        <offset>0</offset>
-      </actuator>
-      <joint name="joint1">
-        <hardwareInterface>hardware_interface/EffortJointInterface</hardwareInterface>
-      </joint>
-    </transmission>
-    <transmission name="trans_joint2">
-      <type>transmission_interface/SimpleTransmission</type>
-      <actuator name="joint2_motor">
-        <hardwareInterface>hardware_interface/EffortJointInterface</hardwareInterface>
-        <mechanicalReduction>1</mechanicalReduction>
-        <offset>0</offset>
-      </actuator>
-      <joint name="joint2">
-        <hardwareInterface>hardware_interface/EffortJointInterface</hardwareInterface>
-      </joint>
-    </transmission>
-    <transmission name="trans_joint3">
-      <type>transmission_interface/SimpleTransmission</type>
-      <actuator name="joint3_motor">
-        <hardwareInterface>hardware_interface/EffortJointInterface</hardwareInterface>
-        <mechanicalReduction>1</mechanicalReduction>
-        <offset>0</offset>
-      </actuator>
-      <joint name="joint3">
-        <hardwareInterface>hardware_interface/EffortJointInterface</hardwareInterface>
-      </joint>
-    </transmission>
-    <transmission name="trans_joint4">
-      <type>transmission_interface/SimpleTransmission</type>
-      <actuator name="joint4_motor">
-        <hardwareInterface>hardware_interface/EffortJointInterface</hardwareInterface>
-        <mechanicalReduction>1</mechanicalReduction>
-        <offset>0</offset>
-      </actuator>
-      <joint name="joint4">
-        <hardwareInterface>hardware_interface/EffortJointInterface</hardwareInterface>
-      </joint>
-    </transmission>
-    <transmission name="trans_joint5">
-      <type>transmission_interface/SimpleTransmission</type>
-      <actuator name="joint5_motor">
-        <hardwareInterface>hardware_interface/EffortJointInterface</hardwareInterface>
-        <mechanicalReduction>1</mechanicalReduction>
-        <offset>0</offset>
-      </actuator>
-      <joint name="joint5">
-        <hardwareInterface>hardware_interface/EffortJointInterface</hardwareInterface>
-      </joint>
-    </transmission>
+    <!-- extensions -->
+    <xacro:include filename="$(find rm_description)/urdf/engineer/arm.transmission.xacro"/>
+    <xacro:arm_transmission/>
+    <!--TODO: Add gazebo-->
   </xacro:macro>
 </robot>
