Commit message: change engineer parameter

File: urdf/engineer/arm.urdf.xacro (robot description, xacro)
@@ -3,28 +3,9 @@
   <xacro:macro name="arm" params="connected_to">
     <!--  link  -->
-    <link name="link0">
-      <inertial>
-        <mass value="0.293"/>
-        <origin xyz="0 0 0.00608"/>
-        <inertia ixx="2.916e-4" ixy="0" ixz="869.776e-9" iyy="2.9134e-4" iyz="0." izz="5.507e-4"/>
-      </inertial>
-      <visual>
-        <origin xyz="0 0 0" rpy="0 0 0"/>
-        <geometry>
-          <mesh filename="package://rm_description/meshes/engineer/link0.stl" scale="0.001 0.001 0.001"/>
-        </geometry>
-      </visual>
-      <collision>
-        <origin xyz="0 0 0.008"/>
-        <geometry>
-          <box size="0.12 0.12 0.016"/>
-        </geometry>
-      </collision>
-    </link>
     <link name="link1">
       <inertial>
-        <mass value="2.775151"/>
-        <origin xyz="0.00286 0.00018 0.05209"/>
-        <inertia ixx="1.962e-2" ixy="4573.477e-9" ixz="-3.727e-3" iyy="2.223e-2" iyz="-2536.137e-9" izz="1.949e-2"/>
+        <mass value="1.7056"/>
+        <origin xyz="0.004 0 0.0571"/>
+        <inertia ixx="1.542e-2" ixy="0" ixz="-1.332e-3" iyy="1.028e-2" iyz="0" izz="1.017e-2"/>
       </inertial>
       <visual>
@@ -35,7 +16,13 @@
       </visual>
       <collision>
-        <origin xyz="-0.02 0 0.05" rpy="0 0 0"/>
+        <origin xyz="-0.045 0 0.035" rpy="0 0 0"/>
         <geometry>
-          <box size="0.200 0.182 0.100"/>
+          <box size="0.15 0.188 0.07"/>
+        </geometry>
+      </collision>
+      <collision>
+        <origin xyz="0.040 0 0.1" rpy="0 -0.95993 0"/>
+        <geometry>
+          <box size="0.17 0.188 0.095"/>
         </geometry>
       </collision>
@@ -43,7 +30,7 @@
     <link name="link2">
       <inertial>
-        <mass value="1.372"/>
-        <origin xyz="0.07668 -0.001679 0"/>
-        <inertia ixx="2.04e-3" ixy="1.959e-4" ixz="-235.828e-9" iyy="1.496e-2" iyz="0." izz="1.564e-2"/>
+        <mass value="1.4763"/>
+        <origin xyz="0.05652 0 0"/>
+        <inertia ixx="1.976e-3" ixy="5.791e-5" ixz="-2.47366e-7" iyy="8.418e-3" iyz="1.0e-7" izz="8.946e-3"/>
       </inertial>
       <visual>
@@ -54,7 +41,7 @@
       </visual>
       <collision>
-        <origin xyz="0.115 0 0"/>
+        <origin xyz="0.062 0 0"/>
         <geometry>
-          <box size="0.335 0.100 0.094"/>
+          <box size="0.225 0.096 0.094"/>
         </geometry>
       </collision>
@@ -62,7 +49,7 @@
     <link name="link3">
       <inertial>
-        <mass value="0.697"/>
-        <origin xyz="0.079837 -0.00581 0.000299"/>
-        <inertia ixx="8.905e-4" ixy="6.123e-5" ixz="-3.193e-5" iyy="6.036e-3" iyz="1936.328e-9" izz="6.588e-3"/>
+        <mass value="0.5946"/>
+        <origin xyz="0.0471 -0.0094 0.0003"/>
+        <inertia ixx="6.49e-4" ixy="5.036e-5" ixz="-2.372e-5" iyy="2.739e-3" iyz="1.795e-6" izz="3.077e-3"/>
       </inertial>
       <visual>
@@ -73,7 +60,7 @@
       </visual>
       <collision>
-        <origin xyz="0.060 0 0"/>
+        <origin xyz="0.063 0 0"/>
         <geometry>
-          <box size="0.200 0.08 0.07"/>
+          <box size="0.216 0.084 0.09"/>
         </geometry>
       </collision>
@@ -81,7 +68,7 @@
     <link name="link4">
       <inertial>
-        <mass value="0.367"/>
+        <mass value="0.361"/>
         <origin xyz="0 0 0"/>
-        <inertia ixx="2.803e-4" ixy="0.15e-9" ixz="0" iyy="19.296e-5" iyz="0." izz="2.798e-4"/>
+        <inertia ixx="2.593e-4" ixy="5.907e-3" ixz="2.629e-2" iyy="8.662e-5" iyz="0." izz="2.589e-4"/>
       </inertial>
       <visual>
@@ -94,5 +81,5 @@
         <origin xyz="0 0 0" rpy="0 0 0"/>
         <geometry>
-          <box size="0.0513 0.0882 0.0513"/>
+          <box size="0.0513 0.074 0.0513"/>
         </geometry>
       </collision>
@@ -100,7 +87,7 @@
     <link name="link5">
       <inertial>
-        <mass value="0.257"/>
-        <origin xyz="0.02803 0.00084 -0.00089"/>
-        <inertia ixx="6.485e-5" ixy="-754.967e-9" ixz="-793.024e-9" iyy="2.477e-4" iyz="0." izz="2.477e-4"/>
+        <mass value="0.249"/>
+        <origin xyz="0.02737 0.0 0.0"/>
+        <inertia ixx="6.090e-5" ixy="7.70024e-7" ixz="7.35489e-7" iyy="2.293e-4" iyz="0." izz=" 2.293e-4"/>
       </inertial>
       <visual>
@@ -113,26 +100,21 @@
         <origin xyz="0.015 0 0" rpy="0 0 0"/>
         <geometry>
-          <box size="0.057 0.0513 0.0513"/>
+          <box size="0.056 0.0513 0.0513"/>
         </geometry>
       </collision>
     </link>
     <!--  joint  -->
-    <joint name="joint0" type="fixed">
-      <origin xyz="0 0 0.35"/>
-      <parent link="${connected_to}"/>
-      <child link="link0"/>
-    </joint>
     <joint name="joint1" type="revolute">
       <axis xyz="0 0 1"/>
-      <origin xyz="0 0 0.019"/>
+      <origin xyz="0.133 0 0.1"/>
       <!--      limit not work while type="continuous"-->
       <limit effort="20" velocity="25" lower="-${pi}" upper="${pi}"/>
       <dynamics damping="0.0" friction="0.1"/>
-      <parent link="link0"/>
+      <parent link="${connected_to}"/>
       <child link="link1"/>
     </joint>
     <joint name="joint2" type="revolute">
       <axis xyz="0 1 0"/>
-      <origin xyz="0.11341 0 0.1380"/>
+      <origin xyz="0.05909 0 0.1280"/>
       <limit effort="30" velocity="10" lower="-${pi}" upper="${0.44*pi}"/>
       <dynamics damping="0.0" friction="0.8"/>
@@ -142,5 +124,5 @@
     <joint name="joint3" type="revolute">
       <axis xyz="0 1 0"/>
-      <origin xyz="0.250 0 0"/>
+      <origin xyz="0.16 0 0"/>
       <limit effort="30" velocity="10" lower="-${0.722*pi}" upper="${0.722*pi}"/>
       <dynamics damping="0.0" friction="0.5"/>
@@ -150,5 +132,5 @@
     <joint name="joint4" type="revolute">
       <axis xyz="0 1 0"/>
-      <origin xyz="0.180 0 0"/>
+      <origin xyz="0.145 0 0"/>
       <limit effort="1.2" velocity="34" lower="-${0.55*pi}" upper="${0.55*pi}"/>
       <dynamics damping="0.0" friction="0.05"/>

File: urdf/engineer/engineer.urdf.xacro (robot description, xacro)
@@ -6,5 +6,5 @@
     <xacro:arg name="roller_type" default="realistic"/>
     <xacro:if value="$(arg load_chassis)">
-        <xacro:include filename="$(find rm_description)/urdf/hero/chassis.urdf.xacro"/>
+        <xacro:include filename="$(find rm_description)/urdf/engineer/chassis.urdf.xacro"/>
         <xacro:chassis roller_type="$(arg roller_type)"/>
     </xacro:if>
@@ -20,6 +20,6 @@
         </xacro:unless>
         <xacro:arm_transmission simulation="$(arg use_simulation)"/>
-        <!--    <xacro:include filename="$(find rm_description)/urdf/engineer/hand.urdf.xacro"/>-->
-        <!--    <xacro:hand connected_to="link5" xyz="0.039 0 0"/>-->
+            <xacro:include filename="$(find rm_description)/urdf/engineer/hand.urdf.xacro"/>
+            <xacro:hand connected_to="link5" xyz="0.039 0 0"/>
     </xacro:if>
     <xacro:if value="$(arg use_simulation)">

File: urdf/engineer/hand.urdf.xacro (robot description, xacro)
@@ -15,7 +15,7 @@
       </visual>
       <collision>
-        <origin xyz="0.020 0.02 0" rpy="0 0 0"/>
+        <origin xyz="0.0225 0.0 0" rpy="0 0 0"/>
         <geometry>
-          <box size="0.04 0.230 0.06"/>
+          <box size="0.045 0.2658 0.0675"/>
         </geometry>
       </collision>
@@ -33,6 +33,25 @@
       </visual>
       <collision>
+        <origin xyz="0.011 -0.04 0" rpy="0 0 0"/>
         <geometry>
-          <mesh filename="package://rm_description/meshes/engineer/right_finger_convex.stl" scale="0.001 0.001 0.001"/>
+          <box size="0.048 0.026 0.030"/>
+        </geometry>
+      </collision>
+      <collision>
+        <origin xyz="0.0235 -0.0832 0" rpy="0 0 0"/>
+        <geometry>
+          <box size="0.022 0.1123 0.03"/>
+        </geometry>
+      </collision>
+      <collision>
+        <origin xyz="0.069 -0.1307 0" rpy="0 0 0"/>
+        <geometry>
+          <box size="0.112 0.0173 0.03"/>
+        </geometry>
+      </collision>
+      <collision>
+        <origin xyz="0.105 -0.1232 0" rpy="0 0 0"/>
+        <geometry>
+          <box size="0.04 0.0323 0.03"/>
         </geometry>
       </collision>
@@ -50,6 +69,25 @@
       </visual>
       <collision>
+        <origin xyz="0.011 0.04 0" rpy="0 0 0"/>
         <geometry>
-          <mesh filename="package://rm_description/meshes/engineer/left_finger_convex.stl" scale="0.001 0.001 0.001"/>
+          <box size="0.048 0.026 0.030"/>
+        </geometry>
+      </collision>
+      <collision>
+        <origin xyz="0.0235 0.0832 0" rpy="0 0 0"/>
+        <geometry>
+          <box size="0.022 0.1123 0.03"/>
+        </geometry>
+      </collision>
+      <collision>
+        <origin xyz="0.069 0.1307 0" rpy="0 0 0"/>
+        <geometry>
+          <box size="0.112 0.0173 0.03"/>
+        </geometry>
+      </collision>
+      <collision>
+        <origin xyz="0.105 0.1232 0" rpy="0 0 0"/>
+        <geometry>
+          <box size="0.04 0.0323 0.03"/>
         </geometry>
       </collision>
@@ -65,5 +103,5 @@
       <parent link="palm"/>
       <child link="right_finger"/>
-      <origin xyz="0.032 0 0" rpy="0 0 0"/>
+      <origin xyz="0.023 -0.045 0" rpy="0 0 0"/>
       <axis xyz="0 1 0"/>
       <limit effort="588" lower="0.0" upper="0.02" velocity="3.772"/>
@@ -72,8 +110,8 @@
       <parent link="palm"/>
       <child link="left_finger"/>
-      <origin xyz="0.032 0 0" rpy="0 0 0"/>
+      <origin xyz="0.023 0.045 0" rpy="0 0 0"/>
       <axis xyz="0 -1 0"/>
       <limit effort="588" lower="0.0" upper="0.02" velocity="3.772"/>
-      <mimic joint="right_finger_joint"/>
+<!--      <mimic joint="right_finger_joint"/>-->
     </joint>
     <transmission name="trans_right_finger_joint">

Commit message: chancollision

File: urdf/engineer/arm.urdf.xacro (robot description, xacro)
@@ -18,5 +18,5 @@
         <origin xyz="-0.045 0 0.035" rpy="0 0 0"/>
         <geometry>
-          <box size="0.15 0.188 0.07"/>
+          <box size="0.15 0.106 0.07"/>
         </geometry>
       </collision>
@@ -24,5 +24,11 @@
         <origin xyz="0.040 0 0.1" rpy="0 -0.95993 0"/>
         <geometry>
-          <box size="0.17 0.188 0.095"/>
+          <box size="0.17 0.106 0.095"/>
+        </geometry>
+      </collision>
+      <collision>
+        <origin xyz="0 0 0.05" rpy="1.5707963 0 0"/>
+        <geometry>
+           <cylinder length="0.188" radius="0.047"/>
         </geometry>
       </collision>
@@ -43,5 +49,5 @@
         <origin xyz="0.062 0 0"/>
         <geometry>
-          <box size="0.225 0.096 0.094"/>
+          <box size="0.225 0.096 0.070"/>
         </geometry>
       </collision>
@@ -62,5 +68,11 @@
         <origin xyz="0.063 0 0"/>
         <geometry>
-          <box size="0.216 0.084 0.09"/>
+          <box size="0.191 0.084 0.053"/>
+        </geometry>
+      </collision>
+      <collision>
+        <origin xyz="0 0 0" rpy="1.5707963 0 0"/>
+        <geometry>
+          <cylinder length="0.082" radius="0.047"/>
         </geometry>
       </collision>

File: urdf/engineer/chassis.urdf.xacro (robot description, xacro)
@@ -28,25 +28,25 @@
             </collision>
             <collision>
-                <origin xyz="-0.0262 -0.097 0.267" rpy="0 0 0"/>
+                <origin xyz="-0.033 -0.1 0.267" rpy="0 0 0.7853982"/>
                 <geometry>
-                    <box size="0.03 0.03 0.334"/>
+                    <box size="0.0207 0.0207 0.334"/>
                 </geometry>
             </collision>
             <collision>
-                <origin xyz="-0.0262 0.097 0.267" rpy="0 0 0"/>
+                <origin xyz="-0.033 0.10 0.267" rpy="0 0 0.7853982"/>
                 <geometry>
-                    <box size="0.03 0.03 0.334"/>
+                    <box size="0.0207 0.0207 0.334"/>
                 </geometry>
             </collision>
             <collision>
-                <origin xyz="-0.23225 -0.097 0.267" rpy="0 0 0"/>
+                <origin xyz="-0.23225 -0.1 0.267" rpy="0 0 0.7853982"/>
                 <geometry>
-                    <box size="0.03 0.03 0.334"/>
+                    <box size="0.0207 0.0207 0.334"/>
                 </geometry>
             </collision>
             <collision>
-                <origin xyz="-0.23225 0.097 0.267" rpy="0 0 0"/>
+                <origin xyz="-0.23225 0.1 0.267" rpy="0 0 0.7853982"/>
                 <geometry>
-                    <box size="0.03 0.03 0.334"/>
+                    <box size="0.0207 0.0207 0.334"/>
                 </geometry>
             </collision>

File: urdf/engineer/hand.urdf.xacro (robot description, xacro)
@@ -45,7 +45,7 @@
       </collision>
       <collision>
-        <origin xyz="0.069 -0.1307 0" rpy="0 0 0"/>
+        <origin xyz="0.069 -0.13 0" rpy="0 0 0"/>
         <geometry>
-          <box size="0.112 0.0173 0.03"/>
+          <box size="0.112 0.0157 0.03"/>
         </geometry>
       </collision>
@@ -81,7 +81,7 @@
       </collision>
       <collision>
-        <origin xyz="0.069 0.1307 0" rpy="0 0 0"/>
+        <origin xyz="0.069 0.13 0" rpy="0 0 0"/>
         <geometry>
-          <box size="0.112 0.0173 0.03"/>
+          <box size="0.112 0.0157 0.03"/>
         </geometry>
       </collision>
