Commit message: add chassis

File: urdf/engineer/arm.urdf.xacro (robot description, xacro)
@@ -1,129 +1,129 @@
 <?xml version="1.0" encoding="utf-8"?>
 <robot xmlns:xacro="http://www.ros.org/wiki/xacro" name="arm">
-    <xacro:macro name="arm" params="connected_to">
-        <!--  link  -->
-        <link name="link1">
-            <inertial>
-                <mass value="1.7056"/>
-                <origin xyz="0.004 0 0.0571"/>
-                <inertia ixx="1.542e-2" ixy="0" ixz="-1.332e-3" iyy="1.028e-2" iyz="0" izz="1.017e-2"/>
-            </inertial>
-            <visual>
-                <origin xyz="0 0 0" rpy="0 0 0"/>
-                <geometry>
-                    <mesh filename="package://rm_description/meshes/engineer/link1.stl" scale="0.001 0.001 0.001"/>
-                </geometry>
-            </visual>
-            <collision>
-                <origin xyz="-0.045 0 0.035" rpy="0 0 0"/>
-                <geometry>
-                    <box size="0.15 0.106 0.07"/>
-                </geometry>
-            </collision>
-            <collision>
-                <origin xyz="0.040 0 0.1" rpy="0 -0.95993 0"/>
-                <geometry>
-                    <box size="0.17 0.106 0.095"/>
-                </geometry>
-            </collision>
-            <collision>
-                <origin xyz="0 0 0.05" rpy="1.5707963 0 0"/>
-                <geometry>
-                    <cylinder length="0.188" radius="0.047"/>
-                </geometry>
-            </collision>
-        </link>
-        <link name="link2">
-            <inertial>
-                <mass value="1.4763"/>
-                <origin xyz="0.05652 0 0"/>
-                <inertia ixx="1.976e-3" ixy="5.791e-5" ixz="-2.47366e-7" iyy="8.418e-3" iyz="1.0e-7" izz="8.946e-3"/>
-            </inertial>
-            <visual>
-                <origin xyz="0 0 0" rpy="0 0 0"/>
-                <geometry>
-                    <mesh filename="package://rm_description/meshes/engineer/link2.stl" scale="0.001 0.001 0.001"/>
-                </geometry>
-            </visual>
-            <collision>
-                <origin xyz="0.062 0 0"/>
-                <geometry>
-                    <box size="0.225 0.096 0.070"/>
-                </geometry>
-            </collision>
-        </link>
-        <link name="link3">
-            <inertial>
-                <mass value="0.5946"/>
-                <origin xyz="0.0471 -0.0094 0.0003"/>
-                <inertia ixx="6.49e-4" ixy="5.036e-5" ixz="-2.372e-5" iyy="2.739e-3" iyz="1.795e-6" izz="3.077e-3"/>
-            </inertial>
-            <visual>
-                <origin xyz="0 0 0" rpy="0 0 0"/>
-                <geometry>
-                    <mesh filename="package://rm_description/meshes/engineer/link3.stl" scale="0.001 0.001 0.001"/>
-                </geometry>
-            </visual>
-            <collision>
-                <origin xyz="0.063 0 0"/>
-                <geometry>
-                    <box size="0.191 0.084 0.053"/>
-                </geometry>
-            </collision>
-            <collision>
-                <origin xyz="0 0 0" rpy="1.5707963 0 0"/>
-                <geometry>
-                    <cylinder length="0.082" radius="0.047"/>
-                </geometry>
-            </collision>
-        </link>
-        <link name="link4">
-            <inertial>
-                <mass value="0.361"/>
-                <origin xyz="0 0 0"/>
-                <inertia ixx="2.593e-4" ixy="5.907e-3" ixz="2.629e-2" iyy="8.662e-5" iyz="0." izz="2.589e-4"/>
-            </inertial>
-            <visual>
-                <origin xyz="0 0 0" rpy="0 0 0"/>
-                <geometry>
-                    <mesh filename="package://rm_description/meshes/engineer/link4.stl" scale="0.001 0.001 0.001"/>
-                </geometry>
-            </visual>
-            <collision>
-                <origin xyz="0 0 0" rpy="0 0 0"/>
-                <geometry>
-                    <box size="0.0513 0.074 0.0513"/>
-                </geometry>
-            </collision>
-        </link>
-        <link name="link5">
-            <inertial>
-                <mass value="0.249"/>
-                <origin xyz="0.02737 0.0 0.0"/>
-                <inertia ixx="6.090e-5" ixy="7.70024e-7" ixz="7.35489e-7" iyy="2.293e-4" iyz="0." izz=" 2.293e-4"/>
-            </inertial>
-            <visual>
-                <origin xyz="0 0 0" rpy="0 0 0"/>
-                <geometry>
-                    <mesh filename="package://rm_description/meshes/engineer/link5.stl" scale="0.001 0.001 0.001"/>
-                </geometry>
-            </visual>
-            <collision>
-                <origin xyz="0.015 0 0" rpy="0 0 0"/>
-                <geometry>
-                    <box size="0.056 0.0513 0.0513"/>
-                </geometry>
-            </collision>
-        </link>
-        <!--  joint  -->
-        <joint name="joint1" type="revolute">
-            <axis xyz="0 0 1"/>
-            <origin xyz="0.133 0 0.1"/>
-            <!--      limit not work while type="continuous"-->
-            <limit effort="20" velocity="25" lower="-${pi}" upper="${pi}"/>
-            <dynamics damping="0.0" friction="0.1"/>
-            <parent link="${connected_to}"/>
-            <child link="link1"/>
-        </joint>
+  <xacro:macro name="arm" params="connected_to">
+    <!--  link  -->
+    <link name="link1">
+      <inertial>
+        <mass value="1.7056"/>
+        <origin xyz="0.004 0 0.0571"/>
+        <inertia ixx="1.542e-2" ixy="0" ixz="-1.332e-3" iyy="1.028e-2" iyz="0" izz="1.017e-2"/>
+      </inertial>
+      <visual>
+        <origin xyz="0 0 0" rpy="0 0 0"/>
+        <geometry>
+          <mesh filename="package://rm_description/meshes/engineer/link1.stl" scale="0.001 0.001 0.001"/>
+        </geometry>
+      </visual>
+      <collision>
+        <origin xyz="-0.045 0 0.035" rpy="0 0 0"/>
+        <geometry>
+          <box size="0.15 0.106 0.07"/>
+        </geometry>
+      </collision>
+      <collision>
+        <origin xyz="0.040 0 0.1" rpy="0 -0.95993 0"/>
+        <geometry>
+          <box size="0.17 0.106 0.095"/>
+        </geometry>
+      </collision>
+      <collision>
+        <origin xyz="0 0 0.05" rpy="1.5707963 0 0"/>
+        <geometry>
+           <cylinder length="0.188" radius="0.047"/>
+        </geometry>
+      </collision>
+    </link>
+    <link name="link2">
+      <inertial>
+        <mass value="1.4763"/>
+        <origin xyz="0.05652 0 0"/>
+        <inertia ixx="1.976e-3" ixy="5.791e-5" ixz="-2.47366e-7" iyy="8.418e-3" iyz="1.0e-7" izz="8.946e-3"/>
+      </inertial>
+      <visual>
+        <origin xyz="0 0 0" rpy="0 0 0"/>
+        <geometry>
+          <mesh filename="package://rm_description/meshes/engineer/link2.stl" scale="0.001 0.001 0.001"/>
+        </geometry>
+      </visual>
+      <collision>
+        <origin xyz="0.062 0 0"/>
+        <geometry>
+          <box size="0.225 0.096 0.070"/>
+        </geometry>
+      </collision>
+    </link>
+    <link name="link3">
+      <inertial>
+        <mass value="0.5946"/>
+        <origin xyz="0.0471 -0.0094 0.0003"/>
+        <inertia ixx="6.49e-4" ixy="5.036e-5" ixz="-2.372e-5" iyy="2.739e-3" iyz="1.795e-6" izz="3.077e-3"/>
+      </inertial>
+      <visual>
+        <origin xyz="0 0 0" rpy="0 0 0"/>
+        <geometry>
+          <mesh filename="package://rm_description/meshes/engineer/link3.stl" scale="0.001 0.001 0.001"/>
+        </geometry>
+      </visual>
+      <collision>
+        <origin xyz="0.063 0 0"/>
+        <geometry>
+          <box size="0.191 0.084 0.053"/>
+        </geometry>
+      </collision>
+      <collision>
+        <origin xyz="0 0 0" rpy="1.5707963 0 0"/>
+        <geometry>
+          <cylinder length="0.082" radius="0.047"/>
+        </geometry>
+      </collision>
+    </link>
+    <link name="link4">
+      <inertial>
+        <mass value="0.361"/>
+        <origin xyz="0 0 0"/>
+        <inertia ixx="2.593e-4" ixy="5.907e-3" ixz="2.629e-2" iyy="8.662e-5" iyz="0." izz="2.589e-4"/>
+      </inertial>
+      <visual>
+        <origin xyz="0 0 0" rpy="0 0 0"/>
+        <geometry>
+          <mesh filename="package://rm_description/meshes/engineer/link4.stl" scale="0.001 0.001 0.001"/>
+        </geometry>
+      </visual>
+      <collision>
+        <origin xyz="0 0 0" rpy="0 0 0"/>
+        <geometry>
+          <box size="0.0513 0.074 0.0513"/>
+        </geometry>
+      </collision>
+    </link>
+    <link name="link5">
+      <inertial>
+        <mass value="0.249"/>
+        <origin xyz="0.02737 0.0 0.0"/>
+        <inertia ixx="6.090e-5" ixy="7.70024e-7" ixz="7.35489e-7" iyy="2.293e-4" iyz="0." izz=" 2.293e-4"/>
+      </inertial>
+      <visual>
+        <origin xyz="0 0 0" rpy="0 0 0"/>
+        <geometry>
+          <mesh filename="package://rm_description/meshes/engineer/link5.stl" scale="0.001 0.001 0.001"/>
+        </geometry>
+      </visual>
+      <collision>
+        <origin xyz="0.015 0 0" rpy="0 0 0"/>
+        <geometry>
+          <box size="0.056 0.0513 0.0513"/>
+        </geometry>
+      </collision>
+    </link>
+    <!--  joint  -->
+    <joint name="joint1" type="revolute">
+      <axis xyz="0 0 1"/>
+      <origin xyz="0.133 0 0.1"/>
+      <!--      limit not work while type="continuous"-->
+      <limit effort="20" velocity="25" lower="-${pi}" upper="${pi}"/>
+      <dynamics damping="0.0" friction="0.1"/>
+      <parent link="${connected_to}"/>
+      <child link="link1"/>
+    </joint>
     <joint name="joint2" type="revolute">
       <axis xyz="0 1 0"/>
@@ -134,12 +134,4 @@
       <child link="link2"/>
     </joint>
-        <joint name="joint2" type="revolute">
-            <axis xyz="0 1 0"/>
-            <origin xyz="0.05909 0 0.1280"/>
-            <limit effort="30" velocity="10" lower="-${pi}" upper="${0.44*pi}"/>
-            <dynamics damping="0.0" friction="0.8"/>
-            <parent link="link1"/>
-            <child link="link2"/>
-        </joint>
     <joint name="joint3" type="revolute">
       <axis xyz="0 1 0"/>
@@ -150,28 +142,20 @@
       <child link="link3"/>
     </joint>
-        <joint name="joint3" type="revolute">
-            <axis xyz="0 1 0"/>
-            <origin xyz="0.16 0 0"/>
-            <limit effort="30" velocity="10" lower="-${0.722*pi}" upper="${0.722*pi}"/>
-            <dynamics damping="0.0" friction="0.5"/>
-            <parent link="link2"/>
-            <child link="link3"/>
-        </joint>
-        <joint name="joint4" type="revolute">
-            <axis xyz="0 1 0"/>
-            <origin xyz="0.145 0 0"/>
-            <limit effort="1.2" velocity="34" lower="-${0.55*pi}" upper="${0.55*pi}"/>
-            <dynamics damping="0.0" friction="0.05"/>
-            <parent link="link3"/>
-            <child link="link4"/>
-        </joint>
-        <joint name="joint5" type="revolute">
-            <axis xyz="1 0 0"/>
-            <origin xyz="0 0 0"/>
-            <limit effort="1.2" velocity="34" lower="-${2*pi}" upper="${2*pi}"/>
-            <dynamics damping="0.0" friction="0.05"/>
-            <parent link="link4"/>
-            <child link="link5"/>
-        </joint>
-    </xacro:macro>
+    <joint name="joint4" type="revolute">
+      <axis xyz="0 1 0"/>
+      <origin xyz="0.145 0 0"/>
+      <limit effort="1.2" velocity="34" lower="-${0.55*pi}" upper="${0.55*pi}"/>
+      <dynamics damping="0.0" friction="0.05"/>
+      <parent link="link3"/>
+      <child link="link4"/>
+    </joint>
+    <joint name="joint5" type="revolute">
+      <axis xyz="1 0 0"/>
+      <origin xyz="0 0 0"/>
+      <limit effort="1.2" velocity="34" lower="-${2*pi}" upper="${2*pi}"/>
+      <dynamics damping="0.0" friction="0.05"/>
+      <parent link="link4"/>
+      <child link="link5"/>
+    </joint>
+  </xacro:macro>
 </robot>

File: urdf/engineer/hand.urdf.xacro (robot description, xacro)
@@ -1,140 +1,138 @@
 <?xml version="1.0" encoding="utf-8"?>
 <robot xmlns:xacro="http://www.ros.org/wiki/xacro" name="hand">
-    <!-- safety_distance: Minimum safety distance in [m] by which the collision volumes are expanded and which is enforced during robot motions -->
-    <xacro:macro name="hand" params="connected_to:='' xyz:='0 0 0' rpy:='0 0 0' ">
-        <link name="palm">
-            <inertial>
-                <origin xyz="0.01877 0.0475 -0.000028" rpy="0 0 0"/>
-                <mass value="0.406611"/>
-                <inertia ixx="2.719e-3" ixy="-3.243e-4" ixz="228.248e-9" iyy="2.564e-4" iyz="1515.727e-9" izz="2.9e-3"/>
-            </inertial>
-            <visual>
-                <geometry>
-                    <mesh filename="package://rm_description/meshes/engineer/palm.stl" scale="0.001 0.001 0.001"/>
-                </geometry>
-            </visual>
-            <collision>
-                <origin xyz="0.0225 0.0 0" rpy="0 0 0"/>
-                <geometry>
-                    <box size="0.045 0.2658 0.0675"/>
-                </geometry>
-            </collision>
-        </link>
-        <link name="right_finger">
-            <inertial>
-                <origin xyz="0.01491 -0.06058 0" rpy="0 0 0"/>
-                <mass value="0.203967"/>
-                <inertia ixx="1.025e-3" ixy="3.865e-4" ixz="-1.144e-9" iyy="3.051e-4" iyz="4.649e-9" izz="1.295e-3"/>
-            </inertial>
-            <visual>
-                <geometry>
-                    <mesh filename="package://rm_description/meshes/engineer/right_finger.stl"
-                          scale="0.001 0.001 0.001"/>
-                </geometry>
-            </visual>
-            <collision>
-                <origin xyz="0.011 -0.04 0" rpy="0 0 0"/>
-                <geometry>
-                    <box size="0.048 0.026 0.030"/>
-                </geometry>
-            </collision>
-            <collision>
-                <origin xyz="0.0235 -0.0832 0" rpy="0 0 0"/>
-                <geometry>
-                    <box size="0.022 0.1123 0.03"/>
-                </geometry>
-            </collision>
-            <collision>
-                <origin xyz="0.069 -0.13 0" rpy="0 0 0"/>
-                <geometry>
-                    <box size="0.112 0.0157 0.03"/>
-                </geometry>
-            </collision>
-            <collision>
-                <origin xyz="0.105 -0.1232 0" rpy="0 0 0"/>
-                <geometry>
-                    <box size="0.04 0.0323 0.03"/>
-                </geometry>
-            </collision>
-        </link>
-        <link name="left_finger">
-            <inertial>
-                <origin xyz="0.01491 0.061581 0" rpy="0 0 0"/>
-                <mass value="0.203967"/>
-                <inertia ixx="1.053e-3" ixy="-3.865e-4" ixz="-1.144e-9" iyy="3.051e-4" iyz="-4.733e-9" izz="1.323e-3"/>
-            </inertial>
-            <visual>
-                <geometry>
-                    <mesh filename="package://rm_description/meshes/engineer/left_finger.stl"
-                          scale="0.001 0.001 0.001"/>
-                </geometry>
-            </visual>
-            <collision>
-                <origin xyz="0.011 0.04 0" rpy="0 0 0"/>
-                <geometry>
-                    <box size="0.048 0.026 0.030"/>
-                </geometry>
-            </collision>
-            <collision>
-                <origin xyz="0.0235 0.0832 0" rpy="0 0 0"/>
-                <geometry>
-                    <box size="0.022 0.1123 0.03"/>
-                </geometry>
-            </collision>
-            <collision>
-                <origin xyz="0.069 0.13 0" rpy="0 0 0"/>
-                <geometry>
-                    <box size="0.112 0.0157 0.03"/>
-                </geometry>
-            </collision>
-            <collision>
-                <origin xyz="0.105 0.1232 0" rpy="0 0 0"/>
-                <geometry>
-                    <box size="0.04 0.0323 0.03"/>
-                </geometry>
-            </collision>
-        </link>
-        <xacro:unless value="${connected_to == ''}">
-            <joint name="palm_joint" type="fixed">
-                <parent link="${connected_to}"/>
-                <child link="palm"/>
-                <origin xyz="${xyz}" rpy="${rpy}"/>
-            </joint>
-        </xacro:unless>
-        <joint name="right_finger_joint" type="prismatic">
-            <parent link="palm"/>
-            <child link="right_finger"/>
-            <origin xyz="0.032 0 0" rpy="0 0 0"/>
-            <axis xyz="0 1 0"/>
-            <limit effort="588" lower="0.0" upper="0.02" velocity="3.772"/>
-        </joint>
-        <joint name="left_finger_joint" type="prismatic">
-            <parent link="palm"/>
-            <child link="left_finger"/>
-            <origin xyz="0.032 0 0" rpy="0 0 0"/>
-            <axis xyz="0 -1 0"/>
-            <limit effort="588" lower="0.0" upper="0.02" velocity="3.772"/>
-            <mimic joint="right_finger_joint"/>
-        </joint>
-        <transmission name="trans_right_finger_joint">
-            <type>transmission_interface/SimpleTransmission</type>
-            <joint name="right_finger_joint">
-                <hardwareInterface>hardware_interface/EffortJointInterface</hardwareInterface>
-            </joint>
-            <actuator name="right_finger_motor">
-                <hardwareInterface>hardware_interface/EffortJointInterface</hardwareInterface>
-                <mechanicalReduction>1</mechanicalReduction>
-            </actuator>
-        </transmission>
-        <transmission name="trans_left_finger_joint">
-            <type>transmission_interface/SimpleTransmission</type>
-            <joint name="left_finger_joint">
-                <hardwareInterface>hardware_interface/EffortJointInterface</hardwareInterface>
-            </joint>
-            <actuator name="left_finger_motor">
-                <hardwareInterface>hardware_interface/EffortJointInterface</hardwareInterface>
-                <mechanicalReduction>1</mechanicalReduction>
-            </actuator>
-        </transmission>
-    </xacro:macro>
+  <!-- safety_distance: Minimum safety distance in [m] by which the collision volumes are expanded and which is enforced during robot motions -->
+  <xacro:macro name="hand" params="connected_to:='' xyz:='0 0 0' rpy:='0 0 0' ">
+    <link name="palm">
+      <inertial>
+        <origin xyz="0.01877 0.0475 -0.000028" rpy="0 0 0"/>
+        <mass value="0.406611"/>
+        <inertia ixx="2.719e-3" ixy="-3.243e-4" ixz="228.248e-9" iyy="2.564e-4" iyz="1515.727e-9" izz="2.9e-3"/>
+      </inertial>
+      <visual>
+        <geometry>
+          <mesh filename="package://rm_description/meshes/engineer/palm.stl" scale="0.001 0.001 0.001"/>
+        </geometry>
+      </visual>
+      <collision>
+        <origin xyz="0.0225 0.0 0" rpy="0 0 0"/>
+        <geometry>
+          <box size="0.045 0.2658 0.0675"/>
+        </geometry>
+      </collision>
+    </link>
+    <link name="right_finger">
+      <inertial>
+        <origin xyz="0.01491 -0.06058 0" rpy="0 0 0"/>
+        <mass value="0.203967"/>
+        <inertia ixx="1.025e-3" ixy="3.865e-4" ixz="-1.144e-9" iyy="3.051e-4" iyz="4.649e-9" izz="1.295e-3"/>
+      </inertial>
+      <visual>
+        <geometry>
+          <mesh filename="package://rm_description/meshes/engineer/right_finger.stl" scale="0.001 0.001 0.001"/>
+        </geometry>
+      </visual>
+      <collision>
+        <origin xyz="0.011 -0.04 0" rpy="0 0 0"/>
+        <geometry>
+          <box size="0.048 0.026 0.030"/>
+        </geometry>
+      </collision>
+      <collision>
+        <origin xyz="0.0235 -0.0832 0" rpy="0 0 0"/>
+        <geometry>
+          <box size="0.022 0.1123 0.03"/>
+        </geometry>
+      </collision>
+      <collision>
+        <origin xyz="0.069 -0.13 0" rpy="0 0 0"/>
+        <geometry>
+          <box size="0.112 0.0157 0.03"/>
+        </geometry>
+      </collision>
+      <collision>
+        <origin xyz="0.105 -0.1232 0" rpy="0 0 0"/>
+        <geometry>
+          <box size="0.04 0.0323 0.03"/>
+        </geometry>
+      </collision>
+    </link>
+    <link name="left_finger">
+      <inertial>
+        <origin xyz="0.01491 0.061581 0" rpy="0 0 0"/>
+        <mass value="0.203967"/>
+        <inertia ixx="1.053e-3" ixy="-3.865e-4" ixz="-1.144e-9" iyy="3.051e-4" iyz="-4.733e-9" izz="1.323e-3"/>
+      </inertial>
+      <visual>
+        <geometry>
+          <mesh filename="package://rm_description/meshes/engineer/left_finger.stl" scale="0.001 0.001 0.001"/>
+        </geometry>
+      </visual>
+      <collision>
+        <origin xyz="0.011 0.04 0" rpy="0 0 0"/>
+        <geometry>
+          <box size="0.048 0.026 0.030"/>
+        </geometry>
+      </collision>
+      <collision>
+        <origin xyz="0.0235 0.0832 0" rpy="0 0 0"/>
+        <geometry>
+          <box size="0.022 0.1123 0.03"/>
+        </geometry>
+      </collision>
+      <collision>
+        <origin xyz="0.069 0.13 0" rpy="0 0 0"/>
+        <geometry>
+          <box size="0.112 0.0157 0.03"/>
+        </geometry>
+      </collision>
+      <collision>
+        <origin xyz="0.105 0.1232 0" rpy="0 0 0"/>
+        <geometry>
+          <box size="0.04 0.0323 0.03"/>
+        </geometry>
+      </collision>
+    </link>
+    <xacro:unless value="${connected_to == ''}">
+      <joint name="palm_joint" type="fixed">
+        <parent link="${connected_to}"/>
+        <child link="palm"/>
+        <origin xyz="${xyz}" rpy="${rpy}"/>
+      </joint>
+    </xacro:unless>
+    <joint name="right_finger_joint" type="prismatic">
+      <parent link="palm"/>
+      <child link="right_finger"/>
+      <origin xyz="0.032 0 0" rpy="0 0 0"/>
+      <axis xyz="0 1 0"/>
+      <limit effort="588" lower="0.0" upper="0.02" velocity="3.772"/>
+    </joint>
+    <joint name="left_finger_joint" type="prismatic">
+      <parent link="palm"/>
+      <child link="left_finger"/>
+      <origin xyz="0.032 0 0" rpy="0 0 0"/>
+      <axis xyz="0 -1 0"/>
+      <limit effort="588" lower="0.0" upper="0.02" velocity="3.772"/>
+      <mimic joint="right_finger_joint"/>
+    </joint>
+    <transmission name="trans_right_finger_joint">
+      <type>transmission_interface/SimpleTransmission</type>
+      <joint name="right_finger_joint">
+        <hardwareInterface>hardware_interface/EffortJointInterface</hardwareInterface>
+      </joint>
+      <actuator name="right_finger_motor">
+        <hardwareInterface>hardware_interface/EffortJointInterface</hardwareInterface>
+        <mechanicalReduction>1</mechanicalReduction>
+      </actuator>
+    </transmission>
+    <transmission name="trans_left_finger_joint">
+      <type>transmission_interface/SimpleTransmission</type>
+      <joint name="left_finger_joint">
+        <hardwareInterface>hardware_interface/EffortJointInterface</hardwareInterface>
+      </joint>
+      <actuator name="left_finger_motor">
+        <hardwareInterface>hardware_interface/EffortJointInterface</hardwareInterface>
+        <mechanicalReduction>1</mechanicalReduction>
+      </actuator>
+    </transmission>
+  </xacro:macro>
 </robot>
