Commit message: change code style

File: urdf/engineer/arm.urdf.xacro (robot description, xacro)
@@ -1,161 +1,161 @@
 <?xml version="1.0" encoding="utf-8"?>
 <robot xmlns:xacro="http://www.ros.org/wiki/xacro" name="arm">
-  <xacro:macro name="arm" params="connected_to">
-    <!--  link  -->
-    <link name="link1">
-      <inertial>
-        <mass value="1.7056"/>
-        <origin xyz="0.004 0 0.0571"/>
-        <inertia ixx="1.542e-2" ixy="0" ixz="-1.332e-3" iyy="1.028e-2" iyz="0" izz="1.017e-2"/>
-      </inertial>
-      <visual>
-        <origin xyz="0 0 0" rpy="0 0 0"/>
-        <geometry>
-          <mesh filename="package://rm_description/meshes/engineer/link1.stl" scale="0.001 0.001 0.001"/>
-        </geometry>
-      </visual>
-      <collision>
-        <origin xyz="-0.045 0 0.035" rpy="0 0 0"/>
-        <geometry>
-          <box size="0.15 0.106 0.07"/>
-        </geometry>
-      </collision>
-      <collision>
-        <origin xyz="0.040 0 0.1" rpy="0 -0.95993 0"/>
-        <geometry>
-          <box size="0.17 0.106 0.095"/>
-        </geometry>
-      </collision>
-      <collision>
-        <origin xyz="0 0 0.05" rpy="1.5707963 0 0"/>
-        <geometry>
-           <cylinder length="0.188" radius="0.047"/>
-        </geometry>
-      </collision>
-    </link>
-    <link name="link2">
-      <inertial>
-        <mass value="1.4763"/>
-        <origin xyz="0.05652 0 0"/>
-        <inertia ixx="1.976e-3" ixy="5.791e-5" ixz="-2.47366e-7" iyy="8.418e-3" iyz="1.0e-7" izz="8.946e-3"/>
-      </inertial>
-      <visual>
-        <origin xyz="0 0 0" rpy="0 0 0"/>
-        <geometry>
-          <mesh filename="package://rm_description/meshes/engineer/link2.stl" scale="0.001 0.001 0.001"/>
-        </geometry>
-      </visual>
-      <collision>
-        <origin xyz="0.062 0 0"/>
-        <geometry>
-          <box size="0.225 0.096 0.070"/>
-        </geometry>
-      </collision>
-    </link>
-    <link name="link3">
-      <inertial>
-        <mass value="0.5946"/>
-        <origin xyz="0.0471 -0.0094 0.0003"/>
-        <inertia ixx="6.49e-4" ixy="5.036e-5" ixz="-2.372e-5" iyy="2.739e-3" iyz="1.795e-6" izz="3.077e-3"/>
-      </inertial>
-      <visual>
-        <origin xyz="0 0 0" rpy="0 0 0"/>
-        <geometry>
-          <mesh filename="package://rm_description/meshes/engineer/link3.stl" scale="0.001 0.001 0.001"/>
-        </geometry>
-      </visual>
-      <collision>
-        <origin xyz="0.063 0 0"/>
-        <geometry>
-          <box size="0.191 0.084 0.053"/>
-        </geometry>
-      </collision>
-      <collision>
-        <origin xyz="0 0 0" rpy="1.5707963 0 0"/>
-        <geometry>
-          <cylinder length="0.082" radius="0.047"/>
-        </geometry>
-      </collision>
-    </link>
-    <link name="link4">
-      <inertial>
-        <mass value="0.361"/>
-        <origin xyz="0 0 0"/>
-        <inertia ixx="2.593e-4" ixy="5.907e-3" ixz="2.629e-2" iyy="8.662e-5" iyz="0." izz="2.589e-4"/>
-      </inertial>
-      <visual>
-        <origin xyz="0 0 0" rpy="0 0 0"/>
-        <geometry>
-          <mesh filename="package://rm_description/meshes/engineer/link4.stl" scale="0.001 0.001 0.001"/>
-        </geometry>
-      </visual>
-      <collision>
-        <origin xyz="0 0 0" rpy="0 0 0"/>
-        <geometry>
-          <box size="0.0513 0.074 0.0513"/>
-        </geometry>
-      </collision>
-    </link>
-    <link name="link5">
-      <inertial>
-        <mass value="0.249"/>
-        <origin xyz="0.02737 0.0 0.0"/>
-        <inertia ixx="6.090e-5" ixy="7.70024e-7" ixz="7.35489e-7" iyy="2.293e-4" iyz="0." izz=" 2.293e-4"/>
-      </inertial>
-      <visual>
-        <origin xyz="0 0 0" rpy="0 0 0"/>
-        <geometry>
-          <mesh filename="package://rm_description/meshes/engineer/link5.stl" scale="0.001 0.001 0.001"/>
-        </geometry>
-      </visual>
-      <collision>
-        <origin xyz="0.015 0 0" rpy="0 0 0"/>
-        <geometry>
-          <box size="0.056 0.0513 0.0513"/>
-        </geometry>
-      </collision>
-    </link>
-    <!--  joint  -->
-    <joint name="joint1" type="revolute">
-      <axis xyz="0 0 1"/>
-      <origin xyz="0.133 0 0.1"/>
-      <!--      limit not work while type="continuous"-->
-      <limit effort="20" velocity="25" lower="-${pi}" upper="${pi}"/>
-      <dynamics damping="0.0" friction="0.1"/>
-      <parent link="${connected_to}"/>
-      <child link="link1"/>
-    </joint>
-    <joint name="joint2" type="revolute">
-      <axis xyz="0 1 0"/>
-      <origin xyz="0.05909 0 0.1280"/>
-      <limit effort="30" velocity="10" lower="-2.231" upper="0.407"/>
-      <dynamics damping="0.0" friction="0.8"/>
-      <parent link="link1"/>
-      <child link="link2"/>
-    </joint>
-    <joint name="joint3" type="revolute">
-      <axis xyz="0 1 0"/>
-      <origin xyz="0.16 0 0"/>
-      <limit effort="30" velocity="10" lower="-2.1645" upper="2.4078"/>
-      <dynamics damping="0.0" friction="0.5"/>
-      <parent link="link2"/>
-      <child link="link3"/>
-    </joint>
-    <joint name="joint4" type="revolute">
-      <axis xyz="0 1 0"/>
-      <origin xyz="0.145 0 0"/>
-      <limit effort="1.2" velocity="34" lower="-${0.55*pi}" upper="${0.55*pi}"/>
-      <dynamics damping="0.0" friction="0.05"/>
-      <parent link="link3"/>
-      <child link="link4"/>
-    </joint>
-    <joint name="joint5" type="revolute">
-      <axis xyz="1 0 0"/>
-      <origin xyz="0 0 0"/>
-      <limit effort="1.2" velocity="34" lower="-${2*pi}" upper="${2*pi}"/>
-      <dynamics damping="0.0" friction="0.05"/>
-      <parent link="link4"/>
-      <child link="link5"/>
-    </joint>
-  </xacro:macro>
+    <xacro:macro name="arm" params="connected_to">
+        <!--  link  -->
+        <link name="link1">
+            <inertial>
+                <mass value="1.7056"/>
+                <origin xyz="0.004 0 0.0571"/>
+                <inertia ixx="1.542e-2" ixy="0" ixz="-1.332e-3" iyy="1.028e-2" iyz="0" izz="1.017e-2"/>
+            </inertial>
+            <visual>
+                <origin xyz="0 0 0" rpy="0 0 0"/>
+                <geometry>
+                    <mesh filename="package://rm_description/meshes/engineer/link1.stl" scale="0.001 0.001 0.001"/>
+                </geometry>
+            </visual>
+            <collision>
+                <origin xyz="-0.045 0 0.035" rpy="0 0 0"/>
+                <geometry>
+                    <box size="0.15 0.106 0.07"/>
+                </geometry>
+            </collision>
+            <collision>
+                <origin xyz="0.040 0 0.1" rpy="0 -0.95993 0"/>
+                <geometry>
+                    <box size="0.17 0.106 0.095"/>
+                </geometry>
+            </collision>
+            <collision>
+                <origin xyz="0 0 0.05" rpy="1.5707963 0 0"/>
+                <geometry>
+                    <cylinder length="0.188" radius="0.047"/>
+                </geometry>
+            </collision>
+        </link>
+        <link name="link2">
+            <inertial>
+                <mass value="1.4763"/>
+                <origin xyz="0.05652 0 0"/>
+                <inertia ixx="1.976e-3" ixy="5.791e-5" ixz="-2.47366e-7" iyy="8.418e-3" iyz="1.0e-7" izz="8.946e-3"/>
+            </inertial>
+            <visual>
+                <origin xyz="0 0 0" rpy="0 0 0"/>
+                <geometry>
+                    <mesh filename="package://rm_description/meshes/engineer/link2.stl" scale="0.001 0.001 0.001"/>
+                </geometry>
+            </visual>
+            <collision>
+                <origin xyz="0.062 0 0"/>
+                <geometry>
+                    <box size="0.225 0.096 0.070"/>
+                </geometry>
+            </collision>
+        </link>
+        <link name="link3">
+            <inertial>
+                <mass value="0.5946"/>
+                <origin xyz="0.0471 -0.0094 0.0003"/>
+                <inertia ixx="6.49e-4" ixy="5.036e-5" ixz="-2.372e-5" iyy="2.739e-3" iyz="1.795e-6" izz="3.077e-3"/>
+            </inertial>
+            <visual>
+                <origin xyz="0 0 0" rpy="0 0 0"/>
+                <geometry>
+                    <mesh filename="package://rm_description/meshes/engineer/link3.stl" scale="0.001 0.001 0.001"/>
+                </geometry>
+            </visual>
+            <collision>
+                <origin xyz="0.063 0 0"/>
+                <geometry>
+                    <box size="0.191 0.084 0.053"/>
+                </geometry>
+            </collision>
+            <collision>
+                <origin xyz="0 0 0" rpy="1.5707963 0 0"/>
+                <geometry>
+                    <cylinder length="0.082" radius="0.047"/>
+                </geometry>
+            </collision>
+        </link>
+        <link name="link4">
+            <inertial>
+                <mass value="0.361"/>
+                <origin xyz="0 0 0"/>
+                <inertia ixx="2.593e-4" ixy="5.907e-3" ixz="2.629e-2" iyy="8.662e-5" iyz="0." izz="2.589e-4"/>
+            </inertial>
+            <visual>
+                <origin xyz="0 0 0" rpy="0 0 0"/>
+                <geometry>
+                    <mesh filename="package://rm_description/meshes/engineer/link4.stl" scale="0.001 0.001 0.001"/>
+                </geometry>
+            </visual>
+            <collision>
+                <origin xyz="0 0 0" rpy="0 0 0"/>
+                <geometry>
+                    <box size="0.0513 0.074 0.0513"/>
+                </geometry>
+            </collision>
+        </link>
+        <link name="link5">
+            <inertial>
+                <mass value="0.249"/>
+                <origin xyz="0.02737 0.0 0.0"/>
+                <inertia ixx="6.090e-5" ixy="7.70024e-7" ixz="7.35489e-7" iyy="2.293e-4" iyz="0." izz=" 2.293e-4"/>
+            </inertial>
+            <visual>
+                <origin xyz="0 0 0" rpy="0 0 0"/>
+                <geometry>
+                    <mesh filename="package://rm_description/meshes/engineer/link5.stl" scale="0.001 0.001 0.001"/>
+                </geometry>
+            </visual>
+            <collision>
+                <origin xyz="0.015 0 0" rpy="0 0 0"/>
+                <geometry>
+                    <box size="0.056 0.0513 0.0513"/>
+                </geometry>
+            </collision>
+        </link>
+        <!--  joint  -->
+        <joint name="joint1" type="revolute">
+            <axis xyz="0 0 1"/>
+            <origin xyz="0.133 0 0.1"/>
+            <!--      limit not work while type="continuous"-->
+            <limit effort="20" velocity="25" lower="-${pi}" upper="${pi}"/>
+            <dynamics damping="0.0" friction="0.1"/>
+            <parent link="${connected_to}"/>
+            <child link="link1"/>
+        </joint>
+        <joint name="joint2" type="revolute">
+            <axis xyz="0 1 0"/>
+            <origin xyz="0.05909 0 0.1280"/>
+            <limit effort="30" velocity="10" lower="-2.231" upper="0.407"/>
+            <dynamics damping="0.0" friction="0.8"/>
+            <parent link="link1"/>
+            <child link="link2"/>
+        </joint>
+        <joint name="joint3" type="revolute">
+            <axis xyz="0 1 0"/>
+            <origin xyz="0.16 0 0"/>
+            <limit effort="30" velocity="10" lower="-2.1645" upper="2.4078"/>
+            <dynamics damping="0.0" friction="0.5"/>
+            <parent link="link2"/>
+            <child link="link3"/>
+        </joint>
+        <joint name="joint4" type="revolute">
+            <axis xyz="0 1 0"/>
+            <origin xyz="0.145 0 0"/>
+            <limit effort="1.2" velocity="34" lower="-${0.55*pi}" upper="${0.55*pi}"/>
+            <dynamics damping="0.0" friction="0.05"/>
+            <parent link="link3"/>
+            <child link="link4"/>
+        </joint>
+        <joint name="joint5" type="revolute">
+            <axis xyz="1 0 0"/>
+            <origin xyz="0 0 0"/>
+            <limit effort="1.2" velocity="34" lower="-${2*pi}" upper="${2*pi}"/>
+            <dynamics damping="0.0" friction="0.05"/>
+            <parent link="link4"/>
+            <child link="link5"/>
+        </joint>
+    </xacro:macro>
 </robot>

Commit message: Change the hand collision

File: urdf/engineer/arm.urdf.xacro (robot description, xacro)
@@ -145,5 +145,5 @@
             <axis xyz="0 1 0"/>
             <origin xyz="0.145 0 0"/>
-            <limit effort="1.2" velocity="34" lower="-${0.55*pi}" upper="${0.55*pi}"/>
+            <limit effort="2.4" velocity="34" lower="-${0.55*pi}" upper="${0.55*pi}"/>
             <dynamics damping="0.0" friction="0.05"/>
             <parent link="link3"/>

File: urdf/engineer/hand.urdf.xacro (robot description, xacro)
@@ -52,13 +52,7 @@
             </collision>
             <collision>
-                <origin xyz="0.069 -0.13 0" rpy="0 0 0"/>
+                <origin xyz="0.069 -0.12 0" rpy="0 0 0"/>
                 <geometry>
-                    <box size="0.112 0.0157 0.03"/>
-                </geometry>
-            </collision>
-            <collision>
-                <origin xyz="0.105 -0.1232 0" rpy="0 0 0"/>
-                <geometry>
-                    <box size="0.04 0.0323 0.03"/>
+                    <box size="0.112 0.03 0.03"/>
                 </geometry>
             </collision>
@@ -89,13 +83,7 @@
             </collision>
             <collision>
-                <origin xyz="0.069 0.13 0" rpy="0 0 0"/>
+                <origin xyz="0.069 0.12 0" rpy="0 0 0"/>
                 <geometry>
-                    <box size="0.112 0.0157 0.03"/>
-                </geometry>
-            </collision>
-            <collision>
-                <origin xyz="0.105 0.1232 0" rpy="0 0 0"/>
-                <geometry>
-                    <box size="0.04 0.0323 0.03"/>
+                    <box size="0.112 0.03 0.03"/>
                 </geometry>
             </collision>
@@ -159,4 +147,20 @@
                 </plugin>
             </gazebo>
+            <gazebo reference="right_finger">
+                <self_collide>1</self_collide>
+                <mu1 value="200000.0"/>
+                <mu2 value="200000.0"/>
+                <kp value="1000000.0"/>
+                <kd value="100.0"/>
+                <material>Gazebo/Black</material>
+            </gazebo>
+            <gazebo reference="left_finger">
+                <self_collide>1</self_collide>
+                <mu1 value="200000.0"/>
+                <mu2 value="200000.0"/>
+                <kp value="1000000.0"/>
+                <kd value="100.0"/>
+                <material>Gazebo/Black</material>
+            </gazebo>
         </xacro:if>
         <transmission name="trans_right_finger_joint">

Commit message: add camera.urdf.xacro

File: urdf/engineer/arm.urdf.xacro (robot description, xacro)
@@ -101,5 +101,5 @@
                 <mass value="0.249"/>
                 <origin xyz="0.02737 0.0 0.0"/>
-                <inertia ixx="6.090e-5" ixy="7.70024e-7" ixz="7.35489e-7" iyy="2.293e-4" iyz="0." izz=" 2.293e-4"/>
+                <inertia ixx="6.090e-5" ixy="7.70024e-7" ixz="7.35489e-7" iyy="2.293e-4" iyz="0." izz="2.293e-4"/>
             </inertial>
             <visual>

File: urdf/engineer/chassis.urdf.xacro (robot description, xacro)
@@ -12,5 +12,5 @@
                 <mass value="28.19"/>
                 <origin xyz="-0.0206 -0.00126 -0.0164"/>
-                <inertia ixx="1.32e+0" ixy="-8.378e-2" ixz="6.28e-2" iyy=" 1.549e+0"
+                <inertia ixx="1.32e+0" ixy="-8.378e-2" ixz="6.28e-2" iyy="1.549e+0"
                          iyz="5.948e-2" izz="2.024e+0"/>
             </inertial>

Commit message: uate engineer uedf pareters

File: urdf/engineer/arm.urdf.xacro (robot description, xacro)
@@ -5,7 +5,7 @@
         <link name="link1">
             <inertial>
-                <mass value="1.7056"/>
-                <origin xyz="0.004 0 0.0571"/>
-                <inertia ixx="1.542e-2" ixy="0" ixz="-1.332e-3" iyy="1.028e-2" iyz="0" izz="1.017e-2"/>
+                <mass value="1.768"/>
+                <origin xyz="-0.005 0.046 0.0"/>
+                <inertia ixx="9.816e-3" ixy="-2.523e-4" ixz="7.839e-6" iyy="9.203e-3" iyz="9.389e-5" izz="3.735e-3"/>
             </inertial>
             <visual>
@@ -36,7 +36,7 @@
         <link name="link2">
             <inertial>
-                <mass value="1.4763"/>
-                <origin xyz="0.05652 0 0"/>
-                <inertia ixx="1.976e-3" ixy="5.791e-5" ixz="-2.47366e-7" iyy="8.418e-3" iyz="1.0e-7" izz="8.946e-3"/>
+                <mass value="1.256"/>
+                <origin xyz="0.057 0.002 0"/>
+                <inertia ixx="1.678e-3" ixy="1.267e-5" ixz="-4.26e-7" iyy="3.761e-3" iyz="1.345e-6" izz="4.111e-3"/>
             </inertial>
             <visual>
@@ -55,7 +55,7 @@
         <link name="link3">
             <inertial>
-                <mass value="0.5946"/>
-                <origin xyz="0.0471 -0.0094 0.0003"/>
-                <inertia ixx="6.49e-4" ixy="5.036e-5" ixz="-2.372e-5" iyy="2.739e-3" iyz="1.795e-6" izz="3.077e-3"/>
+                <mass value="1.139"/>
+                <origin xyz="0.081 -0.0 0.022"/>
+                <inertia ixx="9.633e-4" ixy="-2.836e-4" ixz="-5.244e-4" iyy="2.739e-3" iyz="-8.552e-5" izz="2.963e-3"/>
             </inertial>
             <visual>
@@ -80,7 +80,7 @@
         <link name="link4">
             <inertial>
-                <mass value="0.361"/>
-                <origin xyz="0 0 0"/>
-                <inertia ixx="2.593e-4" ixy="5.907e-3" ixz="2.629e-2" iyy="8.662e-5" iyz="0." izz="2.589e-4"/>
+                <mass value="0.362"/>
+                <origin xyz="0.035 -0.027 0.06"/>
+                <inertia ixx="8.647e-4" ixy="-5.427e-5" ixz="-1.425e-4" iyy="8.477e-4" iyz="-2.555e-4" izz="5.668e-4"/>
             </inertial>
             <visual>
@@ -99,7 +99,7 @@
         <link name="link5">
             <inertial>
-                <mass value="0.249"/>
-                <origin xyz="0.02737 0.0 0.0"/>
-                <inertia ixx="6.090e-5" ixy="7.70024e-7" ixz="7.35489e-7" iyy="2.293e-4" iyz="0." izz="2.293e-4"/>
+                <mass value="0.85"/>
+                <origin xyz="-0.061 0.0 0.0"/>
+                <inertia ixx="1.761e-4" ixy="6.99e-7" ixz="1.26e-7" iyy="5.874e-4" iyz="2.72e-7" izz="5.863e-4"/>
             </inertial>
             <visual>
@@ -119,5 +119,5 @@
         <joint name="joint1" type="revolute">
             <axis xyz="0 0 1"/>
-            <origin xyz="0.133 0 0.1"/>
+            <origin xyz="0.133 0 1" rpy="1.57 0 0"/>
             <!--      limit not work while type="continuous"-->
             <limit effort="20" velocity="25" lower="-${pi}" upper="${pi}"/>
@@ -128,5 +128,5 @@
         <joint name="joint2" type="revolute">
             <axis xyz="0 1 0"/>
-            <origin xyz="0.05909 0 0.1280"/>
+            <origin xyz="0.005 0.128 0" rpy="-1.57 0 0"/>
             <limit effort="30" velocity="10" lower="-2.231" upper="0.407"/>
             <dynamics damping="0.0" friction="0.8"/>
@@ -136,5 +136,5 @@
         <joint name="joint3" type="revolute">
             <axis xyz="0 1 0"/>
-            <origin xyz="0.16 0 0"/>
+            <origin xyz="0.165 0 0" rpy="0 0 0"/>
             <limit effort="30" velocity="10" lower="-2.1645" upper="2.4078"/>
             <dynamics damping="0.0" friction="0.5"/>
@@ -144,5 +144,5 @@
         <joint name="joint4" type="revolute">
             <axis xyz="0 1 0"/>
-            <origin xyz="0.145 0 0"/>
+            <origin xyz="0.106 0 0.028"/>
             <limit effort="2.4" velocity="34" lower="-${0.55*pi}" upper="${0.55*pi}"/>
             <dynamics damping="0.0" friction="0.05"/>
@@ -152,5 +152,5 @@
         <joint name="joint5" type="revolute">
             <axis xyz="1 0 0"/>
-            <origin xyz="0 0 0"/>
+            <origin xyz="0.097 0 0.055"/>
             <limit effort="1.2" velocity="34" lower="-${pi}" upper="${pi}"/>
             <dynamics damping="0.0" friction="0.05"/>

File: urdf/engineer/engineer.urdf.xacro (robot description, xacro)
@@ -15,5 +15,5 @@
         <xacro:arm_transmission simulation="$(arg use_simulation)"/>
         <xacro:include filename="$(find rm_description)/urdf/engineer/hand.urdf.xacro"/>
-        <xacro:hand connected_to="link5" xyz="0.039 0 0" simulation="$(arg use_simulation)"/>
+        <xacro:hand connected_to="link5" xyz="-0.014 0 0" rpy="0 1.57 0" simulation="$(arg use_simulation)"/>
     </xacro:if>
     <xacro:if value="$(arg use_simulation)">

File: urdf/engineer/hand.urdf.xacro (robot description, xacro)
@@ -11,7 +11,7 @@
         <link name="palm">
             <inertial>
-                <origin xyz="0.01877 0.0475 -0.000028" rpy="0 0 0"/>
-                <mass value="0.406611"/>
-                <inertia ixx="2.719e-3" ixy="-3.243e-4" ixz="228.248e-9" iyy="2.564e-4" iyz="1515.727e-9" izz="2.9e-3"/>
+                <mass value="0.695"/>
+                <origin xyz="0.0 0.0 0.024" rpy="0 0 0"/>
+                <inertia ixx="5.042e-4" ixy="1.20e-7" ixz="-3.142e-6" iyy="2.444e-4" iyz="1.18e-7" izz="4.945e-4"/>
             </inertial>
             <visual>
@@ -29,7 +29,7 @@
         <link name="right_finger">
             <inertial>
-                <origin xyz="0.01491 -0.06058 0" rpy="0 0 0"/>
-                <mass value="0.203967"/>
-                <inertia ixx="1.025e-3" ixy="3.865e-4" ixz="-1.144e-9" iyy="3.051e-4" iyz="4.649e-9" izz="1.295e-3"/>
+                <origin xyz="0.0 0.075 0.021" rpy="0 0 0"/>
+                <mass value="0.284"/>
+                <inertia ixx="7.653e-4" ixy="1.922e-5" ixz="1.589e-5" iyy="3.805e-4" iyz="-3.052e-4" izz="4.364e-4"/>
             </inertial>
             <visual>
@@ -66,7 +66,7 @@
         <link name="left_finger">
             <inertial>
-                <origin xyz="0.01491 0.061581 0" rpy="0 0 0"/>
-                <mass value="0.203967"/>
-                <inertia ixx="1.053e-3" ixy="-3.865e-4" ixz="-1.144e-9" iyy="3.051e-4" iyz="-4.733e-9" izz="1.323e-3"/>
+                <origin xyz="0.0 -0.075 0.021" rpy="0 0 0"/>
+                <mass value="0.284"/>
+                <inertia ixx="7.653e-4" ixy="1.922e-5" ixz="-1.589e-5" iyy="3.805e-4" iyz="3.052e-4" izz="4.364e-4"/>
             </inertial>
             <visual>
@@ -131,5 +131,5 @@
             <parent link="palm"/>
             <child link="right_finger"/>
-            <origin xyz="0.032 0 0" rpy="0 0 0"/>
+            <origin xyz="0 0 0.045" rpy="0 0 0"/>
             <axis xyz="0 1 0"/>
             <limit effort="588" lower="0.0" upper="0.03" velocity="3.772"/>
@@ -138,5 +138,5 @@
             <parent link="palm"/>
             <child link="left_finger"/>
-            <origin xyz="0.032 0 0" rpy="0 0 0"/>
+            <origin xyz="0 0 0.045" rpy="0 0 0"/>
             <axis xyz="0 -1 0"/>
             <limit effort="588" lower="0.0" upper="0.03" velocity="3.772"/>
