Commit message: uate engineer <collision> uedf pareters

File: urdf/engineer/arm.urdf.xacro (robot description, xacro)
@@ -16,19 +16,25 @@
             </visual>
             <collision>
-                <origin xyz="-0.045 0 0.035" rpy="0 0 0"/>
+                <origin xyz="0.004 0.071 0" rpy="0 0 0"/>
                 <geometry>
-                    <box size="0.15 0.106 0.07"/>
+                    <box size="0.088 0.142 0.106"/>
                 </geometry>
             </collision>
             <collision>
-                <origin xyz="0.040 0 0.1" rpy="0 -0.95993 0"/>
+                <origin xyz="-0.032 0.068 0" rpy="0 0 -0.593"/>
                 <geometry>
-                    <box size="0.17 0.106 0.095"/>
+                    <box size="0.097 0.14 0.106"/>
                 </geometry>
             </collision>
             <collision>
-                <origin xyz="0 0 0.05" rpy="1.5707963 0 0"/>
+                <origin xyz="-0.002 0.04 0 " rpy="0 0 0"/>
                 <geometry>
                     <cylinder length="0.188" radius="0.047"/>
+                </geometry>
+            </collision>
+            <collision>
+                <origin xyz="0.005 0.128 0" rpy="0 0 0"/>
+                <geometry>
+                    <cylinder length="0.106" radius="0.047"/>
                 </geometry>
             </collision>
@@ -47,7 +53,13 @@
             </visual>
             <collision>
-                <origin xyz="0.062 0 0"/>
+                <origin xyz="0.072 0 0"/>
                 <geometry>
-                    <box size="0.225 0.096 0.070"/>
+                    <box size="0.215 0.096 0.075"/>
+                </geometry>
+            </collision>
+            <collision>
+                <origin xyz="0.165 0 0" rpy="1.5707963 0 0"/>
+                <geometry>
+                    <cylinder length="0.096" radius="0.047"/>
                 </geometry>
             </collision>
@@ -66,13 +78,13 @@
             </visual>
             <collision>
-                <origin xyz="0.063 0 0"/>
+                <origin xyz="0.006 0 0.007" rpy="0 0.8726 0"/>
                 <geometry>
-                    <box size="0.191 0.084 0.053"/>
+                    <box size="0.072 0.066 0.072"/>
                 </geometry>
             </collision>
             <collision>
-                <origin xyz="0 0 0" rpy="1.5707963 0 0"/>
+                <origin xyz="0.066 0 0.027"/>
                 <geometry>
-                    <cylinder length="0.082" radius="0.047"/>
+                    <box size="0.135 0.066 0.062"/>
                 </geometry>
             </collision>
@@ -91,7 +103,13 @@
             </visual>
             <collision>
-                <origin xyz="0 0 0" rpy="0 0 0"/>
+                <origin xyz="0.02 -0.015 0.017" rpy="0 0.8028 0"/>
                 <geometry>
-                    <box size="0.0513 0.074 0.0513"/>
+                    <box size="0.0582 0.092 0.099"/>
+                </geometry>
+            </collision>
+            <collision>
+                <origin xyz="0.0347 -0.015 0.071"/>
+                <geometry>
+                    <box size="0.08 0.094 0.083"/>
                 </geometry>
             </collision>
@@ -110,7 +128,7 @@
             </visual>
             <collision>
-                <origin xyz="0.015 0 0" rpy="0 0 0"/>
+                <origin xyz="-0.054 0 0" rpy="0 1.57 0"/>
                 <geometry>
-                    <box size="0.056 0.0513 0.0513"/>
+                    <cylinder length="0.108" radius="0.021"/>
                 </geometry>
             </collision>
@@ -118,5 +136,5 @@
         <!--  joint  -->
         <joint name="joint1" type="revolute">
-            <axis xyz="0 0 1"/>
+            <axis xyz="0 1 0"/>
             <origin xyz="0.133 0 1" rpy="1.57 0 0"/>
             <!--      limit not work while type="continuous"-->

File: urdf/engineer/hand.urdf.xacro (robot description, xacro)
@@ -21,7 +21,7 @@
             </visual>
             <collision>
-                <origin xyz="0.0225 0.0 0" rpy="0 0 0"/>
+                <origin xyz="0 0 0.027" rpy="0 0 0"/>
                 <geometry>
-                    <box size="0.045 0.2658 0.0675"/>
+                    <box size="0.055 0.267 0.06"/>
                 </geometry>
             </collision>
@@ -40,25 +40,19 @@
             </visual>
             <collision>
-                <origin xyz="0.011 -0.04 0" rpy="0 0 0"/>
+                <origin xyz="0.0 0.046 0.005" rpy="0 0 0"/>
                 <geometry>
-                    <box size="0.048 0.026 0.030"/>
+                    <box size="0.030 0.027 0.063"/>
                 </geometry>
             </collision>
             <collision>
-                <origin xyz="0.0235 -0.0832 0" rpy="0 0 0"/>
+                <origin xyz="0.0 0.091 0.025" rpy="0 0 0"/>
                 <geometry>
-                    <box size="0.022 0.1123 0.03"/>
+                    <box size="0.03 0.109 0.022"/>
                 </geometry>
             </collision>
             <collision>
-                <origin xyz="0.069 -0.13 0" rpy="0 0 0"/>
+                <origin xyz="0.0 0.133 0.07" rpy="0 0 0"/>
                 <geometry>
-                    <box size="0.112 0.0157 0.03"/>
-                </geometry>
-            </collision>
-            <collision>
-                <origin xyz="0.105 -0.1232 0" rpy="0 0 0"/>
-                <geometry>
-                    <box size="0.04 0.0323 0.03"/>
+                    <box size="0.030 0.017 0.112"/>
                 </geometry>
             </collision>
@@ -77,19 +71,19 @@
             </visual>
             <collision>
-                <origin xyz="0.011 0.04 0" rpy="0 0 0"/>
+                <origin xyz="0.0 -0.043 0.005" rpy="0 0 0"/>
                 <geometry>
-                    <box size="0.048 0.026 0.030"/>
+                    <box size="0.030 0.027 0.063"/>
                 </geometry>
             </collision>
             <collision>
-                <origin xyz="0.0235 0.0832 0" rpy="0 0 0"/>
+                <origin xyz="0.0 -0.088 0.025" rpy="0 0 0"/>
                 <geometry>
-                    <box size="0.022 0.1123 0.03"/>
+                    <box size="0.03 0.109 0.022"/>
                 </geometry>
             </collision>
             <collision>
-                <origin xyz="0.069 0.12 0" rpy="0 0 0"/>
+                <origin xyz="0.0 -0.129 0.07" rpy="0 0 0"/>
                 <geometry>
-                    <box size="0.112 0.03 0.03"/>
+                    <box size="0.030 0.017 0.112"/>
                 </geometry>
             </collision>

Commit message: update engineer  collision and wheel position

File: urdf/engineer/arm.urdf.xacro (robot description, xacro)
@@ -137,5 +137,5 @@
         <joint name="joint1" type="revolute">
             <axis xyz="0 1 0"/>
-            <origin xyz="0.133 0 1" rpy="1.57 0 0"/>
+            <origin xyz="0.122 0 0.124" rpy="1.57 0 0"/>
             <!--      limit not work while type="continuous"-->
             <limit effort="20" velocity="10" lower="-${pi}" upper="${pi}"/>

File: urdf/engineer/chassis.urdf.xacro (robot description, xacro)
@@ -2,7 +2,9 @@
     <xacro:include filename="$(find rm_description)/urdf/common/mecanum_wheel.urdf.xacro"/>
     <!-- https://upload.wikimedia.org/wikipedia/commons/5/52/Wheelbase_and_Track.png -->
-    <xacro:property name="wheel_track" value="0.380"/>
-    <xacro:property name="wheel_base" value="0.420"/>
-    <xacro:property name="wheel_offset_z" value="-0.1090"/>
+    <xacro:property name="wheel_front" value="0.091"/>
+    <xacro:property name="wheel_back" value="-0.178"/>
+    <xacro:property name="wheel_left" value="-0.245"/>
+    <xacro:property name="wheel_right" value="0.245"/>
+    <xacro:property name="wheel_offset_z" value="-0.04"/>
     <xacro:property name="wheel_joint_damping" value="1.0"/>
     <xacro:property name="wheel_joint_friction" value="1.0"/>
@@ -58,5 +60,5 @@
             </collision>
             <collision>
-                <origin xyz="-0.0866 0.238 0.2672" rpy="0 0 -0.5061455"/>
+                <origin xyz="-0.08 0.243 0.258" rpy="0 0 -0.5061455"/>
                 <geometry>
                     <box size="0.08 0.0217 0.3033"/>
@@ -64,5 +66,5 @@
             </collision>
             <collision>
-                <origin xyz="-0.2041 0.1846 0.25833" rpy="0 0 1.0646508"/>
+                <origin xyz="-0.21 0.19 0.25833" rpy="0 0 1.0646508"/>
                 <geometry>
                     <box size="0.08 0.0217 0.3033"/>
@@ -70,5 +72,5 @@
             </collision>
             <collision>
-                <origin xyz="-0.1873 0.0566 0.2672" rpy="0 0 -0.5061455"/>
+                <origin xyz="-0.19 0.05 0.258" rpy="0 0 -0.5061455"/>
                 <geometry>
                     <box size="0.08 0.0217 0.3033"/>
@@ -76,5 +78,5 @@
             </collision>
             <collision>
-                <origin xyz="-0.139 0.0847 0.228" rpy="0 0 1.0646508"/>
+                <origin xyz="-0.023 0.0847 0.228" rpy="0 0 1.0646508"/>
                 <geometry>
                     <box size="0.080 0.003 0.250"/>
@@ -83,17 +85,17 @@
         </link>
         <xacro:mecanum_wheel prefix="left_front" connected_to="base_link"
-                             wheel_x_offset="${wheel_track/2}" wheel_y_offset="${wheel_base/2}"
+                             wheel_x_offset="${wheel_front}" wheel_y_offset="${wheel_left}"
                              wheel_z_offset="${wheel_offset_z}"
                              reflect="1" roller_type="${roller_type}"/>
         <xacro:mecanum_wheel prefix="right_front" connected_to="base_link"
-                             wheel_x_offset="${wheel_track/2}" wheel_y_offset="${-wheel_base/2}"
+                             wheel_x_offset="${wheel_front}" wheel_y_offset="${wheel_right}"
                              wheel_z_offset="${wheel_offset_z}"
                              reflect="-1" roller_type="${roller_type}"/>
         <xacro:mecanum_wheel prefix="left_back" connected_to="base_link"
-                             wheel_x_offset="${-wheel_track/2}" wheel_y_offset="${wheel_base/2}"
+                             wheel_x_offset="${wheel_back}" wheel_y_offset="${wheel_left}"
                              wheel_z_offset="${wheel_offset_z}"
                              reflect="-1" roller_type="${roller_type}"/>
         <xacro:mecanum_wheel prefix="right_back" connected_to="base_link"
-                             wheel_x_offset="${-wheel_track/2}" wheel_y_offset="${-wheel_base/2}"
+                             wheel_x_offset="${wheel_back}" wheel_y_offset="${wheel_right}"
                              wheel_z_offset="${wheel_offset_z}"
                              reflect="1" roller_type="${roller_type}"/>

File: urdf/engineer/engineer.urdf.xacro (robot description, xacro)
@@ -17,5 +17,5 @@
         <xacro:hand connected_to="link5" xyz="-0.014 0 0" rpy="0 1.57 0" simulation="$(arg use_simulation)"/>
         <xacro:include filename="$(find rm_description)/urdf/engineer/mast.urdf.xacro"/>
-        <xacro:mast connected_to="link1" xyz="-0.076 0.484 0.108 " rpy="-1.57 0 0" simulation="$(arg use_simulation)"/>
+        <xacro:mast connected_to="link1" xyz="-0.076 0.582 0.108 " rpy="-1.57 0 0" simulation="$(arg use_simulation)"/>
     </xacro:if>
     <xacro:if value="$(arg use_simulation)">

File: urdf/engineer/hand.urdf.xacro (robot description, xacro)
@@ -89,30 +89,4 @@
             </collision>
         </link>
-        <link name="camera">
-            <inertial>
-                <mass value="0.05"/>
-                <origin xyz="0 0 0"/>
-                <inertia ixx="1.271e-3" ixy="2.07e-7" ixz="8.854e-6" iyy="5.190e-4" iyz="1.001e-6" izz="9.976e-4"/>
-            </inertial>
-            <visual>
-                <origin xyz=" 0 0 0 " rpy="0 0 0"/>
-                <geometry>
-                    <box size="0.022 0.021 0.0226"/>
-                </geometry>
-                <material name="Black"/>
-            </visual>
-            <collision>
-                <origin xyz="0.0 0.0 0.0" rpy="0 0 0"/>
-                <geometry>
-                    <box size="0.01 0.04 0.04"/>
-                </geometry>
-            </collision>
-        </link>
-        <joint name="camera_joint" type="fixed">
-            <parent link="palm"/>
-            <child link="camera"/>
-            <origin xyz="0.055 -0.085 0.0962" rpy="0 0 0"/>
-            <axis xyz="0 0 1"/>
-        </joint>
         <xacro:unless value="${connected_to == ''}">
             <joint name="palm_joint" type="fixed">

File: urdf/engineer/mast.urdf.xacro (robot description, xacro)
@@ -71,5 +71,6 @@
                 <child link="mast"/>
                 <axis xyz="0 0 1"/>
-                <limit effort="1.2" velocity="13.82" lower="-1e10" upper="1e10"/>
+                <dynamics damping="0.0" friction="0.8"/>
+                <limit effort="1.2" velocity="13.82" lower="-0.175" upper="0"/>
             </joint>
         </xacro:unless>

Commit message: del one link1 collision

File: urdf/engineer/arm.urdf.xacro (robot description, xacro)
@@ -19,10 +19,4 @@
                 <geometry>
                     <box size="0.088 0.142 0.106"/>
-                </geometry>
-            </collision>
-            <collision>
-                <origin xyz="-0.002 0.04 0 " rpy="0 0 0"/>
-                <geometry>
-                    <cylinder length="0.188" radius="0.047"/>
                 </geometry>
             </collision>

File: urdf/engineer/mast.urdf.xacro (robot description, xacro)
@@ -17,5 +17,5 @@
                 <origin xyz="0.004 0 -0.259" rpy="0 0 0"/>
                 <geometry>
-                    <box size="0.035 0.035 0.4"/>
+                    <box size="0.053 0.035 0.45"/>
                 </geometry>
             </collision>

Commit message: Change engineer's limit

File: urdf/engineer/arm.urdf.xacro (robot description, xacro)
@@ -127,5 +127,5 @@
             <origin xyz="0.122 0 0.124" rpy="1.57 0 0"/>
             <!--      limit not work while type="continuous"-->
-            <limit effort="20" velocity="10" lower="-${pi}" upper="${pi}"/>
+            <limit effort="20" velocity="10" lower="-0.80" upper="5.20"/>
             <dynamics damping="0.0" friction="0.1"/>
             <parent link="${connected_to}"/>
@@ -135,5 +135,5 @@
             <axis xyz="0 1 0"/>
             <origin xyz="0.005 0.128 0" rpy="-1.57 0 0"/>
-            <limit effort="60" velocity="10" lower="-2.5249" upper="0.042903"/>
+            <limit effort="60" velocity="10" lower="-1.87" upper="-0.12"/>
             <dynamics damping="0.0" friction="0.8"/>
             <parent link="link1"/>
@@ -151,5 +151,5 @@
             <axis xyz="0 1 0"/>
             <origin xyz="0.106 0 0.028"/>
-            <limit effort="7" velocity="30" lower="-0.21556" upper="2.6459"/>
+            <limit effort="7" velocity="30" lower="-0.2252557429" upper="0.108979611"/>
             <dynamics damping="0.0" friction="0.5"/>
             <parent link="link3"/>

Commit message: Update engineer's limit

File: urdf/engineer/arm.urdf.xacro (robot description, xacro)
@@ -151,5 +151,5 @@
             <axis xyz="0 1 0"/>
             <origin xyz="0.106 0 0.028"/>
-            <limit effort="7" velocity="30" lower="-0.2252557429" upper="0.108979611"/>
+            <limit effort="7" velocity="30" lower="-0.24430838" upper="2.65452132"/>
             <dynamics damping="0.0" friction="0.5"/>
             <parent link="link3"/>

Commit message: Update engineer's limit

File: urdf/engineer/arm.urdf.xacro (robot description, xacro)
@@ -127,5 +127,5 @@
             <origin xyz="0.122 0 0.124" rpy="1.57 0 0"/>
             <!--      limit not work while type="continuous"-->
-            <limit effort="20" velocity="10" lower="-0.80" upper="5.20"/>
+            <limit effort="20" velocity="10" lower="-0.8507492" upper="5.2558426"/>
             <dynamics damping="0.0" friction="0.1"/>
             <parent link="${connected_to}"/>
@@ -135,5 +135,5 @@
             <axis xyz="0 1 0"/>
             <origin xyz="0.005 0.128 0" rpy="-1.57 0 0"/>
-            <limit effort="60" velocity="10" lower="-1.87" upper="-0.12"/>
+            <limit effort="60" velocity="10" lower="-2.4451245" upper="-0.171148851"/>
             <dynamics damping="0.0" friction="0.8"/>
             <parent link="link1"/>
@@ -143,5 +143,5 @@
             <axis xyz="0 1 0"/>
             <origin xyz="0.165 0 0" rpy="0 0 0"/>
-            <limit effort="30" velocity="10" lower="-0.7203" upper="2.6055"/>
+            <limit effort="30" velocity="10" lower="-0.7518866" upper="2.6334277"/>
             <dynamics damping="0.0" friction="0.5"/>
             <parent link="link2"/>
@@ -151,5 +151,5 @@
             <axis xyz="0 1 0"/>
             <origin xyz="0.106 0 0.028"/>
-            <limit effort="7" velocity="30" lower="-0.24430838" upper="2.65452132"/>
+            <limit effort="7" velocity="30" lower="-0.251792" upper="2.67008"/>
             <dynamics damping="0.0" friction="0.5"/>
             <parent link="link3"/>
@@ -159,5 +159,5 @@
             <axis xyz="1 0 0"/>
             <origin xyz="0.097 0 0.055"/>
-            <limit effort="13" velocity="18" lower="-3.139" upper="0.5454"/>
+            <limit effort="13" velocity="18" lower="-4.31220" upper="1.3749148"/>
             <dynamics damping="0.0" friction="0.5"/>
             <parent link="link4"/>

Commit message: Update engineer limit

File: urdf/engineer/arm.urdf.xacro (robot description, xacro)
@@ -127,5 +127,5 @@
             <origin xyz="0.122 0 0.124" rpy="1.57 0 0"/>
             <!--      limit not work while type="continuous"-->
-            <limit effort="20" velocity="10" lower="-3.93996572" upper="1.805202294"/>
+            <limit effort="20" velocity="10" lower="-4.0492335499" upper="2.066574686023"/>
             <dynamics damping="0.0" friction="0.1"/>
             <parent link="${connected_to}"/>
@@ -135,5 +135,5 @@
             <axis xyz="0 1 0"/>
             <origin xyz="0.005 0.128 0" rpy="-1.57 0 0"/>
-            <limit effort="60" velocity="10" lower="-2.4451245" upper="-0.171148851"/>
+            <limit effort="60" velocity="10" lower="-2.378679831401" upper="-0.0989819625299"/>
             <dynamics damping="0.0" friction="0.8"/>
             <parent link="link1"/>
@@ -143,5 +143,5 @@
             <axis xyz="0 1 0"/>
             <origin xyz="0.165 0 0" rpy="0 0 0"/>
-            <limit effort="30" velocity="10" lower="-0.7518866" upper="2.6334277"/>
+            <limit effort="30" velocity="10" lower="-0.88921949" upper="2.535032168"/>
             <dynamics damping="0.0" friction="0.5"/>
             <parent link="link2"/>
@@ -151,5 +151,5 @@
             <axis xyz="0 1 0"/>
             <origin xyz="0.106 0 0.028"/>
-            <limit effort="7" velocity="30" lower="-0.251792" upper="2.67008"/>
+            <limit effort="7" velocity="30" lower="-0.2989008" upper="2.614725376878"/>
             <dynamics damping="0.0" friction="0.5"/>
             <parent link="link3"/>
@@ -159,7 +159,7 @@
             <axis xyz="1 0 0"/>
             <origin xyz="0.097 0 0.055"/>
-            <limit effort="13" velocity="18" lower="-4.31220" upper="1.3749148"/>
+            <limit effort="13" velocity="18" lower="-4.27171178" upper="1.40800999"/>
             <dynamics damping="0.0" friction="0.5"/>
-            <parent link="link4"/>
+            <parent link="link4"/>z
             <child link="link5"/>
         </joint>
