Commit message: Add engineer safety controller

File: urdf/engineer/arm.urdf.xacro (robot description, xacro)
@@ -2,4 +2,15 @@
 <robot xmlns:xacro="http://www.ros.org/wiki/xacro" name="arm">
     <xacro:macro name="arm" params="connected_to">
+    <xacro:property name="threshold" value="0.1"/>
+    <xacro:property name="joint1_lower_limit" value="-4.0492335499"/>
+    <xacro:property name="joint1_upper_limit" value="2.066574686023"/>
+    <xacro:property name="joint2_lower_limit" value="-2.378679831401"/>
+    <xacro:property name="joint2_upper_limit" value="-0.0989819625299"/>
+    <xacro:property name="joint3_lower_limit" value="-0.88921949"/>
+    <xacro:property name="joint3_upper_limit" value="2.535032168"/>
+    <xacro:property name="joint4_lower_limit" value="-0.2989008"/>
+    <xacro:property name="joint4_upper_limit" value="2.614725376878"/>
+    <xacro:property name="joint5_lower_limit" value="-4.27171178"/>
+    <xacro:property name="joint5_upper_limit" value="1.40800999"/>
         <!--  link  -->
         <link name="link1">
@@ -127,5 +138,8 @@
             <origin xyz="0.122 0 0.124" rpy="1.57 0 0"/>
             <!--      limit not work while type="continuous"-->
-            <limit effort="20" velocity="10" lower="-4.0492335499" upper="2.066574686023"/>
+            <limit effort="20" velocity="10" lower="${joint1_lower_limit}" upper="${joint1_upper_limit}"/>
+            <safety_controller k_position="150" k_velocity="10"
+                               soft_lower_limit="${joint1_lower_limit+threshold}"
+                               soft_upper_limit="${joint1_upper_limit-threshold}"/>
             <dynamics damping="0.0" friction="0.1"/>
             <parent link="${connected_to}"/>
@@ -135,5 +149,8 @@
             <axis xyz="0 1 0"/>
             <origin xyz="0.005 0.128 0" rpy="-1.57 0 0"/>
-            <limit effort="60" velocity="10" lower="-2.378679831401" upper="-0.0989819625299"/>
+            <limit effort="60" velocity="10" lower="${joint2_lower_limit}" upper="${joint2_upper_limit}"/>
+            <safety_controller k_position="500" k_velocity="10"
+                               soft_lower_limit="${joint2_lower_limit+threshold}"
+                               soft_upper_limit="${joint2_upper_limit-threshold}"/>
             <dynamics damping="0.0" friction="0.8"/>
             <parent link="link1"/>
@@ -143,5 +160,8 @@
             <axis xyz="0 1 0"/>
             <origin xyz="0.165 0 0" rpy="0 0 0"/>
-            <limit effort="30" velocity="10" lower="-0.88921949" upper="2.535032168"/>
+            <limit effort="30" velocity="10" lower="${joint3_lower_limit}" upper="${joint3_upper_limit}"/>
+            <safety_controller k_position="500" k_velocity="6"
+                               soft_lower_limit="${joint3_lower_limit+threshold}"
+                               soft_upper_limit="${joint3_upper_limit-threshold}"/>
             <dynamics damping="0.0" friction="0.5"/>
             <parent link="link2"/>
@@ -151,5 +171,8 @@
             <axis xyz="0 1 0"/>
             <origin xyz="0.106 0 0.028"/>
-            <limit effort="7" velocity="30" lower="-0.2989008" upper="2.614725376878"/>
+            <limit effort="7" velocity="30" lower="${joint4_lower_limit}" upper="${joint4_upper_limit}"/>
+            <safety_controller k_position="20" k_velocity="2.5"
+                               soft_lower_limit="${joint4_lower_limit+threshold}"
+                               soft_upper_limit="${joint4_upper_limit-threshold}"/>
             <dynamics damping="0.0" friction="0.5"/>
             <parent link="link3"/>
@@ -159,5 +182,8 @@
             <axis xyz="1 0 0"/>
             <origin xyz="0.097 0 0.055"/>
-            <limit effort="13" velocity="18" lower="-4.27171178" upper="1.40800999"/>
+            <limit effort="13" velocity="18" lower="${joint5_lower_limit}" upper="${joint5_upper_limit}"/>
+            <safety_controller k_position="50" k_velocity="5"
+                               soft_lower_limit="${joint5_lower_limit+threshold}"
+                               soft_upper_limit="${joint5_upper_limit-threshold}"/>
             <dynamics damping="0.0" friction="0.5"/>
             <parent link="link4"/>z

Commit message: Change the chassis.urdf and arm.urdf.

File: urdf/engineer/arm.urdf.xacro (robot description, xacro)
@@ -27,5 +27,5 @@
             </visual>
             <collision>
-                <origin xyz="0.004 0.071 0" rpy="0 0 0"/>
+                <origin xyz="-0.022768 -0.000245 0.034512" rpy="0 0 0"/>
                 <geometry>
                     <box size="0.088 0.142 0.106"/>
@@ -33,5 +33,5 @@
             </collision>
             <collision>
-                <origin xyz="0.005 0.128 0" rpy="0 0 0"/>
+                <origin xyz="0.02 -0.000245 0.034512" rpy="0 0 0"/>
                 <geometry>
                     <cylinder length="0.106" radius="0.047"/>
@@ -136,5 +136,5 @@
         <joint name="joint1" type="revolute">
             <axis xyz="0 1 0"/>
-            <origin xyz="0.122 0 0.124" rpy="1.57 0 0"/>
+            <origin xyz="0.175 0 0.164" rpy="0 0 0"/>
             <!--      limit not work while type="continuous"-->
             <limit effort="20" velocity="10" lower="${joint1_lower_limit}" upper="${joint1_upper_limit}"/>
@@ -148,5 +148,5 @@
         <joint name="joint2" type="revolute">
             <axis xyz="0 1 0"/>
-            <origin xyz="0.005 0.128 0" rpy="-1.57 0 0"/>
+            <origin xyz="0.005327 0 0.128" rpy="0 0 0"/>
             <limit effort="60" velocity="10" lower="${joint2_lower_limit}" upper="${joint2_upper_limit}"/>
             <safety_controller k_position="500" k_velocity="10"

File: urdf/engineer/chassis.urdf.xacro (robot description, xacro)
@@ -2,9 +2,9 @@
     <xacro:include filename="$(find rm_description)/urdf/common/mecanum_wheel.urdf.xacro"/>
     <!-- https://upload.wikimedia.org/wikipedia/commons/5/52/Wheelbase_and_Track.png -->
-    <xacro:property name="wheel_front" value="0.1"/>
-    <xacro:property name="wheel_back" value="-0.18"/>
-    <xacro:property name="wheel_right" value="-0.24"/>
-    <xacro:property name="wheel_left" value="0.24"/>
-    <xacro:property name="wheel_offset_z" value="-0.06"/>
+    <xacro:property name="wheel_front" value="0.134874"/>
+    <xacro:property name="wheel_back" value="-0.134874"/>
+    <xacro:property name="wheel_right" value="-0.2448"/>
+    <xacro:property name="wheel_left" value="0.2448"/>
+    <xacro:property name="wheel_offset_z" value="0.000072"/>
     <xacro:property name="wheel_joint_damping" value="1.0"/>
     <xacro:property name="wheel_joint_friction" value="1.0"/>
@@ -14,6 +14,6 @@
                 <mass value="11.91"/>
                 <origin xyz="-0.063 -0.010 -0.027"/>
-                <inertia ixx="4.230e-1" ixy="-5.057e-4" ixz="3.328e-2" iyy="3.602e-1"
-                         iyz="1.417e-2" izz="5.140e-1"/>
+                <inertia ixx="4.302e-2" ixy="7.618e-4" ixz="6.881e-3" iyy="3.95e-2"
+                         iyz="-1.841e-4" izz="7.25e-2"/>
             </inertial>
             <visual>
@@ -24,11 +24,11 @@
             </visual>
             <collision>
-                <origin xyz="-0.043 0 0.020" rpy="0 0 0"/>
+                <origin xyz="0.005 0 0.06" rpy="0 0 0"/>
                 <geometry>
-                    <box size="0.486 0.596 0.169"/>
+                    <box size="0.5 0.596 0.169"/>
                 </geometry>
             </collision>
             <collision>
-                <origin xyz="-0.08 0.243 0.258" rpy="0 0 -0.5061455"/>
+                <origin xyz="-0.043688 0.236688 0.284" rpy="0 0 -0.5061455"/>
                 <geometry>
                     <box size="0.08 0.0217 0.3033"/>
@@ -36,5 +36,5 @@
             </collision>
             <collision>
-                <origin xyz="-0.21 0.19 0.25833" rpy="0 0 1.0646508"/>
+                <origin xyz="-0.160269 0.184128 0.284" rpy="0 0 1.0646508"/>
                 <geometry>
                     <box size="0.08 0.0217 0.3033"/>
@@ -42,5 +42,5 @@
             </collision>
             <collision>
-                <origin xyz="-0.19 0.05 0.258" rpy="0 0 -0.5061455"/>
+                <origin xyz="-0.143054 0.057391 0.284" rpy="0 0 -0.5061455"/>
                 <geometry>
                     <box size="0.08 0.0217 0.3033"/>
@@ -48,5 +48,5 @@
             </collision>
             <collision>
-                <origin xyz="-0.0239 0.084 0.228" rpy="0 0 1.0646508"/>
+                <origin xyz="0.019028 0.084742 0.269" rpy="0 0 1.0646508"/>
                 <geometry>
                     <box size="0.080 0.003 0.250"/>
@@ -87,5 +87,5 @@
             </visual>
             <collision>
-                <origin xyz="-0.113 0.134 0.0" rpy="0 0.0 0"/>
+                <origin xyz="-0.08 0 0" rpy="0 0.0 0"/>
                 <geometry>
                     <box size="0.253 0.151 0.011"/>
@@ -95,5 +95,5 @@
         <joint name="card_joint" type="prismatic">
             <axis xyz="1 0 0"/>
-            <origin xyz="0.109 0.001 -0.11"/>
+            <origin xyz="0.209783 0.004 -0.08"/>
             <limit effort="0.1" velocity="30" lower="0" upper="0.05"/>
             <dynamics damping="0.0" friction="0.1"/>

File: urdf/engineer/engineer.urdf.xacro (robot description, xacro)
@@ -17,5 +17,5 @@
         <xacro:hand connected_to="link5" xyz="-0.014 0 0" rpy="0 1.57 0" simulation="$(arg use_simulation)"/>
         <xacro:include filename="$(find rm_description)/urdf/engineer/mast.urdf.xacro"/>
-        <xacro:mast connected_to="link1" xyz="-0.076 0.582 0.108 " rpy="-1.57 0 0" simulation="$(arg use_simulation)"/>
+        <xacro:mast connected_to="link1" xyz="-0.0745 -0.1085 0.5697" rpy="0 0 0" simulation="$(arg use_simulation)"/>
     </xacro:if>
     <xacro:if value="$(arg use_simulation)">

Commit message: Change the chassis.urdf and arm.urdf.

File: urdf/engineer/arm.urdf.xacro (robot description, xacro)
@@ -135,5 +135,5 @@
         <!--  joint  -->
         <joint name="joint1" type="revolute">
-            <axis xyz="0 1 0"/>
+            <axis xyz="0 0 1"/>
             <origin xyz="0.175 0 0.164" rpy="0 0 0"/>
             <!--      limit not work while type="continuous"-->

File: urdf/engineer/chassis.urdf.xacro (robot description, xacro)
@@ -6,5 +6,5 @@
     <xacro:property name="wheel_right" value="-0.2448"/>
     <xacro:property name="wheel_left" value="0.2448"/>
-    <xacro:property name="wheel_offset_z" value="0.000072"/>
+    <xacro:property name="wheel_offset_z" value="-0.029928"/>
     <xacro:property name="wheel_joint_damping" value="1.0"/>
     <xacro:property name="wheel_joint_friction" value="1.0"/>
@@ -12,5 +12,5 @@
         <link name="base_link">
             <inertial>
-                <mass value="11.91"/>
+                <mass value="2.361504"/>
                 <origin xyz="-0.063 -0.010 -0.027"/>
                 <inertia ixx="4.302e-2" ixy="7.618e-4" ixz="6.881e-3" iyy="3.95e-2"
@@ -95,5 +95,5 @@
         <joint name="card_joint" type="prismatic">
             <axis xyz="1 0 0"/>
-            <origin xyz="0.209783 0.004 -0.08"/>
+            <origin xyz="0.209783 0.004 -0.064"/>
             <limit effort="0.1" velocity="30" lower="0" upper="0.05"/>
             <dynamics damping="0.0" friction="0.1"/>
@@ -103,5 +103,5 @@
         <joint name="stone_platform_joint" type="prismatic">
             <axis xyz="0 0 1"/>
-            <origin xyz="-0.113 0.134 0.114"/>
+            <origin xyz="-0.0706 0.134 0.1440"/>
             <limit effort="1" velocity="30" lower="0" upper="0.024"/>
             <dynamics damping="0.0" friction="0.1"/>

Commit message: Update joint4 mechanicalReduction

File: urdf/engineer/arm.urdf.xacro (robot description, xacro)
@@ -171,5 +171,5 @@
             <axis xyz="0 1 0"/>
             <origin xyz="0.106 0 0.028"/>
-            <limit effort="7" velocity="30" lower="${joint4_lower_limit}" upper="${joint4_upper_limit}"/>
+            <limit effort="18.53" velocity="13.5" lower="${joint4_lower_limit}" upper="${joint4_upper_limit}"/>
             <safety_controller k_position="20" k_velocity="2.5"
                                soft_lower_limit="${joint4_lower_limit+threshold}"

Commit message: Add a box.

File: urdf/engineer/arm.urdf.xacro (robot description, xacro)
@@ -33,7 +33,7 @@
             </collision>
             <collision>
-                <origin xyz="0.02 -0.000245 0.034512" rpy="0 0 0"/>
+                <origin xyz="0.001 -0.000245 0.04" rpy="1.57 0 0"/>
                 <geometry>
-                    <cylinder length="0.106" radius="0.047"/>
+                    <cylinder length="0.19" radius="0.047"/>
                 </geometry>
             </collision>

File: urdf/engineer/chassis.urdf.xacro (robot description, xacro)
@@ -73,4 +73,10 @@
                 </geometry>
             </collision>
+            <collision>
+                <origin xyz="-0.08 -0.09 0.02" rpy="0 0 1.0646508"/>
+                <geometry>
+                    <box size="0.03 0.06 0.05"/>
+                </geometry>
+            </collision>
         </link>
         <link name="card">
@@ -95,5 +101,5 @@
         <joint name="card_joint" type="prismatic">
             <axis xyz="1 0 0"/>
-            <origin xyz="0.209783 0.004 -0.064/>
+            <origin xyz="0.209783 0.004 -0.064"/>
             <limit effort="20.0" velocity="1.0" lower="0" upper="0.1"/>
             <dynamics damping="0.0" friction="0.1"/>

Commit message: Update engineer arm URDF

File: urdf/engineer/arm.urdf.xacro (robot description, xacro)
@@ -130,5 +130,5 @@
         <joint name="joint1" type="revolute">
             <axis xyz="0 0 1"/>
-            <origin xyz="0.175 0 0.164" rpy="0 0 0"/>
+            <origin xyz="0.175 0 0.174" rpy="0 0 0"/>
             <!--      limit not work while type="continuous"-->
             <limit effort="20" velocity="13" lower="${joint1_lower_limit}" upper="${joint1_upper_limit}"/>

File: urdf/engineer/chassis.urdf.xacro (robot description, xacro)
@@ -48,7 +48,7 @@
             </collision>
             <collision>
-                <origin xyz="-0.043688 0.236688 0.284" rpy="0 0 -0.5061455"/>
+                <origin xyz="-0.038526 0.245965 0.224" rpy="0 0 -0.507"/>
                 <geometry>
-                    <box size="0.08 0.0217 0.3033"/>
+                    <box size="0.08 0.024213 0.448"/>
                 </geometry>
             </collision>
@@ -60,7 +60,7 @@
             </collision>
             <collision>
-                <origin xyz="-0.143054 0.057391 0.284" rpy="0 0 -0.5061455"/>
+                <origin xyz="-0.148196 0.0485 0.224" rpy="0 0 -0.507"/>
                 <geometry>
-                    <box size="0.08 0.0217 0.3033"/>
+                    <box size="0.08 0.024213 0.448"/>
                 </geometry>
             </collision>
@@ -120,5 +120,5 @@
             <axis xyz="1 0 0"/>
             <origin xyz="0.15205 0. -0.07"/>
-            <limit effort="20.0" velocity="1.0" lower="0" upper="0.1"/>
+            <limit effort="20.0" velocity="1.0" lower="0" upper="0.281"/>
             <dynamics damping="0.0" friction="0.1"/>
             <parent link="base_link"/>

File: urdf/engineer/mast.urdf.xacro (robot description, xacro)
@@ -73,5 +73,5 @@
             <origin xyz="0.  0. 0.059 " rpy="0 0 0"/>
             <dynamics damping="0.0" friction="0.1"/>
-            <limit effort="0.1" velocity="10" lower="-0.47247" upper="1.25862"/>
+            <limit effort="0.2" velocity="10" lower="-0.47247" upper="1.25862"/>
             <parent link="yaw"/>
             <child link="pitch"/>
