Commit message: Add use_simulation to arm cause by gazebo doesn't support transmission has more than one joint.

File: urdf/engineer/arm.transmission.xacro (robot description, xacro)
@@ -1,14 +1,13 @@
 <?xml version="1.0" encoding="utf-8"?>
 <robot xmlns:xacro="http://www.ros.org/wiki/xacro">
-  <xacro:macro name="arm_transmission">
+  <xacro:macro name="arm_transmission" params="differential_wrist">
     <!-- transmission -->
     <transmission name="trans_joint1">
       <type>transmission_interface/SimpleTransmission</type>
       <actuator name="joint1_motor">
-        <hardwareInterface>hardware_interface/EffortJointInterface</hardwareInterface>
         <mechanicalReduction>1</mechanicalReduction>
         <offset>0</offset>
       </actuator>
-      <joint name="joint1">
+      <joint name="joint1">load_chassis
         <hardwareInterface>hardware_interface/EffortJointInterface</hardwareInterface>
       </joint>
@@ -17,5 +16,4 @@
       <type>transmission_interface/SimpleTransmission</type>
       <actuator name="joint2_motor">
-        <hardwareInterface>hardware_interface/EffortJointInterface</hardwareInterface>
         <mechanicalReduction>1</mechanicalReduction>
         <offset>0</offset>
@@ -28,5 +26,4 @@
       <type>transmission_interface/SimpleTransmission</type>
       <actuator name="joint3_motor">
-        <hardwareInterface>hardware_interface/EffortJointInterface</hardwareInterface>
         <mechanicalReduction>1</mechanicalReduction>
         <offset>0</offset>
@@ -36,26 +33,55 @@
       </joint>
     </transmission>
-    <transmission name="trans_joint4">
-      <type>transmission_interface/SimpleTransmission</type>
-      <actuator name="joint4_motor">
-        <hardwareInterface>hardware_interface/EffortJointInterface</hardwareInterface>
-        <mechanicalReduction>1</mechanicalReduction>
-        <offset>0</offset>
-      </actuator>
-      <joint name="joint4">
-        <hardwareInterface>hardware_interface/EffortJointInterface</hardwareInterface>
-      </joint>
-    </transmission>
-    <transmission name="trans_joint5">
-      <type>transmission_interface/SimpleTransmission</type>
-      <actuator name="joint5_motor">
-        <hardwareInterface>hardware_interface/EffortJointInterface</hardwareInterface>
-        <mechanicalReduction>1</mechanicalReduction>
-        <offset>0</offset>
-      </actuator>
-      <joint name="joint5">
-        <hardwareInterface>hardware_interface/EffortJointInterface</hardwareInterface>
-      </joint>
-    </transmission>
+    <xacro:if value="${differential_wrist}">
+      <transmission name="trans_wrist">
+        <type>transmission_interface/DifferentialTransmission</type>
+        <actuator name="left_wrist_motor">
+          <role>actuator1</role>
+          <mechanicalReduction>1.2</mechanicalReduction>
+        </actuator>
+        <actuator name="right_wrist_motor">
+          <role>actuator2</role>
+          <mechanicalReduction>1.2</mechanicalReduction>
+        </actuator>
+        <joint name="joint4">
+          <role>joint1</role>
+          <offset>0</offset>
+          <mechanicalReduction>1</mechanicalReduction>
+          <hardwareInterface>hardware_interface/EffortJointInterface</hardwareInterface>
+          <ignoreTransmissionAbsoluteEncoder>1</ignoreTransmissionAbsoluteEncoder>
+        </joint>
+        <joint name="joint5">
+          <role>joint2</role>
+          <offset>0</offset>
+          <mechanicalReduction>1</mechanicalReduction>
+          <hardwareInterface>hardware_interface/EffortJointInterface</hardwareInterface>
+          <ignoreTransmissionAbsoluteEncoder>1</ignoreTransmissionAbsoluteEncoder>
+        </joint>
+      </transmission>
+    </xacro:if>
+    <xacro:unless value="${differential_wrist}">
+      <transmission name="trans_joint4">
+        <type>transmission_interface/SimpleTransmission</type>
+        <actuator name="joint4_motor">
+          <hardwareInterface>hardware_interface/EffortJointInterface</hardwareInterface>
+          <mechanicalReduction>1</mechanicalReduction>
+          <offset>0</offset>
+        </actuator>
+        <joint name="joint4">
+          <hardwareInterface>hardware_interface/EffortJointInterface</hardwareInterface>
+        </joint>
+      </transmission>
+      <transmission name="trans_joint5">
+        <type>transmission_interface/SimpleTransmission</type>
+        <actuator name="joint5_motor">
+          <hardwareInterface>hardware_interface/EffortJointInterface</hardwareInterface>
+          <mechanicalReduction>1</mechanicalReduction>
+          <offset>0</offset>
+        </actuator>
+        <joint name="joint5">
+          <hardwareInterface>hardware_interface/EffortJointInterface</hardwareInterface>
+        </joint>
+      </transmission>
+    </xacro:unless>
   </xacro:macro>
 </robot>

File: urdf/engineer/arm.urdf.xacro (robot description, xacro)
@@ -165,6 +165,4 @@
     </joint>
     <!-- extensions -->
-    <xacro:include filename="$(find rm_description)/urdf/engineer/arm.transmission.xacro"/>
-    <xacro:arm_transmission/>
     <!--TODO: Add gazebo-->
   </xacro:macro>

File: urdf/engineer/engineer.urdf.xacro (robot description, xacro)
@@ -3,5 +3,5 @@
   <xacro:arg name="load_chassis" default="false"/>
   <xacro:arg name="load_arm" default="true"/>
-  <xacro:arg name="load_gazebo" default="true"/>
+  <xacro:arg name="use_simulation" default="true"/>
   <xacro:arg name="use_rm_gazebo" default="false"/>
   <xacro:arg name="roller_type" default="realistic"/>
@@ -13,4 +13,5 @@
   <xacro:if value="$(arg load_arm)">
     <xacro:include filename="$(find rm_description)/urdf/engineer/arm.urdf.xacro"/>
+    <xacro:include filename="$(find rm_description)/urdf/engineer/arm.transmission.xacro"/>
     <xacro:if value="$(arg fixed_arm)">
       <link name="world"/>
@@ -20,8 +21,14 @@
       <xacro:arm connected_to="base_link"/>
     </xacro:unless>
+    <xacro:if value="$(arg use_simulation)">
+      <xacro:arm_transmission differential_wrist="false"/>
+    </xacro:if>
+    <xacro:unless value="$(arg use_simulation)">
+      <xacro:arm_transmission differential_wrist="true"/>
+    </xacro:unless>
     <xacro:include filename="$(find rm_description)/urdf/engineer/hand.urdf.xacro"/>
     <xacro:hand connected_to="link5" xyz="0.039 0 0"/>
   </xacro:if>
-  <xacro:if value="$(arg load_gazebo)">
+  <xacro:if value="$(arg use_simulation)">
     <xacro:if value="$(arg use_rm_gazebo)">
       <gazebo>

Commit message: Set offset

File: urdf/engineer/arm.transmission.xacro (robot description, xacro)
@@ -6,9 +6,9 @@
       <type>transmission_interface/SimpleTransmission</type>
       <actuator name="joint1_motor">
-        <mechanicalReduction>1</mechanicalReduction>
-        <offset>0</offset>
+        <mechanicalReduction>4</mechanicalReduction>
       </actuator>
       <joint name="joint1">load_chassis
         <hardwareInterface>hardware_interface/EffortJointInterface</hardwareInterface>
+        <offset>0</offset>
       </joint>
     </transmission>
@@ -16,9 +16,9 @@
       <type>transmission_interface/SimpleTransmission</type>
       <actuator name="joint2_motor">
-        <mechanicalReduction>1</mechanicalReduction>
-        <offset>0</offset>
+        <mechanicalReduction>-3</mechanicalReduction>
       </actuator>
       <joint name="joint2">
         <hardwareInterface>hardware_interface/EffortJointInterface</hardwareInterface>
+        <offset>-1.889</offset>
       </joint>
     </transmission>
@@ -26,9 +26,9 @@
       <type>transmission_interface/SimpleTransmission</type>
       <actuator name="joint3_motor">
-        <mechanicalReduction>1</mechanicalReduction>
-        <offset>0</offset>
+        <mechanicalReduction>-3</mechanicalReduction>
       </actuator>
       <joint name="joint3">
         <hardwareInterface>hardware_interface/EffortJointInterface</hardwareInterface>
+        <offset>2.4306</offset>
       </joint>
     </transmission>
@@ -42,9 +42,9 @@
         <actuator name="right_wrist_motor">
           <role>actuator2</role>
-          <mechanicalReduction>1.2</mechanicalReduction>
+          <mechanicalReduction>-1.2</mechanicalReduction>
         </actuator>
         <joint name="joint4">
           <role>joint1</role>
-          <offset>0</offset>
+          <offset>-2.1562</offset>
           <mechanicalReduction>1</mechanicalReduction>
           <hardwareInterface>hardware_interface/EffortJointInterface</hardwareInterface>
@@ -53,5 +53,5 @@
         <joint name="joint5">
           <role>joint2</role>
-          <offset>0</offset>
+          <offset>0.0702</offset>
           <mechanicalReduction>1</mechanicalReduction>
           <hardwareInterface>hardware_interface/EffortJointInterface</hardwareInterface>

File: urdf/engineer/arm.urdf.xacro (robot description, xacro)
@@ -135,5 +135,5 @@
       <axis xyz="0 1 0"/>
       <origin xyz="0.11341 0 0.1380"/>
-      <limit effort="60" velocity="10" lower="-${pi}" upper="${0.44*pi}"/>
+      <limit effort="30" velocity="10" lower="-${pi}" upper="${0.44*pi}"/>
       <dynamics damping="0.0" friction="0.8"/>
       <parent link="link1"/>
@@ -164,6 +164,4 @@
       <child link="link5"/>
     </joint>
-    <!-- extensions -->
-    <!--TODO: Add gazebo-->
   </xacro:macro>
 </robot>

File: urdf/engineer/engineer.urdf.xacro (robot description, xacro)
@@ -27,6 +27,6 @@
       <xacro:arm_transmission differential_wrist="true"/>
     </xacro:unless>
-    <xacro:include filename="$(find rm_description)/urdf/engineer/hand.urdf.xacro"/>
-    <xacro:hand connected_to="link5" xyz="0.039 0 0"/>
+    <!--    <xacro:include filename="$(find rm_description)/urdf/engineer/hand.urdf.xacro"/>-->
+    <!--    <xacro:hand connected_to="link5" xyz="0.039 0 0"/>-->
   </xacro:if>
   <xacro:if value="$(arg use_simulation)">

Commit message: Change differential_wrist to simulation

File: urdf/engineer/arm.transmission.xacro (robot description, xacro)
@@ -1,87 +1,87 @@
 <?xml version="1.0" encoding="utf-8"?>
 <robot xmlns:xacro="http://www.ros.org/wiki/xacro">
-  <xacro:macro name="arm_transmission" params="differential_wrist">
-    <!-- transmission -->
-    <transmission name="trans_joint1">
-      <type>transmission_interface/SimpleTransmission</type>
-      <actuator name="joint1_motor">
-        <mechanicalReduction>4</mechanicalReduction>
-      </actuator>
-      <joint name="joint1">load_chassis
-        <hardwareInterface>hardware_interface/EffortJointInterface</hardwareInterface>
-        <offset>0</offset>
-      </joint>
-    </transmission>
-    <transmission name="trans_joint2">
-      <type>transmission_interface/SimpleTransmission</type>
-      <actuator name="joint2_motor">
-        <mechanicalReduction>-3</mechanicalReduction>
-      </actuator>
-      <joint name="joint2">
-        <hardwareInterface>hardware_interface/EffortJointInterface</hardwareInterface>
-        <offset>-3.1904</offset>
-      </joint>
-    </transmission>
-    <transmission name="trans_joint3">
-      <type>transmission_interface/SimpleTransmission</type>
-      <actuator name="joint3_motor">
-        <mechanicalReduction>-3</mechanicalReduction>
-      </actuator>
-      <joint name="joint3">
-        <hardwareInterface>hardware_interface/EffortJointInterface</hardwareInterface>
-        <offset>2.4306</offset>
-      </joint>
-    </transmission>
-    <xacro:if value="${differential_wrist}">
-      <transmission name="trans_wrist">
-        <type>transmission_interface/DifferentialTransmission</type>
-        <actuator name="left_wrist_motor">
-          <role>actuator1</role>
-          <mechanicalReduction>1.2</mechanicalReduction>
-        </actuator>
-        <actuator name="right_wrist_motor">
-          <role>actuator2</role>
-          <mechanicalReduction>-1.2</mechanicalReduction>
-        </actuator>
-        <joint name="joint4">
-          <role>joint1</role>
-          <offset>-2.1562</offset>
-          <mechanicalReduction>1</mechanicalReduction>
-          <hardwareInterface>hardware_interface/EffortJointInterface</hardwareInterface>
-          <ignoreTransmissionAbsoluteEncoder>1</ignoreTransmissionAbsoluteEncoder>
-        </joint>
-        <joint name="joint5">
-          <role>joint2</role>
-          <offset>0.0702</offset>
-          <mechanicalReduction>1</mechanicalReduction>
-          <hardwareInterface>hardware_interface/EffortJointInterface</hardwareInterface>
-          <ignoreTransmissionAbsoluteEncoder>1</ignoreTransmissionAbsoluteEncoder>
-        </joint>
-      </transmission>
-    </xacro:if>
-    <xacro:unless value="${differential_wrist}">
-      <transmission name="trans_joint4">
-        <type>transmission_interface/SimpleTransmission</type>
-        <actuator name="joint4_motor">
-          <hardwareInterface>hardware_interface/EffortJointInterface</hardwareInterface>
-          <mechanicalReduction>1</mechanicalReduction>
-          <offset>0</offset>
-        </actuator>
-        <joint name="joint4">
-          <hardwareInterface>hardware_interface/EffortJointInterface</hardwareInterface>
-        </joint>
-      </transmission>
-      <transmission name="trans_joint5">
-        <type>transmission_interface/SimpleTransmission</type>
-        <actuator name="joint5_motor">
-          <hardwareInterface>hardware_interface/EffortJointInterface</hardwareInterface>
-          <mechanicalReduction>1</mechanicalReduction>
-          <offset>0</offset>
-        </actuator>
-        <joint name="joint5">
-          <hardwareInterface>hardware_interface/EffortJointInterface</hardwareInterface>
-        </joint>
-      </transmission>
-    </xacro:unless>
-  </xacro:macro>
+    <xacro:macro name="arm_transmission" params="simulation">
+        <!-- transmission -->
+        <transmission name="trans_joint1">
+            <type>transmission_interface/SimpleTransmission</type>
+            <actuator name="joint1_motor">
+                <mechanicalReduction>4</mechanicalReduction>
+            </actuator>
+            <joint name="joint1">load_chassis
+                <hardwareInterface>hardware_interface/EffortJointInterface</hardwareInterface>
+                <offset>0</offset>
+            </joint>
+        </transmission>
+        <transmission name="trans_joint2">
+            <type>transmission_interface/SimpleTransmission</type>
+            <actuator name="joint2_motor">
+                <mechanicalReduction>-3</mechanicalReduction>
+            </actuator>
+            <joint name="joint2">
+                <hardwareInterface>hardware_interface/EffortJointInterface</hardwareInterface>
+                <offset>-3.1904</offset>
+            </joint>
+        </transmission>
+        <transmission name="trans_joint3">
+            <type>transmission_interface/SimpleTransmission</type>
+            <actuator name="joint3_motor">
+                <mechanicalReduction>-3</mechanicalReduction>
+            </actuator>
+            <joint name="joint3">
+                <hardwareInterface>hardware_interface/EffortJointInterface</hardwareInterface>
+                <offset>2.4306</offset>
+            </joint>
+        </transmission>
+        <xacro:unless value="${simulation}">
+            <transmission name="trans_wrist">
+                <type>transmission_interface/DifferentialTransmission</type>
+                <actuator name="left_wrist_motor">
+                    <role>actuator1</role>
+                    <mechanicalReduction>1.2</mechanicalReduction>
+                </actuator>
+                <actuator name="right_wrist_motor">
+                    <role>actuator2</role>
+                    <mechanicalReduction>-1.2</mechanicalReduction>
+                </actuator>
+                <joint name="joint4">
+                    <role>joint1</role>
+                    <offset>-2.1562</offset>
+                    <mechanicalReduction>1</mechanicalReduction>
+                    <hardwareInterface>hardware_interface/EffortJointInterface</hardwareInterface>
+                    <ignoreTransmissionAbsoluteEncoder>1</ignoreTransmissionAbsoluteEncoder>
+                </joint>
+                <joint name="joint5">
+                    <role>joint2</role>
+                    <offset>0.0702</offset>
+                    <mechanicalReduction>1</mechanicalReduction>
+                    <hardwareInterface>hardware_interface/EffortJointInterface</hardwareInterface>
+                    <ignoreTransmissionAbsoluteEncoder>1</ignoreTransmissionAbsoluteEncoder>
+                </joint>
+            </transmission>
+        </xacro:unless>
+        <xacro:if value="${simulation}">
+            <transmission name="trans_joint4">
+                <type>transmission_interface/SimpleTransmission</type>
+                <actuator name="joint4_motor">
+                    <hardwareInterface>hardware_interface/EffortJointInterface</hardwareInterface>
+                    <mechanicalReduction>1</mechanicalReduction>
+                    <offset>0</offset>
+                </actuator>
+                <joint name="joint4">
+                    <hardwareInterface>hardware_interface/EffortJointInterface</hardwareInterface>
+                </joint>
+            </transmission>
+            <transmission name="trans_joint5">
+                <type>transmission_interface/SimpleTransmission</type>
+                <actuator name="joint5_motor">
+                    <hardwareInterface>hardware_interface/EffortJointInterface</hardwareInterface>
+                    <mechanicalReduction>1</mechanicalReduction>
+                    <offset>0</offset>
+                </actuator>
+                <joint name="joint5">
+                    <hardwareInterface>hardware_interface/EffortJointInterface</hardwareInterface>
+                </joint>
+            </transmission>
+        </xacro:if>
+    </xacro:macro>
 </robot>

File: urdf/engineer/engineer.urdf.xacro (robot description, xacro)
@@ -1,38 +1,33 @@
 <?xml version="1.0"?>
 <robot xmlns:xacro="http://www.ros.org/wiki/xacro" name="engineer">
-  <xacro:arg name="load_chassis" default="false"/>
-  <xacro:arg name="load_arm" default="true"/>
-  <xacro:arg name="use_simulation" default="true"/>
-  <xacro:arg name="roller_type" default="realistic"/>
-  <xacro:if value="$(arg load_chassis)">
-    <xacro:include filename="$(find rm_description)/urdf/hero/chassis.urdf.xacro"/>
-    <xacro:chassis roller_type="$(arg roller_type)"/>
-  </xacro:if>
-  <xacro:if value="$(arg load_arm)">
-    <xacro:include filename="$(find rm_description)/urdf/engineer/arm.urdf.xacro"/>
-    <xacro:include filename="$(find rm_description)/urdf/engineer/arm.transmission.xacro"/>
+    <xacro:arg name="load_chassis" default="false"/>
+    <xacro:arg name="load_arm" default="true"/>
+    <xacro:arg name="use_simulation" default="true"/>
+    <xacro:arg name="roller_type" default="realistic"/>
     <xacro:if value="$(arg load_chassis)">
-      <xacro:arm connected_to="base_link"/>
+        <xacro:include filename="$(find rm_description)/urdf/hero/chassis.urdf.xacro"/>
+        <xacro:chassis roller_type="$(arg roller_type)"/>
     </xacro:if>
-    <xacro:unless value="$(arg load_chassis)">
-      <link name="world"/>
-      <xacro:arm connected_to="world"/>
-    </xacro:unless>
+    <xacro:if value="$(arg load_arm)">
+        <xacro:include filename="$(find rm_description)/urdf/engineer/arm.urdf.xacro"/>
+        <xacro:include filename="$(find rm_description)/urdf/engineer/arm.transmission.xacro"/>
+        <xacro:if value="$(arg load_chassis)">
+            <xacro:arm connected_to="base_link"/>
+        </xacro:if>
+        <xacro:unless value="$(arg load_chassis)">
+            <link name="world"/>
+            <xacro:arm connected_to="world"/>
+        </xacro:unless>
+        <xacro:arm_transmission simulation="$(arg use_simulation)"/>
+        <!--    <xacro:include filename="$(find rm_description)/urdf/engineer/hand.urdf.xacro"/>-->
+        <!--    <xacro:hand connected_to="link5" xyz="0.039 0 0"/>-->
+    </xacro:if>
     <xacro:if value="$(arg use_simulation)">
-      <xacro:arm_transmission differential_wrist="false"/>
+        <gazebo>
+            <plugin name="rm_ros_control" filename="librm_robot_hw_sim.so">
+                <robotNamespace>/</robotNamespace>
+                <robotSimType>rm_gazebo/RmRobotHWSim</robotSimType>
+            </plugin>
+        </gazebo>
     </xacro:if>
-    <xacro:unless value="$(arg use_simulation)">
-      <xacro:arm_transmission differential_wrist="true"/>
-    </xacro:unless>
-    <!--    <xacro:include filename="$(find rm_description)/urdf/engineer/hand.urdf.xacro"/>-->
-    <!--    <xacro:hand connected_to="link5" xyz="0.039 0 0"/>-->
-  </xacro:if>
-  <xacro:if value="$(arg use_simulation)">
-    <gazebo>
-      <plugin name="rm_ros_control" filename="librm_robot_hw_sim.so">
-        <robotNamespace>/</robotNamespace>
-        <robotSimType>rm_gazebo/RmRobotHWSim</robotSimType>
-      </plugin>
-    </gazebo>
-  </xacro:if>
 </robot>
