Commit message: add chassis

File: urdf/engineer/arm.transmission.xacro (robot description, xacro)
@@ -8,7 +8,7 @@
                 <mechanicalReduction>4</mechanicalReduction>
             </actuator>
-            <joint name="joint1">load_chassis
+            <joint name="joint1">
                 <hardwareInterface>hardware_interface/EffortJointInterface</hardwareInterface>
-                <offset>0</offset>
+                <offset>-0.0148</offset>
             </joint>
         </transmission>
@@ -16,9 +16,9 @@
             <type>transmission_interface/SimpleTransmission</type>
             <actuator name="joint3_motor">
-                <mechanicalReduction>-3</mechanicalReduction>
+                <mechanicalReduction>3</mechanicalReduction>
             </actuator>
             <joint name="joint3">
                 <hardwareInterface>hardware_interface/EffortJointInterface</hardwareInterface>
-                <offset>2.4306</offset>
+                <offset>0.48517</offset>
             </joint>
         </transmission>
@@ -35,7 +35,7 @@
                 </actuator>
                 <joint name="joint2">
-                    <offset>0</offset>
+                    <hardwareInterface>hardware_interface/EffortJointInterface</hardwareInterface>
+                    <offset>0.49839</offset>
                     <mechanicalReduction>1</mechanicalReduction>
-                    <hardwareInterface>hardware_interface/EffortJointInterface</hardwareInterface>
                 </joint>
             </transmission>
@@ -52,5 +52,5 @@
                 <joint name="joint4">
                     <role>joint1</role>
-                    <offset>-2.1562</offset>
+                    <offset>1.1504</offset>
                     <mechanicalReduction>1</mechanicalReduction>
                     <hardwareInterface>hardware_interface/EffortJointInterface</hardwareInterface>
@@ -59,6 +59,6 @@
                 <joint name="joint5">
                     <role>joint2</role>
-                    <offset>0.0702</offset>
-                    <mechanicalReduction>1</mechanicalReduction>
+                    <offset>-0.0801</offset>
+                    <mechanicalReduction>-1</mechanicalReduction>
                     <hardwareInterface>hardware_interface/EffortJointInterface</hardwareInterface>
                     <ignoreTransmissionAbsoluteEncoder>1</ignoreTransmissionAbsoluteEncoder>

File: urdf/engineer/arm.urdf.xacro (robot description, xacro)
@@ -129,5 +129,5 @@
       <axis xyz="0 1 0"/>
       <origin xyz="0.05909 0 0.1280"/>
-      <limit effort="30" velocity="10" lower="-${pi}" upper="${0.44*pi}"/>
+      <limit effort="30" velocity="10" lower="-${0.694*pi}" upper="${0.12*pi}"/>
       <dynamics damping="0.0" friction="0.8"/>
       <parent link="link1"/>
@@ -137,5 +137,5 @@
       <axis xyz="0 1 0"/>
       <origin xyz="0.16 0 0"/>
-      <limit effort="30" velocity="10" lower="-${0.722*pi}" upper="${0.722*pi}"/>
+      <limit effort="30" velocity="10" lower="-${0.666*pi}" upper="${0.75*pi}"/>
       <dynamics damping="0.0" friction="0.5"/>
       <parent link="link2"/>

File: urdf/engineer/chassis.urdf.xacro (robot description, xacro)
@@ -2,7 +2,7 @@
     <xacro:include filename="$(find rm_description)/urdf/common/mecanum_wheel.urdf.xacro"/>
     <!-- https://upload.wikimedia.org/wikipedia/commons/5/52/Wheelbase_and_Track.png -->
-    <xacro:property name="wheel_track" value="0.500"/>
-    <xacro:property name="wheel_base" value="0.475"/>
-    <xacro:property name="wheel_offset_z" value="-0.036"/>
+    <xacro:property name="wheel_track" value="0.380"/>
+    <xacro:property name="wheel_base" value="0.420"/>
+    <xacro:property name="wheel_offset_z" value="-0.1090"/>
     <xacro:property name="wheel_joint_damping" value="1.0"/>
     <xacro:property name="wheel_joint_friction" value="1.0"/>

Commit message: change limit

File: urdf/engineer/arm.transmission.xacro (robot description, xacro)
@@ -20,5 +20,5 @@
             <joint name="joint3">
                 <hardwareInterface>hardware_interface/EffortJointInterface</hardwareInterface>
-                <offset>0.48517</offset>
+                <offset>2.288</offset>
             </joint>
         </transmission>
@@ -36,5 +36,5 @@
                 <joint name="joint2">
                     <hardwareInterface>hardware_interface/EffortJointInterface</hardwareInterface>
-                    <offset>0.49839</offset>
+                    <offset>-2.3386</offset>
                     <mechanicalReduction>1</mechanicalReduction>
                 </joint>

File: urdf/engineer/arm.urdf.xacro (robot description, xacro)
@@ -129,5 +129,5 @@
       <axis xyz="0 1 0"/>
       <origin xyz="0.05909 0 0.1280"/>
-      <limit effort="30" velocity="10" lower="-${0.694*pi}" upper="${0.12*pi}"/>
+      <limit effort="30" velocity="10" lower="-2.231" upper="0.407"/>
       <dynamics damping="0.0" friction="0.8"/>
       <parent link="link1"/>
@@ -137,5 +137,5 @@
       <axis xyz="0 1 0"/>
       <origin xyz="0.16 0 0"/>
-      <limit effort="30" velocity="10" lower="-${0.666*pi}" upper="${0.75*pi}"/>
+      <limit effort="30" velocity="10" lower="-2.1645" upper="2.4078"/>
       <dynamics damping="0.0" friction="0.5"/>
       <parent link="link2"/>

Commit message: add box

File: urdf/engineer/arm.transmission.xacro (robot description, xacro)
@@ -20,5 +20,5 @@
             <joint name="joint3">
                 <hardwareInterface>hardware_interface/EffortJointInterface</hardwareInterface>
-                <offset>2.288</offset>
+                <offset>2.2875</offset>
             </joint>
         </transmission>
@@ -36,5 +36,5 @@
                 <joint name="joint2">
                     <hardwareInterface>hardware_interface/EffortJointInterface</hardwareInterface>
-                    <offset>-2.3386</offset>
+                    <offset>-2.3289</offset>
                     <mechanicalReduction>1</mechanicalReduction>
                 </joint>
@@ -52,5 +52,5 @@
                 <joint name="joint4">
                     <role>joint1</role>
-                    <offset>1.1504</offset>
+                    <offset>1.2603</offset>
                     <mechanicalReduction>1</mechanicalReduction>
                     <hardwareInterface>hardware_interface/EffortJointInterface</hardwareInterface>
@@ -59,5 +59,5 @@
                 <joint name="joint5">
                     <role>joint2</role>
-                    <offset>-0.0801</offset>
+                    <offset>0.1179</offset>
                     <mechanicalReduction>-1</mechanicalReduction>
                     <hardwareInterface>hardware_interface/EffortJointInterface</hardwareInterface>

File: urdf/engineer/chassis.urdf.xacro (robot description, xacro)
@@ -51,4 +51,16 @@
                 </geometry>
             </collision>
+            <collision>
+                <origin xyz="-0.193 -0.189 0.235" rpy="0 0 0"/>
+                <geometry>
+                    <box size="0.186 0.1 0.3"/>
+                </geometry>
+            </collision>
+            <collision>
+                <origin xyz="-0.0623 -0.2405 0.242" rpy="0 0 0"/>
+                <geometry>
+                    <box size="0.08 0.003 0.06"/>
+                </geometry>
+            </collision>
         </link>
         <xacro:mecanum_wheel prefix="front_left" connected_to="base_link"

File: urdf/engineer/hand.urdf.xacro (robot description, xacro)
@@ -121,4 +121,5 @@
             <joint name="right_finger_joint">
                 <hardwareInterface>hardware_interface/EffortJointInterface</hardwareInterface>
+                <offset>-0.0640</offset>
             </joint>
             <actuator name="right_finger_motor">
@@ -131,4 +132,5 @@
             <joint name="left_finger_joint">
                 <hardwareInterface>hardware_interface/EffortJointInterface</hardwareInterface>
+                <offset>-0.0640</offset>
             </joint>
             <actuator name="left_finger_motor">
