Commit message: engineer parameter

File: urdf/engineer/arm.transmission.xacro (robot description, xacro)
@@ -20,5 +20,5 @@
             <joint name="joint3">
                 <hardwareInterface>hardware_interface/EffortJointInterface</hardwareInterface>
-                <offset>2.4132</offset>
+                <offset>0.364</offset>
             </joint>
         </transmission>
@@ -36,5 +36,5 @@
                 <joint name="joint2">
                     <hardwareInterface>hardware_interface/EffortJointInterface</hardwareInterface>
-                    <offset>-2.269</offset>
+                    <offset>0.494</offset>
                     <mechanicalReduction>1</mechanicalReduction>
                 </joint>
@@ -52,5 +52,5 @@
                 <joint name="joint4">
                     <role>joint1</role>
-                    <offset>1.14294</offset>
+                    <offset>1.215</offset>
                     <mechanicalReduction>1</mechanicalReduction>
                     <hardwareInterface>hardware_interface/EffortJointInterface</hardwareInterface>
@@ -59,5 +59,5 @@
                 <joint name="joint5">
                     <role>joint2</role>
-                    <offset>0.0583</offset>
+                    <offset>0.065</offset>
                     <mechanicalReduction>-1</mechanicalReduction>
                     <hardwareInterface>hardware_interface/EffortJointInterface</hardwareInterface>

File: urdf/engineer/hand.urdf.xacro (robot description, xacro)
@@ -149,64 +149,53 @@
             <mimic joint="right_finger_joint"/>
         </joint>
-        <xacro:if value="${simulation}">
-            <gazebo reference="camera">
-                <sensor type="camera" name="camera_node">
-                    <update_rate>30.0</update_rate>
-                    <camera name="head">
-                        <horizontal_fov>1.3962634</horizontal_fov>
-                        <image>
-                            <width>1920</width>
-                            <height>1080</height>
-                            <format>R8G8B8</format>
-                        </image>
-                        <clip>
-                            <near>0.02</near>
-                            <far>300</far>
-                        </clip>
-                        <noise>
-                            <type>gaussian</type>
-                            <mean>0.0</mean>
-                            <stddev>0.007</stddev>
-                        </noise>
-                    </camera>
-                    <plugin name="gazebo_camera" filename="libgazebo_ros_camera.so">
-                        <alwaysOn>true</alwaysOn>
-                        <updateRate>0.0</updateRate>
-                        <cameraName>/camera</cameraName>
-                        <imageTopicName>image_raw</imageTopicName>
-                        <cameraInfoTopicName>camera_info</cameraInfoTopicName>
-                        <frameName>camera</frameName>
-                        <hackBaseline>0.07</hackBaseline>
-                        <distortionK1>0.0</distortionK1>
-                        <distortionK2>0.0</distortionK2>
-                        <distortionK3>0.0</distortionK3>
-                        <distortionT1>0.0</distortionT1>
-                        <distortionT2>0.0</distortionT2>
-                    </plugin>
-                </sensor>
-            </gazebo>
-        </xacro:if>
         <transmission name="trans_right_finger_joint">
             <type>transmission_interface/SimpleTransmission</type>
             <joint name="right_finger_joint">
                 <hardwareInterface>hardware_interface/EffortJointInterface</hardwareInterface>
-                <offset>-0.0640</offset>
+                <offset>0.0</offset>
             </joint>
             <actuator name="right_finger_motor">
                 <hardwareInterface>hardware_interface/EffortJointInterface</hardwareInterface>
-                <mechanicalReduction>1</mechanicalReduction>
+                <mechanicalReduction>-4712.388</mechanicalReduction>
             </actuator>
         </transmission>
-        <transmission name="trans_left_finger_joint">
-            <type>transmission_interface/SimpleTransmission</type>
-            <joint name="left_finger_joint">
-                <hardwareInterface>hardware_interface/EffortJointInterface</hardwareInterface>
-                <offset>-0.0640</offset>
-            </joint>
-            <actuator name="left_finger_motor">
-                <hardwareInterface>hardware_interface/EffortJointInterface</hardwareInterface>
-                <mechanicalReduction>1</mechanicalReduction>
-            </actuator>
-        </transmission>
+        <xacro:if value="${simulation}">
+            <!--            <gazebo reference="camera">-->
+            <!--                <sensor type="camera" name="camera_node">-->
+            <!--                    <update_rate>30.0</update_rate>-->
+            <!--                    <camera name="head">-->
+            <!--                        <horizontal_fov>1.3962634</horizontal_fov>-->
+            <!--                        <image>-->
+            <!--                            <width>1920</width>-->
+            <!--                            <height>1080</height>-->
+            <!--                            <format>R8G8B8</format>-->
+            <!--                        </image>-->
+            <!--                        <clip>-->
+            <!--                            <near>0.02</near>-->
+            <!--                            <far>300</far>-->
+            <!--                        </clip>-->
+            <!--                        <noise>-->
+            <!--                            <type>gaussian</type>-->
+            <!--                            <mean>0.0</mean>-->
+            <!--                            <stddev>0.007</stddev>-->
+            <!--                        </noise>-->
+            <!--                    </camera>-->
+            <!--                    <plugin name="gazebo_camera" filename="libgazebo_ros_camera.so">-->
+            <!--                        <alwaysOn>true</alwaysOn>-->
+            <!--                        <updateRate>0.0</updateRate>-->
+            <!--                        <cameraName>/camera</cameraName>-->
+            <!--                        <imageTopicName>image_raw</imageTopicName>-->
+            <!--                        <cameraInfoTopicName>camera_info</cameraInfoTopicName>-->
+            <!--                        <frameName>camera</frameName>-->
+            <!--                        <hackBaseline>0.07</hackBaseline>-->
+            <!--                        <distortionK1>0.0</distortionK1>-->
+            <!--                        <distortionK2>0.0</distortionK2>-->
+            <!--                        <distortionK3>0.0</distortionK3>-->
+            <!--                        <distortionT1>0.0</distortionT1>-->
+            <!--                        <distortionT2>0.0</distortionT2>-->
+            <!--                    </plugin>-->
+            <!--                </sensor>-->
+            <!--            </gazebo>-->
+        </xacro:if>
     </xacro:macro>
 </robot>

Commit message: Change offset

File: urdf/engineer/arm.transmission.xacro (robot description, xacro)
@@ -10,5 +10,5 @@
             <joint name="joint1">
                 <hardwareInterface>hardware_interface/EffortJointInterface</hardwareInterface>
-                <offset>0.0573</offset>
+                <offset>-0.02552</offset>
             </joint>
         </transmission>
@@ -20,5 +20,5 @@
             <joint name="joint3">
                 <hardwareInterface>hardware_interface/EffortJointInterface</hardwareInterface>
-                <offset>2.4715</offset>
+                <offset>-0.6104</offset>
             </joint>
         </transmission>
@@ -36,5 +36,5 @@
                 <joint name="joint2">
                     <hardwareInterface>hardware_interface/EffortJointInterface</hardwareInterface>
-                    <offset>-2.231</offset>
+                    <offset>-0.86486</offset>
                     <mechanicalReduction>1</mechanicalReduction>
                 </joint>
@@ -52,5 +52,5 @@
                 <joint name="joint4">
                     <role>joint1</role>
-                    <offset>1.0621</offset>
+                    <offset>1.192744</offset>
                     <mechanicalReduction>1</mechanicalReduction>
                     <hardwareInterface>hardware_interface/EffortJointInterface</hardwareInterface>
@@ -59,5 +59,5 @@
                 <joint name="joint5">
                     <role>joint2</role>
-                    <offset>0.1548</offset>
+                    <offset>0.04641</offset>
                     <mechanicalReduction>-1</mechanicalReduction>
                     <hardwareInterface>hardware_interface/EffortJointInterface</hardwareInterface>

File: urdf/engineer/arm.urdf.xacro (robot description, xacro)
@@ -153,5 +153,5 @@
             <axis xyz="1 0 0"/>
             <origin xyz="0 0 0"/>
-            <limit effort="1.2" velocity="34" lower="-${2*pi}" upper="${2*pi}"/>
+            <limit effort="1.2" velocity="34" lower="-${pi}" upper="${pi}"/>
             <dynamics damping="0.0" friction="0.05"/>
             <parent link="link4"/>

File: urdf/engineer/hand.urdf.xacro (robot description, xacro)
@@ -155,6 +155,6 @@
             <gazebo reference="right_finger">
                 <self_collide>1</self_collide>
-                <mu1 value="200000.0"/>
-                <mu2 value="200000.0"/>
+                <mu1 value="2000000000.0"/>
+                <mu2 value="2000000000.0"/>
                 <kp value="1000000.0"/>
                 <kd value="100.0"/>
@@ -163,6 +163,6 @@
             <gazebo reference="left_finger">
                 <self_collide>1</self_collide>
-                <mu1 value="200000.0"/>
-                <mu2 value="200000.0"/>
+                <mu1 value="2000000000.0"/>
+                <mu2 value="2000000000.0"/>
                 <kp value="1000000.0"/>
                 <kd value="100.0"/>

Commit message: uate engineer   and hand offset nd  mechanicalReduction

File: urdf/engineer/arm.transmission.xacro (robot description, xacro)
@@ -6,9 +6,9 @@
             <type>transmission_interface/SimpleTransmission</type>
             <actuator name="joint1_motor">
-                <mechanicalReduction>4</mechanicalReduction>
+                <mechanicalReduction>76.8128</mechanicalReduction>
             </actuator>
             <joint name="joint1">
                 <hardwareInterface>hardware_interface/EffortJointInterface</hardwareInterface>
-                <offset>-0.02552</offset>
+                <offset>-0.004</offset>
             </joint>
         </transmission>
@@ -20,5 +20,25 @@
             <joint name="joint3">
                 <hardwareInterface>hardware_interface/EffortJointInterface</hardwareInterface>
-                <offset>-0.6104</offset>
+                <offset>0.3592</offset>
+            </joint>
+        </transmission>
+        <transmission name="trans_joint4">
+            <type>transmission_interface/SimpleTransmission</type>
+            <actuator name="joint4_motor">
+                <mechanicalReduction>-27</mechanicalReduction>
+            </actuator>
+            <joint name="joint4">
+                <hardwareInterface>hardware_interface/EffortJointInterface</hardwareInterface>
+                <offset>1.454</offset>
+            </joint>
+        </transmission>
+        <transmission name="trans_joint5">
+            <type>transmission_interface/SimpleTransmission</type>
+            <actuator name="joint5_motor">
+                <mechanicalReduction>51</mechanicalReduction>
+            </actuator>
+            <joint name="joint5">
+                <hardwareInterface>hardware_interface/EffortJointInterface</hardwareInterface>
+                <offset>-0.1264</offset>
             </joint>
         </transmission>
@@ -36,33 +56,33 @@
                 <joint name="joint2">
                     <hardwareInterface>hardware_interface/EffortJointInterface</hardwareInterface>
-                    <offset>-0.86486</offset>
+                    <offset>0.0979</offset>
                     <mechanicalReduction>1</mechanicalReduction>
                 </joint>
             </transmission>
-            <transmission name="trans_wrist">
-                <type>transmission_interface/DifferentialTransmission</type>
-                <actuator name="left_wrist_motor">
-                    <role>actuator1</role>
-                    <mechanicalReduction>1.2</mechanicalReduction>
-                </actuator>
-                <actuator name="right_wrist_motor">
-                    <role>actuator2</role>
-                    <mechanicalReduction>-1.2</mechanicalReduction>
-                </actuator>
-                <joint name="joint4">
-                    <role>joint1</role>
-                    <offset>1.192744</offset>
-                    <mechanicalReduction>1</mechanicalReduction>
-                    <hardwareInterface>hardware_interface/EffortJointInterface</hardwareInterface>
-                    <ignoreTransmissionAbsoluteEncoder>1</ignoreTransmissionAbsoluteEncoder>
-                </joint>
-                <joint name="joint5">
-                    <role>joint2</role>
-                    <offset>0.04641</offset>
-                    <mechanicalReduction>-1</mechanicalReduction>
-                    <hardwareInterface>hardware_interface/EffortJointInterface</hardwareInterface>
-                    <ignoreTransmissionAbsoluteEncoder>1</ignoreTransmissionAbsoluteEncoder>
-                </joint>
-            </transmission>
+<!--            <transmission name="trans_wrist">-->
+<!--                <type>transmission_interface/DifferentialTransmission</type>-->
+<!--                <actuator name="left_wrist_motor">-->
+<!--                    <role>actuator1</role>-->
+<!--                    <mechanicalReduction>1.2</mechanicalReduction>-->
+<!--                </actuator>-->
+<!--                <actuator name="right_wrist_motor">-->
+<!--                    <role>actuator2</role>-->
+<!--                    <mechanicalReduction>-1.2</mechanicalReduction>-->
+<!--                </actuator>-->
+<!--                <joint name="joint4">-->
+<!--                    <role>joint1</role>-->
+<!--                    <offset>1.192744</offset>-->
+<!--                    <mechanicalReduction>1</mechanicalReduction>-->
+<!--                    <hardwareInterface>hardware_interface/EffortJointInterface</hardwareInterface>-->
+<!--                    <ignoreTransmissionAbsoluteEncoder>1</ignoreTransmissionAbsoluteEncoder>-->
+<!--                </joint>-->
+<!--                <joint name="joint5">-->
+<!--                    <role>joint2</role>-->
+<!--                    <offset>0.04641</offset>-->
+<!--                    <mechanicalReduction>-1</mechanicalReduction>-->
+<!--                    <hardwareInterface>hardware_interface/EffortJointInterface</hardwareInterface>-->
+<!--                    <ignoreTransmissionAbsoluteEncoder>1</ignoreTransmissionAbsoluteEncoder>-->
+<!--                </joint>-->
+<!--            </transmission>-->
         </xacro:unless>
         <xacro:if value="${simulation}">
@@ -77,22 +97,4 @@
                 </joint>
             </transmission>
-            <transmission name="trans_joint4">
-                <type>transmission_interface/SimpleTransmission</type>
-                <actuator name="joint4_motor">
-                    <mechanicalReduction>1</mechanicalReduction>
-                </actuator>
-                <joint name="joint4">
-                    <hardwareInterface>hardware_interface/EffortJointInterface</hardwareInterface>
-                </joint>
-            </transmission>
-            <transmission name="trans_joint5">
-                <type>transmission_interface/SimpleTransmission</type>
-                <actuator name="joint5_motor">
-                    <mechanicalReduction>1</mechanicalReduction>
-                </actuator>
-                <joint name="joint5">
-                    <hardwareInterface>hardware_interface/EffortJointInterface</hardwareInterface>
-                </joint>
-            </transmission>
         </xacro:if>
     </xacro:macro>

File: urdf/engineer/arm.urdf.xacro (robot description, xacro)
@@ -147,5 +147,5 @@
             <axis xyz="0 1 0"/>
             <origin xyz="0.005 0.128 0" rpy="-1.57 0 0"/>
-            <limit effort="30" velocity="10" lower="-2.231" upper="0.407"/>
+            <limit effort="30" velocity="10" lower="-2.5249" upper="0.042903"/>
             <dynamics damping="0.0" friction="0.8"/>
             <parent link="link1"/>
@@ -155,5 +155,5 @@
             <axis xyz="0 1 0"/>
             <origin xyz="0.165 0 0" rpy="0 0 0"/>
-            <limit effort="30" velocity="10" lower="-2.1645" upper="2.4078"/>
+            <limit effort="30" velocity="10" lower="-0.7203" upper="2.6055"/>
             <dynamics damping="0.0" friction="0.5"/>
             <parent link="link2"/>
@@ -163,6 +163,6 @@
             <axis xyz="0 1 0"/>
             <origin xyz="0.106 0 0.028"/>
-            <limit effort="2.4" velocity="34" lower="-${0.55*pi}" upper="${0.55*pi}"/>
-            <dynamics damping="0.0" friction="0.05"/>
+            <limit effort="10" velocity="25" lower="-0.21556" upper="2.6459"/>
+            <dynamics damping="0.0" friction="0.5"/>
             <parent link="link3"/>
             <child link="link4"/>
@@ -171,6 +171,6 @@
             <axis xyz="1 0 0"/>
             <origin xyz="0.097 0 0.055"/>
-            <limit effort="1.2" velocity="34" lower="-${pi}" upper="${pi}"/>
-            <dynamics damping="0.0" friction="0.05"/>
+            <limit effort="10" velocity="25" lower="-3.139" upper="0.5454"/>
+            <dynamics damping="0.0" friction="0.5"/>
             <parent link="link4"/>
             <child link="link5"/>

File: urdf/engineer/hand.urdf.xacro (robot description, xacro)
@@ -171,5 +171,5 @@
             </joint>
             <actuator name="right_finger_motor">
-                <mechanicalReduction>2356.194</mechanicalReduction>
+                <mechanicalReduction>-2356.194</mechanicalReduction>
             </actuator>
         </transmission>

Commit message: update engineer transmission offset

File: urdf/engineer/arm.transmission.xacro (robot description, xacro)
@@ -20,5 +20,5 @@
             <joint name="joint3">
                 <hardwareInterface>hardware_interface/EffortJointInterface</hardwareInterface>
-                <offset>0.3592</offset>
+                <offset>2.4659</offset>
             </joint>
         </transmission>
@@ -56,33 +56,8 @@
                 <joint name="joint2">
                     <hardwareInterface>hardware_interface/EffortJointInterface</hardwareInterface>
-                    <offset>0.0979</offset>
+                    <offset>-2.3884</offset>
                     <mechanicalReduction>1</mechanicalReduction>
                 </joint>
             </transmission>
-<!--            <transmission name="trans_wrist">-->
-<!--                <type>transmission_interface/DifferentialTransmission</type>-->
-<!--                <actuator name="left_wrist_motor">-->
-<!--                    <role>actuator1</role>-->
-<!--                    <mechanicalReduction>1.2</mechanicalReduction>-->
-<!--                </actuator>-->
-<!--                <actuator name="right_wrist_motor">-->
-<!--                    <role>actuator2</role>-->
-<!--                    <mechanicalReduction>-1.2</mechanicalReduction>-->
-<!--                </actuator>-->
-<!--                <joint name="joint4">-->
-<!--                    <role>joint1</role>-->
-<!--                    <offset>1.192744</offset>-->
-<!--                    <mechanicalReduction>1</mechanicalReduction>-->
-<!--                    <hardwareInterface>hardware_interface/EffortJointInterface</hardwareInterface>-->
-<!--                    <ignoreTransmissionAbsoluteEncoder>1</ignoreTransmissionAbsoluteEncoder>-->
-<!--                </joint>-->
-<!--                <joint name="joint5">-->
-<!--                    <role>joint2</role>-->
-<!--                    <offset>0.04641</offset>-->
-<!--                    <mechanicalReduction>-1</mechanicalReduction>-->
-<!--                    <hardwareInterface>hardware_interface/EffortJointInterface</hardwareInterface>-->
-<!--                    <ignoreTransmissionAbsoluteEncoder>1</ignoreTransmissionAbsoluteEncoder>-->
-<!--                </joint>-->
-<!--            </transmission>-->
         </xacro:unless>
         <xacro:if value="${simulation}">

File: urdf/engineer/hand.urdf.xacro (robot description, xacro)
@@ -127,5 +127,5 @@
             <origin xyz="0 0 0.045" rpy="0 0 0"/>
             <axis xyz="0 1 0"/>
-            <limit effort="588" lower="0.0" upper="0.03" velocity="3.772"/>
+            <limit effort="588" lower="-0.025" upper="0.0" velocity="3.772"/>
         </joint>
         <joint name="left_finger_joint" type="prismatic">
@@ -134,5 +134,5 @@
             <origin xyz="0 0 0.045" rpy="0 0 0"/>
             <axis xyz="0 -1 0"/>
-            <limit effort="588" lower="0.0" upper="0.03" velocity="3.772"/>
+            <limit effort="588" lower="-0.025" upper="0.0" velocity="3.772"/>
             <mimic joint="right_finger_joint"/>
         </joint>
