Commit message: update limit d accurate mechanicalReduction

File: urdf/engineer/arm.transmission.xacro (robot description, xacro)
@@ -26,5 +26,5 @@
             <type>transmission_interface/SimpleTransmission</type>
             <actuator name="joint4_motor">
-                <mechanicalReduction>-27</mechanicalReduction>
+                <mechanicalReduction>-26.851</mechanicalReduction>
             </actuator>
             <joint name="joint4">
@@ -36,5 +36,5 @@
             <type>transmission_interface/SimpleTransmission</type>
             <actuator name="joint5_motor">
-                <mechanicalReduction>51</mechanicalReduction>
+                <mechanicalReduction>50.895</mechanicalReduction>
             </actuator>
             <joint name="joint5">

File: urdf/engineer/arm.urdf.xacro (robot description, xacro)
@@ -139,5 +139,5 @@
             <origin xyz="0.133 0 1" rpy="1.57 0 0"/>
             <!--      limit not work while type="continuous"-->
-            <limit effort="20" velocity="25" lower="-${pi}" upper="${pi}"/>
+            <limit effort="20" velocity="10" lower="-${pi}" upper="${pi}"/>
             <dynamics damping="0.0" friction="0.1"/>
             <parent link="${connected_to}"/>
@@ -163,5 +163,5 @@
             <axis xyz="0 1 0"/>
             <origin xyz="0.106 0 0.028"/>
-            <limit effort="10" velocity="25" lower="-0.21556" upper="2.6459"/>
+            <limit effort="7" velocity="30" lower="-0.21556" upper="2.6459"/>
             <dynamics damping="0.0" friction="0.5"/>
             <parent link="link3"/>
@@ -171,5 +171,5 @@
             <axis xyz="1 0 0"/>
             <origin xyz="0.097 0 0.055"/>
-            <limit effort="10" velocity="25" lower="-3.139" upper="0.5454"/>
+            <limit effort="13" velocity="18" lower="-3.139" upper="0.5454"/>
             <dynamics damping="0.0" friction="0.5"/>
             <parent link="link4"/>

Commit message: update engineer collision

File: urdf/engineer/arm.transmission.xacro (robot description, xacro)
@@ -69,5 +69,5 @@
                 <joint name="joint2">
                     <hardwareInterface>hardware_interface/EffortJointInterface</hardwareInterface>
-                    <offset>0</offset>
+                    <offset>-2.3764</offset>
                 </joint>
             </transmission>

File: urdf/engineer/arm.urdf.xacro (robot description, xacro)
@@ -19,10 +19,4 @@
                 <geometry>
                     <box size="0.088 0.142 0.106"/>
-                </geometry>
-            </collision>
-            <collision>
-                <origin xyz="-0.032 0.068 0" rpy="0 0 -0.593"/>
-                <geometry>
-                    <box size="0.097 0.14 0.106"/>
                 </geometry>
             </collision>
@@ -127,10 +121,10 @@
                 </geometry>
             </visual>
-            <collision>
-                <origin xyz="-0.054 0 0" rpy="0 1.57 0"/>
-                <geometry>
-                    <cylinder length="0.108" radius="0.021"/>
-                </geometry>
-            </collision>
+<!--            <collision>-->
+<!--                <origin xyz="-0.054 0 0" rpy="0 1.57 0"/>-->
+<!--                <geometry>-->
+<!--                    <cylinder length="0.108" radius="0.021"/>-->
+<!--                </geometry>-->
+<!--            </collision>-->
         </link>
         <!--  joint  -->

File: urdf/engineer/chassis.urdf.xacro (robot description, xacro)
@@ -78,5 +78,5 @@
             </collision>
             <collision>
-                <origin xyz="0.0 0 0" rpy="0 0 1.0646508"/>
+                <origin xyz="-0.0239 0.084 0.228" rpy="0 0 1.0646508"/>
                 <geometry>
                     <box size="0.080 0.003 0.250"/>
@@ -103,8 +103,35 @@
             </collision>
         </link>
+        <link name="card">
+            <inertial>
+                <mass value="0.26"/>
+                <origin xyz="-0.071 -0.006 0.003"/>
+                <inertia ixx="1.078e-3" ixy="6.486e-5" ixz="1.454e-5" iyy="1.142e-4" iyz="5.143e-6" izz="2.215e-3"/>
+            </inertial>
+            <visual>
+                <origin xyz="0 0 0" rpy="0 0 0"/>
+                <geometry>
+                    <mesh filename="package://rm_description/meshes/engineer/card.stl" scale="0.001 0.001 0.001"/>
+                </geometry>
+            </visual>
+            <collision>
+                <origin xyz="-0.113 0.134 0.0" rpy="0 0.0 0"/>
+                <geometry>
+                    <box size="0.253 0.151 0.011"/>
+                </geometry>
+            </collision>
+        </link>
+        <joint name="card_joint" type="prismatic">
+            <axis xyz="1 0 0"/>
+            <origin xyz="0.109 0.001 -0.11"/>
+            <limit effort="0.1" velocity="30" lower="0" upper="0.05"/>
+            <dynamics damping="0.0" friction="0.1"/>
+            <parent link="base_link"/>
+            <child link="card"/>
+        </joint>
         <joint name="stone_platform_joint" type="prismatic">
             <axis xyz="0 0 1"/>
             <origin xyz="-0.113 0.134 0.114"/>
-            <limit effort="7" velocity="30" lower="0" upper="2.6459"/>
+            <limit effort="1" velocity="30" lower="0" upper="0.024"/>
             <dynamics damping="0.0" friction="0.1"/>
             <parent link="base_link"/>
@@ -117,4 +144,14 @@
             </actuator>
             <joint name="stone_platform_joint">
+                <hardwareInterface>hardware_interface/EffortJointInterface</hardwareInterface>
+                <offset>0</offset>
+            </joint>
+        </transmission>
+        <transmission name="trans_card_joint">
+            <type>transmission_interface/SimpleTransmission</type>
+            <actuator name="card_joint_motor">
+                <mechanicalReduction>49.97</mechanicalReduction>
+            </actuator>
+            <joint name="card_joint">
                 <hardwareInterface>hardware_interface/EffortJointInterface</hardwareInterface>
                 <offset>0</offset>

File: urdf/engineer/hand.urdf.xacro (robot description, xacro)
@@ -23,8 +23,11 @@
                 <origin xyz="0 0 0.027" rpy="0 0 0"/>
                 <geometry>
-                    <box size="0.055 0.267 0.06"/>
+                    <box size="0.055 0.267 0.055"/>
                 </geometry>
             </collision>
         </link>
+        <gazebo reference="palm">
+            <self_collide>1</self_collide>
+        </gazebo>
         <link name="right_finger">
             <inertial>
@@ -39,14 +42,14 @@
                 </geometry>
             </visual>
+<!--            <collision>-->
+<!--                <origin xyz="0.0 0.046 0.005" rpy="0 0 0"/>-->
+<!--                <geometry>-->
+<!--                    <box size="0.030 0.027 0.063"/>-->
+<!--                </geometry>-->
+<!--            </collision>-->
             <collision>
-                <origin xyz="0.0 0.046 0.005" rpy="0 0 0"/>
+                <origin xyz="0.0 0.088 0.025" rpy="0 0 0"/>
                 <geometry>
-                    <box size="0.030 0.027 0.063"/>
-                </geometry>
-            </collision>
-            <collision>
-                <origin xyz="0.0 0.091 0.025" rpy="0 0 0"/>
-                <geometry>
-                    <box size="0.03 0.109 0.022"/>
+                    <box size="0.03 0.112 0.022"/>
                 </geometry>
             </collision>
@@ -70,14 +73,14 @@
                 </geometry>
             </visual>
-            <collision>
-                <origin xyz="0.0 -0.043 0.005" rpy="0 0 0"/>
-                <geometry>
-                    <box size="0.030 0.027 0.063"/>
-                </geometry>
-            </collision>
+<!--            <collision>-->
+<!--                <origin xyz="0.0 -0.043 0.005" rpy="0 0 0"/>-->
+<!--                <geometry>-->
+<!--                    <box size="0.030 0.027 0.063"/>-->
+<!--                </geometry>-->
+<!--            </collision>-->
             <collision>
                 <origin xyz="0.0 -0.088 0.025" rpy="0 0 0"/>
                 <geometry>
-                    <box size="0.03 0.109 0.022"/>
+                    <box size="0.03 0.112 0.022"/>
                 </geometry>
             </collision>

File: urdf/engineer/mast.urdf.xacro (robot description, xacro)
@@ -17,5 +17,5 @@
                 <origin xyz="0.004 0 -0.259" rpy="0 0 0"/>
                 <geometry>
-                    <box size="0.053 0.035 0.45"/>
+                    <box size="0.035 0.035 0.4"/>
                 </geometry>
             </collision>
@@ -38,10 +38,4 @@
                 </geometry>
             </visual>
-<!--            <collision>-->
-<!--                <origin xyz="0.0 0.004 0.03" rpy="0 0 0"/>-->
-<!--                <geometry>-->
-<!--                    <cylinder length="0.14" radius="0.01"/>-->
-<!--                </geometry>-->
-<!--            </collision>-->
         </link>
         <link name="pitch">
@@ -56,10 +50,4 @@
                 </geometry>
             </visual>
-<!--            <collision>-->
-<!--                <origin xyz="-0.005 -0.04 0.014" rpy="0 0 0"/>-->
-<!--                <geometry>-->
-<!--                    <box size="0.1 0.048 0.036"/>-->
-<!--                </geometry>-->
-<!--            </collision>-->
         </link>
 <!--        <link name="camera_telephoto"/>-->
@@ -94,4 +82,7 @@
             <axis xyz="0 1 0 "/>
         </joint>
+        <gazebo reference="mast">
+            <self_collide>1</self_collide>
+        </gazebo>
 <!--        <joint name="camera_wideangle_joint" type="fixed">-->
 <!--            <parent link="pitch"/>-->

Commit message: update engineer offset

File: urdf/engineer/arm.transmission.xacro (robot description, xacro)
@@ -10,5 +10,5 @@
             <joint name="joint1">
                 <hardwareInterface>hardware_interface/EffortJointInterface</hardwareInterface>
-                <offset>-0.004</offset>
+                <offset>0</offset>
             </joint>
         </transmission>
@@ -20,5 +20,5 @@
             <joint name="joint3">
                 <hardwareInterface>hardware_interface/EffortJointInterface</hardwareInterface>
-                <offset>2.3713</offset>
+                <offset>-0.82513</offset>
             </joint>
         </transmission>
@@ -30,5 +30,5 @@
             <joint name="joint4">
                 <hardwareInterface>hardware_interface/EffortJointInterface</hardwareInterface>
-                <offset>1.454</offset>
+                <offset>-0.28587</offset>
             </joint>
         </transmission>
@@ -40,5 +40,5 @@
             <joint name="joint5">
                 <hardwareInterface>hardware_interface/EffortJointInterface</hardwareInterface>
-                <offset>-0.1264</offset>
+                <offset>0.886556</offset>
             </joint>
         </transmission>
@@ -56,5 +56,5 @@
                 <joint name="joint2">
                     <hardwareInterface>hardware_interface/EffortJointInterface</hardwareInterface>
-                    <offset>-2.3764</offset>
+                    <offset>-2.45428</offset>
                     <mechanicalReduction>1</mechanicalReduction>
                 </joint>

File: urdf/engineer/arm.urdf.xacro (robot description, xacro)
@@ -135,5 +135,5 @@
             <axis xyz="0 1 0"/>
             <origin xyz="0.005 0.128 0" rpy="-1.57 0 0"/>
-            <limit effort="30" velocity="10" lower="-2.5249" upper="0.042903"/>
+            <limit effort="60" velocity="10" lower="-2.5249" upper="0.042903"/>
             <dynamics damping="0.0" friction="0.8"/>
             <parent link="link1"/>

Commit message: Update joint1 offset and limit

File: urdf/engineer/arm.transmission.xacro (robot description, xacro)
@@ -10,5 +10,5 @@
             <joint name="joint1">
                 <hardwareInterface>hardware_interface/EffortJointInterface</hardwareInterface>
-                <offset>-0.86371</offset>
+                <offset>-0.9260763</offset>
             </joint>
         </transmission>
@@ -40,5 +40,5 @@
             <joint name="joint5">
                 <hardwareInterface>hardware_interface/EffortJointInterface</hardwareInterface>
-                <offset>0</offset>
+                <offset>2.099906</offset>
             </joint>
         </transmission>

File: urdf/engineer/arm.urdf.xacro (robot description, xacro)
@@ -127,5 +127,5 @@
             <origin xyz="0.122 0 0.124" rpy="1.57 0 0"/>
             <!--      limit not work while type="continuous"-->
-            <limit effort="20" velocity="10" lower="-0.8507492" upper="5.2558426"/>
+            <limit effort="20" velocity="10" lower="-3.93996572" upper="1.805202294"/>
             <dynamics damping="0.0" friction="0.1"/>
             <parent link="${connected_to}"/>

Commit message: Change joint1 calibration controller toward

File: urdf/engineer/arm.transmission.xacro (robot description, xacro)
@@ -10,5 +10,5 @@
             <joint name="joint1">
                 <hardwareInterface>hardware_interface/EffortJointInterface</hardwareInterface>
-                <offset>-4.0653796</offset>
+                <offset>5.2446903</offset>
             </joint>
         </transmission>

File: urdf/engineer/arm.urdf.xacro (robot description, xacro)
@@ -3,6 +3,6 @@
     <xacro:macro name="arm" params="connected_to">
     <xacro:property name="threshold" value="0.1"/>
-    <xacro:property name="joint1_lower_limit" value="-4.0492335499"/>
-    <xacro:property name="joint1_upper_limit" value="2.066574686023"/>
+    <xacro:property name="joint1_lower_limit" value="-0.88190193"/>
+    <xacro:property name="joint1_upper_limit" value="5.233317170108"/>
     <xacro:property name="joint2_lower_limit" value="-2.378679831401"/>
     <xacro:property name="joint2_upper_limit" value="-0.0989819625299"/>

Commit message: Update joint1 limit and offset

File: urdf/engineer/arm.transmission.xacro (robot description, xacro)
@@ -10,5 +10,5 @@
             <joint name="joint1">
                 <hardwareInterface>hardware_interface/EffortJointInterface</hardwareInterface>
-                <offset>5.2446903</offset>
+                <offset>2.092296433</offset>
             </joint>
         </transmission>

File: urdf/engineer/arm.urdf.xacro (robot description, xacro)
@@ -3,6 +3,6 @@
     <xacro:macro name="arm" params="connected_to">
     <xacro:property name="threshold" value="0.1"/>
-    <xacro:property name="joint1_lower_limit" value="-0.88190193"/>
-    <xacro:property name="joint1_upper_limit" value="5.233317170108"/>
+    <xacro:property name="joint1_lower_limit" value="-4.02409094"/>
+    <xacro:property name="joint1_upper_limit" value="2.074442915664"/>
     <xacro:property name="joint2_lower_limit" value="-2.378679831401"/>
     <xacro:property name="joint2_upper_limit" value="-0.0989819625299"/>

Commit message: Change the offset and limit of engineer's joint1

File: urdf/engineer/arm.transmission.xacro (robot description, xacro)
@@ -6,9 +6,9 @@
             <type>transmission_interface/SimpleTransmission</type>
             <actuator name="joint1_motor">
-                <mechanicalReduction>76.8128</mechanicalReduction>
+                <mechanicalReduction>71.75</mechanicalReduction>
             </actuator>
             <joint name="joint1">
                 <hardwareInterface>hardware_interface/EffortJointInterface</hardwareInterface>
-                <offset>2.092296433</offset>
+                <offset>2.068</offset>
             </joint>
         </transmission>

File: urdf/engineer/arm.urdf.xacro (robot description, xacro)
@@ -2,15 +2,15 @@
 <robot xmlns:xacro="http://www.ros.org/wiki/xacro" name="arm">
     <xacro:macro name="arm" params="connected_to">
-    <xacro:property name="threshold" value="0.1"/>
-    <xacro:property name="joint1_lower_limit" value="-4.02409094"/>
-    <xacro:property name="joint1_upper_limit" value="2.074442915664"/>
-    <xacro:property name="joint2_lower_limit" value="-2.378679831401"/>
-    <xacro:property name="joint2_upper_limit" value="-0.0989819625299"/>
-    <xacro:property name="joint3_lower_limit" value="-0.88921949"/>
-    <xacro:property name="joint3_upper_limit" value="2.535032168"/>
-    <xacro:property name="joint4_lower_limit" value="-0.2989008"/>
-    <xacro:property name="joint4_upper_limit" value="2.614725376878"/>
-    <xacro:property name="joint5_lower_limit" value="-4.27171178"/>
-    <xacro:property name="joint5_upper_limit" value="1.40800999"/>
+        <xacro:property name="threshold" value="0.1"/>
+        <xacro:property name="joint1_lower_limit" value="-4.0246823"/>
+        <xacro:property name="joint1_upper_limit" value="2.05507607"/>
+        <xacro:property name="joint2_lower_limit" value="-2.378679831401"/>
+        <xacro:property name="joint2_upper_limit" value="-0.0989819625299"/>
+        <xacro:property name="joint3_lower_limit" value="-0.88921949"/>
+        <xacro:property name="joint3_upper_limit" value="2.535032168"/>
+        <xacro:property name="joint4_lower_limit" value="-0.2989008"/>
+        <xacro:property name="joint4_upper_limit" value="2.614725376878"/>
+        <xacro:property name="joint5_lower_limit" value="-4.27171178"/>
+        <xacro:property name="joint5_upper_limit" value="1.40800999"/>
         <!--  link  -->
         <link name="link1">
@@ -126,10 +126,4 @@
                 </geometry>
             </visual>
-<!--            <collision>-->
-<!--                <origin xyz="-0.054 0 0" rpy="0 1.57 0"/>-->
-<!--                <geometry>-->
-<!--                    <cylinder length="0.108" radius="0.021"/>-->
-<!--                </geometry>-->
-<!--            </collision>-->
         </link>
         <!--  joint  -->
@@ -138,5 +132,5 @@
             <origin xyz="0.175 0 0.164" rpy="0 0 0"/>
             <!--      limit not work while type="continuous"-->
-            <limit effort="20" velocity="10" lower="${joint1_lower_limit}" upper="${joint1_upper_limit}"/>
+            <limit effort="20" velocity="13" lower="${joint1_lower_limit}" upper="${joint1_upper_limit}"/>
             <safety_controller k_position="37.5" k_velocity="10"
                                soft_lower_limit="${joint1_lower_limit+threshold}"

Commit message: Update engineer arm URDF

File: urdf/engineer/arm.transmission.xacro (robot description, xacro)
@@ -20,5 +20,5 @@
             <joint name="joint3">
                 <hardwareInterface>hardware_interface/EffortJointInterface</hardwareInterface>
-                <offset>-0.9671676701</offset>
+                <offset>-0.85</offset>
             </joint>
         </transmission>

File: urdf/engineer/chassis.urdf.xacro (robot description, xacro)
@@ -62,5 +62,5 @@
                 <origin xyz="-0.148196 0.0485 0.224" rpy="0 0 -0.507"/>
                 <geometry>
-                    <box size="0.08 0.024213 0.448"/>
+                    <box size="0.08 0.05 0.448"/>
                 </geometry>
             </collision>

File: urdf/engineer/mast.urdf.xacro (robot description, xacro)
@@ -65,5 +65,5 @@
                     rpy="0 0 0"/>
             <dynamics damping="0.0" friction="0.1"/>
-            <limit effort="0.1" velocity="10" lower="-0.23087" upper="3.496015"/>
+            <limit effort="0.2" velocity="10" lower="-0.6197" upper="3.4545"/>
             <parent link="mast"/>
             <child link="yaw"/>
@@ -87,5 +87,5 @@
             </actuator>
             <joint name="yaw_joint">
-                <offset>-0.2538</offset>
+                <offset>-0.60668</offset>
                 <hardwareInterface>hardware_interface/EffortJointInterface</hardwareInterface>
             </joint>
