Commit message: move some collision

File: urdf/engineer/chassis.urdf.xacro (robot description, xacro)
@@ -27,16 +27,16 @@
                 </geometry>
             </collision>
-            <collision>
-                <origin xyz="-0.033 -0.1 0.267" rpy="0 0 0.7853982"/>
-                <geometry>
-                    <box size="0.0207 0.0207 0.334"/>
-                </geometry>
-            </collision>
-            <collision>
-                <origin xyz="-0.033 0.10 0.267" rpy="0 0 0.7853982"/>
-                <geometry>
-                    <box size="0.0207 0.0207 0.334"/>
-                </geometry>
-            </collision>
+            <!--            <collision>
+                            <origin xyz="-0.033 -0.1 0.267" rpy="0 0 0.7853982"/>
+                            <geometry>
+                                <box size="0.0207 0.0207 0.334"/>
+                            </geometry>
+                        </collision>
+                        <collision>
+                            <origin xyz="-0.033 0.10 0.267" rpy="0 0 0.7853982"/>
+                            <geometry>
+                                <box size="0.0207 0.0207 0.334"/>
+                            </geometry>
+                        </collision>-->
             <collision>
                 <origin xyz="-0.23225 -0.1 0.267" rpy="0 0 0.7853982"/>

Commit message: Add the camera model in description

File: urdf/engineer/chassis.urdf.xacro (robot description, xacro)
@@ -10,8 +10,8 @@
         <link name="base_link">
             <inertial>
-                <mass value="137.6"/>
-                <origin xyz="-0.12101 -0.0025 0.25321"/>
-                <inertia ixx="1.254e+1" ixy="-8.377e-2" ixz="4.560e+0" iyy=" 1.480e+1"
-                         iyz="5.948e-2" izz="4.106e+0"/>
+                <mass value="28.19"/>
+                <origin xyz="-0.0206 -0.00126 -0.0164"/>
+                <inertia ixx="1.32e+0" ixy="-8.378e-2" ixz="6.28e-2" iyy=" 1.549e+0"
+                         iyz="5.948e-2" izz="2.024e+0"/>
             </inertial>
             <visual>

File: urdf/engineer/hand.urdf.xacro (robot description, xacro)
@@ -95,4 +95,33 @@
             </collision>
         </link>
+        <link name="camera">
+            <inertial>
+                <mass value="0.04"/>
+                <origin xyz="0 0 0"/>
+                <inertia ixx="0.01" ixy="0.0" ixz="0.0" iyy="0.01" iyz="0.0" izz="0.01"/>
+            </inertial>
+            <visual>
+                <origin xyz=" 0 0 0 " rpy="0 0 0"/>
+                <geometry>
+                    <box size="0.022 0.021 0.0226"/>
+                </geometry>
+                <material name="Black"/>
+            </visual>
+            <collision>
+                <origin xyz="0.0 0.0 0.0" rpy="0 0 0"/>
+                <geometry>
+                    <box size="0.01 0.04 0.04"/>
+                </geometry>
+            </collision>
+        </link>
+        <!--        <gazebo reference="camera">-->
+        <!--            <masterial>Gazebo/White</masterial>-->
+        <!--        </gazebo>-->
+        <joint name="camera_joint" type="fixed">
+            <parent link="palm"/>
+            <child link="camera"/>
+            <origin xyz="0.055 -0.085 0.0962" rpy="0 0 0"/>
+            <axis xyz="0 1 0"/>
+        </joint>
         <xacro:unless value="${connected_to == ''}">
             <joint name="palm_joint" type="fixed">
@@ -139,4 +168,40 @@
             </actuator>
         </transmission>
+        <gazebo reference="camera">
+            <sensor type="camera" name="camera_node">
+                <update_rate>30.0</update_rate>
+                <camera name="head">
+                    <horizontal_fov>1.3962634</horizontal_fov>
+                    <image>
+                        <width>800</width>
+                        <height>800</height>
+                        <format>R8G8B8</format>
+                    </image>
+                    <clip>
+                        <near>0.02</near>
+                        <far>300</far>
+                    </clip>
+                    <noise>
+                        <type>gaussian</type>
+                        <mean>0.0</mean>
+                        <stddev>0.007</stddev>
+                    </noise>
+                </camera>
+                <plugin name="gazebo_camera" filename="libgazebo_ros_camera.so">
+                    <alwaysOn>true</alwaysOn>
+                    <updateRate>0.0</updateRate>
+                    <cameraName>/camera</cameraName>
+                    <imageTopicName>image_raw</imageTopicName>
+                    <cameraInfoTopicName>camera_info</cameraInfoTopicName>
+                    <frameName>camera</frameName>
+                    <hackBaseline>0.07</hackBaseline>
+                    <distortionK1>0.0</distortionK1>
+                    <distortionK2>0.0</distortionK2>
+                    <distortionK3>0.0</distortionK3>
+                    <distortionT1>0.0</distortionT1>
+                    <distortionT2>0.0</distortionT2>
+                </plugin>
+            </sensor>
+        </gazebo>
     </xacro:macro>
 </robot>

Commit message: update baselink parameter

File: urdf/engineer/chassis.urdf.xacro (robot description, xacro)
@@ -10,8 +10,8 @@
         <link name="base_link">
             <inertial>
-                <mass value="28.19"/>
-                <origin xyz="-0.0206 -0.00126 -0.0164"/>
-                <inertia ixx="1.32e+0" ixy="-8.378e-2" ixz="6.28e-2" iyy="1.549e+0"
-                         iyz="5.948e-2" izz="2.024e+0"/>
+                <mass value="11.91"/>
+                <origin xyz="-0.063 -0.010 -0.027"/>
+                <inertia ixx="4.230e-1" ixy="-5.057e-4" ixz="3.328e-2" iyy="3.602e-1"
+                         iyz="1.417e-2" izz="5.140e-1"/>
             </inertial>
             <visual>
@@ -22,43 +22,61 @@
             </visual>
             <collision>
-                <origin xyz="0 0 0" rpy="0 0 0"/>
+                <origin xyz="-0.043 0 0.020" rpy="0 0 0"/>
                 <geometry>
-                    <box size="0.5845 0.526 0.2"/>
+                    <box size="0.486 0.596 0.169"/>
                 </geometry>
             </collision>
-            <!--            <collision>
-                            <origin xyz="-0.033 -0.1 0.267" rpy="0 0 0.7853982"/>
+                        <collision>
+                            <origin xyz="-0.130 -0.132 0.255" rpy="0 0 0.8377580"/>
                             <geometry>
-                                <box size="0.0207 0.0207 0.334"/>
+                                <box size="0.106 0.186 0.3"/>
                             </geometry>
                         </collision>
                         <collision>
-                            <origin xyz="-0.033 0.10 0.267" rpy="0 0 0.7853982"/>
+                            <origin xyz="-0.0336 -0.27 0.262" rpy="0 0 -0.7853982"/>
                             <geometry>
-                                <box size="0.0207 0.0207 0.334"/>
+                                <box size="0.01 0.033 0.06"/>
                             </geometry>
-                        </collision>-->
+                        </collision>
             <collision>
-                <origin xyz="-0.23225 -0.1 0.267" rpy="0 0 0.7853982"/>
+                <origin xyz="-0.083 -0.225 0.262" rpy="0 0 -0.7853982"/>
                 <geometry>
-                    <box size="0.0207 0.0207 0.334"/>
+                    <box size="0.01 0.033 0.06"/>
                 </geometry>
             </collision>
             <collision>
-                <origin xyz="-0.23225 0.1 0.267" rpy="0 0 0.7853982"/>
+                <origin xyz="-0.0685 -0.259 0.287" rpy="0 0 0.8377580"/>
                 <geometry>
-                    <box size="0.0207 0.0207 0.334"/>
+                    <box size="0.003 0.057 0.01"/>
                 </geometry>
             </collision>
             <collision>
-                <origin xyz="-0.193 -0.189 0.235" rpy="0 0 0"/>
+                <origin xyz="-0.0685 -0.259 0.237" rpy="0 0 0.8377580"/>
                 <geometry>
-                    <box size="0.186 0.1 0.3"/>
+                    <box size="0.003 0.057 0.01"/>
                 </geometry>
             </collision>
             <collision>
-                <origin xyz="-0.0623 -0.2405 0.242" rpy="0 0 0"/>
+                <origin xyz="-0.0866 0.238 0.2672" rpy="0 0 -0.5061455"/>
                 <geometry>
-                    <box size="0.08 0.003 0.06"/>
+                    <box size="0.08 0.0217 0.3033"/>
+                </geometry>
+            </collision>
+            <collision>
+                <origin xyz="-0.2041 0.1846 0.25833" rpy="0 0 1.0646508"/>
+                <geometry>
+                    <box size="0.08 0.0217 0.3033"/>
+                </geometry>
+            </collision>
+            <collision>
+                <origin xyz="-0.1873 0.0566 0.2672" rpy="0 0 -0.5061455"/>
+                <geometry>
+                    <box size="0.08 0.0217 0.3033"/>
+                </geometry>
+            </collision>
+            <collision>
+                <origin xyz="-0.139 0.0847 0.228" rpy="0 0 1.0646508"/>
+                <geometry>
+                    <box size="0.080 0.003 0.250"/>
                 </geometry>
             </collision>

Commit message: update chassis platform

File: urdf/engineer/chassis.urdf.xacro (robot description, xacro)
@@ -84,4 +84,41 @@
             </collision>
         </link>
+        <link name="platform">
+            <inertial>
+                <mass value="0.073"/>
+                <origin xyz="-0.037 -0.005 0.009"/>
+                <inertia ixx="5.874e-4" ixy="-2.845e-4" ixz="1.882e-5" iyy=" 2.133e-4" iyz="2.682e-5" izz="7.780e-4"/>
+            </inertial>
+            <visual>
+                <origin xyz="0 0 0" rpy="0 0 0"/>
+                <geometry>
+                    <mesh filename="package://rm_description/meshes/engineer/platform.stl" scale="0.001 0.001 0.001"/>
+                </geometry>
+            </visual>
+            <collision>
+                <origin xyz="-0.113 0.134 0.114" rpy="0 0.0 0"/>
+                <geometry>
+                    <box size="0.106 0.105 0.002"/>
+                </geometry>
+            </collision>
+        </link>
+        <joint name="platform_joint" type="prismatic">
+            <axis xyz="0 1 0"/>
+            <origin xyz="-0.113 0.134 0.114"/>
+            <limit effort="7" velocity="30" lower="0" upper="2.6459"/>
+            <dynamics damping="0.0" friction="0.1"/>
+            <parent link="base_link"/>
+            <child link="platform"/>
+        </joint>
+        <transmission name="trans_platform_joint">
+            <type>transmission_interface/SimpleTransmission</type>
+            <actuator name="platform_joint_motor">
+                <mechanicalReduction>1</mechanicalReduction>
+            </actuator>
+            <joint name="platform_joint">
+                <hardwareInterface>hardware_interface/EffortJointInterface</hardwareInterface>
+                <offset>0</offset>
+            </joint>
+        </transmission>
         <xacro:mecanum_wheel prefix="left_front" connected_to="base_link"
                              wheel_x_offset="${wheel_front}" wheel_y_offset="${wheel_left}"

File: urdf/engineer/mast.urdf.xacro (robot description, xacro)
@@ -72,5 +72,5 @@
                 <axis xyz="0 0 1"/>
                 <dynamics damping="0.0" friction="0.8"/>
-                <limit effort="1.2" velocity="13.82" lower="-0.175" upper="0"/>
+                <limit effort="30" velocity="13.82" lower="-0.175" upper="0"/>
             </joint>
         </xacro:unless>
