Commit message: update collision of engineer

File: urdf/engineer/chassis.urdf.xacro (robot description, xacro)
@@ -78,5 +78,5 @@
             </collision>
             <collision>
-                <origin xyz="-0.023 0.0847 0.228" rpy="0 0 1.0646508"/>
+                <origin xyz="0.0 0 0" rpy="0 0 1.0646508"/>
                 <geometry>
                     <box size="0.080 0.003 0.250"/>

File: urdf/engineer/mast.urdf.xacro (robot description, xacro)
@@ -21,7 +21,7 @@
             </collision>
             <collision>
-                <origin xyz="-0.013 0 -0.021" rpy="0 0 0"/>
-                <geometry>
-                    <box size="0.075 0.059 0.043"/>
+                <origin xyz="0. 0.004 0.03" rpy="0 0 0"/>
+                <geometry>
+                    <cylinder length="0.14" radius="0.07"/>
                 </geometry>
             </collision>
@@ -38,10 +38,10 @@
                 </geometry>
             </visual>
-            <collision>
-                <origin xyz="0. 0.004 0.04" rpy="0 0 0"/>
-                <geometry>
-                    <box size="0.054 0.120 0.081"/>
-                </geometry>
-            </collision>
+<!--            <collision>-->
+<!--                <origin xyz="0.0 0.004 0.03" rpy="0 0 0"/>-->
+<!--                <geometry>-->
+<!--                    <cylinder length="0.14" radius="0.01"/>-->
+<!--                </geometry>-->
+<!--            </collision>-->
         </link>
         <link name="pitch">
@@ -56,15 +56,15 @@
                 </geometry>
             </visual>
-            <collision>
-                <origin xyz="-0.005 -0.04 0.014" rpy="0 0 0"/>
-                <geometry>
-                    <box size="0.1 0.048 0.036"/>
-                </geometry>
-            </collision>
+<!--            <collision>-->
+<!--                <origin xyz="-0.005 -0.04 0.014" rpy="0 0 0"/>-->
+<!--                <geometry>-->
+<!--                    <box size="0.1 0.048 0.036"/>-->
+<!--                </geometry>-->
+<!--            </collision>-->
         </link>
-        <link name="camera_telephoto"/>
-        <link name="camera_wideangle"/>
-        <link name="camera_wideangle_optical_frame"/>
-        <link name="camera_telephoto_optical_frame"/>
+<!--        <link name="camera_telephoto"/>-->
+<!--        <link name="camera_wideangle"/>-->
+<!--        <link name="camera_wideangle_optical_frame"/>-->
+<!--        <link name="camera_telephoto_optical_frame"/>-->
         <xacro:unless value="${connected_to == ''}">
             <joint name="mast_joint" type="prismatic">
@@ -81,5 +81,5 @@
                     rpy="0 0 0"/>
             <dynamics damping="0.0" friction="0.1"/>
-            <limit effort="1.2" velocity="13.82" lower="-1e10" upper="1e10"/>
+            <limit effort="1.2" velocity="13.82" lower="-3.14" upper="3.14"/>
             <parent link="mast"/>
             <child link="yaw"/>
@@ -94,26 +94,26 @@
             <axis xyz="0 1 0 "/>
         </joint>
-        <joint name="camera_wideangle_joint" type="fixed">
-            <parent link="pitch"/>
-            <child link="camera_wideangle"/>
-            <origin xyz="0.006 0.028 0.021" rpy="0 0 0"/>
-            <axis xyz="0 0 1"/>
-        </joint>
-        <joint name="camera_telephoto_joint" type="fixed">
-            <parent link="pitch"/>
-            <child link="camera_telephoto"/>
-            <origin xyz="0.006 0.052 0.021" rpy="0 0 0"/>
-            <axis xyz="0 0 1"/>
-        </joint>
-        <joint name="camera_wideangle_optical_frame_joint" type="fixed">
-            <origin xyz="0.026 0 -0.0145" rpy="-1.57 0 -1.57"/>
-            <parent link="camera_wideangle"/>
-            <child link="camera_wideangle_optical_frame"/>
-        </joint>
-        <joint name="camera_telephoto_optical_frame_joint" type="fixed">
-            <origin xyz="0.026 0 -0.0145" rpy="-1.57 0 -1.57"/>
-            <parent link="camera_telephoto"/>
-            <child link="camera_telephoto_optical_frame"/>
-        </joint>
+<!--        <joint name="camera_wideangle_joint" type="fixed">-->
+<!--            <parent link="pitch"/>-->
+<!--            <child link="camera_wideangle"/>-->
+<!--            <origin xyz="0.006 0.028 0.021" rpy="0 0 0"/>-->
+<!--            <axis xyz="0 0 1"/>-->
+<!--        </joint>-->
+<!--        <joint name="camera_telephoto_joint" type="fixed">-->
+<!--            <parent link="pitch"/>-->
+<!--            <child link="camera_telephoto"/>-->
+<!--            <origin xyz="0.006 0.052 0.021" rpy="0 0 0"/>-->
+<!--            <axis xyz="0 0 1"/>-->
+<!--        </joint>-->
+<!--        <joint name="camera_wideangle_optical_frame_joint" type="fixed">-->
+<!--            <origin xyz="0.026 0 -0.0145" rpy="-1.57 0 -1.57"/>-->
+<!--            <parent link="camera_wideangle"/>-->
+<!--            <child link="camera_wideangle_optical_frame"/>-->
+<!--        </joint>-->
+<!--        <joint name="camera_telephoto_optical_frame_joint" type="fixed">-->
+<!--            <origin xyz="0.026 0 -0.0145" rpy="-1.57 0 -1.57"/>-->
+<!--            <parent link="camera_telephoto"/>-->
+<!--            <child link="camera_telephoto_optical_frame"/>-->
+<!--        </joint>-->
         <transmission name="trans_yaw_joint">
             <type>transmission_interface/SimpleTransmission</type>
@@ -147,76 +147,76 @@
         </transmission>
         <xacro:if value="${simulation}">
-            <gazebo reference="camera_wideangle">
-                <sensor type="camera" name="camera_wideangle">
-                    <update_rate>100.0</update_rate>
-                    <camera name="wideangle">
-                        <horizontal_fov>2.0934</horizontal_fov>
-                        <image>
-                            <width>1920</width>
-                            <height>1080</height>
-                            <format>R8G8B8</format>
-                        </image>
-                        <clip>
-                            <near>0.05</near>
-                            <far>5</far>
-                        </clip>
-                        <noise>
-                            <type>gaussian</type>
-                            <mean>0.0</mean>
-                            <stddev>0.007</stddev>
-                        </noise>
-                    </camera>
-                    <plugin name="camera_controller" filename="libgazebo_ros_camera.so">
-                        <alwaysOn>true</alwaysOn>
-                        <updateRate>0.0</updateRate>
-                        <cameraName>usb_camera/camera_wideangle</cameraName>
-                        <imageTopicName>image_raw</imageTopicName>
-                        <cameraInfoTopicName>camera_info</cameraInfoTopicName>
-                        <frameName>camera_wideangle_optical_frame</frameName>
-                        <hackBaseline>0.07</hackBaseline>
-                        <distortionK1>0.0</distortionK1>
-                        <distortionK2>0.0</distortionK2>
-                        <distortionK3>0.0</distortionK3>
-                        <distortionT1>0.0</distortionT1>
-                        <distortionT2>0.0</distortionT2>
-                    </plugin>
-                </sensor>
-            </gazebo>
-            <gazebo reference="camera_telephoto">
-                <sensor type="camera" name="camera_telephoto">
-                    <update_rate>100.0</update_rate>
-                    <camera name="telephoto">
-                        <horizontal_fov>1.919</horizontal_fov>
-                        <image>
-                            <width>1920</width>
-                            <height>1080</height>
-                            <format>R8G8B8</format>
-                        </image>
-                        <clip>
-                            <near>0.05</near>
-                            <far>5</far>
-                        </clip>
-                        <noise>
-                            <type>gaussian</type>
-                            <mean>0.0</mean>
-                            <stddev>0.007</stddev>
-                        </noise>
-                    </camera>
-                    <plugin name="camera_controller" filename="libgazebo_ros_camera.so">
-                        <alwaysOn>true</alwaysOn>
-                        <updateRate>0.0</updateRate>
-                        <cameraName>usb_camera/camera_telephoto</cameraName>
-                        <imageTopicName>image_raw</imageTopicName>
-                        <cameraInfoTopicName>camera_info</cameraInfoTopicName>
-                        <frameName>camera_telephoto_optical_frame</frameName>
-                        <hackBaseline>0.07</hackBaseline>
-                        <distortionK1>0.0</distortionK1>
-                        <distortionK2>0.0</distortionK2>
-                        <distortionK3>0.0</distortionK3>
-                        <distortionT1>0.0</distortionT1>
-                        <distortionT2>0.0</distortionT2>
-                    </plugin>
-                </sensor>
-            </gazebo>
+<!--            <gazebo reference="camera_wideangle">-->
+<!--                <sensor type="camera" name="camera_wideangle">-->
+<!--                    <update_rate>100.0</update_rate>-->
+<!--                    <camera name="wideangle">-->
+<!--                        <horizontal_fov>2.0934</horizontal_fov>-->
+<!--                        <image>-->
+<!--                            <width>1920</width>-->
+<!--                            <height>1080</height>-->
+<!--                            <format>R8G8B8</format>-->
+<!--                        </image>-->
+<!--                        <clip>-->
+<!--                            <near>0.05</near>-->
+<!--                            <far>5</far>-->
+<!--                        </clip>-->
+<!--                        <noise>-->
+<!--                            <type>gaussian</type>-->
+<!--                            <mean>0.0</mean>-->
+<!--                            <stddev>0.007</stddev>-->
+<!--                        </noise>-->
+<!--                    </camera>-->
+<!--                    <plugin name="camera_controller" filename="libgazebo_ros_camera.so">-->
+<!--                        <alwaysOn>true</alwaysOn>-->
+<!--                        <updateRate>0.0</updateRate>-->
+<!--                        <cameraName>usb_camera/camera_wideangle</cameraName>-->
+<!--                        <imageTopicName>image_raw</imageTopicName>-->
+<!--                        <cameraInfoTopicName>camera_info</cameraInfoTopicName>-->
+<!--                        <frameName>camera_wideangle_optical_frame</frameName>-->
+<!--                        <hackBaseline>0.07</hackBaseline>-->
+<!--                        <distortionK1>0.0</distortionK1>-->
+<!--                        <distortionK2>0.0</distortionK2>-->
+<!--                        <distortionK3>0.0</distortionK3>-->
+<!--                        <distortionT1>0.0</distortionT1>-->
+<!--                        <distortionT2>0.0</distortionT2>-->
+<!--                    </plugin>-->
+<!--                </sensor>-->
+<!--            </gazebo>-->
+<!--            <gazebo reference="camera_telephoto">-->
+<!--                <sensor type="camera" name="camera_telephoto">-->
+<!--                    <update_rate>100.0</update_rate>-->
+<!--                    <camera name="telephoto">-->
+<!--                        <horizontal_fov>1.919</horizontal_fov>-->
+<!--                        <image>-->
+<!--                            <width>1920</width>-->
+<!--                            <height>1080</height>-->
+<!--                            <format>R8G8B8</format>-->
+<!--                        </image>-->
+<!--                        <clip>-->
+<!--                            <near>0.05</near>-->
+<!--                            <far>5</far>-->
+<!--                        </clip>-->
+<!--                        <noise>-->
+<!--                            <type>gaussian</type>-->
+<!--                            <mean>0.0</mean>-->
+<!--                            <stddev>0.007</stddev>-->
+<!--                        </noise>-->
+<!--                    </camera>-->
+<!--                    <plugin name="camera_controller" filename="libgazebo_ros_camera.so">-->
+<!--                        <alwaysOn>true</alwaysOn>-->
+<!--                        <updateRate>0.0</updateRate>-->
+<!--                        <cameraName>usb_camera/camera_telephoto</cameraName>-->
+<!--                        <imageTopicName>image_raw</imageTopicName>-->
+<!--                        <cameraInfoTopicName>camera_info</cameraInfoTopicName>-->
+<!--                        <frameName>camera_telephoto_optical_frame</frameName>-->
+<!--                        <hackBaseline>0.07</hackBaseline>-->
+<!--                        <distortionK1>0.0</distortionK1>-->
+<!--                        <distortionK2>0.0</distortionK2>-->
+<!--                        <distortionK3>0.0</distortionK3>-->
+<!--                        <distortionT1>0.0</distortionT1>-->
+<!--                        <distortionT2>0.0</distortionT2>-->
+<!--                    </plugin>-->
+<!--                </sensor>-->
+<!--            </gazebo>-->
         </xacro:if>
     </xacro:macro>

Commit message: change platform to stone_platform

File: urdf/engineer/chassis.urdf.xacro (robot description, xacro)
@@ -84,5 +84,5 @@
             </collision>
         </link>
-        <link name="platform">
+        <link name="stone_platform">
             <inertial>
                 <mass value="0.073"/>
@@ -93,5 +93,5 @@
                 <origin xyz="0 0 0" rpy="0 0 0"/>
                 <geometry>
-                    <mesh filename="package://rm_description/meshes/engineer/platform.stl" scale="0.001 0.001 0.001"/>
+                    <mesh filename="package://rm_description/meshes/engineer/stone_platform.stl" scale="0.001 0.001 0.001"/>
                 </geometry>
             </visual>
@@ -103,5 +103,5 @@
             </collision>
         </link>
-        <joint name="platform_joint" type="prismatic">
+        <joint name="stone_platform_joint" type="prismatic">
             <axis xyz="0 1 0"/>
             <origin xyz="-0.113 0.134 0.114"/>
@@ -109,12 +109,12 @@
             <dynamics damping="0.0" friction="0.1"/>
             <parent link="base_link"/>
-            <child link="platform"/>
+            <child link="stone_platform"/>
         </joint>
-        <transmission name="trans_platform_joint">
+        <transmission name="trans_stone_platform_joint">
             <type>transmission_interface/SimpleTransmission</type>
-            <actuator name="platform_joint_motor">
+            <actuator name="stone_platform_joint_motor">
                 <mechanicalReduction>1</mechanicalReduction>
             </actuator>
-            <joint name="platform_joint">
+            <joint name="stone_platform_joint">
                 <hardwareInterface>hardware_interface/EffortJointInterface</hardwareInterface>
                 <offset>0</offset>

Commit message: update mechanicalReduction of stone_platform_joint

File: urdf/engineer/chassis.urdf.xacro (robot description, xacro)
@@ -104,5 +104,5 @@
         </link>
         <joint name="stone_platform_joint" type="prismatic">
-            <axis xyz="0 1 0"/>
+            <axis xyz="0 0 1"/>
             <origin xyz="-0.113 0.134 0.114"/>
             <limit effort="7" velocity="30" lower="0" upper="2.6459"/>
@@ -114,5 +114,5 @@
             <type>transmission_interface/SimpleTransmission</type>
             <actuator name="stone_platform_joint_motor">
-                <mechanicalReduction>1</mechanicalReduction>
+                <mechanicalReduction>49.97</mechanicalReduction>
             </actuator>
             <joint name="stone_platform_joint">

Commit message: update chassis xyz to wheeel

File: urdf/engineer/chassis.urdf.xacro (robot description, xacro)
@@ -2,9 +2,9 @@
     <xacro:include filename="$(find rm_description)/urdf/common/mecanum_wheel.urdf.xacro"/>
     <!-- https://upload.wikimedia.org/wikipedia/commons/5/52/Wheelbase_and_Track.png -->
-    <xacro:property name="wheel_front" value="0.091"/>
-    <xacro:property name="wheel_back" value="-0.178"/>
-    <xacro:property name="wheel_left" value="-0.245"/>
-    <xacro:property name="wheel_right" value="0.245"/>
-    <xacro:property name="wheel_offset_z" value="-0.04"/>
+    <xacro:property name="wheel_front" value="0.1"/>
+    <xacro:property name="wheel_back" value="-0.18"/>
+    <xacro:property name="wheel_left" value="-0.24"/>
+    <xacro:property name="wheel_right" value="0.24"/>
+    <xacro:property name="wheel_offset_z" value="-0.06"/>
     <xacro:property name="wheel_joint_damping" value="1.0"/>
     <xacro:property name="wheel_joint_friction" value="1.0"/>

Commit message: change the cover parent to base_link

File: urdf/engineer/chassis.urdf.xacro (robot description, xacro)
@@ -97,5 +97,5 @@
             </visual>
             <collision>
-                <origin xyz="-0.113 0.134 0.114" rpy="0 0.0 0"/>
+                <origin xyz="0.0 0.0 0.0" rpy="0 0.0 0"/>
                 <geometry>
                     <box size="0.106 0.105 0.002"/>

File: urdf/hero/chassis.urdf.xacro (robot description, xacro)
@@ -50,5 +50,5 @@
             <limit effort="1" velocity="30" lower="-3.14" upper="3.14"/>
             <dynamics damping="0.0" friction="0.1"/>
-            <parent link="pitch"/>
+            <parent link="base_link"/>
             <child link="cover"/>
         </joint>

Commit message: Fix engineer left wheel and right wheel are opposite

File: urdf/engineer/chassis.urdf.xacro (robot description, xacro)
@@ -4,6 +4,6 @@
     <xacro:property name="wheel_front" value="0.1"/>
     <xacro:property name="wheel_back" value="-0.18"/>
-    <xacro:property name="wheel_left" value="-0.24"/>
-    <xacro:property name="wheel_right" value="0.24"/>
+    <xacro:property name="wheel_right" value="-0.24"/>
+    <xacro:property name="wheel_left" value="0.24"/>
     <xacro:property name="wheel_offset_z" value="-0.06"/>
     <xacro:property name="wheel_joint_damping" value="1.0"/>

Commit message: Delete magazine collision box.

File: urdf/engineer/chassis.urdf.xacro (robot description, xacro)
@@ -27,34 +27,4 @@
                 <geometry>
                     <box size="0.486 0.596 0.169"/>
-                </geometry>
-            </collision>
-                        <collision>
-                            <origin xyz="-0.130 -0.132 0.255" rpy="0 0 0.8377580"/>
-                            <geometry>
-                                <box size="0.106 0.186 0.3"/>
-                            </geometry>
-                        </collision>
-                        <collision>
-                            <origin xyz="-0.0336 -0.27 0.262" rpy="0 0 -0.7853982"/>
-                            <geometry>
-                                <box size="0.01 0.033 0.06"/>
-                            </geometry>
-                        </collision>
-            <collision>
-                <origin xyz="-0.083 -0.225 0.262" rpy="0 0 -0.7853982"/>
-                <geometry>
-                    <box size="0.01 0.033 0.06"/>
-                </geometry>
-            </collision>
-            <collision>
-                <origin xyz="-0.0685 -0.259 0.287" rpy="0 0 0.8377580"/>
-                <geometry>
-                    <box size="0.003 0.057 0.01"/>
-                </geometry>
-            </collision>
-            <collision>
-                <origin xyz="-0.0685 -0.259 0.237" rpy="0 0 0.8377580"/>
-                <geometry>
-                    <box size="0.003 0.057 0.01"/>
                 </geometry>
             </collision>
@@ -93,5 +63,6 @@
                 <origin xyz="0 0 0" rpy="0 0 0"/>
                 <geometry>
-                    <mesh filename="package://rm_description/meshes/engineer/stone_platform.stl" scale="0.001 0.001 0.001"/>
+                    <mesh filename="package://rm_description/meshes/engineer/stone_platform.stl"
+                          scale="0.001 0.001 0.001"/>
                 </geometry>
             </visual>

Commit message: Update card controller limit

File: urdf/engineer/chassis.urdf.xacro (robot description, xacro)
@@ -96,5 +96,5 @@
             <axis xyz="1 0 0"/>
             <origin xyz="0.109 0.001 -0.11"/>
-            <limit effort="0.1" velocity="30" lower="0" upper="0.05"/>
+            <limit effort="15" velocity="0.8708" lower="0" upper="0.15899"/>
             <dynamics damping="0.0" friction="0.1"/>
             <parent link="base_link"/>
@@ -104,5 +104,5 @@
             <axis xyz="0 0 1"/>
             <origin xyz="-0.113 0.134 0.114"/>
-            <limit effort="1" velocity="30" lower="0" upper="0.024"/>
+            <limit effort="30" velocity="0.8708" lower="0" upper="0.024"/>
             <dynamics damping="0.0" friction="0.1"/>
             <parent link="base_link"/>
@@ -112,5 +112,5 @@
             <type>transmission_interface/SimpleTransmission</type>
             <actuator name="stone_platform_joint_motor">
-                <mechanicalReduction>49.97</mechanicalReduction>
+                <mechanicalReduction>50</mechanicalReduction>
             </actuator>
             <joint name="stone_platform_joint">
@@ -122,5 +122,5 @@
             <type>transmission_interface/SimpleTransmission</type>
             <actuator name="card_joint_motor">
-                <mechanicalReduction>49.97</mechanicalReduction>
+                <mechanicalReduction>50</mechanicalReduction>
             </actuator>
             <joint name="card_joint">
