Commit message: Change the chassis collision box.

File: urdf/engineer/chassis.urdf.xacro (robot description, xacro)
@@ -2,9 +2,9 @@
     <xacro:include filename="$(find rm_description)/urdf/common/mecanum_wheel.urdf.xacro"/>
     <!-- https://upload.wikimedia.org/wikipedia/commons/5/52/Wheelbase_and_Track.png -->
-    <xacro:property name="wheel_front" value="0.1"/>
-    <xacro:property name="wheel_back" value="-0.18"/>
-    <xacro:property name="wheel_right" value="-0.24"/>
-    <xacro:property name="wheel_left" value="0.24"/>
-    <xacro:property name="wheel_offset_z" value="-0.06"/>
+    <xacro:property name="wheel_front" value="0.134874"/>
+    <xacro:property name="wheel_back" value="-0.134874"/>
+    <xacro:property name="wheel_right" value="-0.2448"/>
+    <xacro:property name="wheel_left" value="0.2448"/>
+    <xacro:property name="wheel_offset_z" value="0.000072"/>
     <xacro:property name="wheel_joint_damping" value="1.0"/>
     <xacro:property name="wheel_joint_friction" value="1.0"/>
@@ -24,5 +24,5 @@
             </visual>
             <collision>
-                <origin xyz="-0.043 0 0.020" rpy="0 0 0"/>
+                <origin xyz="0 0 0.05" rpy="0 0 0"/>
                 <geometry>
                     <box size="0.486 0.596 0.169"/>
@@ -30,5 +30,5 @@
             </collision>
             <collision>
-                <origin xyz="-0.08 0.243 0.258" rpy="0 0 -0.5061455"/>
+                <origin xyz="-0.043668 0.236688 0.284" rpy="0 0 -0.5061455"/>
                 <geometry>
                     <box size="0.08 0.0217 0.3033"/>
@@ -36,5 +36,5 @@
             </collision>
             <collision>
-                <origin xyz="-0.21 0.19 0.25833" rpy="0 0 1.0646508"/>
+                <origin xyz="-0.160269 0.184128 0.284" rpy="0 0 1.0646508"/>
                 <geometry>
                     <box size="0.08 0.0217 0.3033"/>
@@ -42,5 +42,5 @@
             </collision>
             <collision>
-                <origin xyz="-0.19 0.05 0.258" rpy="0 0 -0.5061455"/>
+                <origin xyz="-0.143054 0.057391 0.284" rpy="0 0 -0.5061455"/>
                 <geometry>
                     <box size="0.08 0.0217 0.3033"/>
@@ -48,5 +48,5 @@
             </collision>
             <collision>
-                <origin xyz="-0.0239 0.084 0.228" rpy="0 0 1.0646508"/>
+                <origin xyz="0.019028 0.084742 0.269" rpy="0 0 1.0646508"/>
                 <geometry>
                     <box size="0.080 0.003 0.250"/>
@@ -74,31 +74,4 @@
             </collision>
         </link>
-        <link name="card">
-            <inertial>
-                <mass value="0.26"/>
-                <origin xyz="-0.071 -0.006 0.003"/>
-                <inertia ixx="1.078e-3" ixy="6.486e-5" ixz="1.454e-5" iyy="1.142e-4" iyz="5.143e-6" izz="2.215e-3"/>
-            </inertial>
-            <visual>
-                <origin xyz="0 0 0" rpy="0 0 0"/>
-                <geometry>
-                    <mesh filename="package://rm_description/meshes/engineer/card.stl" scale="0.001 0.001 0.001"/>
-                </geometry>
-            </visual>
-            <collision>
-                <origin xyz="-0.113 0.134 0.0" rpy="0 0.0 0"/>
-                <geometry>
-                    <box size="0.253 0.151 0.011"/>
-                </geometry>
-            </collision>
-        </link>
-        <joint name="card_joint" type="prismatic">
-            <axis xyz="1 0 0"/>
-            <origin xyz="0.109 0.001 -0.11"/>
-            <limit effort="0.1" velocity="30" lower="0" upper="0.05"/>
-            <dynamics damping="0.0" friction="0.1"/>
-            <parent link="base_link"/>
-            <child link="card"/>
-        </joint>
         <joint name="stone_platform_joint" type="prismatic">
             <axis xyz="0 0 1"/>

Commit message: Update chassis.urdf.xacro

File: urdf/engineer/chassis.urdf.xacro (robot description, xacro)
@@ -12,5 +12,5 @@
         <link name="base_link">
             <inertial>
-                <mass value="11.91"/>
+                <mass value="2.361504/>
                 <origin xyz="-0.063 -0.010 -0.027"/>
                 <inertia ixx="4.302e-2" ixy="7.618e-4" ixz="6.881e-3" iyy="3.95e-2"

Commit message: solve the problem of one of the inertia elements is not a valid double

File: urdf/engineer/chassis.urdf.xacro (robot description, xacro)
@@ -58,5 +58,5 @@
                 <mass value="0.073"/>
                 <origin xyz="-0.037 -0.005 0.009"/>
-                <inertia ixx="5.874e-4" ixy="-2.845e-4" ixz="1.882e-5" iyy=" 2.133e-4" iyz="2.682e-5" izz="7.780e-4"/>
+                <inertia ixx="5.874e-4" ixy="-2.845e-4" ixz="1.882e-5" iyy="2.133e-4" iyz="2.682e-5" izz="7.780e-4"/>
             </inertial>
             <visual>

Commit message: Set limit of mast and card

File: urdf/engineer/chassis.urdf.xacro (robot description, xacro)
@@ -96,5 +96,5 @@
             <axis xyz="1 0 0"/>
             <origin xyz="0.209783 0.004 -0.08"/>
-            <limit effort="0.1" velocity="30" lower="0" upper="0.05"/>
+            <limit effort="20.0" velocity="1.0" lower="0" upper="0.1"/>
             <dynamics damping="0.0" friction="0.1"/>
             <parent link="base_link"/>

File: urdf/engineer/mast.urdf.xacro (robot description, xacro)
@@ -62,5 +62,5 @@
                 <axis xyz="0 0 1"/>
                 <dynamics damping="0.0" friction="0.8"/>
-                <limit effort="10" velocity="13.82" lower="-0.175" upper="0"/>
+                <limit effort="20.0" velocity="1.0" lower="-0.37" upper="0"/>
             </joint>
         </xacro:unless>

Commit message: collect some erros

File: urdf/engineer/chassis.urdf.xacro (robot description, xacro)
@@ -6,5 +6,5 @@
     <xacro:property name="wheel_right" value="-0.2448"/>
     <xacro:property name="wheel_left" value="0.2448"/>
-    <xacro:property name="wheel_offset_z" value="0.000072"/>
+    <xacro:property name="wheel_offset_z" value="-0.029928"/>
     <xacro:property name="wheel_joint_damping" value="1.0"/>
     <xacro:property name="wheel_joint_friction" value="1.0"/>
@@ -12,5 +12,5 @@
         <link name="base_link">
             <inertial>
-                <mass value="11.91"/>
+                <mass value="2.361504"/>
                 <origin xyz="-0.063 -0.010 -0.027"/>
                 <inertia ixx="4.302e-2" ixy="7.618e-4" ixz="6.881e-3" iyy="3.95e-2"
@@ -95,5 +95,5 @@
         <joint name="card_joint" type="prismatic">
             <axis xyz="1 0 0"/>
-            <origin xyz="0.209783 0.004 -0.08"/>
+            <origin xyz="0.209783 0.004 -0.064/>
             <limit effort="20.0" velocity="1.0" lower="0" upper="0.1"/>
             <dynamics damping="0.0" friction="0.1"/>
@@ -103,5 +103,5 @@
         <joint name="stone_platform_joint" type="prismatic">
             <axis xyz="0 0 1"/>
-            <origin xyz="-0.113 0.134 0.114"/>
+            <origin xyz="-0.0706 0.134 0.114"/>
             <limit effort="1" velocity="30" lower="0" upper="0.024"/>
             <dynamics damping="0.0" friction="0.1"/>

Commit message: Change the chassis box.

File: urdf/engineer/chassis.urdf.xacro (robot description, xacro)
@@ -24,7 +24,25 @@
             </visual>
             <collision>
-                <origin xyz="0.005 0 0.06" rpy="0 0 0"/>
+                <origin xyz="-0.125 0. 0.06" rpy="0 0 0"/>
                 <geometry>
-                    <box size="0.5 0.596 0.169"/>
+                    <box size="0.25 0.596 0.169"/>
+                </geometry>
+            </collision>
+            <collision>
+                <origin xyz="0.15 -0.15 0.015" rpy="0 0 0"/>
+                <geometry>
+                    <box size="0.255 0.29 0.06"/>
+                </geometry>
+            </collision>
+            <collision>
+                <origin xyz="0.15 0.144 0.015" rpy="0 0 0"/>
+                <geometry>
+                    <box size="0.255 0.29 0.06"/>
+                </geometry>
+            </collision>
+            <collision>
+                <origin xyz="0.16 0. 0.1" rpy="0 0 0"/>
+                <geometry>
+                    <box size="0.12 0.2 0.1"/>
                 </geometry>
             </collision>
@@ -101,5 +119,5 @@
         <joint name="card_joint" type="prismatic">
             <axis xyz="1 0 0"/>
-            <origin xyz="0.209783 0.004 -0.064"/>
+            <origin xyz="0.15205 0. -0.07"/>
             <limit effort="20.0" velocity="1.0" lower="0" upper="0.1"/>
             <dynamics damping="0.0" friction="0.1"/>

Commit message: Correct the chassis mass.

File: urdf/engineer/chassis.urdf.xacro (robot description, xacro)
@@ -12,5 +12,5 @@
         <link name="base_link">
             <inertial>
-                <mass value="2.361504"/>
+                <mass value="13"/>
                 <origin xyz="-0.063 -0.010 -0.027"/>
                 <inertia ixx="4.302e-2" ixy="7.618e-4" ixz="6.881e-3" iyy="3.95e-2"
@@ -127,5 +127,5 @@
         <joint name="stone_platform_joint" type="prismatic">
             <axis xyz="0 0 1"/>
-            <origin xyz="-0.0706 0.134 0.114"/>
+            <origin xyz="-0.0706 0.134 0.144"/>
             <limit effort="1" velocity="30" lower="0" upper="0.024"/>
             <dynamics damping="0.0" friction="0.1"/>

Commit message: Set limit of stone_platform_joint

File: urdf/engineer/chassis.urdf.xacro (robot description, xacro)
@@ -127,6 +127,6 @@
         <joint name="stone_platform_joint" type="prismatic">
             <axis xyz="0 0 1"/>
-            <origin xyz="-0.0706 0.134 0.144"/>
-            <limit effort="1" velocity="30" lower="0" upper="0.024"/>
+            <origin xyz="-0.0706 0.134 0.114"/>
+            <limit effort="20.0" velocity="1.0" lower="0" upper="0.19"/>
             <dynamics damping="0.0" friction="0.1"/>
             <parent link="base_link"/>

Commit message: Update collision box of engineer arm

File: urdf/engineer/chassis.urdf.xacro (robot description, xacro)
@@ -62,5 +62,5 @@
                 <origin xyz="-0.148196 0.0485 0.224" rpy="0 0 -0.507"/>
                 <geometry>
-                    <box size="0.08 0.05 0.448"/>
+                    <box size="0.08 0.03 0.448"/>
                 </geometry>
             </collision>
