Commit message: Fix inertia element iyy is not a valid double

File: urdf/engineer/hand.urdf.xacro (robot description, xacro)
@@ -25,5 +25,5 @@
         <origin xyz="0.01491 -0.06058 0" rpy="0 0 0"/>
         <mass value="0.203967"/>
-        <inertia ixx="1.025e-3" ixy="3.865e-4" ixz="-1.144e-9" iyy="3.051e-4e-4" iyz="4.649e-9" izz="1.295e-3"/>
+        <inertia ixx="1.025e-3" ixy="3.865e-4" ixz="-1.144e-9" iyy="3.051e-4" iyz="4.649e-9" izz="1.295e-3"/>
       </inertial>
       <visual>
@@ -42,5 +42,5 @@
         <origin xyz="0.01491 0.061581 0" rpy="0 0 0"/>
         <mass value="0.203967"/>
-        <inertia ixx="1.053e-3" ixy="-3.865e-4" ixz="-1.144e-9" iyy="3.051e-4e-4" iyz="-4.733e-9" izz="1.323e-3"/>
+        <inertia ixx="1.053e-3" ixy="-3.865e-4" ixz="-1.144e-9" iyy="3.051e-4" iyz="-4.733e-9" izz="1.323e-3"/>
       </inertial>
       <visual>

Commit message: Fix some small error

File: urdf/engineer/hand.urdf.xacro (robot description, xacro)
@@ -56,5 +56,5 @@
     </link>
     <xacro:unless value="${connected_to == ''}">
-      <joint name="$palm_joint" type="fixed">
+      <joint name="palm_joint" type="fixed">
         <parent link="${connected_to}"/>
         <child link="palm"/>
@@ -73,5 +73,5 @@
       <child link="left_finger"/>
       <origin xyz="0.032 0 0" rpy="0 0 0"/>
-      <axis xyz="0 1- 0"/>
+      <axis xyz="0 -1 0"/>
       <limit effort="20" lower="0.0" upper="0.02" velocity="0.5"/>
       <mimic joint="right_finger_joint"/>

Commit message: change finger_joint xyz

File: urdf/engineer/hand.urdf.xacro (robot description, xacro)
@@ -103,5 +103,5 @@
       <parent link="palm"/>
       <child link="right_finger"/>
-      <origin xyz="0.023 -0.045 0" rpy="0 0 0"/>
+      <origin xyz="0.032 0 0" rpy="0 0 0"/>
       <axis xyz="0 1 0"/>
       <limit effort="588" lower="0.0" upper="0.02" velocity="3.772"/>
@@ -110,8 +110,8 @@
       <parent link="palm"/>
       <child link="left_finger"/>
-      <origin xyz="0.023 0.045 0" rpy="0 0 0"/>
+      <origin xyz="0.032 0 0" rpy="0 0 0"/>
       <axis xyz="0 -1 0"/>
       <limit effort="588" lower="0.0" upper="0.02" velocity="3.772"/>
-<!--      <mimic joint="right_finger_joint"/>-->
+      <mimic joint="right_finger_joint"/>
     </joint>
     <transmission name="trans_right_finger_joint">

Commit message: Add mimic_joint plugin to left_finger_joint

File: urdf/engineer/hand.urdf.xacro (robot description, xacro)
@@ -150,39 +150,12 @@
         </joint>
         <xacro:if value="${simulation}">
-            <gazebo reference="camera">
-                <sensor type="camera" name="camera_node">
-                    <update_rate>30.0</update_rate>
-                    <camera name="head">
-                        <horizontal_fov>1.3962634</horizontal_fov>
-                        <image>
-                            <width>1920</width>
-                            <height>1080</height>
-                            <format>R8G8B8</format>
-                        </image>
-                        <clip>
-                            <near>0.02</near>
-                            <far>300</far>
-                        </clip>
-                        <noise>
-                            <type>gaussian</type>
-                            <mean>0.0</mean>
-                            <stddev>0.007</stddev>
-                        </noise>
-                    </camera>
-                    <plugin name="gazebo_camera" filename="libgazebo_ros_camera.so">
-                        <alwaysOn>true</alwaysOn>
-                        <updateRate>0.0</updateRate>
-                        <cameraName>/camera</cameraName>
-                        <imageTopicName>image_raw</imageTopicName>
-                        <cameraInfoTopicName>camera_info</cameraInfoTopicName>
-                        <frameName>camera</frameName>
-                        <hackBaseline>0.07</hackBaseline>
-                        <distortionK1>0.0</distortionK1>
-                        <distortionK2>0.0</distortionK2>
-                        <distortionK3>0.0</distortionK3>
-                        <distortionT1>0.0</distortionT1>
-                        <distortionT2>0.0</distortionT2>
-                    </plugin>
-                </sensor>
+            <gazebo>
+                <plugin name="left_finger_mimic_joint_plugin"
+                        filename="libroboticsgroup_upatras_gazebo_mimic_joint_plugin.so">
+                    <joint>right_finger_joint</joint>
+                    <mimicJoint>left_finger_joint</mimicJoint>
+                    <hasPID/>
+                    <maxEffort>588.0</maxEffort>
+                </plugin>
             </gazebo>
         </xacro:if>

Commit message: Remove comment

File: urdf/engineer/hand.urdf.xacro (robot description, xacro)
@@ -42,10 +42,4 @@
                 </geometry>
             </visual>
-<!--            <collision>-->
-<!--                <origin xyz="0.0 0.046 0.005" rpy="0 0 0"/>-->
-<!--                <geometry>-->
-<!--                    <box size="0.030 0.027 0.063"/>-->
-<!--                </geometry>-->
-<!--            </collision>-->
             <collision>
                 <origin xyz="0.0 0.088 0.025" rpy="0 0 0"/>
@@ -73,10 +67,4 @@
                 </geometry>
             </visual>
-<!--            <collision>-->
-<!--                <origin xyz="0.0 -0.043 0.005" rpy="0 0 0"/>-->
-<!--                <geometry>-->
-<!--                    <box size="0.030 0.027 0.063"/>-->
-<!--                </geometry>-->
-<!--            </collision>-->
             <collision>
                 <origin xyz="0.0 -0.088 0.025" rpy="0 0 0"/>

Commit message: Fix can not grasp resource

File: urdf/engineer/hand.urdf.xacro (robot description, xacro)
@@ -49,5 +49,5 @@
             </collision>
             <collision>
-                <origin xyz="0.0 0.133 0.07" rpy="0 0 0"/>
+                <origin xyz="0.0 0.130 0.07" rpy="0 0 0"/>
                 <geometry>
                     <box size="0.030 0.017 0.112"/>
@@ -74,5 +74,5 @@
             </collision>
             <collision>
-                <origin xyz="0.0 -0.129 0.07" rpy="0 0 0"/>
+                <origin xyz="0.0 -0.130 0.07" rpy="0 0 0"/>
                 <geometry>
                     <box size="0.030 0.017 0.112"/>
@@ -92,5 +92,5 @@
             <origin xyz="0 0 0.045" rpy="0 0 0"/>
             <axis xyz="0 1 0"/>
-            <limit effort="588" lower="-0.025" upper="0.0" velocity="3.772"/>
+            <limit effort="588" lower="-0.04" upper="0.0" velocity="3.772"/>
         </joint>
         <joint name="left_finger_joint" type="prismatic">
@@ -99,5 +99,5 @@
             <origin xyz="0 0 0.045" rpy="0 0 0"/>
             <axis xyz="0 -1 0"/>
-            <limit effort="588" lower="-0.025" upper="0.0" velocity="3.772"/>
+            <limit effort="588" lower="-0.04" upper="0.0" velocity="3.772"/>
             <mimic joint="right_finger_joint"/>
         </joint>
@@ -114,16 +114,17 @@
             <gazebo reference="right_finger">
                 <self_collide>1</self_collide>
-                <mu1 value="8000000000.0"/>
-                <mu2 value="8000000000.0"/>
+                <mu1 value="2000"/>
+                <mu2 value="2000"/>
                 <kp value="1000000.0"/>
                 <kd value="100.0"/>
+                <maxContacts>2</maxContacts>
                 <material>Gazebo/Black</material>
             </gazebo>
             <gazebo reference="left_finger">
-                <self_collide>1</self_collide>
-                <mu1 value="8000000000.0"/>
-                <mu2 value="8000000000.0"/>
+                <mu1 value="2000"/>
+                <mu2 value="2000"/>
                 <kp value="1000000.0"/>
                 <kd value="100.0"/>
+                <maxContacts>2</maxContacts>
                 <material>Gazebo/Black</material>
             </gazebo>

Commit message: Adjust the hands inertial.

File: urdf/engineer/hand.urdf.xacro (robot description, xacro)
@@ -12,6 +12,6 @@
             <inertial>
                 <mass value="0.695"/>
-                <origin xyz="0.0 0.0 0.024" rpy="0 0 0"/>
-                <inertia ixx="5.042e-4" ixy="1.20e-7" ixz="-3.142e-6" iyy="2.444e-4" iyz="1.18e-7" izz="4.945e-4"/>
+                <origin xyz="0.0 0.0 -0.024" rpy="0 0 0"/>
+                <inertia ixx="4.945e-4" ixy="1.180e-7" ixz="3.142e-6" iyy="2.444e-4" iyz="-1.2e-7" izz="5.042e-4"/>
             </inertial>
             <visual>
@@ -32,7 +32,7 @@
         <link name="right_finger">
             <inertial>
-                <origin xyz="0.0 0.075 0.021" rpy="0 0 0"/>
+                <origin xyz="0.0 0.075 -0.021" rpy="0 0 0"/>
                 <mass value="0.284"/>
-                <inertia ixx="7.653e-4" ixy="1.922e-5" ixz="1.589e-5" iyy="3.805e-4" iyz="-3.052e-4" izz="4.364e-4"/>
+                <inertia ixx="4.364e-4" ixy="-3.052e-5" ixz="-1.589e-5" iyy="3.805e-4" iyz="-1.922e-5" izz="7.653e-4"/>
             </inertial>
             <visual>
@@ -58,7 +58,7 @@
         <link name="left_finger">
             <inertial>
-                <origin xyz="0.0 -0.075 0.021" rpy="0 0 0"/>
+                <origin xyz="0.0 -0.075 -0.021" rpy="0 0 0"/>
                 <mass value="0.284"/>
-                <inertia ixx="7.653e-4" ixy="1.922e-5" ixz="-1.589e-5" iyy="3.805e-4" iyz="3.052e-4" izz="4.364e-4"/>
+                <inertia ixx="4.364e-4" ixy="3.052e-4" ixz="1.589e-5" iyy="3.805e-4" iyz="-1.922e-5" izz="7.653e-4"/>
             </inertial>
             <visual>

Commit message: Decrease the hand limit effort to 200N

File: urdf/engineer/hand.urdf.xacro (robot description, xacro)
@@ -13,5 +13,6 @@
                 <mass value="0.705"/>
                 <origin xyz="0.0 0.0 0" rpy="0 0 0"/>
-                <inertia ixx="1.483e-3" ixy="-3.268e-4" ixz="-1.279015e-5" iyy="1.014e-4" iyz="-5.7349231e-5" izz="1.553e-3"/>
+                <inertia ixx="1.483e-3" ixy="-3.268e-4" ixz="-1.279015e-5" iyy="1.014e-4" iyz="-5.7349231e-5"
+                         izz="1.553e-3"/>
             </inertial>
             <visual>
@@ -43,5 +44,5 @@
             </inertial>
             <visual>
-<!--                <origin xyz="0 0 0" rpy="0 0 0"/>-->
+                <!--                <origin xyz="0 0 0" rpy="0 0 0"/>-->
                 <geometry>
                     <mesh filename="package://rm_description/meshes/engineer/right_finger.stl"
@@ -60,8 +61,9 @@
                 <origin xyz="0.015 0.062 8e-6" rpy="0 0 0"/>
                 <mass value="0.211439"/>
-                <inertia ixx="1.107e-3" ixy="-4.148e-4" ixz="4.1265e-8" iyy="3.139e-4" iyz="-0.071221e-8" izz="1.39e-3"/>
+                <inertia ixx="1.107e-3" ixy="-4.148e-4" ixz="4.1265e-8" iyy="3.139e-4" iyz="-0.071221e-8"
+                         izz="1.39e-3"/>
             </inertial>
             <visual>
-<!--                <origin xyz="0 0 0" rpy="0 1.57 0"/>-->
+                <!--                <origin xyz="0 0 0" rpy="0 1.57 0"/>-->
                 <geometry>
                     <mesh filename="package://rm_description/meshes/engineer/left_finger.stl"
@@ -69,10 +71,10 @@
                 </geometry>
             </visual>
-<!--            <collision>-->
-<!--                <origin xyz="0.0 -0.088 0.025" rpy="0 0 0"/>-->
-<!--                <geometry>-->
-<!--                    <box size="0.03 0.112 0.022"/>-->
-<!--                </geometry>-->
-<!--            </collision>-->
+            <!--            <collision>-->
+            <!--                <origin xyz="0.0 -0.088 0.025" rpy="0 0 0"/>-->
+            <!--                <geometry>-->
+            <!--                    <box size="0.03 0.112 0.022"/>-->
+            <!--                </geometry>-->
+            <!--            </collision>-->
             <collision>
                 <origin xyz="0.068474 0.126453 0.0" rpy="0 0 0"/>
@@ -94,5 +96,5 @@
             <origin xyz="0.045 0 0" rpy="0 0 0"/>
             <axis xyz="0 1 0"/>
-            <limit effort="588" lower="-0.04" upper="0.0" velocity="3.772"/>
+            <limit effort="200" lower="-0.04" upper="0.0" velocity="3.772"/>
         </joint>
         <joint name="left_finger_joint" type="prismatic">

Commit message: Add countdown to improve accuracy

File: urdf/engineer/hand.urdf.xacro (robot description, xacro)
@@ -103,5 +103,5 @@
             <origin xyz="0.045 0 0" rpy="0 0 0"/>
             <axis xyz="0 -1 0"/>
-            <limit effort="588" lower="-0.04" upper="0.0" velocity="3.772"/>
+            <limit effort="200" lower="-0.04" upper="0.0" velocity="3.772"/>
             <mimic joint="right_finger_joint"/>
         </joint>

Commit message: Decrease engineer's hand limit

File: urdf/engineer/hand.urdf.xacro (robot description, xacro)
@@ -96,5 +96,5 @@
             <origin xyz="0.045 0 0" rpy="0 0 0"/>
             <axis xyz="0 1 0"/>
-            <limit effort="200" lower="-0.04" upper="0.0" velocity="3.772"/>
+            <limit effort="150" lower="-0.04" upper="0.0" velocity="3.772"/>
         </joint>
         <joint name="left_finger_joint" type="prismatic">
@@ -103,5 +103,5 @@
             <origin xyz="0.045 0 0" rpy="0 0 0"/>
             <axis xyz="0 -1 0"/>
-            <limit effort="200" lower="-0.04" upper="0.0" velocity="3.772"/>
+            <limit effort="150" lower="-0.04" upper="0.0" velocity="3.772"/>
             <mimic joint="right_finger_joint"/>
         </joint>
