Commit message: Simplify engineer arm

File: urdf/engineer/engineer.urdf.xacro (robot description, xacro)
@@ -1,26 +1,14 @@
 <?xml version="1.0"?>
 <robot xmlns:xacro="http://www.ros.org/wiki/xacro" name="engineer">
-    <xacro:arg name="load_chassis" default="true"/>
-    <xacro:arg name="load_arm" default="true"/>
     <xacro:arg name="use_simulation" default="false"/>
     <xacro:arg name="roller_type" default="none"/>
-    <xacro:if value="$(arg load_chassis)">
-        <xacro:include filename="$(find rm_description)/urdf/engineer/chassis.urdf.xacro"/>
-        <xacro:chassis roller_type="$(arg roller_type)"/>
-    </xacro:if>
-    <xacro:if value="$(arg load_arm)">
-        <xacro:include filename="$(find rm_description)/urdf/engineer/arm.urdf.xacro"/>
-        <xacro:include filename="$(find rm_description)/urdf/engineer/arm.transmission.xacro"/>
-        <xacro:if value="$(arg load_chassis)">
-            <xacro:arm connected_to="base_link"/>
-        </xacro:if>
-        <xacro:unless value="$(arg load_chassis)">
-            <link name="world"/>
-            <xacro:arm connected_to="world"/>
-        </xacro:unless>
-        <xacro:arm_transmission simulation="$(arg use_simulation)"/>
-        <xacro:include filename="$(find rm_description)/urdf/engineer/hand.urdf.xacro"/>
-        <xacro:hand connected_to="link5" xyz="0.039 0 0"/>
-    </xacro:if>
+    <xacro:include filename="$(find rm_description)/urdf/engineer/chassis.urdf.xacro"/>
+    <xacro:chassis roller_type="$(arg roller_type)"/>
+    <xacro:include filename="$(find rm_description)/urdf/engineer/arm.urdf.xacro"/>
+    <xacro:include filename="$(find rm_description)/urdf/engineer/arm.transmission.xacro"/>
+    <xacro:arm connected_to="base_link"/>
+    <xacro:arm_transmission simulation="$(arg use_simulation)"/>
+    <xacro:include filename="$(find rm_description)/urdf/engineer/hand.urdf.xacro"/>
+    <xacro:hand connected_to="link5" xyz="0.039 0 0"/>
     <xacro:if value="$(arg use_simulation)">
         <gazebo>

Commit message: add engineer simulation condition

File: urdf/engineer/engineer.urdf.xacro (robot description, xacro)
@@ -10,5 +10,5 @@
     <xacro:arm_transmission simulation="$(arg use_simulation)"/>
     <xacro:include filename="$(find rm_description)/urdf/engineer/hand.urdf.xacro"/>
-    <xacro:hand connected_to="link5" xyz="0.039 0 0"/>
+    <xacro:hand connected_to="link5" xyz="0.039 0 0" simulation="$(arg use_simulation)"/>
     <xacro:if value="$(arg use_simulation)">
         <gazebo>

File: urdf/engineer/hand.urdf.xacro (robot description, xacro)
@@ -2,5 +2,11 @@
 <robot xmlns:xacro="http://www.ros.org/wiki/xacro" name="hand">
     <!-- safety_distance: Minimum safety distance in [m] by which the collision volumes are expanded and which is enforced during robot motions -->
-    <xacro:macro name="hand" params="connected_to:='' xyz:='0 0 0' rpy:='0 0 0' ">
+    <xacro:macro name="hand" params="connected_to:='' xyz:='0 0 0' rpy:='0 0 0' simulation ">
+        <material name="Black">
+            <color rgba="0 0 0 1"/>
+        </material>
+        <material name="White">
+            <color rgba="1 1 1 1"/>
+        </material>
         <link name="palm">
             <inertial>
@@ -97,7 +103,7 @@
         <link name="camera">
             <inertial>
-                <mass value="0.04"/>
+                <mass value="0.05"/>
                 <origin xyz="0 0 0"/>
-                <inertia ixx="0.01" ixy="0.0" ixz="0.0" iyy="0.01" iyz="0.0" izz="0.01"/>
+                <inertia ixx="1.271e-3" ixy="2.07e-7" ixz="8.854e-6" iyy="5.190e-4" iyz="1.001e-6" izz="9.976e-4"/>
             </inertial>
             <visual>
@@ -115,12 +121,9 @@
             </collision>
         </link>
-        <!--        <gazebo reference="camera">-->
-        <!--            <masterial>Gazebo/White</masterial>-->
-        <!--        </gazebo>-->
         <joint name="camera_joint" type="fixed">
             <parent link="palm"/>
             <child link="camera"/>
             <origin xyz="0.055 -0.085 0.0962" rpy="0 0 0"/>
-            <axis xyz="0 1 0"/>
+            <axis xyz="0 0 1"/>
         </joint>
         <xacro:unless value="${connected_to == ''}">
@@ -146,4 +149,42 @@
             <mimic joint="right_finger_joint"/>
         </joint>
+        <xacro:if value="${simulation}">
+            <gazebo reference="camera">
+                <sensor type="camera" name="camera_node">
+                    <update_rate>30.0</update_rate>
+                    <camera name="head">
+                        <horizontal_fov>1.3962634</horizontal_fov>
+                        <image>
+                            <width>1920</width>
+                            <height>1080</height>
+                            <format>R8G8B8</format>
+                        </image>
+                        <clip>
+                            <near>0.02</near>
+                            <far>300</far>
+                        </clip>
+                        <noise>
+                            <type>gaussian</type>
+                            <mean>0.0</mean>
+                            <stddev>0.007</stddev>
+                        </noise>
+                    </camera>
+                    <plugin name="gazebo_camera" filename="libgazebo_ros_camera.so">
+                        <alwaysOn>true</alwaysOn>
+                        <updateRate>0.0</updateRate>
+                        <cameraName>/camera</cameraName>
+                        <imageTopicName>image_raw</imageTopicName>
+                        <cameraInfoTopicName>camera_info</cameraInfoTopicName>
+                        <frameName>camera</frameName>
+                        <hackBaseline>0.07</hackBaseline>
+                        <distortionK1>0.0</distortionK1>
+                        <distortionK2>0.0</distortionK2>
+                        <distortionK3>0.0</distortionK3>
+                        <distortionT1>0.0</distortionT1>
+                        <distortionT2>0.0</distortionT2>
+                    </plugin>
+                </sensor>
+            </gazebo>
+        </xacro:if>
         <transmission name="trans_right_finger_joint">
             <type>transmission_interface/SimpleTransmission</type>
@@ -168,40 +209,4 @@
             </actuator>
         </transmission>
-        <gazebo reference="camera">
-            <sensor type="camera" name="camera_node">
-                <update_rate>30.0</update_rate>
-                <camera name="head">
-                    <horizontal_fov>1.3962634</horizontal_fov>
-                    <image>
-                        <width>800</width>
-                        <height>800</height>
-                        <format>R8G8B8</format>
-                    </image>
-                    <clip>
-                        <near>0.02</near>
-                        <far>300</far>
-                    </clip>
-                    <noise>
-                        <type>gaussian</type>
-                        <mean>0.0</mean>
-                        <stddev>0.007</stddev>
-                    </noise>
-                </camera>
-                <plugin name="gazebo_camera" filename="libgazebo_ros_camera.so">
-                    <alwaysOn>true</alwaysOn>
-                    <updateRate>0.0</updateRate>
-                    <cameraName>/camera</cameraName>
-                    <imageTopicName>image_raw</imageTopicName>
-                    <cameraInfoTopicName>camera_info</cameraInfoTopicName>
-                    <frameName>camera</frameName>
-                    <hackBaseline>0.07</hackBaseline>
-                    <distortionK1>0.0</distortionK1>
-                    <distortionK2>0.0</distortionK2>
-                    <distortionK3>0.0</distortionK3>
-                    <distortionT1>0.0</distortionT1>
-                    <distortionT2>0.0</distortionT2>
-                </plugin>
-            </sensor>
-        </gazebo>
     </xacro:macro>
 </robot>

Commit message: update mast parameter

File: urdf/engineer/engineer.urdf.xacro (robot description, xacro)
@@ -16,4 +16,6 @@
         <xacro:include filename="$(find rm_description)/urdf/engineer/hand.urdf.xacro"/>
         <xacro:hand connected_to="link5" xyz="-0.014 0 0" rpy="0 1.57 0" simulation="$(arg use_simulation)"/>
+        <xacro:include filename="$(find rm_description)/urdf/engineer/mast.urdf.xacro"/>
+        <xacro:mast connected_to="link1" xyz="0.076 0.484 0.108 " rpy="-1.57 0 0" simulation="$(arg use_simulation)"/>
     </xacro:if>
     <xacro:if value="$(arg use_simulation)">

File: urdf/engineer/mast.urdf.xacro (robot description, xacro)
@@ -1,15 +1,15 @@
 <?xml version="1.0" encoding="utf-8"?>
-<robot xmlns:xacro="http://www.ros.org/wiki/xacro" name="hand">
+<robot xmlns:xacro="http://www.ros.org/wiki/xacro" name="mast">
     <!-- safety_distance: Minimum safety distance in [m] by which the collision volumes are expanded and which is enforced during robot motions -->
-    <xacro:macro name="gimbal" params="connected_to:='' xyz:='0 0 0' rpy:='0 0 0' simulation ">
+    <xacro:macro name="mast" params="connected_to:='' xyz:='0 0 0' rpy:='0 0 0' simulation">
         <link name="mast">
             <inertial>
-                <mass value="0.348"/>
-                <origin xyz="0.029 0.042 0.096" rpy="0 0 0"/>
-                <inertia ixx="1.221e-2" ixy="1.727e-5" ixz="6.890e-4" iyy="1.237e-2" iyz="7.284e-5" izz="3.043e-4"/>
+                <mass value="0.517"/>
+                <origin xyz="0.009 -0.002 -0.190" rpy="0 0 0"/>
+                <inertia ixx="1.221e-2" ixy="1.727e-5" ixz="6.890e-4" iyy="1.237e-2" iyz="-7.284e-5" izz="3.043e-4"/>
             </inertial>
             <visual>
                 <geometry>
-                    <mesh filename="package://rm_description/meshes/gineer/mast.stl" scale="0.001 0.001 0.001"/>
+                    <mesh filename="package://rm_description/meshes/engineer/mast.stl" scale="0.001 0.001 0.001"/>
                 </geometry>
             </visual>
@@ -23,11 +23,11 @@
         <link name="yaw">
             <inertial>
-                <origin xyz="0.0 0.075 0.021" rpy="0 0 0"/>
-                <mass value="0.284"/>
-                <inertia ixx="7.653e-4" ixy="1.922e-5" ixz="1.589e-5" iyy="3.805e-4" iyz="-3.052e-4" izz="4.364e-4"/>
+                <origin xyz="0.0 0.029 0.035" rpy="0 0 0"/>
+                <mass value="0.175"/>
+                <inertia ixx="3.583e-4" ixy="-4.2e-7" ixz="2.42e-7" iyy="1.473e-4" iyz="-4.618e-5" izz="2.568e-4"/>
             </inertial>
             <visual>
                 <geometry>
-                    <box size="0.030 0.027 0.063"/>
+                    <mesh filename="package://rm_description/meshes/engineer/yaw.stl" scale="0.001 0.001 0.001"/>
                 </geometry>
             </visual>
@@ -41,11 +41,11 @@
         <link name="pitch">
             <inertial>
-                <origin xyz="0.0 -0.075 0.021" rpy="0 0 0"/>
-                <mass value="0.284"/>
-                <inertia ixx="7.653e-4" ixy="1.922e-5" ixz="-1.589e-5" iyy="3.805e-4" iyz="3.052e-4" izz="4.364e-4"/>
+                <origin xyz="0.0 -0.04 0.002" rpy="0 0 0"/>
+                <mass value="0.246"/>
+                <inertia ixx="1.883e-4" ixy="1.22e-7" ixz="-7.56e-6" iyy="2.304e-4" iyz="-2.18e-7" izz="2.662e-4"/>
             </inertial>
             <visual>
                 <geometry>
-                    <box size="0.030 0.027 0.063"/>
+                    <mesh filename="package://rm_description/meshes/engineer/pitch.stl" scale="0.001 0.001 0.001"/>
                 </geometry>
             </visual>
@@ -57,53 +57,17 @@
             </collision>
         </link>
-        <link name="camera1">
-            <inertial>
-                <mass value="0.05"/>
-                <origin xyz="0 0 0"/>
-                <inertia ixx="1.271e-3" ixy="2.07e-7" ixz="8.854e-6" iyy="5.190e-4" iyz="1.001e-6" izz="9.976e-4"/>
-            </inertial>
-            <visual>
-                <origin xyz=" 0 0 0 " rpy="0 0 0"/>
-                <geometry>
-                    <box size="0.022 0.021 0.0226"/>
-                </geometry>
-                <material name="Black"/>
-            </visual>
-            <collision>
-                <origin xyz="0.0 0.0 0.0" rpy="0 0 0"/>
-                <geometry>
-                    <box size="0.01 0.04 0.04"/>
-                </geometry>
-            </collision>
-        </link>
-        <link name="camera2">
-            <inertial>
-                <mass value="0.05"/>
-                <origin xyz="0 0 0"/>
-                <inertia ixx="1.271e-3" ixy="2.07e-7" ixz="8.854e-6" iyy="5.190e-4" iyz="1.001e-6" izz="9.976e-4"/>
-            </inertial>
-            <visual>
-                <origin xyz=" 0 0 0 " rpy="0 0 0"/>
-                <geometry>
-                    <box size="0.022 0.021 0.0226"/>
-                </geometry>
-                <material name="Black"/>
-            </visual>
-            <collision>
-                <origin xyz="0.0 0.0 0.0" rpy="0 0 0"/>
-                <geometry>
-                    <box size="0.01 0.04 0.04"/>
-                </geometry>
-            </collision>
-        </link>
+        <link name="camera1"/>
+        <link name="camera2"/>
         <xacro:unless value="${connected_to == ''}">
             <joint name="mast_joint" type="prismatic">
+                <origin xyz="${xyz}" rpy="${rpy}"/>
                 <parent link="${connected_to}"/>
                 <child link="mast"/>
-                <origin xyz="${xyz}" rpy="${rpy}"/>
+                <axis xyz="0 0 1"/>
+                <limit effort="1.2" velocity="13.82" lower="-1e10" upper="1e10"/>
             </joint>
         </xacro:unless>
         <joint name="yaw_joint" type="revolute">
-            <origin xyz="0 0 0.129"
+            <origin xyz="0 0 0"
                     rpy="0 0 0"/>
             <dynamics damping="0.0" friction="0.1"/>
@@ -114,11 +78,7 @@
         </joint>
         <joint name="pitch_joint" type="revolute">
-            <origin xyz="-0.06  0 0.191 " rpy="0 0 0"/>
+            <origin xyz="0.0  0.029 0.059 " rpy="0 0 0"/>
             <dynamics damping="0.0" friction="0.1"/>
             <limit effort="1.2" velocity="13.82" lower="-1e10" upper="1e10"/>
-            <safety_controller k_velocity="0.1"
-                               k_position="100"
-                               soft_lower_limit="${pitch_lower_limit+threshold}"
-                               soft_upper_limit="${pitch_upper_limit-threshold}"/>
             <parent link="yaw"/>
             <child link="pitch"/>
@@ -128,5 +88,5 @@
             <parent link="pitch"/>
             <child link="camera1"/>
-            <origin xyz="0.055 -0.85 0.0962" rpy="0 0 0"/>
+            <origin xyz="0.006 0.028 0.021" rpy="0 0 0"/>
             <axis xyz="0 0 1"/>
         </joint>
@@ -134,5 +94,5 @@
             <parent link="pitch"/>
             <child link="camera2"/>
-            <origin xyz="0.055 0.85 0.0962" rpy="0 0 0"/>
+            <origin xyz="0.006 0.052 0.021" rpy="0 0 0"/>
             <axis xyz="0 0 1"/>
         </joint>
@@ -169,6 +129,6 @@
         </transmission>
         <xacro:if value="${simulation}">
-            <gazebo reference="camera_link">
-                <sensor type="camera" name="camera">
+            <gazebo reference="camera1_link">
+                <sensor type="camera" name="camera1">
                     <update_rate>30.0</update_rate>
                     <camera name="head">

Commit message: update engineer collision

File: urdf/engineer/engineer.urdf.xacro (robot description, xacro)
@@ -17,5 +17,5 @@
         <xacro:hand connected_to="link5" xyz="-0.014 0 0" rpy="0 1.57 0" simulation="$(arg use_simulation)"/>
         <xacro:include filename="$(find rm_description)/urdf/engineer/mast.urdf.xacro"/>
-        <xacro:mast connected_to="link1" xyz="0.076 0.484 0.108 " rpy="-1.57 0 0" simulation="$(arg use_simulation)"/>
+        <xacro:mast connected_to="link1" xyz="-0.076 0.484 0.108 " rpy="-1.57 0 0" simulation="$(arg use_simulation)"/>
     </xacro:if>
     <xacro:if value="$(arg use_simulation)">

File: urdf/engineer/mast.urdf.xacro (robot description, xacro)
@@ -15,7 +15,13 @@
             </visual>
             <collision>
-                <origin xyz="0 0 0" rpy="0 0 0"/>
+                <origin xyz="0.004 0 -0.259" rpy="0 0 0"/>
                 <geometry>
-                    <box size="0.055 0.267 0.06"/>
+                    <box size="0.053 0.035 0.45"/>
+                </geometry>
+            </collision>
+            <collision>
+                <origin xyz="-0.013 0 -0.021" rpy="0 0 0"/>
+                <geometry>
+                    <box size="0.075 0.059 0.043"/>
                 </geometry>
             </collision>
@@ -33,7 +39,7 @@
             </visual>
             <collision>
-                <origin xyz="0 0 0" rpy="0 0 0"/>
+                <origin xyz="0. 0.004 0.04" rpy="0 0 0"/>
                 <geometry>
-                    <box size="0.030 0.027 0.063"/>
+                    <box size="0.054 0.120 0.081"/>
                 </geometry>
             </collision>
@@ -51,7 +57,7 @@
             </visual>
             <collision>
-                <origin xyz="0 0 0" rpy="0 0 0"/>
+                <origin xyz="-0.005 -0.04 0.014" rpy="0 0 0"/>
                 <geometry>
-                    <box size="0.030 0.027 0.063"/>
+                    <box size="0.1 0.048 0.036"/>
                 </geometry>
             </collision>
@@ -111,5 +117,4 @@
             <actuator name="pitch_joint_motor">
                 <mechanicalReduction>-1</mechanicalReduction>
-                <mechanicalReduction>1</mechanicalReduction>
             </actuator>
             <joint name="pitch_joint">
@@ -125,5 +130,5 @@
             </joint>
             <actuator name="mast_motor">
-                <mechanicalReduction>30</mechanicalReduction>
+                <mechanicalReduction>71.44</mechanicalReduction>
             </actuator>
         </transmission>

Commit message: Change the hands coordinates.

File: urdf/engineer/engineer.urdf.xacro (robot description, xacro)
@@ -15,5 +15,5 @@
         <xacro:arm_transmission simulation="$(arg use_simulation)"/>
         <xacro:include filename="$(find rm_description)/urdf/engineer/hand.urdf.xacro"/>
-        <xacro:hand connected_to="link5" xyz="-0.014 0 0" rpy="0 1.57 0" simulation="$(arg use_simulation)"/>
+        <xacro:hand connected_to="link5" xyz="-0.014 0 0" rpy="0 -1.57 0" simulation="$(arg use_simulation)"/>
         <xacro:include filename="$(find rm_description)/urdf/engineer/mast.urdf.xacro"/>
         <xacro:mast connected_to="link1" xyz="-0.0745 -0.1085 0.5697" rpy="0 0 0" simulation="$(arg use_simulation)"/>

File: urdf/engineer/hand.urdf.xacro (robot description, xacro)
@@ -37,4 +37,5 @@
             </inertial>
             <visual>
+                <origin xyz="0 0 0" rpy="0 1.57 0"/>
                 <geometry>
                     <mesh filename="package://rm_description/meshes/engineer/right_finger.stl"
@@ -42,12 +43,12 @@
                 </geometry>
             </visual>
+<!--            <collision>-->
+<!--                <origin xyz="0.0 0.088 0.025" rpy="0 0 0"/>-->
+<!--                <geometry>-->
+<!--                    <box size="0.03 0.112 0.022"/>-->
+<!--                </geometry>-->
+<!--            </collision>-->
             <collision>
-                <origin xyz="0.0 0.088 0.025" rpy="0 0 0"/>
-                <geometry>
-                    <box size="0.03 0.112 0.022"/>
-                </geometry>
-            </collision>
-            <collision>
-                <origin xyz="0.0 0.130 0.07" rpy="0 0 0"/>
+                <origin xyz="0.07 0.130 0.0" rpy="0 1.57 0"/>
                 <geometry>
                     <box size="0.030 0.017 0.112"/>
@@ -62,4 +63,5 @@
             </inertial>
             <visual>
+                <origin xyz="0 0 0" rpy="0 1.57 0"/>
                 <geometry>
                     <mesh filename="package://rm_description/meshes/engineer/left_finger.stl"
@@ -67,12 +69,12 @@
                 </geometry>
             </visual>
+<!--            <collision>-->
+<!--                <origin xyz="0.0 -0.088 0.025" rpy="0 0 0"/>-->
+<!--                <geometry>-->
+<!--                    <box size="0.03 0.112 0.022"/>-->
+<!--                </geometry>-->
+<!--            </collision>-->
             <collision>
-                <origin xyz="0.0 -0.088 0.025" rpy="0 0 0"/>
-                <geometry>
-                    <box size="0.03 0.112 0.022"/>
-                </geometry>
-            </collision>
-            <collision>
-                <origin xyz="0.0 -0.130 0.07" rpy="0 0 0"/>
+                <origin xyz="0.07 -0.130 0.0" rpy="0 1.57 0"/>
                 <geometry>
                     <box size="0.030 0.017 0.112"/>
@@ -90,5 +92,5 @@
             <parent link="palm"/>
             <child link="right_finger"/>
-            <origin xyz="0 0 0.045" rpy="0 0 0"/>
+            <origin xyz="0 0 0.045" rpy="0 1.57 0"/>
             <axis xyz="0 1 0"/>
             <limit effort="588" lower="-0.04" upper="0.0" velocity="3.772"/>
@@ -97,5 +99,5 @@
             <parent link="palm"/>
             <child link="left_finger"/>
-            <origin xyz="0 0 0.045" rpy="0 0 0"/>
+            <origin xyz="0 0 0.045" rpy="0 1.57 0"/>
             <axis xyz="0 -1 0"/>
             <limit effort="588" lower="-0.04" upper="0.0" velocity="3.772"/>
