Commit message: Adjust the hands inertial.

File: urdf/engineer/engineer.urdf.xacro (robot description, xacro)
@@ -15,5 +15,5 @@
         <xacro:arm_transmission simulation="$(arg use_simulation)"/>
         <xacro:include filename="$(find rm_description)/urdf/engineer/hand.urdf.xacro"/>
-        <xacro:hand connected_to="link5" xyz="-0.014 0 0" rpy="0 -1.57 0" simulation="$(arg use_simulation)"/>
+        <xacro:hand connected_to="link5" xyz="-0.014 0 0" rpy="0 0 0" simulation="$(arg use_simulation)"/>
         <xacro:include filename="$(find rm_description)/urdf/engineer/mast.urdf.xacro"/>
         <xacro:mast connected_to="link1" xyz="-0.0745 -0.1085 0.5697" rpy="0 0 0" simulation="$(arg use_simulation)"/>

File: urdf/engineer/hand.urdf.xacro (robot description, xacro)
@@ -11,7 +11,7 @@
         <link name="palm">
             <inertial>
-                <mass value="0.695"/>
-                <origin xyz="0.0 0.0 -0.024" rpy="0 0 0"/>
-                <inertia ixx="4.945e-4" ixy="1.180e-7" ixz="3.142e-6" iyy="2.444e-4" iyz="-1.2e-7" izz="5.042e-4"/>
+                <mass value="0.705"/>
+                <origin xyz="0.0 0.0 0" rpy="0 0 0"/>
+                <inertia ixx="1.483e-3" ixy="-3.268e-4" ixz="-1.279015e-5" iyy="1.014e-4" iyz="-5.7349231e-5" izz="1.553e-3"/>
             </inertial>
             <visual>
@@ -21,7 +21,13 @@
             </visual>
             <collision>
-                <origin xyz="0 0 0.027" rpy="0 0 0"/>
+                <origin xyz="0.026 0. 0." rpy="0 0 0"/>
                 <geometry>
-                    <box size="0.055 0.267 0.055"/>
+                    <box size="0.056 0.2748 0.062"/>
+                </geometry>
+            </collision>
+            <collision>
+                <origin xyz="0.023 0.117985 0." rpy="0 0 0"/>
+                <geometry>
+                    <box size="0.064 0.045 0.09"/>
                 </geometry>
             </collision>
@@ -32,10 +38,10 @@
         <link name="right_finger">
             <inertial>
-                <origin xyz="0.0 0.075 -0.021" rpy="0 0 0"/>
-                <mass value="0.284"/>
-                <inertia ixx="4.364e-4" ixy="-3.052e-5" ixz="-1.589e-5" iyy="3.805e-4" iyz="-1.922e-5" izz="7.653e-4"/>
+                <origin xyz="0.015044 -0.0622 8e-6" rpy="0 0 0"/>
+                <mass value="0.211439"/>
+                <inertia ixx="1.107e-3" ixy="4.148e-4" ixz="4.1265e-8" iyy="3.139e-4" iyz="7.1221e-8" izz="1.39e-3"/>
             </inertial>
             <visual>
-                <origin xyz="0 0 0" rpy="0 1.57 0"/>
+<!--                <origin xyz="0 0 0" rpy="0 0 0"/>-->
                 <geometry>
                     <mesh filename="package://rm_description/meshes/engineer/right_finger.stl"
@@ -43,14 +49,8 @@
                 </geometry>
             </visual>
-<!--            <collision>-->
-<!--                <origin xyz="0.0 0.088 0.025" rpy="0 0 0"/>-->
-<!--                <geometry>-->
-<!--                    <box size="0.03 0.112 0.022"/>-->
-<!--                </geometry>-->
-<!--            </collision>-->
             <collision>
-                <origin xyz="0.07 0.130 0.0" rpy="0 1.57 0"/>
+                <origin xyz="0.066 -0.126453 0.0" rpy="0 0 0"/>
                 <geometry>
-                    <box size="0.030 0.017 0.112"/>
+                    <box size="0.113 0.0178 0.036"/>
                 </geometry>
             </collision>
@@ -58,10 +58,10 @@
         <link name="left_finger">
             <inertial>
-                <origin xyz="0.0 -0.075 -0.021" rpy="0 0 0"/>
-                <mass value="0.284"/>
-                <inertia ixx="4.364e-4" ixy="3.052e-4" ixz="1.589e-5" iyy="3.805e-4" iyz="-1.922e-5" izz="7.653e-4"/>
+                <origin xyz="0.015 0.062 8e-6" rpy="0 0 0"/>
+                <mass value="0.211439"/>
+                <inertia ixx="1.107e-3" ixy="-4.148e-4" ixz="4.1265e-8" iyy="3.139e-4" iyz="-0.071221e-8" izz="1.39e-3"/>
             </inertial>
             <visual>
-                <origin xyz="0 0 0" rpy="0 1.57 0"/>
+<!--                <origin xyz="0 0 0" rpy="0 1.57 0"/>-->
                 <geometry>
                     <mesh filename="package://rm_description/meshes/engineer/left_finger.stl"
@@ -76,7 +76,7 @@
 <!--            </collision>-->
             <collision>
-                <origin xyz="0.07 -0.130 0.0" rpy="0 1.57 0"/>
+                <origin xyz="0.068474 0.126453 0.0" rpy="0 0 0"/>
                 <geometry>
-                    <box size="0.030 0.017 0.112"/>
+                    <box size="0.113 0.0178 0.036"/>
                 </geometry>
             </collision>
@@ -92,5 +92,5 @@
             <parent link="palm"/>
             <child link="right_finger"/>
-            <origin xyz="0 0 0.045" rpy="0 1.57 0"/>
+            <origin xyz="0.045 0 0" rpy="0 0 0"/>
             <axis xyz="0 1 0"/>
             <limit effort="588" lower="-0.04" upper="0.0" velocity="3.772"/>
@@ -99,5 +99,5 @@
             <parent link="palm"/>
             <child link="left_finger"/>
-            <origin xyz="0 0 0.045" rpy="0 1.57 0"/>
+            <origin xyz="0.045 0 0" rpy="0 0 0"/>
             <axis xyz="0 -1 0"/>
             <limit effort="588" lower="-0.04" upper="0.0" velocity="3.772"/>

Commit message: Update mast URDF

File: urdf/engineer/engineer.urdf.xacro (robot description, xacro)
@@ -17,5 +17,5 @@
         <xacro:hand connected_to="link5" xyz="-0.014 0 0" rpy="0 0 0" simulation="$(arg use_simulation)"/>
         <xacro:include filename="$(find rm_description)/urdf/engineer/mast.urdf.xacro"/>
-        <xacro:mast connected_to="link1" xyz="-0.0745 -0.1085 0.5697" rpy="0 0 0" simulation="$(arg use_simulation)"/>
+        <xacro:mast connected_to="link1" xyz="-0.0745 -0.1085 0.53" rpy="0 0 0" simulation="$(arg use_simulation)"/>
     </xacro:if>
     <xacro:if value="$(arg use_simulation)">

File: urdf/engineer/mast.urdf.xacro (robot description, xacro)
@@ -17,5 +17,5 @@
                 <origin xyz="0.004 0 -0.259" rpy="0 0 0"/>
                 <geometry>
-                    <box size="0.053 0.035 0.45"/>
+                    <box size="0.035 0.035 0.45"/>
                 </geometry>
             </collision>
