Commit message: Add camera in mast of engineer

File: urdf/engineer/mast.urdf.xacro (robot description, xacro)
@@ -57,6 +57,44 @@
             </collision>
         </link>
-        <link name="camera1"/>
-        <link name="camera2"/>
+        <link name="camera_wideangle">
+            <visual>
+                <origin xyz="0 0 0" rpy="0 0 0"/>
+                <geometry>
+                    <mesh filename="package://rm_description/meshes/common/camera.stl" scale="0.001 0.001 0.001"/>
+                </geometry>
+            </visual>
+            <inertial>
+                <mass value="0.17671"/>
+                <origin xyz="0.022 0.0 0.0"/>
+                <inertia ixx="2.129e-5" ixy="7.329e-8" ixz="-1.11e-7" iyy="2.198e-4" iyz="-8.04e-7" izz="2.197e-4"/>
+            </inertial>
+            <collision>
+                <origin xyz="0 0 0" rpy="0 0 0"/>
+                <geometry>
+                    <mesh filename="package://rm_description/meshes/common/camera.stl" scale="0.001 0.001 0.001"/>
+                </geometry>
+            </collision>
+        </link>
+        <link name="camera_telephoto">
+            <visual>
+                <origin xyz="0 0 0" rpy="0 0 0"/>
+                <geometry>
+                    <mesh filename="package://rm_description/meshes/common/camera.stl" scale="0.001 0.001 0.001"/>
+                </geometry>
+            </visual>
+            <inertial>
+                <mass value="0.17671"/>
+                <origin xyz="0.022 0.0 0.0"/>
+                <inertia ixx="2.129e-5" ixy="7.329e-8" ixz="-1.11e-7" iyy="2.198e-4" iyz="-8.04e-7" izz="2.197e-4"/>
+            </inertial>
+            <collision>
+                <origin xyz="0 0 0" rpy="0 0 0"/>
+                <geometry>
+                    <mesh filename="package://rm_description/meshes/common/camera.stl" scale="0.001 0.001 0.001"/>
+                </geometry>
+            </collision>
+        </link>
+        <link name="camera_wideangle_optical_frame"/>
+        <link name="camera_telephoto_optical_frame"/>
         <xacro:unless value="${connected_to == ''}">
             <joint name="mast_joint" type="prismatic">
@@ -85,15 +123,25 @@
             <axis xyz="0 1 0 "/>
         </joint>
-        <joint name="camera1_joint" type="fixed">
+        <joint name="camera_wideangle_joint" type="fixed">
             <parent link="pitch"/>
-            <child link="camera1"/>
+            <child link="camera_wideangle"/>
             <origin xyz="0.006 0.028 0.021" rpy="0 0 0"/>
             <axis xyz="0 0 1"/>
         </joint>
-        <joint name="camera2_joint" type="fixed">
+        <joint name="camera_telephoto_joint" type="fixed">
             <parent link="pitch"/>
-            <child link="camera2"/>
+            <child link="camera_telephoto"/>
             <origin xyz="0.006 0.052 0.021" rpy="0 0 0"/>
             <axis xyz="0 0 1"/>
+        </joint>
+        <joint name="camera_wideangle_optical_frame_joint" type="fixed">
+            <origin xyz="0.026 0 -0.0145" rpy="-1.57 0 -1.57"/>
+            <parent link="camera_wideangle"/>
+            <child link="camera_wideangle_optical_frame"/>
+        </joint>
+        <joint name="camera_telephoto_optical_frame_joint" type="fixed">
+            <origin xyz="0.026 0 -0.0145" rpy="-1.57 0 -1.57"/>
+            <parent link="camera_telephoto"/>
+            <child link="camera_telephoto_optical_frame"/>
         </joint>
         <transmission name="trans_yaw_joint">
@@ -129,7 +177,7 @@
         </transmission>
         <xacro:if value="${simulation}">
-            <gazebo reference="camera1_link">
-                <sensor type="camera" name="camera1">
-                    <update_rate>30.0</update_rate>
+            <gazebo reference="camera_wideangle">
+                <sensor type="camera" name="camera_wideangle">
+                    <update_rate>100.0</update_rate>
                     <camera name="head">
                         <horizontal_fov>1.3962634</horizontal_fov>
@@ -152,8 +200,44 @@
                         <alwaysOn>true</alwaysOn>
                         <updateRate>0.0</updateRate>
-                        <cameraName>galaxy_camera</cameraName>
+                        <cameraName>galaxy_camera/camera_wideangle</cameraName>
                         <imageTopicName>image_raw</imageTopicName>
                         <cameraInfoTopicName>camera_info</cameraInfoTopicName>
-                        <frameName>camera_link</frameName>
+                        <frameName>camera_wideangle_optical_frame</frameName>
+                        <hackBaseline>0.07</hackBaseline>
+                        <distortionK1>0.0</distortionK1>
+                        <distortionK2>0.0</distortionK2>
+                        <distortionK3>0.0</distortionK3>
+                        <distortionT1>0.0</distortionT1>
+                        <distortionT2>0.0</distortionT2>
+                    </plugin>
+                </sensor>
+            </gazebo>
+            <gazebo reference="camera_telephoto">
+                <sensor type="camera" name="camera_telephoto">
+                    <update_rate>100.0</update_rate>
+                    <camera name="head">
+                        <horizontal_fov>1.3962634</horizontal_fov>
+                        <image>
+                            <width>1920</width>
+                            <height>1080</height>
+                            <format>R8G8B8</format>
+                        </image>
+                        <clip>
+                            <near>0.05</near>
+                            <far>5</far>
+                        </clip>
+                        <noise>
+                            <type>gaussian</type>
+                            <mean>0.0</mean>
+                            <stddev>0.007</stddev>
+                        </noise>
+                    </camera>
+                    <plugin name="camera_controller" filename="libgazebo_ros_camera.so">
+                        <alwaysOn>true</alwaysOn>
+                        <updateRate>0.0</updateRate>
+                        <cameraName>galaxy_camera/camera_telephoto</cameraName>
+                        <imageTopicName>image_raw</imageTopicName>
+                        <cameraInfoTopicName>camera_info</cameraInfoTopicName>
+                        <frameName>camera_telephoto_optical_frame</frameName>
                         <hackBaseline>0.07</hackBaseline>
                         <distortionK1>0.0</distortionK1>

Commit message: change mast camera frame

File: urdf/engineer/mast.urdf.xacro (robot description, xacro)
@@ -63,42 +63,6 @@
             </collision>
         </link>
-        <link name="camera_wideangle">
-            <visual>
-                <origin xyz="0 0 0" rpy="0 0 0"/>
-                <geometry>
-                    <mesh filename="package://rm_description/meshes/common/camera.stl" scale="0.001 0.001 0.001"/>
-                </geometry>
-            </visual>
-            <inertial>
-                <mass value="0.17671"/>
-                <origin xyz="0.022 0.0 0.0"/>
-                <inertia ixx="2.129e-5" ixy="7.329e-8" ixz="-1.11e-7" iyy="2.198e-4" iyz="-8.04e-7" izz="2.197e-4"/>
-            </inertial>
-            <collision>
-                <origin xyz="0 0 0" rpy="0 0 0"/>
-                <geometry>
-                    <mesh filename="package://rm_description/meshes/common/camera.stl" scale="0.001 0.001 0.001"/>
-                </geometry>
-            </collision>
-        </link>
-        <link name="camera_telephoto">
-            <visual>
-                <origin xyz="0 0 0" rpy="0 0 0"/>
-                <geometry>
-                    <mesh filename="package://rm_description/meshes/common/camera.stl" scale="0.001 0.001 0.001"/>
-                </geometry>
-            </visual>
-            <inertial>
-                <mass value="0.17671"/>
-                <origin xyz="0.022 0.0 0.0"/>
-                <inertia ixx="2.129e-5" ixy="7.329e-8" ixz="-1.11e-7" iyy="2.198e-4" iyz="-8.04e-7" izz="2.197e-4"/>
-            </inertial>
-            <collision>
-                <origin xyz="0 0 0" rpy="0 0 0"/>
-                <geometry>
-                    <mesh filename="package://rm_description/meshes/common/camera.stl" scale="0.001 0.001 0.001"/>
-                </geometry>
-            </collision>
-        </link>
+        <link name="camera_telephoto"/>
+        <link name="camera_wideangle"/>
         <link name="camera_wideangle_optical_frame"/>
         <link name="camera_telephoto_optical_frame"/>

Commit message: ix mast limit and add engineer.yaml

File: urdf/engineer/mast.urdf.xacro (robot description, xacro)
@@ -81,5 +81,5 @@
                     rpy="0 0 0"/>
             <dynamics damping="0.0" friction="0.1"/>
-            <limit effort="1.2" velocity="13.82" lower="-3.14" upper="3.14"/>
+            <limit effort="0.1" velocity="10" lower="-3.14" upper="3.14"/>
             <parent link="mast"/>
             <child link="yaw"/>
@@ -89,5 +89,5 @@
             <origin xyz="0.0  0.029 0.059 " rpy="0 0 0"/>
             <dynamics damping="0.0" friction="0.1"/>
-            <limit effort="1.2" velocity="13.82" lower="-1e10" upper="1e10"/>
+            <limit effort="0.1" velocity="10" lower="-0.38" upper="0.52"/>
             <parent link="yaw"/>
             <child link="pitch"/>
@@ -119,8 +119,8 @@
             <type>transmission_interface/SimpleTransmission</type>
             <actuator name="yaw_joint_motor">
-                <mechanicalReduction>1</mechanicalReduction>
+                <mechanicalReduction>-1</mechanicalReduction>
             </actuator>
             <joint name="yaw_joint">
-                <offset>-2.160</offset>
+                <offset>2.52493</offset>
                 <hardwareInterface>hardware_interface/EffortJointInterface</hardwareInterface>
             </joint>
@@ -132,5 +132,5 @@
             </actuator>
             <joint name="pitch_joint">
-                <offset>0.902</offset>
+                <offset>2.9038</offset>
                 <hardwareInterface>hardware_interface/EffortJointInterface</hardwareInterface>
             </joint>
@@ -142,5 +142,5 @@
                 <offset>0.0</offset>
             </joint>
-            <actuator name="mast_motor">
+            <actuator name="mast_joint_motor">
                 <mechanicalReduction>71.44</mechanicalReduction>
             </actuator>

Commit message: Delete lots commented code

File: urdf/engineer/mast.urdf.xacro (robot description, xacro)
@@ -51,8 +51,8 @@
             </visual>
         </link>
-<!--        <link name="camera_telephoto"/>-->
-<!--        <link name="camera_wideangle"/>-->
-<!--        <link name="camera_wideangle_optical_frame"/>-->
-<!--        <link name="camera_telephoto_optical_frame"/>-->
+        <!--        <link name="camera_telephoto"/>-->
+        <!--        <link name="camera_wideangle"/>-->
+        <!--        <link name="camera_wideangle_optical_frame"/>-->
+        <!--        <link name="camera_telephoto_optical_frame"/>-->
         <xacro:unless value="${connected_to == ''}">
             <joint name="mast_joint" type="prismatic">
@@ -62,5 +62,5 @@
                 <axis xyz="0 0 1"/>
                 <dynamics damping="0.0" friction="0.8"/>
-                <limit effort="30" velocity="13.82" lower="-0.175" upper="0"/>
+                <limit effort="10" velocity="13.82" lower="-0.175" upper="0"/>
             </joint>
         </xacro:unless>
@@ -85,26 +85,4 @@
             <self_collide>1</self_collide>
         </gazebo>
-<!--        <joint name="camera_wideangle_joint" type="fixed">-->
-<!--            <parent link="pitch"/>-->
-<!--            <child link="camera_wideangle"/>-->
-<!--            <origin xyz="0.006 0.028 0.021" rpy="0 0 0"/>-->
-<!--            <axis xyz="0 0 1"/>-->
-<!--        </joint>-->
-<!--        <joint name="camera_telephoto_joint" type="fixed">-->
-<!--            <parent link="pitch"/>-->
-<!--            <child link="camera_telephoto"/>-->
-<!--            <origin xyz="0.006 0.052 0.021" rpy="0 0 0"/>-->
-<!--            <axis xyz="0 0 1"/>-->
-<!--        </joint>-->
-<!--        <joint name="camera_wideangle_optical_frame_joint" type="fixed">-->
-<!--            <origin xyz="0.026 0 -0.0145" rpy="-1.57 0 -1.57"/>-->
-<!--            <parent link="camera_wideangle"/>-->
-<!--            <child link="camera_wideangle_optical_frame"/>-->
-<!--        </joint>-->
-<!--        <joint name="camera_telephoto_optical_frame_joint" type="fixed">-->
-<!--            <origin xyz="0.026 0 -0.0145" rpy="-1.57 0 -1.57"/>-->
-<!--            <parent link="camera_telephoto"/>-->
-<!--            <child link="camera_telephoto_optical_frame"/>-->
-<!--        </joint>-->
         <transmission name="trans_yaw_joint">
             <type>transmission_interface/SimpleTransmission</type>
@@ -134,81 +112,7 @@
             </joint>
             <actuator name="mast_joint_motor">
-                <mechanicalReduction>52.63</mechanicalReduction>
+                <mechanicalReduction>-50.0</mechanicalReduction>
             </actuator>
         </transmission>
-        <xacro:if value="${simulation}">
-<!--            <gazebo reference="camera_wideangle">-->
-<!--                <sensor type="camera" name="camera_wideangle">-->
-<!--                    <update_rate>100.0</update_rate>-->
-<!--                    <camera name="wideangle">-->
-<!--                        <horizontal_fov>2.0934</horizontal_fov>-->
-<!--                        <image>-->
-<!--                            <width>1920</width>-->
-<!--                            <height>1080</height>-->
-<!--                            <format>R8G8B8</format>-->
-<!--                        </image>-->
-<!--                        <clip>-->
-<!--                            <near>0.05</near>-->
-<!--                            <far>5</far>-->
-<!--                        </clip>-->
-<!--                        <noise>-->
-<!--                            <type>gaussian</type>-->
-<!--                            <mean>0.0</mean>-->
-<!--                            <stddev>0.007</stddev>-->
-<!--                        </noise>-->
-<!--                    </camera>-->
-<!--                    <plugin name="camera_controller" filename="libgazebo_ros_camera.so">-->
-<!--                        <alwaysOn>true</alwaysOn>-->
-<!--                        <updateRate>0.0</updateRate>-->
-<!--                        <cameraName>usb_camera/camera_wideangle</cameraName>-->
-<!--                        <imageTopicName>image_raw</imageTopicName>-->
-<!--                        <cameraInfoTopicName>camera_info</cameraInfoTopicName>-->
-<!--                        <frameName>camera_wideangle_optical_frame</frameName>-->
-<!--                        <hackBaseline>0.07</hackBaseline>-->
-<!--                        <distortionK1>0.0</distortionK1>-->
-<!--                        <distortionK2>0.0</distortionK2>-->
-<!--                        <distortionK3>0.0</distortionK3>-->
-<!--                        <distortionT1>0.0</distortionT1>-->
-<!--                        <distortionT2>0.0</distortionT2>-->
-<!--                    </plugin>-->
-<!--                </sensor>-->
-<!--            </gazebo>-->
-<!--            <gazebo reference="camera_telephoto">-->
-<!--                <sensor type="camera" name="camera_telephoto">-->
-<!--                    <update_rate>100.0</update_rate>-->
-<!--                    <camera name="telephoto">-->
-<!--                        <horizontal_fov>1.919</horizontal_fov>-->
-<!--                        <image>-->
-<!--                            <width>1920</width>-->
-<!--                            <height>1080</height>-->
-<!--                            <format>R8G8B8</format>-->
-<!--                        </image>-->
-<!--                        <clip>-->
-<!--                            <near>0.05</near>-->
-<!--                            <far>5</far>-->
-<!--                        </clip>-->
-<!--                        <noise>-->
-<!--                            <type>gaussian</type>-->
-<!--                            <mean>0.0</mean>-->
-<!--                            <stddev>0.007</stddev>-->
-<!--                        </noise>-->
-<!--                    </camera>-->
-<!--                    <plugin name="camera_controller" filename="libgazebo_ros_camera.so">-->
-<!--                        <alwaysOn>true</alwaysOn>-->
-<!--                        <updateRate>0.0</updateRate>-->
-<!--                        <cameraName>usb_camera/camera_telephoto</cameraName>-->
-<!--                        <imageTopicName>image_raw</imageTopicName>-->
-<!--                        <cameraInfoTopicName>camera_info</cameraInfoTopicName>-->
-<!--                        <frameName>camera_telephoto_optical_frame</frameName>-->
-<!--                        <hackBaseline>0.07</hackBaseline>-->
-<!--                        <distortionK1>0.0</distortionK1>-->
-<!--                        <distortionK2>0.0</distortionK2>-->
-<!--                        <distortionK3>0.0</distortionK3>-->
-<!--                        <distortionT1>0.0</distortionT1>-->
-<!--                        <distortionT2>0.0</distortionT2>-->
-<!--                    </plugin>-->
-<!--                </sensor>-->
-<!--            </gazebo>-->
-        </xacro:if>
     </xacro:macro>
 </robot>

Commit message: Increase mast_joint effort limit

File: urdf/engineer/mast.urdf.xacro (robot description, xacro)
@@ -62,5 +62,5 @@
                 <axis xyz="0 0 1"/>
                 <dynamics damping="0.0" friction="0.8"/>
-                <limit effort="20.0" velocity="1.0" lower="-0.37" upper="0"/>
+                <limit effort="25.0" velocity="1.0" lower="-0.37" upper="0"/>
             </joint>
         </xacro:unless>

Commit message: Update mast limit and offset

File: urdf/engineer/mast.urdf.xacro (robot description, xacro)
@@ -51,8 +51,4 @@
             </visual>
         </link>
-        <!--        <link name="camera_telephoto"/>-->
-        <!--        <link name="camera_wideangle"/>-->
-        <!--        <link name="camera_wideangle_optical_frame"/>-->
-        <!--        <link name="camera_telephoto_optical_frame"/>-->
         <xacro:unless value="${connected_to == ''}">
             <joint name="mast_joint" type="prismatic">
@@ -69,5 +65,5 @@
                     rpy="0 0 0"/>
             <dynamics damping="0.0" friction="0.1"/>
-            <limit effort="0.1" velocity="10" lower="-3.14" upper="3.14"/>
+            <limit effort="0.1" velocity="10" lower="-0.23087" upper="3.496015"/>
             <parent link="mast"/>
             <child link="yaw"/>
@@ -75,7 +71,7 @@
         </joint>
         <joint name="pitch_joint" type="revolute">
-            <origin xyz="0.0  0.029 0.059 " rpy="0 0 0"/>
+            <origin xyz="0.  0. 0.059 " rpy="0 0 0"/>
             <dynamics damping="0.0" friction="0.1"/>
-            <limit effort="0.1" velocity="10" lower="-0.38" upper="0.52"/>
+            <limit effort="0.1" velocity="10" lower="-0.47247" upper="1.25862"/>
             <parent link="yaw"/>
             <child link="pitch"/>
@@ -91,5 +87,5 @@
             </actuator>
             <joint name="yaw_joint">
-                <offset>3.959203</offset>
+                <offset>-0.2538</offset>
                 <hardwareInterface>hardware_interface/EffortJointInterface</hardwareInterface>
             </joint>
@@ -101,5 +97,5 @@
             </actuator>
             <joint name="pitch_joint">
-                <offset>3.34561</offset>
+                <offset>1.26553</offset>
                 <hardwareInterface>hardware_interface/EffortJointInterface</hardwareInterface>
             </joint>

Commit message: Delete safety_controller of mast

File: urdf/engineer/mast.urdf.xacro (robot description, xacro)
@@ -21,7 +21,7 @@
             </collision>
             <collision>
-                <origin xyz="0. 0.004 0.03" rpy="0 0 0"/>
+                <origin xyz="0. 0.004 0.04" rpy="0 0 0"/>
                 <geometry>
-                    <cylinder length="0.14" radius="0.07"/>
+                    <cylinder length="0.1" radius="0.07"/>
                 </geometry>
             </collision>
@@ -66,5 +66,5 @@
             <dynamics damping="0.0" friction="0.1"/>
             <limit effort="0.2" velocity="10" lower="-0.6197" upper="3.4545"/>
-            <safety_controller k_position="0.2" k_velocity="0.04" soft_lower_limit="-0.519" soft_upper_limit="3.35"/>
+            <!--            <safety_controller k_position="2" k_velocity="0.02" soft_lower_limit="-0.519" soft_upper_limit="3.35"/>-->
             <parent link="mast"/>
             <child link="yaw"/>
