Commit message: Modify the origin data of pitch_joint

File: rm_description/urdf/hero/gimbal.transmission.urdf.xacro (robot description, xacro)
@@ -7,5 +7,5 @@
         </actuator>
         <joint name="yaw_joint">
-            <offset>-5.990</offset>
+            <offset>-3.607</offset>
             <hardwareInterface>hardware_interface/EffortJointInterface</hardwareInterface>
         </joint>
@@ -17,5 +17,5 @@
         </actuator>
         <joint name="pitch_joint">
-            <offset>4.888</offset>
+            <offset>0.876</offset>
             <hardwareInterface>hardware_interface/EffortJointInterface</hardwareInterface>
         </joint>

File: rm_description/urdf/hero/gimbal.urdf.xacro (robot description, xacro)
@@ -54,5 +54,5 @@
     </link>
     <joint name="pitch_joint" type="revolute">
-        <origin xyz="0 0 0.191 " rpy="0 0 0"/>
+        <origin xyz="-0.05 0 0.151 " rpy="0 0 0"/>
         <dynamics damping="0.0" friction="0.1"/>
         <limit effort="1.2" velocity="13.82" lower="${pitch_lower_limit}" upper="${pitch_upper_limit}"/>

File: rm_description/urdf/hero/shooter.transmission.urdf.xacro (robot description, xacro)
@@ -7,5 +7,4 @@
         </actuator>
         <joint name="trigger_joint">
-            <offset>-0.036</offset>>
             <hardwareInterface>hardware_interface/EffortJointInterface</hardwareInterface>
         </joint>
