Commit message: Update standard3 config

File: rm_description/urdf/standard/shooter.urdf.xacro (robot description, xacro)
@@ -31,8 +31,8 @@
         </collision>
     </link>
-    <joint name="trigger_joint" type="continuous">
+    <joint name="trigger_joint" type="revolute">
         <origin xyz="-0.064 0 0" rpy="0 0 0"/>
         <dynamics damping="0.0" friction="0.01"/>
-        <limit effort="1.0" velocity="43.54" lower="-1e16" upper="1e16"/>
+        <limit effort="3.0" velocity="43.54" lower="-1e16" upper="1e16"/>
         <parent link="pitch"/>
         <child link="trigger"/>

File: rm_description/urdf/standard3/shooter.transmission.urdf.xacro (robot description, xacro)
@@ -4,5 +4,5 @@
         <type>transmission_interface/SimpleTransmission</type>
         <actuator name="trigger_joint_motor">
-            <mechanicalReduction>1</mechanicalReduction>
+            <mechanicalReduction>3</mechanicalReduction>
         </actuator>
         <joint name="trigger_joint">
