Commit message: Update standard3 config.

File: rm_description/urdf/standard/gimbal.urdf.xacro (robot description, xacro)
@@ -2,25 +2,25 @@
 <robot xmlns:xacro="http://www.ros.org/wiki/xacro">
     <xacro:property name="threshold" value="0.1"/>
-    <xacro:property name="pitch_lower_limit" value="-0.7"/>
-    <xacro:property name="pitch_upper_limit" value="0.45"/>
-        <link name="yaw">
-            <inertial>
-                <mass value="1.337"/>
-                <origin xyz="0.00072 0.000098 0.00976"/>
-                <inertia ixx="4.777e-3" ixy="-1.108e-5" ixz="1.574e-5" iyy="4.902e-3"
-                         iyz="-1.234e-5" izz="3.643e-3"/>
-            </inertial>
-            <visual>
-                <origin xyz="0 0 0" rpy="0 0 0"/>
-                <geometry>
-                    <mesh filename="package://rm_description/meshes/standard/yaw.stl" scale="0.001 0.001 0.001"/>
-                </geometry>
-            </visual>
-            <collision>
-                <origin xyz="0 0 0" rpy="0 0 0"/>
-                <geometry>
-                    <mesh filename="package://rm_description/meshes/standard/yaw.stl" scale="0.001 0.001 0.001"/>
-                </geometry>
-            </collision>
+    <xacro:property name="pitch_lower_limit" value="-0.421"/>
+    <xacro:property name="pitch_upper_limit" value="0.39"/>
+    <link name="yaw">
+        <inertial>
+            <mass value="1.337"/>
+            <origin xyz="0.00072 0.000098 0.00976"/>
+            <inertia ixx="4.777e-3" ixy="-1.108e-5" ixz="1.574e-5" iyy="4.902e-3"
+                     iyz="-1.234e-5" izz="3.643e-3"/>
+        </inertial>
+        <visual>
+            <origin xyz="0 0 0" rpy="0 0 0"/>
+            <geometry>
+                <mesh filename="package://rm_description/meshes/standard/yaw.stl" scale="0.001 0.001 0.001"/>
+            </geometry>
+        </visual>
+        <collision>
+            <origin xyz="0 0 0" rpy="0 0 0"/>
+            <geometry>
+                <mesh filename="package://rm_description/meshes/standard/yaw.stl" scale="0.001 0.001 0.001"/>
+            </geometry>
+        </collision>
         </link>
         <joint name="yaw_joint" type="revolute">

File: rm_description/urdf/standard3/gimbal.transmission.urdf.xacro (robot description, xacro)
@@ -7,5 +7,5 @@
         </actuator>
         <joint name="yaw_joint">
-            <offset>0.417</offset>
+            <offset>-3.678</offset>
             <hardwareInterface>hardware_interface/EffortJointInterface</hardwareInterface>
         </joint>
@@ -14,8 +14,8 @@
         <type>transmission_interface/SimpleTransmission</type>
         <actuator name="pitch_joint_motor">
-            <mechanicalReduction>-1</mechanicalReduction>
+            <mechanicalReduction>-14</mechanicalReduction>
         </actuator>
         <joint name="pitch_joint">
-            <offset>1.559</offset>
+            <offset>0.162</offset>
             <hardwareInterface>hardware_interface/EffortJointInterface</hardwareInterface>
         </joint>
@@ -24,5 +24,5 @@
         <type>transmission_interface/SimpleTransmission</type>
         <actuator name="cover_joint_motor">
-            <mechanicalReduction>1</mechanicalReduction>
+            <mechanicalReduction>-1</mechanicalReduction>
         </actuator>
         <joint name="cover_joint">

File: rm_description/urdf/standard3/shooter.transmission.urdf.xacro (robot description, xacro)
@@ -13,5 +13,5 @@
         <type>transmission_interface/SimpleTransmission</type>
         <actuator name="left_friction_wheel_joint_motor">
-            <mechanicalReduction>-1</mechanicalReduction>
+            <mechanicalReduction>1</mechanicalReduction>
         </actuator>
         <joint name="left_friction_wheel_joint">
@@ -22,5 +22,5 @@
         <type>transmission_interface/SimpleTransmission</type>
         <actuator name="right_friction_wheel_joint_motor">
-            <mechanicalReduction>-1</mechanicalReduction>
+            <mechanicalReduction>1</mechanicalReduction>
         </actuator>
         <joint name="right_friction_wheel_joint">
