Commit message: Update standard3 urdf.

File: rm_description/urdf/standard/chassis.urdf.xacro (robot description, xacro)
@@ -1,9 +1,8 @@
 <robot xmlns:xacro="http://www.ros.org/wiki/xacro">
-    <xacro:include filename="$(find rm_description)/urdf/common/mecanum_wheel.urdf.xacro"/>
+    <xacro:include filename="$(find rm_description)/urdf/common/omni_wheel.urdf.xacro"/>
     <!-- https://upload.wikimedia.org/wikipedia/commons/5/52/Wheelbase_and_Track.png -->
-    <xacro:property name="wheel_track" value="0.380"/>
-    <xacro:property name="wheel_base" value="0.395"/>
+    <xacro:property name="chassis_radius" value="0.208"/>
     <xacro:property name="wheel_offset_z" value="0.0"/>
-    <xacro:macro name="chassis" params="roller_type">
+    <xacro:macro name="chassis">
         <link name="base_link">
             <inertial>
@@ -26,20 +25,20 @@
             </collision>
         </link>
-        <xacro:mecanum_wheel prefix="left_front" connected_to="base_link"
-                             wheel_x_offset="${wheel_track/2}" wheel_y_offset="${wheel_base/2}"
-                             wheel_z_offset="${wheel_offset_z}"
-                             reflect="1" roller_type="${roller_type}"/>
-        <xacro:mecanum_wheel prefix="right_front" connected_to="base_link"
-                             wheel_x_offset="${wheel_track/2}" wheel_y_offset="${-wheel_base/2}"
-                             wheel_z_offset="${wheel_offset_z}"
-                             reflect="-1" roller_type="${roller_type}"/>
-        <xacro:mecanum_wheel prefix="left_back" connected_to="base_link"
-                             wheel_x_offset="${-wheel_track/2}" wheel_y_offset="${wheel_base/2}"
-                             wheel_z_offset="${wheel_offset_z}"
-                             reflect="-1" roller_type="${roller_type}"/>
-        <xacro:mecanum_wheel prefix="right_back" connected_to="base_link"
-                             wheel_x_offset="${-wheel_track/2}" wheel_y_offset="${-wheel_base/2}"
-                             wheel_z_offset="${wheel_offset_z}"
-                             reflect="1" roller_type="${roller_type}"/>
+        <xacro:omni_wheel prefix="left_front" connected_to="base_link"
+                          wheel_x_offset="${chassis_radius/sqrt(2)}" wheel_y_offset="${chassis_radius/sqrt(2)}"
+                          wheel_z_offset="${wheel_offset_z}" rotation_degree="${3*pi/4}"
+        />
+        <xacro:omni_wheel prefix="right_front" connected_to="base_link"
+                          wheel_x_offset="${chassis_radius/sqrt(2)}" wheel_y_offset="${-chassis_radius/sqrt(2)}"
+                          wheel_z_offset="${wheel_offset_z}" rotation_degree="${pi/4}"
+        />
+        <xacro:omni_wheel prefix="left_back" connected_to="base_link"
+                          wheel_x_offset="${-chassis_radius/sqrt(2)}" wheel_y_offset="${chassis_radius/sqrt(2)}"
+                          wheel_z_offset="${wheel_offset_z}" rotation_degree="${-3*pi/4}"
+        />
+        <xacro:omni_wheel prefix="right_back" connected_to="base_link"
+                          wheel_x_offset="${-chassis_radius/sqrt(2)}" wheel_y_offset="${-chassis_radius/sqrt(2)}"
+                          wheel_z_offset="${wheel_offset_z}" rotation_degree="${-pi/4}"
+        />
         <xacro:wheel_transmission prefix="left_front" mechanical_reduction="19.2032"/>
         <xacro:wheel_transmission prefix="right_front" mechanical_reduction="-19.2032"/>

File: rm_description/urdf/standard3/standard3.urdf.xacro (robot description, xacro)
@@ -7,18 +7,13 @@
     <xacro:arg name="camera_optical_frame" default="camera_optical_frame"/>
     <xacro:arg name="use_simulation" default="true"/>
-    <xacro:arg name="roller_type" default="realistic"/>
     <xacro:if value="$(arg load_chassis)">
         <xacro:include filename="$(find rm_description)/urdf/standard/chassis.urdf.xacro"/>
-        <xacro:chassis roller_type="$(arg roller_type)"/>
+        <xacro:chassis/>
         <xacro:if value="$(arg load_gimbal)">
             <xacro:include filename="$(find rm_description)/urdf/standard/gimbal.urdf.xacro"/>
             <xacro:include filename="$(find rm_description)/urdf/standard3/gimbal.transmission.urdf.xacro"/>
             <xacro:include filename="$(find rm_description)/urdf/common/camera.urdf.xacro"/>
-            <xacro:camera_sensor xyz="0.127 0 -0.038" rpy="0 0 0" frame_id="$(arg camera_link)" parent="pitch"
-                                 camera_sim="$(arg use_simulation)"/>
-            <xacro:camera_optical_frame xyz="0.089 -0.004 -0.053" rpy="1.593 0.0 1.567"
-                                        frame_id="$(arg camera_optical_frame)" parent="pitch"
-                                        camera_sim="$(arg use_simulation)"/>
-            <xacro:IMU connected_to="pitch" imu_name="gimbal_imu" xyz="0.08 0. 0.08" rpy="0 0 -${pi/2}"/>
+            <xacro:include filename="$(find rm_description)/urdf/common/imu.urdf.xacro"/>
+            <xacro:IMU connected_to="pitch" imu_name="gimbal_imu" xyz="0 0 0" rpy="0 0 0"/>
             <xacro:if value="$(arg load_shooter)">
                 <xacro:include filename="$(find rm_description)/urdf/standard/shooter.urdf.xacro"/>

Commit message: Update standard3 urdf.

File: rm_description/urdf/standard/chassis.urdf.xacro (robot description, xacro)
@@ -7,8 +7,8 @@
         <link name="base_link">
             <inertial>
-                <mass value="1.737"/>
-                <origin xyz="0.000425  -0.000733  0.00762"/>
-                <inertia ixx="4.088e-2" ixy="9.103e-5" ixz="-1.697e-4" iyy="4.498e-2"
-                         iyz="6.472e-5" izz="8.107e-2"/>
+                <mass value="8.472226"/>
+                <origin xyz="0.009872  0.010973  0.001286"/>
+                <inertia ixx="1.131e-1" ixy="-4.480e-4" ixz="-9.581e-3" iyy="1.473e-1"
+                         iyz="3.352e-3" izz="2.048e-1"/>
             </inertial>
             <visual>

File: rm_description/urdf/standard/gimbal.urdf.xacro (robot description, xacro)
@@ -2,12 +2,12 @@
 <robot xmlns:xacro="http://www.ros.org/wiki/xacro">
     <xacro:property name="threshold" value="0.1"/>
-    <xacro:property name="pitch_lower_limit" value="-0.421"/>
-    <xacro:property name="pitch_upper_limit" value="0.39"/>
+    <xacro:property name="pitch_lower_limit" value="-0.583"/>
+    <xacro:property name="pitch_upper_limit" value="0.562"/>
     <link name="yaw">
         <inertial>
-            <mass value="1.337"/>
-            <origin xyz="0.00072 0.000098 0.00976"/>
-            <inertia ixx="4.777e-3" ixy="-1.108e-5" ixz="1.574e-5" iyy="4.902e-3"
-                     iyz="-1.234e-5" izz="3.643e-3"/>
+            <mass value="2.497"/>
+            <origin xyz="0.014616 -0.007729 -0.004103"/>
+            <inertia ixx="1.039e-2" ixy="1.575e-3" ixz="-2.149e-3" iyy="1.181e-2"
+                     iyz="1.267e-3" izz="6.380e-3"/>
         </inertial>
         <visual>
@@ -25,5 +25,5 @@
         </link>
         <joint name="yaw_joint" type="revolute">
-            <origin xyz="0 0 0.0696"
+            <origin xyz="0 0 0.162"
                     rpy="0 0 0"/>
             <dynamics damping="0.0" friction="0.1"/>
@@ -35,8 +35,8 @@
         <link name="pitch">
             <inertial>
-                <mass value="1.175"/>
-                <origin xyz="-0.00439 0.0113 -0.00970"/>
-                <inertia ixx="4.716e-3" ixy="-1.511e-4" ixz="-1.134e-4" iyy="5.220e-3"
-                         iyz="1.192e-5" izz="6.046e-3"/>
+                <mass value="2.244065"/>
+                <origin xyz="0.00115 -0.0128 0.0253"/>
+                <inertia ixx="9.63e-3" ixy="-4.829e-3" ixz="-1.382e-3" iyy="1.723e-2"
+                         iyz="-1.088e-3" izz="1.867e-2"/>
             </inertial>
             <visual>
@@ -54,5 +54,5 @@
         </link>
         <joint name="pitch_joint" type="revolute">
-            <origin xyz="0 0 0.189" rpy="0 0 0"/>
+            <origin xyz="0 0 0.129897" rpy="0 0 0"/>
             <dynamics damping="0.0" friction="0.1"/>
             <limit effort="1.2" velocity="13.82" lower="${pitch_lower_limit}" upper="${pitch_upper_limit}"/>

File: rm_description/urdf/standard/shooter.urdf.xacro (robot description, xacro)
@@ -1,8 +1,8 @@
 <robot xmlns:xacro="http://www.ros.org/wiki/xacro">
     <xacro:include filename="$(find rm_description)/urdf/common/friction.urdf.xacro"/>
-<!--    <xacro:include filename="$(find rm_description)/urdf/standard/gimbal.urdf.xacro"/>-->
-    <xacro:property name="wheel_offset_x" value="0.00884"/>
-    <xacro:property name="wheel_offset_y" value="0.036564"/>
-    <xacro:property name="wheel_offset_z" value="0.0"/>
+    <!--    <xacro:include filename="$(find rm_description)/urdf/standard/gimbal.urdf.xacro"/>-->
+    <xacro:property name="wheel_offset_x" value="0.055"/>
+    <xacro:property name="wheel_offset_y" value="0.0365"/>
+    <xacro:property name="wheel_offset_z" value="0.022375"/>
     <xacro:friction_wheel prefixs="left" connected_to="pitch"
                           wheel_x_offset="${wheel_offset_x}" wheel_y_offset="${wheel_offset_y}"
@@ -13,8 +13,8 @@
     <link name="trigger">
         <inertial>
-            <mass value="0.2972"/>
-            <origin xyz="-0.00549 -0.00233 0.00344"/>
-            <inertia ixx="1.955e-4" ixy="-2.402e-5" ixz="-2.718e-5" iyy="3.514e-4"
-                     iyz="-6.239e-6" izz="4.209e-4"/>
+            <mass value="0.952"/>
+            <origin xyz="-0.012227 -0.000055 0.010137"/>
+            <inertia ixx="8.90e-4" ixy="2.012e-6" ixz="1.911e-4" iyy="1.768e-3"
+                     iyz="-7.72e-7" izz="2.067e-3"/>
         </inertial>
         <visual>
@@ -32,8 +32,8 @@
     </link>
     <joint name="trigger_joint" type="revolute">
-        <origin xyz="-0.064 0 0" rpy="0 0 0"/>
+        <origin xyz="0 0 -0.011" rpy="0 0 0"/>
         <dynamics damping="0.0" friction="0.01"/>
         <limit effort="3.0" velocity="43.54" lower="-1e16" upper="1e16"/>
-        <parent link="pitch"/>
+        <parent link="base_link"/>
         <child link="trigger"/>
         <axis xyz="0 0 1 "/>
@@ -41,7 +41,7 @@
     <link name="cover">
         <inertial>
-            <mass value="0.149"/>
-            <origin xyz="-0.008 -0.005 0.019"/>
-            <inertia ixx="2.366e-3" ixy="-2.372e-4" ixz="-7.983e-4" iyy="2.959e-3" iyz="-2.826e-4" izz="9.090e-4"/>
+            <mass value="0.0246"/>
+            <origin xyz="-0.064 -0.000225 0.02447"/>
+            <inertia ixx="5.40e-5" ixy="-1.30e-7" ixz="5.13e-5" iyy="1.54e-4" iyz="4.7e-8" izz="1.688e-4"/>
         </inertial>
         <visual>
@@ -59,9 +59,9 @@
     </link>
     <joint name="cover_joint" type="revolute">
-        <axis xyz="0 0 1"/>
-        <origin xyz="0.037 0.042 0.122"/>
-        <limit effort="1.0" velocity="30" lower="-3.14" upper="3.14"/>
+        <axis xyz="0 1 0"/>
+        <origin xyz="0.187014 0 0.113269"/>
+        <limit effort="1.0" velocity="30" lower="0" upper="3.14"/>
         <dynamics damping="0.0" friction="0.1"/>
-        <parent link="pitch"/>
+        <parent link="base_link"/>
         <child link="cover"/>
     </joint>

File: rm_description/urdf/standard3/gimbal.transmission.urdf.xacro (robot description, xacro)
@@ -14,8 +14,8 @@
         <type>transmission_interface/SimpleTransmission</type>
         <actuator name="pitch_joint_motor">
-            <mechanicalReduction>-14</mechanicalReduction>
+            <mechanicalReduction>1</mechanicalReduction>
         </actuator>
         <joint name="pitch_joint">
-            <offset>0.162</offset>
+            <offset>-2.208</offset>
             <hardwareInterface>hardware_interface/EffortJointInterface</hardwareInterface>
         </joint>

File: rm_description/urdf/standard3/shooter.transmission.urdf.xacro (robot description, xacro)
@@ -4,5 +4,5 @@
         <type>transmission_interface/SimpleTransmission</type>
         <actuator name="trigger_joint_motor">
-            <mechanicalReduction>3</mechanicalReduction>
+            <mechanicalReduction>-3</mechanicalReduction>
         </actuator>
         <joint name="trigger_joint">

File: rm_description/urdf/standard3/standard3.urdf.xacro (robot description, xacro)
@@ -15,5 +15,4 @@
             <xacro:include filename="$(find rm_description)/urdf/common/camera.urdf.xacro"/>
             <xacro:include filename="$(find rm_description)/urdf/common/imu.urdf.xacro"/>
-            <xacro:IMU connected_to="pitch" imu_name="gimbal_imu" xyz="0 0 0" rpy="0 0 0"/>
             <xacro:if value="$(arg load_shooter)">
                 <xacro:include filename="$(find rm_description)/urdf/standard/shooter.urdf.xacro"/>
